File: magic-donut/magic-donut.sch (EAGLE design)
At the start: 21 parts

Commit message: wip
Parts:
- added PRIB, T1, T2, T3, T4: (no value), con-phoenix-500:MSTBV2
Connections:
- net N$1: now also T1-1.SK
- net N$11: now also PRIB-1.SK
- net N$12: now also PRIB-2.SK
- net N$2: now also T2-1.SK
- net N$3: now also T4-2.SK
- net N$4: now also T4-1.SK
- net N$5: now also T3-2.SK
- net N$6: now also T3-1.SK
- net N$7: now also T2-2.SK
- net N$9: now also T1-2.SK
