File: cdf-interrupter/cdf-interrupter.brd (EAGLE design)
At the start: 66 x 58.4 mm, 28 parts, among them IC1 7805T, Q1 16MHz, U1 ATMEGA328P_PDIP

Commit message: cdf interrupter sent to fab
Parts:
- added H5, H6: MOUNT-HOLE3.3, holes:3,3
- added JP1: (no value), pinhead:1X02
- BAT: value (none) -> KEYSTONE-9V-BAT-HOLDER-1291; device con-ptr500:AK500/2 -> keves:KEYSTONE-9V-BAT-HOLDER-1291
- C1, C2: device rcl:C025-025X050 -> rcl:C050-025X075
- FREQ, PW: value PTV111-4220A-B104 -> (none); device keves:PTV111-4 -> Bourns:PTV09A-4
- moved BAT 29.3 mm to (82.5, 5.84), flipped to the top, turned to 270 degrees
- moved FREQ 6.16 mm to (38.5, 9.14)
- moved PW 5.18 mm to (38.5, 28.4)
- moved C2 1.02 mm to (15.0, 21.6)
Connections:
- net +5V: now also FREQ.3, PW.3; no longer FREQ.P3, PW.P3
- net FREQ: now also FREQ.2; no longer FREQ.P2
- net GND: now also BAT.P_NEG, FREQ.1, JP1.2, PW.1; no longer BAT.2, FREQ.P1, PW.P1
- net N$10: now also BAT.P_POS, JP1.1; no longer BAT.1
- net PW: now also PW.2; no longer PW.P2
Routing:
- net GND: track 0.00 -> 49.4 mm
- net N$10: track 14.6 -> 34.7 mm
- net SCK: track 27.2 -> 24.4 mm
- net MISO: track 29.7 -> 27.0 mm
- net PW: track 28.0 -> 30.1 mm
- net N$6: track 12.5 -> 13.4 mm
- net FREQ: track 41.9 -> 42.9 mm
- net MOSI: track 44.0 -> 43.1 mm
- net N$5: track 11.0 -> 11.5 mm
Other:
- board size 66 x 58.4 mm -> 99.1 x 58.4 mm
- board text added: "+"
- board text added: "FREQ"
- board text added: "PW"
