File: cdf-interrupter/cdf-interrupter.sch (EAGLE design)
At the start: 13 parts, among them IC1 7805T, U1 ATMEGA328P_PDIP

Commit message: interrupter
Parts:
- removed U$5: 100SP1T1B4M2QE, keves:100SP1T1B4M2QE
- added BAT: (no value), con-ptr500:AK500/2
- added C1, C2: 18pF, rcl:C-EU025-025X050
- added C3, C4: 1uF, rcl:CPOL-USE2-4
- added H1, H2, H3, H4: MOUNT-PAD-SQUARE4.3, holes:MOUNT-PAD-SQUARE4.3
- added LED1: (no value), adafruit:LED5MM
- added PWR_SW: 100SP1T1B4M2QE, keves:100SP1T1B4M2QE
- added Q1: 16MHz, adafruit:CRYSTALHC49UP
- added R3: 3.3K, rcl:R-US_0204/7
- added R4: 4.7K, rcl:R-US_0204/7
- added R5: 100, rcl:R-US_0204/7
- added R6: 330, rcl:R-US_0204/7
- renumbered U$2 to PW, U$3 to FREQ, U$4 to MODE
Connections:
- new net +5V: C3.+, FREQ.E, IC1.VO, ISP1.VCC, MODE.1, PW.E, R3.2, R4.2, R6.1, U1.AVCC, U1.VCC
- new net FREQ: FREQ.S, U1.PC0(ADC0)
- new net GND: BAT-2.KL, C1.1, C2.2, C3.-, C4.-, FREQ.A, IC1.GND, ISP1.GND, LED1.C, MODE.3, OK1.EMI, PW.A, R2.2, U$6.C, U1.GND@1, U1.GND@2
- new net MISO: ISP1.MISO, U1.PB4(MISO)
- new net MODE: MODE.2, U1.PD3(INT1)
- new net MOSI: ISP1.MOSI, U1.PB3(MOSI/OC2)
- new net N$10: BAT-1.KL, PWR_SW.2
- new net N$11: C4.+, IC1.VI, PWR_SW.3
- new net N$4: OK1.BAS, R2.1
- new net N$5: C1.2, Q1.2, U1.PB6(XTAL1/TOSC1)
- new net N$6: C2.1, Q1.1, U1.PB7(XTAL2/TOSC2)
- new net N$7: R5.2, U1.PD2(INT0)
- new net N$8: R5.1, U$6.A
- new net N$9: LED1.A, R6.2
- new net PW: PW.S, U1.PC1(ADC1)
- new net RESET: ISP1.RST, R4.1, U1.PC6(/RESET)
- new net RX: OK1.COL, R3.1, U1.PD0(RXD)
- new net SCK: ISP1.SCK, U1.PB5(SCK)
Other:
- moved on the sheet: IC1, ISP1, U$6, U1

Commit message: wip
Parts:
- H1, H2, H3, H4: value MOUNT-PAD-SQUARE4.3 -> MOUNT-HOLE3.3; device holes:MOUNT-PAD-SQUARE4.3 -> holes:MOUNT-HOLE3.3
Changed lines of the file:
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@@
 <part name="P+9" library="supply1" deviceset="+5V" device=""/>
 <part name="BAT" library="con-ptr500" deviceset="AK500/2" device=""/>
-<part name="H1" library="holes" deviceset="MOUNT-PAD-SQUARE" device="4.3"/>
-<part name="H2" library="holes" deviceset="MOUNT-PAD-SQUARE" device="4.3"/>
-<part name="H3" library="holes" deviceset="MOUNT-PAD-SQUARE" device="4.3"/>
-<part name="H4" library="holes" deviceset="MOUNT-PAD-SQUARE" device="4.3"/>
+<part name="H1" library="holes" deviceset="MOUNT-HOLE" device="3.3"/>
+<part name="H2" library="holes" deviceset="MOUNT-HOLE" device="3.3"/>
+<part name="H3" library="holes" deviceset="MOUNT-HOLE" device="3.3"/>
+<part name="H4" library="holes" deviceset="MOUNT-HOLE" device="3.3"/>
 </parts>
 <sheets>
@@
 <instance part="BAT" gate="-1" x="-76.2" y="15.24"/>
 <instance part="BAT" gate="-2" x="-76.2" y="10.16"/>
-<instance part="H1" gate="G$1" x="-78.74" y="106.68"/>
-<instance part="H2" gate="G$1" x="-78.74" y="99.06"/>
-<instance part="H3" gate="G$1" x="-78.74" y="91.44"/>
-<instance part="H4" gate="G$1" x="-78.74" y="83.82"/>
+<instance part="H1" gate="G$1" x="-73.66" y="116.84"/>
+<instance part="H2" gate="G$1" x="-73.66" y="111.76"/>
+<instance part="H3" gate="G$1" x="-73.66" y="106.68"/>
+<instance part="H4" gate="G$1" x="-73.66" y="101.6"/>
 </instances>
 <busses>

Commit message: cdf interrupter sent to fab
Parts:
- added H5, H6: MOUNT-HOLE3.3, holes:MOUNT-HOLE3.3
- added JP1: (no value), pinhead:PINHD-1X2
- BAT: value (none) -> KEYSTONE-9V-BAT-HOLDER-1291; device con-ptr500:AK500/2 -> keves:KEYSTONE-9V-BAT-HOLDER-1291
- C1, C2: device rcl:C-EU025-025X050 -> rcl:C-EU050-025X075
- FREQ, PW: value PTV111-4220A-B104 -> (none); device keves:PTV111-4220A-B104 -> Bourns:POTENTIOMETERPTV09A_VERTICAL
Connections:
- net +5V: now also FREQ.CW, PW.CW; no longer FREQ.E, PW.E
- net FREQ: now also FREQ.WIPER; no longer FREQ.S
- net GND: now also BATG_NEG.1, FREQ.CCW, JP1.2, PW.CCW; no longer BAT-2.KL, FREQ.A, PW.A
- net N$10: now also BATG_POS.1, JP1.1; no longer BAT-1.KL
- net PW: now also PW.WIPER; no longer PW.S
Changed lines of the file:
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@@
 <part name="U$1" library="keves" deviceset="MIDIJACK" device=""/>
 <part name="ISP1" library="adafruit" deviceset="AVRISP" device="-BOX"/>
-<part name="PW" library="keves" deviceset="PTV111-4220A-B104" device=""/>
-<part name="FREQ" library="keves" deviceset="PTV111-4220A-B104" device=""/>
 <part name="MODE" library="keves" deviceset="100SP1T1B4M2QE" device=""/>
 <part name="PWR_SW" library="keves" deviceset="100SP1T1B4M2QE" device=""/>
@@
 <part name="P+3" library="supply1" deviceset="+5V" device=""/>
 <part name="Q1" library="adafruit" deviceset="CRYSTAL" device="HC49UP" value="16MHz"/>
-<part name="C1" library="rcl" deviceset="C-EU" device="025-025X050" value="18pF"/>
-<part name="C2" library="rcl" deviceset="C-EU" device="025-025X050" value="18pF"/>
+<part name="C1" library="rcl" deviceset="C-EU" device="050-025X075" value="18pF"/>
+<part name="C2" library="rcl" deviceset="C-EU" device="050-025X075" value="18pF"/>
 <part name="GND5" library="supply1" deviceset="GND" device=""/>
 <part name="GND6" library="supply1" deviceset="GND" device=""/>
@@
 <part name="GND13" library="supply1" deviceset="GND" device=""/>
 <part name="P+9" library="supply1" deviceset="+5V" device=""/>
-<part name="BAT" library="con-ptr500" deviceset="AK500/2" device=""/>
 <part name="H1" library="holes" deviceset="MOUNT-HOLE" device="3.3"/>
 <part name="H2" library="holes" deviceset="MOUNT-HOLE" device="3.3"/>
 <part name="H3" library="holes" deviceset="MOUNT-HOLE" device="3.3"/>
 <part name="H4" library="holes" deviceset="MOUNT-HOLE" device="3.3"/>
+<part name="BAT" library="keves" deviceset="KEYSTONE-9V-BAT-HOLDER-1291" device=""/>
+<part name="H5" library="holes" deviceset="MOUNT-HOLE" device="3.3"/>
+<part name="H6" library="holes" deviceset="MOUNT-HOLE" device="3.3"/>
+<part name="JP1" library="pinhead" deviceset="PINHD-1X2" device=""/>
+<part name="PW" library="Bourns" deviceset="POTENTIOMETER" device="PTV09A_VERTICAL"/>
+<part name="FREQ" library="Bourns" deviceset="POTENTIOMETER" device="PTV09A_VERTICAL"/>
 </parts>
 <sheets>
@@
 <instance part="U$1" gate="G$1" x="-30.48" y="83.82"/>
 <instance part="ISP1" gate="G$1" x="83.82" y="88.9" rot="R180"/>
-<instance part="PW" gate="G$1" x="127" y="81.28" rot="R270"/>
-<instance part="FREQ" gate="G$1" x="160.02" y="81.28" rot="R270"/>
 <instance part="MODE" gate="G$1" x="127" y="66.04" rot="R270"/>
 <instance part="PWR_SW" gate="G$1" x="-55.88" y="15.24" rot="R270"/>
@@
 <instance part="P+4" gate="1" x="66.04" y="86.36" rot="R90"/>
 <instance part="GND7" gate="1" x="66.04" y="91.44" rot="R270"/>
-<instance part="GND8" gate="1" x="134.62" y="81.28" rot="R90"/>
-<instance part="GND9" gate="1" x="167.64" y="81.28" rot="R90"/>
-<instance part="P+5" gate="1" x="119.38" y="81.28" rot="R90"/>
-<instance part="P+6" gate="1" x="152.4" y="81.28" rot="R90"/>
+<instance part="GND8" gate="1" x="139.7" y="96.52" rot="R90"/>
+<instance part="GND9" gate="1" x="167.64" y="96.52" rot="R90"/>
+<instance part="P+5" gate="1" x="119.38" y="96.52" rot="R90"/>
+<instance part="P+6" gate="1" x="147.32" y="96.52" rot="R90"/>
 <instance part="P+7" gate="1" x="134.62" y="68.58" rot="R270"/>
 <instance part="GND10" gate="1" x="134.62" y="63.5" rot="R90"/>
@@
 <instance part="GND13" gate="1" x="-20.32" y="-2.54"/>
 <instance part="P+9" gate="1" x="-2.54" y="20.32"/>
-<instance part="BAT" gate="-1" x="-76.2" y="15.24"/>
-<instance part="BAT" gate="-2" x="-76.2" y="10.16"/>
 <instance part="H1" gate="G$1" x="-73.66" y="116.84"/>
 <instance part="H2" gate="G$1" x="-73.66" y="111.76"/>
 <instance part="H3" gate="G$1" x="-73.66" y="106.68"/>
 <instance part="H4" gate="G$1" x="-73.66" y="101.6"/>
+<instance part="BAT" gate="G_POS" x="-73.66" y="15.24" rot="R180"/>
+<instance part="BAT" gate="G_NEG" x="-73.66" y="10.16" rot="R180"/>
+<instance part="H5" gate="G$1" x="-73.66" y="96.52"/>
+<instance part="H6" gate="G$1" x="-73.66" y="91.44"/>
+<instance part="JP1" gate="G$1" x="-63.5" y="30.48" rot="R90"/>
+<instance part="PW" gate="G$1" x="129.54" y="96.52" rot="R180"/>
+<instance part="FREQ" gate="G$1" x="157.48" y="96.52" rot="R180"/>
 </instances>
 <busses>
@@
 <pinref part="ISP1" gate="G$1" pin="GND"/>
 <pinref part="GND7" gate="1" pin="GND"/>
-</segment>
-<segment>
-<pinref part="PW" gate="G$1" pin="A"/>
-<pinref part="GND8" gate="1" pin="GND"/>
-</segment>
-<segment>
-<pinref part="FREQ" gate="G$1" pin="A"/>
-<pinref part="GND9" gate="1" pin="GND"/>
 </segment>
 <segment>
@@
 <wire x1="-2.54" y1="2.54" x2="-2.54" y2="5.08" width="0.1524" layer="91"/>
 <junction x="-20.32" y="2.54"/>
-<pinref part="BAT" gate="-2" pin="KL"/>
-<wire x1="-40.64" y1="2.54" x2="-71.12" y2="2.54" width="0.1524" layer="91"/>
+<wire x1="-40.64" y1="2.54" x2="-63.5" y2="2.54" width="0.1524" layer="91"/>
+<wire x1="-63.5" y1="2.54" x2="-71.12" y2="2.54" width="0.1524" layer="91"/>
 <wire x1="-71.12" y1="2.54" x2="-71.12" y2="10.16" width="0.1524" layer="91"/>
 <junction x="-40.64" y="2.54"/>
+<pinref part="BAT" gate="G_NEG" pin="1"/>
+<pinref part="JP1" gate="G$1" pin="2"/>
+<wire x1="-63.5" y1="27.94" x2="-63.5" y2="2.54" width="0.1524" layer="91"/>
+<junction x="-63.5" y="2.54"/>
 </segment>
 <segment>
@@
 <pinref part="R2" gate="G$1" pin="2"/>
 <wire x1="22.86" y1="99.06" x2="22.86" y2="96.52" width="0.1524" layer="91"/>
+</segment>
+<segment>
+<pinref part="PW" gate="G$1" pin="CCW"/>
+<pinref part="GND8" gate="1" pin="GND"/>
+</segment>
+<segment>
+<pinref part="FREQ" gate="G$1" pin="CCW"/>
+<pinref part="GND9" gate="1" pin="GND"/>
 </segment>
 </net>
@@
 </segment>
 <segment>
-<pinref part="PW" gate="G$1" pin="E"/>
-<pinref part="P+5" gate="1" pin="+5V"/>
-</segment>
-<segment>
-<pinref part="FREQ" gate="G$1" pin="E"/>
-<pinref part="P+6" gate="1" pin="+5V"/>
-</segment>
-<segment>
 <pinref part="MODE" gate="G$1" pin="1"/>
 <pinref part="P+7" gate="1" pin="+5V"/>
@@
 <wire x1="-2.54" y1="12.7" x2="-2.54" y2="17.78" width="0.1524" layer="91"/>
 <junction x="-2.54" y="12.7"/>
+</segment>
+<segment>
+<pinref part="PW" gate="G$1" pin="CW"/>
+<pinref part="P+5" gate="1" pin="+5V"/>
+</segment>
+<segment>
+<pinref part="FREQ" gate="G$1" pin="CW"/>
+<pinref part="P+6" gate="1" pin="+5V"/>
 </segment>
 </net>
@@
 <net name="PW" class="0">
 <segment>
-<pinref part="PW" gate="G$1" pin="S"/>
-<wire x1="127" y1="76.2" x2="127" y2="73.66" width="0.1524" layer="91"/>
-<label x="127" y="73.66" size="1.778" layer="95"/>
+<wire x1="129.54" y1="91.44" x2="129.54" y2="88.9" width="0.1524" layer="91"/>
+<label x="129.54" y="88.9" size="1.778" layer="95"/>
+<pinref part="PW" gate="G$1" pin="WIPER"/>
 </segment>
 <segment>
@@
 <net name="FREQ" class="0">
 <segment>
-<pinref part="FREQ" gate="G$1" pin="S"/>
-<wire x1="160.02" y1="76.2" x2="160.02" y2="73.66" width="0.1524" layer="91"/>
-<label x="160.02" y="73.66" size="1.778" layer="95"/>
+<wire x1="157.48" y1="91.44" x2="157.48" y2="88.9" width="0.1524" layer="91"/>
+<label x="157.48" y="88.9" size="1.778" layer="95"/>
+<pinref part="FREQ" gate="G$1" pin="WIPER"/>
 </segment>
 <segment>
@@
 <segment>
 <pinref part="PWR_SW" gate="G$1" pin="2"/>
-<wire x1="-60.96" y1="15.24" x2="-71.12" y2="15.24" width="0.1524" layer="91"/>
-<pinref part="BAT" gate="-1" pin="KL"/>
-</segment>
-</net>
+<wire x1="-60.96" y1="15.24" x2="-66.04" y2="15.24" width="0.1524" layer="91"/>
+<pinref part="BAT" gate="G_POS" pin="1"/>
+<pinref part="JP1" gate="G$1" pin="1"/>
+<wire x1="-66.04" y1="15.24" x2="-71.12" y2="15.24" width="0.1524" layer="91"/>
+<wire x1="-66.04" y1="27.94" x2="-66.04" y2="15.24" width="0.1524" layer="91"/>
+<junction x="-66.04" y="15.24"/>
+</segment>
+</net>
