File: led-cube/led-cube.brd (EAGLE design)
At the start: 53.2 x 53.2 mm, 36 parts

Commit message: wip
Parts:
- moved C5 5.53 mm to (5.85, 19.4), turned to 90 degrees
- moved C13 5.28 mm to (5.92, 39.8), turned to 90 degrees
- moved C9 5.05 mm to (5.88, 29.4), turned to 90 degrees
Routing:
- net N$30: track 50.2 -> 41.9 mm
- net N$28: track 49.7 -> 42.5 mm
- net N$29: track 47.1 -> 41.0 mm
- net N$27: track 46.8 -> 41.6 mm
- net DI: vias 4 -> 3
- net CI: vias 4 -> 3
Other:
- outline, holes or cut-outs redrawn
