File: led-cube/led-cube.brd (EAGLE design)
At the start: 53.2 x 53.2 mm, 36 parts

Commit message: wip
Changed lines of the file:
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@@
 <?xml version="1.0" encoding="utf-8"?>
 <!DOCTYPE eagle SYSTEM "eagle.dtd">
-<eagle version="7.6.0">
+<eagle version="7.5.0">
 <drawing>
 <settings>
@@
 <element name="C16" library="microbuilder" package="0603" value="0.1uF" x="40" y="36.5"/>
 <element name="IN1" library="keves" package="1X04" value="" x="25.5" y="1.2"/>
-<element name="IN2" library="keves" package="1X04" value="" x="1.2" y="25" rot="R90"/>
-<element name="OUT1" library="keves" package="1X04" value="" x="25.5" y="48.8"/>
+<element name="IN2" library="keves" package="1X04" value="" x="1.2" y="25" smashed="yes" rot="R90">
+<attribute name="NAME" x="1.5302" y="30.5118" size="1.27" layer="25" ratio="10" rot="R90"/>
+<attribute name="VALUE" x="4.375" y="19.92" size="1.27" layer="27" rot="R90"/>
+</element>
+<element name="OUT1" library="keves" package="1X04" value="" x="25.5" y="48.8" smashed="yes">
+<attribute name="NAME" x="20.5978" y="45.9298" size="1.27" layer="25" ratio="10"/>
+<attribute name="VALUE" x="20.42" y="45.625" size="1.27" layer="27"/>
+</element>
 <element name="OUT2" library="keves" package="1X04" value="" x="48.8" y="25" rot="R90"/>
 </elements>
