File: ab-berry/ab-berry.brd (EAGLE design)
At the start: 100 x 80 mm, 19 parts, among them U1 LM1117MPX-3.3/NOPB or AP2114H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

Commit message: wip
Parts:
- added ROT1, ROT2, ROT3, ROT4: PEC12R-4225F-S0024, keves:PEC111-4XXXK-SXXXX
Connections:
- new net ROT1_A: ROT1.A
- new net ROT1_B: ROT1.B
- new net ROT1_SW: ROT1.S2
- new net ROT2_A: ROT2.A
- new net ROT2_B: ROT2.B
- new net ROT2_SW: ROT2.S2
- new net ROT3_A: ROT3.A
- new net ROT3_B: ROT3.B
- new net ROT3_SW: ROT3.S2
- new net ROT4_A: ROT4.A
- new net ROT4_B: ROT4.B
- new net ROT4_SW: ROT4.S2
- net GND: now also ROT1.C, ROT1.S1, ROT2.C, ROT2.S1, ROT3.C, ROT3.S1, ROT4.C, ROT4.S1
Changed lines of the file:
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@@
 <layer number="121" name="sName" color="7" fill="1" visible="yes" active="yes"/>
 <layer number="122" name="_bPlace" color="7" fill="1" visible="yes" active="yes"/>
+<layer number="123" name="tTestmark" color="7" fill="1" visible="no" active="yes"/>
+<layer number="124" name="bTestmark" color="7" fill="1" visible="no" active="yes"/>
 <layer number="125" name="_tNames" color="7" fill="1" visible="yes" active="yes"/>
 <layer number="126" name="_bNames" color="7" fill="1" visible="yes" active="yes"/>
 <layer number="127" name="_tValues" color="7" fill="1" visible="yes" active="yes"/>
 <layer number="128" name="_bValues" color="7" fill="1" visible="yes" active="yes"/>
+<layer number="131" name="tAdjust" color="7" fill="1" visible="no" active="yes"/>
+<layer number="132" name="bAdjust" color="7" fill="1" visible="no" active="yes"/>
 <layer number="144" name="Drill_legend" color="7" fill="1" visible="yes" active="yes"/>
 <layer number="151" name="HeatSink" color="7" fill="1" visible="yes" active="yes"/>
 <layer number="152" name="_bDocu" color="7" fill="1" visible="yes" active="yes"/>
+<layer number="199" name="Contour" color="7" fill="1" visible="yes" active="yes"/>
 <layer number="200" name="200bmp" color="1" fill="10" visible="yes" active="yes"/>
 <layer number="201" name="201bmp" color="7" fill="1" visible="yes" active="yes"/>
@@
 <layer number="207" name="207bmp" color="8" fill="10" visible="yes" active="yes"/>
 <layer number="208" name="208bmp" color="9" fill="10" visible="yes" active="yes"/>
+<layer number="209" name="209bmp" color="7" fill="1" visible="no" active="yes"/>
+<layer number="210" name="210bmp" color="7" fill="1" visible="no" active="yes"/>
+<layer number="211" name="211bmp" color="7" fill="1" visible="no" active="yes"/>
+<layer number="212" name="212bmp" color="7" fill="1" visible="no" active="yes"/>
+<layer number="213" name="213bmp" color="7" fill="1" visible="no" active="yes"/>
+<layer number="214" name="214bmp" color="7" fill="1" visible="no" active="yes"/>
+<layer number="215" name="215bmp" color="7" fill="1" visible="no" active="yes"/>
+<layer number="216" name="216bmp" color="7" fill="1" visible="no" active="yes"/>
+<layer number="217" name="217bmp" color="18" fill="1" visible="no" active="no"/>
+<layer number="218" name="218bmp" color="19" fill="1" visible="no" active="no"/>
+<layer number="219" name="219bmp" color="20" fill="1" visible="no" active="no"/>
+<layer number="220" name="220bmp" color="21" fill="1" visible="no" active="no"/>
+<layer number="221" name="221bmp" color="22" fill="1" visible="no" active="no"/>
+<layer number="222" name="222bmp" color="23" fill="1" visible="no" active="no"/>
+<layer number="223" name="223bmp" color="24" fill="1" visible="no" active="no"/>
+<layer number="224" name="224bmp" color="25" fill="1" visible="no" active="no"/>
 <layer number="231" name="Eagle3D_PG1" color="14" fill="1" visible="yes" active="yes"/>
 <layer number="232" name="Eagle3D_PG2" color="14" fill="2" visible="yes" active="yes"/>
@@
 <element name="LED1" library="microbuilder" package="CHIPLED_0603" value="" x="-41.91" y="-45.72"/>
 <element name="R5" library="microbuilder" package="0603" value="330" x="-41.91" y="-49.53"/>
+<element name="ROT1" library="keves" package="PEC111-4XXXK-SXXXX" value="PEC12R-4225F-S0024" x="-52.07" y="-41.91"/>
+<element name="ROT2" library="keves" package="PEC111-4XXXK-SXXXX" value="PEC12R-4225F-S0024" x="-52.07" y="-59.69"/>
+<element name="ROT3" library="keves" package="PEC111-4XXXK-SXXXX" value="PEC12R-4225F-S0024" x="-52.07" y="-77.47"/>
+<element name="ROT4" library="keves" package="PEC111-4XXXK-SXXXX" value="PEC12R-4225F-S0024" x="-52.07" y="-95.25"/>
 </elements>
 <signals>
@@
 <contactref element="C9" pad="2"/>
 <contactref element="U1" pad="1"/>
+<contactref element="ROT1" pad="C"/>
+<contactref element="ROT1" pad="S1"/>
+<contactref element="ROT2" pad="C"/>
+<contactref element="ROT2" pad="S1"/>
+<contactref element="ROT3" pad="C"/>
+<contactref element="ROT3" pad="S1"/>
+<contactref element="ROT4" pad="C"/>
+<contactref element="ROT4" pad="S1"/>
+<wire x1="-54.57" y1="-88.25" x2="-52.07" y2="-102.75" width="0" layer="19" extent="1-1"/>
+<wire x1="-52.07" y1="-84.97" x2="-54.57" y2="-88.25" width="0" layer="19" extent="1-1"/>
+<wire x1="-54.57" y1="-70.47" x2="-52.07" y2="-84.97" width="0" layer="19" extent="1-1"/>
+<wire x1="-52.07" y1="-67.19" x2="-54.57" y2="-70.47" width="0" layer="19" extent="1-1"/>
+<wire x1="-54.57" y1="-52.69" x2="-52.07" y2="-67.19" width="0" layer="19" extent="1-1"/>
+<wire x1="-52.07" y1="-49.41" x2="-54.57" y2="-52.69" width="0" layer="19" extent="1-1"/>
+<wire x1="-41.91" y1="-44.97" x2="-52.07" y2="-49.41" width="0" layer="19" extent="1-1"/>
 <wire x1="-37.68" y1="-44.45" x2="-41.91" y2="-44.97" width="0" layer="19" extent="1-1"/>
 <wire x1="-37.86" y1="-42.42" x2="-37.68" y2="-44.45" width="0" layer="19" extent="1-1"/>
@@
 <wire x1="-28.92" y1="11.77" x2="-22.52" y2="9.87" width="0" layer="19" extent="1-1"/>
 <wire x1="-30.82" y1="6.87" x2="-28.92" y2="11.77" width="0" layer="19" extent="1-1"/>
+<wire x1="-54.57" y1="-34.91" x2="-52.07" y2="-49.41" width="0" layer="19" extent="1-1"/>
 </signal>
 <signal name="3.3V">
@@
 <wire x1="-33.26" y1="-42.42" x2="-35.98" y2="-44.45" width="0" layer="19" extent="1-1"/>
 </signal>
+<signal name="ROT1_A">
+<contactref element="ROT1" pad="A"/>
+</signal>
+<signal name="ROT1_B">
+<contactref element="ROT1" pad="B"/>
+</signal>
+<signal name="ROT1_SW">
+<contactref element="ROT1" pad="S2"/>
+</signal>
+<signal name="ROT2_A">
+<contactref element="ROT2" pad="A"/>
+</signal>
+<signal name="ROT2_B">
+<contactref element="ROT2" pad="B"/>
+</signal>
+<signal name="ROT2_SW">
+<contactref element="ROT2" pad="S2"/>
+</signal>
+<signal name="ROT3_A">
+<contactref element="ROT3" pad="A"/>
+</signal>
+<signal name="ROT3_B">
+<contactref element="ROT3" pad="B"/>
+</signal>
+<signal name="ROT3_SW">
+<contactref element="ROT3" pad="S2"/>
+</signal>
+<signal name="ROT4_A">
+<contactref element="ROT4" pad="A"/>
+</signal>
+<signal name="ROT4_B">
+<contactref element="ROT4" pad="B"/>
+</signal>
+<signal name="ROT4_SW">
+<contactref element="ROT4" pad="S2"/>
+</signal>
 </signals>

Commit message: wip
Parts:
- added C10, C11: 0.1uF, microbuilder:0603
- added LCD1, LCD2: SSD1306-7PIN, keves:SSD1306-7PIN
Connections:
- new net LCD_CS1: LCD1.CS
- new net LCD_CS2: LCD2.CS
- new net LCD_DC: LCD1.DC, LCD2.DC
- new net LCD_RST: LCD1.RES, LCD2.RES
- new net SPI1_CLK: LCD1.CLK, LCD2.CLK, STM32F072CBT6.15
- new net SPI1_MOSI: LCD1.MOSI, LCD2.MOSI, STM32F072CBT6.17
- net 3.3V: now also C10.1, C11.1, LCD1.VCC, LCD2.VCC
- net GND: now also C10.2, C11.2, LCD1.GND, LCD2.GND
Changed lines of the file:
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@@
 <element name="ROT3" library="keves" package="PEC111-4XXXK-SXXXX" value="PEC12R-4225F-S0024" x="-52.07" y="-77.47"/>
 <element name="ROT4" library="keves" package="PEC111-4XXXK-SXXXX" value="PEC12R-4225F-S0024" x="-52.07" y="-95.25"/>
+<element name="LCD1" library="keves" package="SSD1306-7PIN" value="SSD1306-7PIN" x="-73.66" y="-100.33"/>
+<element name="C10" library="microbuilder" package="0603" value="0.1uF" x="-85.09" y="-105.41"/>
+<element name="LCD2" library="keves" package="SSD1306-7PIN" value="SSD1306-7PIN" x="-73.66" y="-133.35"/>
+<element name="C11" library="microbuilder" package="0603" value="0.1uF" x="-85.09" y="-137.16"/>
 </elements>
 <signals>
@@
 <contactref element="ROT4" pad="C"/>
 <contactref element="ROT4" pad="S1"/>
-<wire x1="-54.57" y1="-88.25" x2="-52.07" y2="-102.75" width="0" layer="19" extent="1-1"/>
-<wire x1="-52.07" y1="-84.97" x2="-54.57" y2="-88.25" width="0" layer="19" extent="1-1"/>
-<wire x1="-54.57" y1="-70.47" x2="-52.07" y2="-84.97" width="0" layer="19" extent="1-1"/>
+<contactref element="C10" pad="2"/>
+<contactref element="LCD1" pad="GND"/>
+<contactref element="C11" pad="2"/>
+<contactref element="LCD2" pad="GND"/>
+<wire x1="-81.28" y1="-109.05" x2="-84.24" y2="-137.16" width="0" layer="19" extent="1-1"/>
+<wire x1="-84.24" y1="-105.41" x2="-81.28" y2="-109.05" width="0" layer="19" extent="1-1"/>
+<wire x1="-81.28" y1="-76.03" x2="-84.24" y2="-105.41" width="0" layer="19" extent="1-1"/>
+<wire x1="-54.57" y1="-70.47" x2="-81.28" y2="-76.03" width="0" layer="19" extent="1-1"/>
 <wire x1="-52.07" y1="-67.19" x2="-54.57" y2="-70.47" width="0" layer="19" extent="1-1"/>
+<wire x1="-52.07" y1="-84.97" x2="-54.57" y2="-70.47" width="0" layer="19" extent="1-1"/>
+<wire x1="-54.57" y1="-88.25" x2="-52.07" y2="-84.97" width="0" layer="19" extent="1-1"/>
+<wire x1="-52.07" y1="-102.75" x2="-54.57" y2="-88.25" width="0" layer="19" extent="1-1"/>
 <wire x1="-54.57" y1="-52.69" x2="-52.07" y2="-67.19" width="0" layer="19" extent="1-1"/>
 <wire x1="-52.07" y1="-49.41" x2="-54.57" y2="-52.69" width="0" layer="19" extent="1-1"/>
@@
 <contactref element="R5" pad="2"/>
 <contactref element="C9" pad="1"/>
+<contactref element="LCD1" pad="VCC"/>
+<contactref element="C10" pad="1"/>
+<contactref element="LCD2" pad="VCC"/>
+<contactref element="C11" pad="1"/>
+<wire x1="-78.74" y1="-109.05" x2="-85.94" y2="-137.16" width="0" layer="19" extent="1-1"/>
+<wire x1="-85.94" y1="-105.41" x2="-78.74" y2="-109.05" width="0" layer="19" extent="1-1"/>
+<wire x1="-78.74" y1="-76.03" x2="-85.94" y2="-105.41" width="0" layer="19" extent="1-1"/>
+<wire x1="-41.06" y1="-49.53" x2="-78.74" y2="-76.03" width="0" layer="19" extent="1-1"/>
 <wire x1="-37.68" y1="-46.99" x2="-41.06" y2="-49.53" width="0" layer="19" extent="1-1"/>
 <wire x1="-35.56" y1="-42.42" x2="-37.68" y2="-46.99" width="0" layer="19" extent="1-1"/>
@@
 <contactref element="ROT4" pad="S2"/>
 </signal>
+<signal name="SPI1_MOSI">
+<contactref element="LCD1" pad="MOSI"/>
+<contactref element="LCD2" pad="MOSI"/>
+<contactref element="STM32F072CBT6" pad="17"/>
+<wire x1="-73.66" y1="-76.03" x2="-73.66" y2="-109.05" width="0" layer="19" extent="1-1"/>
+<wire x1="-27.42" y1="3.47" x2="-73.66" y2="-76.03" width="0" layer="19" extent="1-1"/>
+</signal>
+<signal name="LCD_CS1">
+<contactref element="LCD1" pad="CS"/>
+</signal>
+<signal name="LCD_DC">
+<contactref element="LCD1" pad="DC"/>
+<contactref element="LCD2" pad="DC"/>
+<wire x1="-68.58" y1="-76.03" x2="-68.58" y2="-109.05" width="0" layer="19" extent="1-1"/>
+</signal>
+<signal name="LCD_RST">
+<contactref element="LCD1" pad="RES"/>
+<contactref element="LCD2" pad="RES"/>
+<wire x1="-71.12" y1="-76.03" x2="-71.12" y2="-109.05" width="0" layer="19" extent="1-1"/>
+</signal>
+<signal name="SPI1_CLK">
+<contactref element="LCD1" pad="CLK"/>
+<contactref element="LCD2" pad="CLK"/>
+<contactref element="STM32F072CBT6" pad="15"/>
+<wire x1="-76.2" y1="-76.03" x2="-76.2" y2="-109.05" width="0" layer="19" extent="1-1"/>
+<wire x1="-28.42" y1="3.47" x2="-76.2" y2="-76.03" width="0" layer="19" extent="1-1"/>
+</signal>
+<signal name="LCD_CS2">
+<contactref element="LCD2" pad="CS"/>
+</signal>
 </signals>

Commit message: wip
Parts:
- added H1, H2, H3, H4: MOUNT-HOLE3.6, holes:3,6
- added JP1, JP2: (no value), keves:1X04
- added JP3: (no value), pinhead:1X02
- moved C11 207.6 mm to (28.8, 36.4), flipped to the bottom, turned to 90 degrees
- moved C10 201.7 mm to (58.3, 36.4), flipped to the bottom, turned to 90 degrees
- moved LCD2 182.3 mm to (6.35, 30.5), turned to 270 degrees
- moved LCD1 170.6 mm to (35.8, 30.5), turned to 270 degrees
- moved ROT3 164.1 mm to (47.8, 52.8)
- moved ROT4 144.3 mm to (47.8, 8.89)
- moved ROT2 132.7 mm to (18.3, 52.8)
- moved R5 130.5 mm to (29.8, 59.4), flipped to the bottom, turned to 90 degrees
- moved LED1 124.4 mm to (29.8, 55.9), flipped to the bottom, turned to 180 degrees
- moved C8 118.2 mm to (63.8, 17.7), flipped to the bottom, turned to 180 degrees
- moved U1 110.9 mm to (62.4, 12.7), flipped to the bottom, turned to 180 degrees
- moved C9 110.8 mm to (58.4, 9.65), flipped to the bottom
- moved ROT1 86.8 mm to (18.3, 8.89)
- moved C7 86.6 mm to (8.26, 36.2), flipped to the bottom, turned to 180 degrees
- moved R4 83.6 mm to (4.95, 37.0), flipped to the bottom, turned to 90 degrees
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Connections:
- net 3.3V: now also JP3.1
- net 5.0V: now also JP1.1, JP2.1
- net CAN_H: now also JP1.2, JP2.2
- net CAN_L: now also JP1.3, JP2.3
- net GND: now also JP1.4, JP2.4, JP3.2
Routing:
- net CAN_L: track 0.00 -> 80.9 mm
- net CAN_H: track 0.00 -> 76.6 mm
- net 5.0V: track 0.00 -> 76.5 mm
- net SPI1_CLK: track 0.00 -> 45.3 mm, vias 0 -> 1
- net SPI1_MOSI: track 0.00 -> 43.9 mm, vias 0 -> 1
- net LCD_RST: track 0.00 -> 29.5 mm
- net LCD_DC: track 0.00 -> 29.5 mm
- net 3.3V: track 0.00 -> 27.3 mm, vias 0 -> 5
- net RST: track 0.00 -> 24.1 mm, vias 0 -> 2
- net DBG_TX: track 0.00 -> 23.5 mm, vias 0 -> 2
- net DBG_RX: track 0.00 -> 21.5 mm, vias 0 -> 2
- net SWDIO: track 0.00 -> 21.5 mm
- net SWCLK: track 0.00 -> 19.6 mm
- net CAN_TX: track 0.00 -> 13.6 mm
- net CAN_RX: track 0.00 -> 4.64 mm
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- added copper zone on layer 1, net 3.3V
- added copper zone on layer 16, net GND
Other:
- board size 100 x 80 mm -> 66 x 62.2 mm

Commit message: wip
Parts:
- H1, H2, H3, H4: value MOUNT-HOLE3.6 -> MOUNT-HOLE3.2; device holes:3,6 -> holes:3,2
- moved U1 33.2 mm to (30.2, 4.45), turned to 270 degrees
- moved C8 32.1 mm to (35.2, 3.05), turned to 270 degrees
- moved C9 31.3 mm to (27.2, 8.38), turned to 90 degrees
- moved JP2 19.7 mm to (57.1, 11.8)
- moved JP1 18.7 mm to (1.27, 11.8)
- moved H3 7.73 mm to (55.9, 58.4)
- moved H4 7.62 mm to (55.9, 2.54)
- moved JP3 5.93 mm to (29.7, 56.3)
- moved LED1 5.93 mm to (25.5, 51.8)
- moved R5 5.93 mm to (25.5, 55.4)
- moved R2 5.24 mm to (1.52, 24.4), turned to 270 degrees
- moved ROT3 3.82 mm to (43.9, 52.6)
- moved ROT2 3.82 mm to (14.5, 52.6)
- moved C10 3.81 mm to (54.5, 36.4)
- moved C11 3.81 mm to (25.0, 36.4)
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Connections:
- net CAN_H: now also JP1.3, JP2.3; no longer JP1.2, JP2.2
- net CAN_L: now also JP1.2, JP2.2; no longer JP1.3, JP2.3
Routing:
- net 5.0V: track 76.5 -> 61.7 mm
- net GND: track 0.00 -> 10.7 mm, vias 0 -> 2
- net RST: track 24.1 -> 28.3 mm
- net CAN_L: track 80.9 -> 77.1 mm
- net SWDIO: track 21.5 -> 17.7 mm
- net DBG_TX: track 23.5 -> 26.6 mm
- net CAN_H: track 76.6 -> 73.8 mm
- net SWCLK: track 19.6 -> 18.0 mm
- net DBG_RX: track 21.5 -> 22.8 mm
- net N$2: track 2.25 -> 3.37 mm
Other:
- board size 66 x 62.2 mm -> 58.4 x 61 mm

Commit message: ab-berry
Parts:
- added LED2: (no value), microbuilder:CHIPLED_0603
- added R6: 330, microbuilder:0603
- C8, C9: value (none) -> 10uF Tantalum
- moved C3 2.01 mm to (11.9, 24.0), turned to 90 degrees
- moved R1 1.52 mm to (17.0, 41.4), turned to 0 degrees
- moved C2 1.37 mm to (19.7, 35.9)
- moved C6 1.37 mm to (19.7, 37.7)
Connections:
- new net N$6: R6.2, STM32F072CBT6.18
- new net N$7: LED2.A, R6.1
- net GND: now also LED2.C
- net LCD_CS1: now also STM32F072CBT6.20
- net LCD_CS2: now also STM32F072CBT6.19
- net LCD_DC: now also STM32F072CBT6.14
- net LCD_RST: now also STM32F072CBT6.13
- net ROT1_A: now also STM32F072CBT6.28
- net ROT1_B: now also STM32F072CBT6.27
- net ROT1_SW: now also STM32F072CBT6.25
- net ROT2_A: now also STM32F072CBT6.40
- net ROT2_B: now also STM32F072CBT6.41
- net ROT2_SW: now also STM32F072CBT6.39
- net ROT3_A: now also STM32F072CBT6.43
- net ROT3_B: now also STM32F072CBT6.45
- net ROT3_SW: now also STM32F072CBT6.42
- net ROT4_A: now also STM32F072CBT6.26
- net ROT4_B: now also STM32F072CBT6.22
- net ROT4_SW: now also STM32F072CBT6.21
Routing:
- net ROT4_A: track 0.00 -> 53.7 mm, vias 0 -> 1
- net ROT4_B: track 0.00 -> 51.1 mm, vias 0 -> 1
- net LCD_CS1: track 0.00 -> 46.9 mm, vias 0 -> 1
- net ROT3_SW: track 0.00 -> 46.1 mm, vias 0 -> 1
- net ROT4_SW: track 0.00 -> 39.8 mm
- net ROT3_B: track 0.00 -> 37.7 mm, vias 0 -> 1
- net ROT3_A: track 0.00 -> 34.5 mm, vias 0 -> 1
- net ROT1_B: track 0.00 -> 34.4 mm, vias 0 -> 1
- net 3.3V: track 27.7 -> 61.4 mm, vias 5 -> 14
- net ROT1_A: track 0.00 -> 33.0 mm, vias 0 -> 1
- net ROT2_SW: track 0.00 -> 28.1 mm, vias 0 -> 1
- net ROT1_SW: track 0.00 -> 17.1 mm
- net LCD_CS2: track 0.00 -> 16.0 mm
- net ROT2_B: track 0.00 -> 11.3 mm
- net LCD_DC: track 29.5 -> 40.7 mm, vias 0 -> 1
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
Commit message: ab-berry: added xtal :/
Parts:
- added C12, C13: 18pF, microbuilder:0603
- added U$36: ABM7-8.000MHZ-D2Y-T, keves:ABM7-8.000MHZ-D2Y-T
- moved C1 14.0 mm to (8.76, 36.1), turned to 270 degrees
- moved C4 13.3 mm to (18.8, 26.4), turned to 90 degrees
- moved R4 4.95 mm to (1.14, 32.0)
- moved D1 4.95 mm to (3.05, 26.3)
- moved C7 4.62 mm to (2.79, 31.9), turned to 90 degrees
- moved C11 4.45 mm to (29.5, 36.4)
- moved C3 3.66 mm to (8.89, 26.0)
- moved R2 3.39 mm to (2.29, 21.1), turned to 180 degrees
- moved C5 2.98 mm to (20.6, 26.4)
- moved R3 2.09 mm to (4.57, 31.9), turned to 90 degrees
- moved C2 1.70 mm to (18.2, 36.7)
- moved C6 1.70 mm to (18.2, 38.5)
- moved STM32F072CBT6 1.52 mm to (13.2, 31.4)
- moved LED2 1.27 mm to (21.6, 23.4)
- moved R6 0.92 mm to (17.8, 23.4)
Connections:
- new net N$8: C12.2, STM32F072CBT6.5, U$36.P$2
- new net N$9: C13.1, STM32F072CBT6.6, U$36.P$1
- net DBG_RX: now also TC1.8; no longer TC1.6
- net DBG_TX: now also TC1.6; no longer TC1.8
- net GND: now also C12.1, C13.2
- net ROT1_A: now also STM32F072CBT6.27; no longer STM32F072CBT6.28
- net ROT1_B: now also STM32F072CBT6.28; no longer STM32F072CBT6.27
Routing:
- net ROT4_A: track 53.7 -> 44.6 mm
- net N$8: track 0.00 -> 7.94 mm
- net N$9: track 0.00 -> 7.83 mm
- net ROT2_B: track 11.3 -> 3.88 mm
- net ROT3_SW: track 46.1 -> 39.0 mm
- net ROT3_A: track 34.5 -> 27.6 mm
- net ROT2_A: track 10.2 -> 3.59 mm
- net ROT3_B: track 37.7 -> 32.1 mm
- net N$1: track 6.17 -> 0.97 mm
- net ROT2_SW: track 28.1 -> 23.0 mm
- net CAN_L: track 77.1 -> 72.8 mm
- net CAN_H: track 73.5 -> 69.3 mm
- net CAN_TX: track 13.6 -> 9.88 mm
- net 3.3V: track 61.4 -> 58.1 mm
- net N$6: track 3.69 -> 6.87 mm
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
Commit message: ab-berry: silkscreen
Routing:
- net ROT4_A: track 44.6 -> 55.5 mm, vias 1 -> 3
- net ROT2_B: track 3.88 -> 11.9 mm
- net ROT3_SW: track 39.0 -> 46.7 mm
- net ROT3_A: track 27.6 -> 35.1 mm
- net ROT3_B: track 32.1 -> 39.2 mm
- net ROT2_A: track 3.59 -> 9.58 mm
- net N$1: track 0.97 -> 6.80 mm
- net ROT2_SW: track 23.0 -> 27.5 mm
- net 3.3V: track 58.1 -> 59.3 mm
Other:
- board text added: "ab-berry v1.0 2016 Designed by Eran Rundstein"
