File: ab-berry/ab-berry-rev2.brd (EAGLE design)
At the start: 58.4 x 61 mm, 70 parts, among them IC1 STM32F303CCT6, U1 LM1117MPX-3.3/NOPB or AP2114H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, U2 PRTR5V0U2X

Commit message: wip
Parts:
- moved LED2 0.40 mm to (21.5, 23.7)
- moved R6 0.38 mm to (17.8, 23.7)
Connections:
- net ROT3_B: now also IC1.18
Routing:
- net ROT3_B: track 41.3 -> 61.2 mm, vias 4 -> 2
- net N$16: track 1.93 -> 3.71 mm
- net N$18: track 50.5 -> 51.3 mm
- net N$19: track 49.3 -> 50.1 mm
Changed lines of the file:
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@@
 <element name="H4" library="holes" package="3,2" value="MOUNT-HOLE3.2" x="55.88" y="2.54"/>
 <element name="JP3" library="pinhead" package="1X02" value="" x="55.626" y="50.546" rot="MR90"/>
-<element name="R6" library="microbuilder" package="0603" value="330" x="17.78" y="23.368" rot="MR0"/>
-<element name="LED2" library="microbuilder" package="CHIPLED_0603" value="" x="21.59" y="23.368" rot="MR90"/>
+<element name="R6" library="microbuilder" package="0603" value="330" x="17.78" y="23.749" rot="MR0"/>
+<element name="LED2" library="microbuilder" package="CHIPLED_0603" value="" x="21.463" y="23.749" rot="MR90"/>
 <element name="C12" library="microbuilder" package="0603" value="18pF" x="24.257" y="33.782" rot="MR90"/>
 <element name="C13" library="microbuilder" package="0603" value="18pF" x="24.257" y="30.226" smashed="yes" rot="MR90">
@@
 <wire x1="8.382" y1="48.602" x2="8.167" y2="48.602" width="0.254" layer="16"/>
 <wire x1="8.167" y1="48.602" x2="5.969" y2="50.8" width="0.254" layer="16"/>
-<wire x1="2.794" y1="51.562" x2="5.969" y2="50.8" width="0" layer="19" extent="16-16"/>
 </signal>
 <signal name="3.3V">
@@
 <signal name="ROT1_SW">
 <contactref element="ROT1" pad="S2"/>
-<wire x1="7.283" y1="28.619" x2="6.858" y2="28.194" width="0.254" layer="16"/>
-<wire x1="6.858" y1="28.194" x2="6.858" y2="24.765" width="0.254" layer="16"/>
 <via x="11.43" y="20.193" extent="1-16" drill="0.6"/>
 <wire x1="16.978" y1="15.89" x2="15.733" y2="15.89" width="0.254" layer="1"/>
@@
 <contactref element="IC1" pad="25"/>
 <wire x1="9.058" y1="28.619" x2="7.283" y2="28.619" width="0.254" layer="16"/>
+<wire x1="7.283" y1="28.619" x2="6.35" y2="27.686" width="0.254" layer="16"/>
+<wire x1="6.35" y1="27.686" x2="6.35" y2="25.273" width="0.254" layer="16"/>
+<wire x1="6.35" y1="25.273" x2="6.858" y2="24.765" width="0.254" layer="16"/>
 </signal>
 <signal name="ROT2_A">
@@
 </signal>
 <signal name="ROT3_B">
-<wire x1="46.442" y1="42.886" x2="45.72" y2="42.164" width="0.254" layer="1"/>
-<via x="21.59" y="40.386" extent="1-16" drill="0.6"/>
-<wire x1="21.59" y1="40.386" x2="15.875" y2="40.386" width="0.254" layer="16"/>
-<wire x1="14.458" y1="38.969" x2="15.875" y2="40.386" width="0.254" layer="16"/>
 <contactref element="R20" pad="1"/>
 <contactref element="C21" pad="1"/>
@@
 <wire x1="50.038" y1="46.902" x2="48.182" y2="46.902" width="0.254" layer="16"/>
 <wire x1="48.182" y1="46.902" x2="48.094" y2="46.99" width="0.254" layer="16"/>
-<wire x1="21.59" y1="40.386" x2="34.544" y2="40.386" width="0.254" layer="1"/>
-<wire x1="34.544" y1="40.386" x2="36.322" y2="42.164" width="0.254" layer="1"/>
-<via x="36.322" y="42.164" extent="1-16" drill="0.6"/>
-<wire x1="36.322" y1="42.164" x2="39.751" y2="42.164" width="0.254" layer="16"/>
-<via x="39.751" y="42.164" extent="1-16" drill="0.6"/>
-<wire x1="39.751" y1="42.164" x2="45.72" y2="42.164" width="0.254" layer="1"/>
+<contactref element="IC1" pad="18"/>
+<wire x1="13.458" y1="27.219" x2="13.458" y2="24.134" width="0.254" layer="16"/>
+<wire x1="13.458" y1="24.134" x2="14.732" y2="22.86" width="0.254" layer="16"/>
+<wire x1="14.732" y1="22.86" x2="24.384" y2="22.86" width="0.254" layer="16"/>
+<wire x1="24.384" y1="22.86" x2="25.781" y2="24.257" width="0.254" layer="16"/>
+<wire x1="25.781" y1="24.257" x2="41.021" y2="24.257" width="0.254" layer="16"/>
+<via x="41.021" y="24.257" extent="1-16" drill="0.6"/>
+<wire x1="41.021" y1="24.257" x2="42.545" y2="24.257" width="0.254" layer="1"/>
+<wire x1="42.545" y1="24.257" x2="44.323" y2="26.035" width="0.254" layer="1"/>
+<wire x1="44.323" y1="26.035" x2="44.323" y2="40.767" width="0.254" layer="1"/>
+<wire x1="44.323" y1="40.767" x2="46.442" y2="42.886" width="0.254" layer="1"/>
 </signal>
 <signal name="ROT3_SW">
@@
 <signal name="ROT4_A">
 <wire x1="8.89" y1="21.59" x2="17.272" y2="13.208" width="0.254" layer="16"/>
-<wire x1="7.021" y1="29.119" x2="6.35" y2="28.448" width="0.254" layer="16"/>
+<wire x1="7.021" y1="29.119" x2="5.715" y2="27.813" width="0.254" layer="16"/>
 <via x="6.985" y="23.495" extent="1-16" drill="0.6"/>
 <wire x1="6.985" y1="23.495" x2="8.89" y2="21.59" width="0.254" layer="1"/>
-<wire x1="6.096" y1="24.384" x2="6.985" y2="23.495" width="0.254" layer="16"/>
+<wire x1="5.715" y1="24.765" x2="6.985" y2="23.495" width="0.254" layer="16"/>
 <via x="8.89" y="21.59" extent="1-16" drill="0.6"/>
 <wire x1="19.177" y1="6.35" x2="18.034" y2="6.35" width="0.254" layer="1"/>
@@
 <wire x1="37.553" y1="3.302" x2="37.553" y2="1.475" width="0.3048" layer="16"/>
 <wire x1="37.553" y1="1.475" x2="37.631" y2="1.397" width="0.3048" layer="16"/>
-<wire x1="6.35" y1="28.448" x2="6.35" y2="25.527" width="0.254" layer="16"/>
-<wire x1="6.35" y1="25.527" x2="6.096" y2="25.273" width="0.254" layer="16"/>
-<wire x1="6.096" y1="25.273" x2="6.096" y2="24.384" width="0.254" layer="16"/>
 <contactref element="IC1" pad="26"/>
 <wire x1="9.058" y1="29.119" x2="7.021" y2="29.119" width="0.254" layer="16"/>
+<wire x1="5.715" y1="24.765" x2="5.715" y2="27.813" width="0.254" layer="16"/>
 </signal>
 <signal name="ROT4_B">
@@
 <contactref element="LCD2" pad="RES"/>
 <wire x1="56.304" y1="27.94" x2="26.84" y2="27.94" width="0.254" layer="16"/>
-<wire x1="16.551" y1="27.219" x2="17.018" y2="27.686" width="0.254" layer="16"/>
-<via x="17.018" y="27.686" extent="1-16" drill="0.6"/>
-<wire x1="17.018" y1="27.686" x2="20.574" y2="27.686" width="0.254" layer="1"/>
-<wire x1="20.574" y1="27.686" x2="20.828" y2="27.94" width="0.254" layer="1"/>
+<via x="17.145" y="27.305" extent="1-16" drill="0.6"/>
 <wire x1="20.828" y1="27.94" x2="26.84" y2="27.94" width="0.254" layer="1"/>
 <contactref element="IC1" pad="13"/>
-<wire x1="15.958" y1="27.219" x2="16.551" y2="27.219" width="0.254" layer="16"/>
+<wire x1="15.958" y1="27.219" x2="17.059" y2="27.219" width="0.254" layer="16"/>
+<wire x1="17.059" y1="27.219" x2="17.145" y2="27.305" width="0.254" layer="16"/>
+<wire x1="17.145" y1="27.305" x2="20.193" y2="27.305" width="0.254" layer="1"/>
+<wire x1="20.193" y1="27.305" x2="20.828" y2="27.94" width="0.254" layer="1"/>
 </signal>
 <signal name="SPI1_CLK">
@@
 <contactref element="R6" pad="1"/>
 <contactref element="LED2" pad="A"/>
-<wire x1="18.63" y1="23.368" x2="20.84" y2="23.368" width="0.254" layer="16"/>
+<wire x1="18.63" y1="23.749" x2="20.713" y2="23.749" width="0.254" layer="16"/>
 </signal>
 <signal name="N$8">
@@
 <wire x1="46.394" y1="46.99" x2="46.394" y2="45.126" width="0.254" layer="16"/>
 <wire x1="46.394" y1="45.126" x2="46.442" y2="45.078" width="0.254" layer="16"/>
-<wire x1="46.394" y1="46.99" x2="46.394" y2="48.768" width="0" layer="19" extent="16-16"/>
+<wire x1="46.394" y1="46.99" x2="46.394" y2="48.768" width="0.254" layer="16"/>
 </signal>
 <signal name="N$17">
@@
 <contactref element="R23" pad="1"/>
 <contactref element="U2" pad="3"/>
-<wire x1="1.524" y1="54.229" x2="4.826" y2="54.229" width="0.254" layer="16"/>
-<wire x1="1.016" y1="53.721" x2="1.524" y2="54.229" width="0.254" layer="16"/>
+<wire x1="1.397" y1="54.61" x2="5.207" y2="54.61" width="0.254" layer="16"/>
 <wire x1="8.255" y1="57.658" x2="19.812" y2="57.658" width="0.254" layer="16"/>
 <wire x1="19.812" y1="57.658" x2="21.59" y2="59.436" width="0.254" layer="16"/>
@@
 <wire x1="27.96" y1="52.059" x2="27.96" y2="51.101" width="0.254" layer="16"/>
 <wire x1="27.96" y1="51.101" x2="26.958" y2="50.099" width="0.254" layer="16"/>
-<wire x1="4.826" y1="54.229" x2="8.255" y2="57.658" width="0.254" layer="16"/>
-<wire x1="1.016" y1="53.721" x2="1.016" y2="42.252" width="0.254" layer="16"/>
+<wire x1="5.207" y1="54.61" x2="8.255" y2="57.658" width="0.254" layer="16"/>
+<wire x1="0.381" y1="53.594" x2="0.381" y2="42.887" width="0.254" layer="16"/>
+<wire x1="0.381" y1="42.887" x2="1.016" y2="42.252" width="0.254" layer="16"/>
+<wire x1="1.397" y1="54.61" x2="0.381" y2="53.594" width="0.254" layer="16"/>
 </signal>
 <signal name="N$19">
@@
 <contactref element="R24" pad="1"/>
 <contactref element="U2" pad="2"/>
-<wire x1="1.524" y1="53.467" x2="1.778" y2="53.721" width="0.254" layer="16"/>
-<wire x1="1.778" y1="53.721" x2="4.953" y2="53.721" width="0.254" layer="16"/>
+<wire x1="1.651" y1="54.102" x2="5.334" y2="54.102" width="0.254" layer="16"/>
 <wire x1="8.382" y1="57.15" x2="20.066" y2="57.15" width="0.254" layer="16"/>
 <wire x1="20.066" y1="57.15" x2="21.844" y2="58.928" width="0.254" layer="16"/>
@@
 <wire x1="24.892" y1="50.927" x2="24.892" y2="50.133" width="0.254" layer="16"/>
 <wire x1="24.892" y1="50.133" x2="24.858" y2="50.099" width="0.254" layer="16"/>
-<wire x1="1.524" y1="53.467" x2="1.524" y2="43.522" width="0.254" layer="16"/>
-<wire x1="4.953" y1="53.721" x2="8.382" y2="57.15" width="0.254" layer="16"/>
-<wire x1="1.524" y1="43.522" x2="2.794" y2="42.252" width="0.254" layer="16"/>
+<wire x1="0.889" y1="44.157" x2="2.794" y2="42.252" width="0.254" layer="16"/>
+<wire x1="5.334" y1="54.102" x2="8.382" y2="57.15" width="0.254" layer="16"/>
+<wire x1="0.889" y1="53.34" x2="0.889" y2="44.157" width="0.254" layer="16"/>
+<wire x1="1.651" y1="54.102" x2="0.889" y2="53.34" width="0.254" layer="16"/>
 </signal>
 <signal name="USB_DM">

Commit message: wip
Parts:
- moved LED2 21.4 mm to (9.40, 41.4)
- moved R6 18.0 mm to (9.40, 39.6), turned to 180 degrees
Connections:
- new net N$6: IC1.38, R6.2
Routing:
- net N$6: track 0.00 -> 4.40 mm
Other:
- board text added: "Designed by"
- board text added: "Eran Rundstein"
- board text added: "ab-berry"
- board text added: "ver 2.0 - 2017"
- board text removed: "ab-berry v1.0 2016 Designed by Eran Rundstein"
Changed lines of the file:
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@@
 <grid distance="5" unitdist="mil" unit="mil" style="lines" multiple="1" display="no" altdistance="0.025" altunitdist="inch" altunit="inch"/>
 <layers>
-<layer number="1" name="Top" color="4" fill="1" visible="yes" active="yes"/>
+<layer number="1" name="Top" color="4" fill="1" visible="no" active="yes"/>
 <layer number="2" name="Route2" color="1" fill="3" visible="no" active="no"/>
 <layer number="3" name="Route3" color="4" fill="3" visible="no" active="no"/>
@@
 <layer number="14" name="Route14" color="1" fill="6" visible="no" active="no"/>
 <layer number="15" name="Route15" color="4" fill="6" visible="no" active="no"/>
-<layer number="16" name="Bottom" color="1" fill="1" visible="yes" active="yes"/>
+<layer number="16" name="Bottom" color="1" fill="1" visible="no" active="yes"/>
 <layer number="17" name="Pads" color="2" fill="1" visible="yes" active="yes"/>
 <layer number="18" name="Vias" color="2" fill="1" visible="yes" active="yes"/>
@@
 <layer number="20" name="Dimension" color="15" fill="1" visible="yes" active="yes"/>
 <layer number="21" name="tPlace" color="7" fill="1" visible="yes" active="yes"/>
-<layer number="22" name="bPlace" color="7" fill="1" visible="yes" active="yes"/>
+<layer number="22" name="bPlace" color="7" fill="1" visible="no" active="yes"/>
 <layer number="23" name="tOrigins" color="15" fill="1" visible="yes" active="yes"/>
-<layer number="24" name="bOrigins" color="15" fill="1" visible="yes" active="yes"/>
+<layer number="24" name="bOrigins" color="15" fill="1" visible="no" active="yes"/>
 <layer number="25" name="tNames" color="7" fill="1" visible="yes" active="yes"/>
-<layer number="26" name="bNames" color="7" fill="1" visible="yes" active="yes"/>
+<layer number="26" name="bNames" color="7" fill="1" visible="no" active="yes"/>
 <layer number="27" name="tValues" color="7" fill="1" visible="yes" active="yes"/>
-<layer number="28" name="bValues" color="7" fill="1" visible="yes" active="yes"/>
+<layer number="28" name="bValues" color="7" fill="1" visible="no" active="yes"/>
 <layer number="29" name="tStop" color="7" fill="3" visible="no" active="yes"/>
 <layer number="30" name="bStop" color="7" fill="6" visible="no" active="yes"/>
@@
 <layer number="50" name="dxf" color="7" fill="1" visible="yes" active="yes"/>
 <layer number="51" name="tDocu" color="7" fill="1" visible="yes" active="yes"/>
-<layer number="52" name="bDocu" color="7" fill="1" visible="yes" active="yes"/>
+<layer number="52" name="bDocu" color="7" fill="1" visible="no" active="yes"/>
 <layer number="53" name="tGND_GNDA" color="7" fill="9" visible="no" active="no"/>
 <layer number="54" name="bGND_GNDA" color="1" fill="9" visible="no" active="no"/>
@@
 <wire x1="58.42" y1="60.96" x2="0" y2="60.96" width="0" layer="20"/>
 <wire x1="0" y1="60.96" x2="0" y2="0" width="0" layer="20"/>
-<text x="40.259" y="46.609" size="0.762" layer="21" font="vector" rot="R180">ab-berry v1.0 2016
-Designed by Eran Rundstein</text>
+<text x="23.241" y="12.065" size="1.778" layer="21" font="vector">ab-berry</text>
+<text x="22.733" y="5.842" size="0.508" layer="21" font="vector">Designed by</text>
+<text x="23.114" y="4.318" size="1.016" layer="21" font="vector">Eran Rundstein</text>
+<text x="23.114" y="8.001" size="1.016" layer="21" font="vector">ver 2.0 - 2017</text>
 </plain>
 <attributes>
@@
 <elements>
 <element name="C1" library="microbuilder" package="0603" value="0.1uF" x="8.763" y="36.068" smashed="yes" rot="MR270">
-<attribute name="NAME" x="8.89" y="39.497" size="0.8128" layer="26" font="vector" ratio="18" rot="MR270"/>
-<attribute name="VALUE" x="9.525" y="39.497" size="0.4064" layer="28" font="vector" ratio="10" rot="MR270"/>
+<attribute name="NAME" x="7.747" y="35.814" size="0.8128" layer="26" font="vector" ratio="18" rot="MR270"/>
+<attribute name="VALUE" x="6.731" y="35.814" size="0.4064" layer="28" font="vector" ratio="10" rot="MR270"/>
 </element>
 <element name="C2" library="microbuilder" package="0603" value="0.1uF" x="18.161" y="36.703" rot="MR0"/>
@@
 <element name="R5" library="microbuilder" package="0603" value="330" x="50.673" y="39.37" rot="MR90"/>
 <element name="ROT1" library="keves" package="PEC111-4XXXK-SXXXX" value="PEC12R-4225F-S0024" x="14.478" y="8.89" smashed="yes">
-<attribute name="NAME" x="21.209" y="5.715" size="1.27" layer="25" rot="R270"/>
+<attribute name="NAME" x="26.289" y="2.794" size="1.27" layer="25" rot="R180"/>
 </element>
 <element name="LCD1" library="keves" package="SSD1306-7PIN-NO-HOLES" value="SSD1306-7PINWITHOUT-HOLES" x="32.004" y="30.48" rot="R270"/>
@@
 <element name="H4" library="holes" package="3,2" value="MOUNT-HOLE3.2" x="55.88" y="2.54"/>
 <element name="JP3" library="pinhead" package="1X02" value="" x="55.626" y="50.546" rot="MR90"/>
-<element name="R6" library="microbuilder" package="0603" value="330" x="17.78" y="23.749" rot="MR0"/>
-<element name="LED2" library="microbuilder" package="CHIPLED_0603" value="" x="21.463" y="23.749" rot="MR90"/>
+<element name="R6" library="microbuilder" package="0603" value="330" x="9.398" y="39.624" rot="MR180"/>
+<element name="LED2" library="microbuilder" package="CHIPLED_0603" value="" x="9.398" y="41.402" rot="MR90"/>
 <element name="C12" library="microbuilder" package="0603" value="18pF" x="24.257" y="33.782" rot="MR90"/>
 <element name="C13" library="microbuilder" package="0603" value="18pF" x="24.257" y="30.226" smashed="yes" rot="MR90">
@@
 </element>
 <element name="ROT4" library="keves" package="PEC111-4XXXK-SXXXX" value="PEC12R-4225F-S0024" x="43.942" y="8.89" smashed="yes">
-<attribute name="NAME" x="37.084" y="1.778" size="1.27" layer="25" rot="R90"/>
+<attribute name="NAME" x="31.877" y="1.778" size="1.27" layer="25"/>
 </element>
 <element name="R11" library="microbuilder" package="0603" value="10K" x="38.481" y="1.397" smashed="yes" rot="MR180">
@@
 </element>
 <element name="ROT2" library="keves" package="PEC111-4XXXK-SXXXX" value="PEC12R-4225F-S0024" x="14.478" y="52.578" smashed="yes">
-<attribute name="NAME" x="7.62" y="45.466" size="1.27" layer="25" rot="R90"/>
+<attribute name="NAME" x="21.717" y="45.974" size="1.27" layer="25"/>
 </element>
 <element name="R15" library="microbuilder" package="0603" value="10K" x="11.176" y="46.99" smashed="yes" rot="MR180">
@@
 </element>
 <element name="ROT3" library="keves" package="PEC111-4XXXK-SXXXX" value="PEC12R-4225F-S0024" x="43.942" y="52.578" smashed="yes">
-<attribute name="NAME" x="52.324" y="45.212" size="1.27" layer="25" rot="R90"/>
+<attribute name="NAME" x="32.512" y="45.847" size="1.27" layer="25"/>
 </element>
 <element name="R19" library="microbuilder" package="0603" value="10K" x="38.481" y="45.085" smashed="yes" rot="MR180">
@@
 <wire x1="5.334" y1="43.307" x2="6.096" y2="42.545" width="0.254" layer="16"/>
 <wire x1="6.096" y1="42.545" x2="6.096" y2="39.624" width="0.254" layer="16"/>
-<wire x1="6.096" y1="39.624" x2="6.477" y2="39.243" width="0.254" layer="16"/>
-<wire x1="6.477" y1="39.243" x2="8.89" y2="39.243" width="0.254" layer="16"/>
 <wire x1="5.334" y1="46.482" x2="5.334" y2="43.307" width="0.254" layer="16"/>
 <wire x1="4.064" y1="47.752" x2="5.334" y2="46.482" width="0.254" layer="16"/>
-<wire x1="10.458" y1="37.675" x2="8.89" y2="39.243" width="0.254" layer="16"/>
 <contactref element="IC1" pad="37"/>
-<wire x1="10.458" y1="37.675" x2="10.458" y2="35.519" width="0.254" layer="16"/>
+<wire x1="10.458" y1="37.802" x2="10.458" y2="35.519" width="0.254" layer="16"/>
+<wire x1="10.458" y1="37.802" x2="9.906" y2="38.354" width="0.254" layer="16"/>
+<wire x1="9.906" y1="38.354" x2="7.366" y2="38.354" width="0.254" layer="16"/>
+<wire x1="7.366" y1="38.354" x2="6.096" y2="39.624" width="0.254" layer="16"/>
 </signal>
 <signal name="RST">
@@
 <contactref element="R6" pad="1"/>
 <contactref element="LED2" pad="A"/>
-<wire x1="18.63" y1="23.749" x2="20.713" y2="23.749" width="0.254" layer="16"/>
+<wire x1="8.548" y1="39.624" x2="8.548" y2="41.302" width="0.254" layer="16"/>
+<wire x1="8.548" y1="41.302" x2="8.648" y2="41.402" width="0.254" layer="16"/>
 </signal>
 <signal name="N$8">
@@
 <wire x1="33.108" y1="54.647" x2="35.23" y2="56.769" width="0.254" layer="16"/>
 </signal>
+<signal name="N$6">
+<contactref element="IC1" pad="38"/>
+<contactref element="R6" pad="2"/>
+<wire x1="10.958" y1="35.519" x2="10.958" y2="38.914" width="0.254" layer="16"/>
+<wire x1="10.958" y1="38.914" x2="10.248" y2="39.624" width="0.254" layer="16"/>
+</signal>
 </signals>
 <errors>
@@
 </board>
 </drawing>
-<compatibility>
-<note version="6.3" minversion="6.2.2" severity="warning">
-Since Version 6.2.2 text objects can contain more than one line,
-which will not be processed correctly with this version.
-</note>
-</compatibility>
 </eagle>

Commit message: wip
Parts:
- added C23: 0.1uF, microbuilder:0603
- added IC2: AT45DB161D-SU, atmel:8S2
Connections:
- new net FLASH_CS: IC1.12, IC2.4
- new net SPI1_MISO: IC1.16, IC2.8
- net 3.3V: now also C23.1, IC2.3, IC2.5, IC2.6
- net GND: now also C23.2, IC2.7
- net SPI1_CLK: now also IC2.2
- net SPI1_MOSI: now also IC2.1
Routing:
- net SPI1_MISO: track 0.00 -> 44.1 mm, vias 0 -> 4
- net FLASH_CS: track 0.00 -> 30.6 mm, vias 0 -> 2
- net 3.3V: track 75.9 -> 85.3 mm, vias 20 -> 23
- net ROT4_B: track 54.2 -> 55.7 mm
- net SPI1_CLK: track 45.8 -> 46.9 mm
- net LCD_RST: track 40.6 -> 41.4 mm
- net SPI1_MOSI: track 44.8 -> 45.3 mm
