File: ab-berry/ab-berry-rev2.sch (EAGLE design)
At the start: 64 parts, among them IC1 STM32F302_F303_B_C_LQFP48, U1 LM1117MPX-3.3/NOPB or AP2114H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

Commit message: wip
Parts:
- added C22: 4.7nF, microbuilder:CAP_CERAMIC0603
- added R23, R24: 22, microbuilder:RESISTOR0603
- added R25: 1M, microbuilder:RESISTOR0603
- added U2: PRTR5V0U2X, Volks73-NXPSemiconductors:PRTR5V0U2X
- added X1: (no value), keves:TE-292304-1
- IC1: value STM32F302_F303_B_C_LQFP48 -> STM32F303CCT6
- LCD1, LCD2: value SSD1306-7PIN -> SSD1306-7PINWITHOUT-HOLES; device keves:SSD1306-7PIN -> keves:SSD1306-7PINWITHOUT-HOLES
Connections:
- removed net N$6: IC1.PB0, R6.2
- new net N$18: R23.1, U2U$1.IO2, X1_CONN.2
- new net N$19: R24.1, U2U$1.IO1, X1_CONN.3
- new net N$20: C22.P$1, R25.1, X1SHIELD.S1, X1SHIELD.S2
- new net USB_DM: IC1.PA11, R23.2
- new net USB_DP: IC1.PA12, R24.2
- net 5.0V: now also U2-SUPPLY.VCC, X1_CONN.1
- net CAN_RX: now also IC1.PB8; no longer IC1.PA11
- net CAN_TX: now also IC1.PB9; no longer IC1.PA12
- net GND: now also C22.P$2, R25.2, U2-SUPPLY.GND, X1_CONN.4
- net ROT3_B: no longer IC1.PB8
Changed lines of the file:
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@@
 <part name="U$16" library="microbuilder" deviceset="GND" device=""/>
 <part name="U$17" library="microbuilder" deviceset="GND" device=""/>
-<part name="LCD1" library="keves" deviceset="SSD1306-7PIN" device=""/>
+<part name="LCD1" library="keves" deviceset="SSD1306-7PIN" device="WITHOUT-HOLES"/>
 <part name="C10" library="microbuilder" deviceset="CAP_CERAMIC" device="0603" value="0.1uF"/>
 <part name="U$23" library="microbuilder" deviceset="GND" device=""/>
 <part name="U$24" library="microbuilder" deviceset="GND" device=""/>
 <part name="U$25" library="microbuilder" deviceset="3.3V" device=""/>
-<part name="LCD2" library="keves" deviceset="SSD1306-7PIN" device=""/>
+<part name="LCD2" library="keves" deviceset="SSD1306-7PIN" device="WITHOUT-HOLES"/>
 <part name="C11" library="microbuilder" deviceset="CAP_CERAMIC" device="0603" value="0.1uF"/>
 <part name="U$26" library="microbuilder" deviceset="GND" device=""/>
@@
 <part name="C8" library="SparkFun-Capacitors" deviceset="10UF-6.3V-20%(0603)(TANT)" device="&quot;" value="10uF TANT"/>
 <part name="C9" library="SparkFun-Capacitors" deviceset="10UF-6.3V-20%(0603)(TANT)" device="&quot;" value="10uF TANT"/>
-<part name="IC1" library="keves" deviceset="STM32F302_F303_B_C_LQFP48" device=""/>
+<part name="IC1" library="keves" deviceset="STM32F302_F303_B_C_LQFP48" device="" value="STM32F303CCT6"/>
+<part name="X1" library="keves" deviceset="TE-292304-1" device=""/>
+<part name="R23" library="microbuilder" deviceset="RESISTOR" device="0603" value="22"/>
+<part name="R24" library="microbuilder" deviceset="RESISTOR" device="0603" value="22"/>
+<part name="U$54" library="microbuilder" deviceset="5.0V" device=""/>
+<part name="U$55" library="microbuilder" deviceset="GND" device=""/>
+<part name="R25" library="microbuilder" deviceset="RESISTOR" device="0603" value="1M"/>
+<part name="C22" library="microbuilder" deviceset="CAP_CERAMIC" device="0603" value="4.7nF"/>
+<part name="U$56" library="microbuilder" deviceset="GND" device=""/>
+<part name="U2" library="Volks73-NXPSemiconductors" deviceset="PRTR5V0U2X?" device=""/>
+<part name="U$57" library="microbuilder" deviceset="GND" device=""/>
+<part name="U$58" library="microbuilder" deviceset="5.0V" device=""/>
 </parts>
 <sheets>
@@
 <instance part="C9" gate="G$1" x="-45.72" y="78.74"/>
 <instance part="IC1" gate="G$1" x="53.34" y="58.42"/>
+<instance part="X1" gate="_CONN" x="132.08" y="106.68"/>
+<instance part="X1" gate="SHIELD" x="132.08" y="109.22"/>
+<instance part="R23" gate="G$1" x="114.3" y="109.22" rot="R180"/>
+<instance part="R24" gate="G$1" x="101.6" y="106.68" rot="R180"/>
+<instance part="U$54" gate="G$1" x="129.54" y="121.92"/>
+<instance part="U$55" gate="G$1" x="129.54" y="96.52"/>
+<instance part="R25" gate="G$1" x="134.62" y="86.36" rot="R270"/>
+<instance part="C22" gate="G$1" x="142.24" y="86.36"/>
+<instance part="U$56" gate="G$1" x="134.62" y="76.2"/>
+<instance part="U2" gate="U$1" x="124.46" y="132.08" rot="R90"/>
+<instance part="U2" gate="-SUPPLY" x="104.14" y="132.08" rot="R180"/>
+<instance part="U$57" gate="G$1" x="104.14" y="147.32" rot="R180"/>
+<instance part="U$58" gate="G$1" x="104.14" y="116.84" rot="R180"/>
 </instances>
 <busses>
@@
 <pinref part="C21" gate="G$1" pin="P$2"/>
 <pinref part="U$51" gate="G$1" pin="GND"/>
+</segment>
+<segment>
+<pinref part="X1" gate="_CONN" pin="4"/>
+<pinref part="U$55" gate="G$1" pin="GND"/>
+<wire x1="129.54" y1="99.06" x2="129.54" y2="104.14" width="0.1524" layer="91"/>
+</segment>
+<segment>
+<pinref part="C22" gate="G$1" pin="P$2"/>
+<wire x1="142.24" y1="83.82" x2="142.24" y2="81.28" width="0.1524" layer="91"/>
+<pinref part="U$56" gate="G$1" pin="GND"/>
+<wire x1="142.24" y1="81.28" x2="134.62" y2="81.28" width="0.1524" layer="91"/>
+<wire x1="134.62" y1="81.28" x2="134.62" y2="78.74" width="0.1524" layer="91"/>
+<pinref part="R25" gate="G$1" pin="2"/>
+<junction x="134.62" y="81.28"/>
+</segment>
+<segment>
+<pinref part="U2" gate="-SUPPLY" pin="GND"/>
+<pinref part="U$57" gate="G$1" pin="GND"/>
 </segment>
 </net>
@@
 </segment>
 <segment>
-<wire x1="83.82" y1="55.88" x2="93.98" y2="55.88" width="0.1524" layer="91"/>
-<label x="91.44" y="55.88" size="1.778" layer="95"/>
-<pinref part="IC1" gate="G$1" pin="PA12"/>
+<pinref part="IC1" gate="G$1" pin="PB9"/>
+<wire x1="83.82" y1="17.78" x2="93.98" y2="17.78" width="0.1524" layer="91"/>
+<label x="91.44" y="17.78" size="1.778" layer="95"/>
 </segment>
 </net>
@@
 </segment>
 <segment>
-<wire x1="83.82" y1="58.42" x2="93.98" y2="58.42" width="0.1524" layer="91"/>
-<label x="91.44" y="58.42" size="1.778" layer="95"/>
-<pinref part="IC1" gate="G$1" pin="PA11"/>
+<wire x1="83.82" y1="20.32" x2="93.98" y2="20.32" width="0.1524" layer="91"/>
+<label x="91.44" y="20.32" size="1.778" layer="95"/>
+<pinref part="IC1" gate="G$1" pin="PB8"/>
 </segment>
 </net>
@@
 <junction x="-68.58" y="43.18"/>
 </segment>
+<segment>
+<pinref part="X1" gate="_CONN" pin="1"/>
+<pinref part="U$54" gate="G$1" pin="5.0V"/>
+<wire x1="129.54" y1="119.38" x2="129.54" y2="111.76" width="0.1524" layer="91"/>
+</segment>
+<segment>
+<pinref part="U2" gate="-SUPPLY" pin="VCC"/>
+<pinref part="U$58" gate="G$1" pin="5.0V"/>
+</segment>
 </net>
 <net name="ROT1_A" class="0">
@@
 <net name="ROT3_B" class="0">
 <segment>
-<wire x1="83.82" y1="20.32" x2="93.98" y2="20.32" width="0.1524" layer="91"/>
-<label x="91.44" y="20.32" size="1.778" layer="95"/>
-<pinref part="IC1" gate="G$1" pin="PB8"/>
-</segment>
-<segment>
 <pinref part="R20" gate="G$1" pin="1"/>
 <wire x1="-132.08" y1="5.08" x2="-144.78" y2="5.08" width="0.1524" layer="91"/>
@@
 <label x="91.44" y="38.1" size="1.778" layer="95"/>
 <pinref part="IC1" gate="G$1" pin="PB1"/>
-</segment>
-</net>
-<net name="N$6" class="0">
-<segment>
-<pinref part="R6" gate="G$1" pin="2"/>
-<wire x1="101.6" y1="40.64" x2="83.82" y2="40.64" width="0.1524" layer="91"/>
-<pinref part="IC1" gate="G$1" pin="PB0"/>
 </segment>
 </net>
@@
 </segment>
 </net>
+<net name="N$18" class="0">
+<segment>
+<pinref part="X1" gate="_CONN" pin="2"/>
+<pinref part="R23" gate="G$1" pin="1"/>
+<wire x1="119.38" y1="109.22" x2="124.46" y2="109.22" width="0.1524" layer="91"/>
+<pinref part="U2" gate="U$1" pin="IO2"/>
+<wire x1="124.46" y1="109.22" x2="129.54" y2="109.22" width="0.1524" layer="91"/>
+<wire x1="124.46" y1="121.92" x2="124.46" y2="109.22" width="0.1524" layer="91"/>
+<junction x="124.46" y="109.22"/>
+</segment>
+</net>
+<net name="N$19" class="0">
+<segment>
+<pinref part="X1" gate="_CONN" pin="3"/>
+<pinref part="R24" gate="G$1" pin="1"/>
+<wire x1="106.68" y1="106.68" x2="121.92" y2="106.68" width="0.1524" layer="91"/>
+<pinref part="U2" gate="U$1" pin="IO1"/>
+<wire x1="121.92" y1="106.68" x2="129.54" y2="106.68" width="0.1524" layer="91"/>
+<wire x1="121.92" y1="121.92" x2="121.92" y2="106.68" width="0.1524" layer="91"/>
+<junction x="121.92" y="106.68"/>
+</segment>
+</net>
+<net name="USB_DM" class="0">
+<segment>
+<pinref part="R23" gate="G$1" pin="2"/>
+<wire x1="109.22" y1="109.22" x2="81.28" y2="109.22" width="0.1524" layer="91"/>
+<label x="81.28" y="109.22" size="1.778" layer="95"/>
+</segment>
+<segment>
+<wire x1="83.82" y1="58.42" x2="93.98" y2="58.42" width="0.1524" layer="91"/>
+<label x="91.44" y="58.42" size="1.778" layer="95"/>
+<pinref part="IC1" gate="G$1" pin="PA11"/>
+</segment>
+</net>
+<net name="USB_DP" class="0">
+<segment>
+<pinref part="R24" gate="G$1" pin="2"/>
+<wire x1="96.52" y1="106.68" x2="81.28" y2="106.68" width="0.1524" layer="91"/>
+<label x="81.28" y="106.68" size="1.778" layer="95"/>
+</segment>
+<segment>
+<wire x1="83.82" y1="55.88" x2="93.98" y2="55.88" width="0.1524" layer="91"/>
+<label x="91.44" y="55.88" size="1.778" layer="95"/>
+<pinref part="IC1" gate="G$1" pin="PA12"/>
+</segment>
+</net>
+<net name="N$20" class="0">
+<segment>
+<pinref part="X1" gate="SHIELD" pin="S2"/>
+<pinref part="R25" gate="G$1" pin="1"/>
+<wire x1="132.08" y1="96.52" x2="134.62" y2="96.52" width="0.1524" layer="91"/>
+<wire x1="134.62" y1="96.52" x2="134.62" y2="91.44" width="0.1524" layer="91"/>
+<pinref part="C22" gate="G$1" pin="P$1"/>
+<wire x1="134.62" y1="91.44" x2="142.24" y2="91.44" width="0.1524" layer="91"/>
+<junction x="134.62" y="91.44"/>
+<pinref part="X1" gate="SHIELD" pin="S1"/>
+<junction x="134.62" y="96.52"/>
+</segment>
+</net>

Commit message: wip
Connections:
- net ROT3_B: now also IC1.PB0
Changed lines of the file:
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@@
 <label x="-152.4" y="5.08" size="1.778" layer="95"/>
+</segment>
+<segment>
+<pinref part="IC1" gate="G$1" pin="PB0"/>
+<wire x1="83.82" y1="40.64" x2="93.98" y2="40.64" width="0.1524" layer="91"/>
+<label x="91.44" y="40.64" size="1.778" layer="95"/>
 </segment>
 </net>

Commit message: wip
Connections:
- new net N$6: IC1.PA15, R6.2
Other:
- moved on the sheet: LED2, R6
Changed lines of the file:
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@@
 <instance part="U$31" gate="G$1" x="-71.12" y="58.42" rot="R90"/>
 <instance part="U$32" gate="G$1" x="-71.12" y="55.88" rot="R270"/>
-<instance part="R6" gate="G$1" x="106.68" y="40.64" rot="R180"/>
-<instance part="LED2" gate="G$1" x="119.38" y="40.64"/>
-<instance part="U$33" gate="G$1" x="129.54" y="40.64" rot="R90"/>
+<instance part="R6" gate="G$1" x="106.68" y="48.26" rot="R180"/>
+<instance part="LED2" gate="G$1" x="119.38" y="48.26"/>
+<instance part="U$33" gate="G$1" x="127" y="48.26" rot="R90"/>
 <instance part="C12" gate="G$1" x="12.7" y="20.32" rot="R90"/>
 <instance part="C13" gate="G$1" x="10.16" y="15.24" rot="R270"/>
@@
 <pinref part="LED2" gate="G$1" pin="C"/>
 <pinref part="U$33" gate="G$1" pin="GND"/>
-<wire x1="127" y1="40.64" x2="121.92" y2="40.64" width="0.1524" layer="91"/>
+<wire x1="124.46" y1="48.26" x2="121.92" y2="48.26" width="0.1524" layer="91"/>
 </segment>
 <segment>
@@
 <pinref part="R6" gate="G$1" pin="1"/>
 <pinref part="LED2" gate="G$1" pin="A"/>
-<wire x1="114.3" y1="40.64" x2="111.76" y2="40.64" width="0.1524" layer="91"/>
+<wire x1="114.3" y1="48.26" x2="111.76" y2="48.26" width="0.1524" layer="91"/>
 </segment>
 </net>
@@
 </segment>
 </net>
+<net name="N$6" class="0">
+<segment>
+<pinref part="IC1" gate="G$1" pin="PA15"/>
+<pinref part="R6" gate="G$1" pin="2"/>
+<wire x1="101.6" y1="48.26" x2="83.82" y2="48.26" width="0.1524" layer="91"/>
+</segment>
+</net>

Commit message: wip
Parts:
- added C23: 0.1uF, microbuilder:CAP_CERAMIC0603
- added IC2: AT45DB161D-SU, atmel:AT45DB161D-SU
Connections:
- new net FLASH_CS: IC1.PA2, IC2.!CS
- new net SPI1_MISO: IC1.PA6, IC2.SO
- net 3.3V: now also C23.P$1, IC2.!RESET, IC2.!WP, IC2.VCC
- net GND: now also C23.P$2, IC2.GND
- net SPI1_CLK: now also IC2.SCK
- net SPI1_MOSI: now also IC2.SI
Changed lines of the file:
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@@
 <part name="U$57" library="microbuilder" deviceset="GND" device=""/>
 <part name="U$58" library="microbuilder" deviceset="5.0V" device=""/>
+<part name="IC2" library="atmel" deviceset="AT45DB161D" device="-SU"/>
+<part name="C23" library="microbuilder" deviceset="CAP_CERAMIC" device="0603" value="0.1uF"/>
+<part name="U$59" library="microbuilder" deviceset="GND" device=""/>
+<part name="U$60" library="microbuilder" deviceset="GND" device=""/>
+<part name="U$61" library="microbuilder" deviceset="3.3V" device=""/>
+<part name="U$62" library="microbuilder" deviceset="3.3V" device=""/>
+<part name="U$63" library="microbuilder" deviceset="3.3V" device=""/>
 </parts>
 <sheets>
@@
 <instance part="U$57" gate="G$1" x="104.14" y="147.32" rot="R180"/>
 <instance part="U$58" gate="G$1" x="104.14" y="116.84" rot="R180"/>
+<instance part="IC2" gate="G$1" x="147.32" y="15.24"/>
+<instance part="C23" gate="G$1" x="160.02" y="30.48" rot="R180"/>
+<instance part="U$59" gate="G$1" x="160.02" y="38.1" rot="R180"/>
+<instance part="U$60" gate="G$1" x="165.1" y="10.16" rot="R90"/>
+<instance part="U$61" gate="G$1" x="165.1" y="20.32" rot="R270"/>
+<instance part="U$62" gate="G$1" x="116.84" y="15.24" rot="R90"/>
+<instance part="U$63" gate="G$1" x="116.84" y="20.32" rot="R90"/>
 </instances>
 <busses>
@@
 <pinref part="U2" gate="-SUPPLY" pin="GND"/>
 <pinref part="U$57" gate="G$1" pin="GND"/>
+</segment>
+<segment>
+<pinref part="IC2" gate="G$1" pin="GND"/>
+<pinref part="U$60" gate="G$1" pin="GND"/>
+<wire x1="162.56" y1="10.16" x2="160.02" y2="10.16" width="0.1524" layer="91"/>
+</segment>
+<segment>
+<pinref part="C23" gate="G$1" pin="P$2"/>
+<pinref part="U$59" gate="G$1" pin="GND"/>
+<wire x1="160.02" y1="33.02" x2="160.02" y2="35.56" width="0.1524" layer="91"/>
 </segment>
 </net>
@@
 <pinref part="U$53" gate="G$1" pin="3.3V"/>
 </segment>
+<segment>
+<pinref part="IC2" gate="G$1" pin="VCC"/>
+<pinref part="U$61" gate="G$1" pin="3.3V"/>
+<wire x1="162.56" y1="20.32" x2="160.02" y2="20.32" width="0.1524" layer="91"/>
+<pinref part="C23" gate="G$1" pin="P$1"/>
+<wire x1="160.02" y1="25.4" x2="160.02" y2="20.32" width="0.1524" layer="91"/>
+<junction x="160.02" y="20.32"/>
+</segment>
+<segment>
+<pinref part="IC2" gate="G$1" pin="!WP"/>
+<pinref part="U$62" gate="G$1" pin="3.3V"/>
+<wire x1="119.38" y1="15.24" x2="137.16" y2="15.24" width="0.1524" layer="91"/>
+</segment>
+<segment>
+<pinref part="IC2" gate="G$1" pin="!RESET"/>
+<pinref part="U$63" gate="G$1" pin="3.3V"/>
+<wire x1="119.38" y1="20.32" x2="137.16" y2="20.32" width="0.1524" layer="91"/>
+</segment>
 </net>
 <net name="SWDIO" class="0">
@@
 <pinref part="IC1" gate="G$1" pin="PA7"/>
 </segment>
+<segment>
+<pinref part="IC2" gate="G$1" pin="SI"/>
+<wire x1="137.16" y1="17.78" x2="124.46" y2="17.78" width="0.1524" layer="91"/>
+<label x="121.92" y="17.78" size="1.778" layer="95"/>
+</segment>
 </net>
 <net name="LCD_CS1" class="0">
@@
 <label x="91.44" y="73.66" size="1.778" layer="95"/>
 <pinref part="IC1" gate="G$1" pin="PA5"/>
+</segment>
+<segment>
+<pinref part="IC2" gate="G$1" pin="SCK"/>
+<wire x1="137.16" y1="12.7" x2="124.46" y2="12.7" width="0.1524" layer="91"/>
+<label x="121.92" y="12.7" size="1.778" layer="95"/>
 </segment>
 </net>
@@
 </segment>
 </net>
+<net name="FLASH_CS" class="0">
+<segment>
+<pinref part="IC2" gate="G$1" pin="!CS"/>
+<wire x1="137.16" y1="10.16" x2="124.46" y2="10.16" width="0.1524" layer="91"/>
+<label x="121.92" y="10.16" size="1.778" layer="95"/>
+</segment>
+<segment>
+<pinref part="IC1" gate="G$1" pin="PA2"/>
+<wire x1="83.82" y1="81.28" x2="93.98" y2="81.28" width="0.1524" layer="91"/>
+<label x="91.44" y="81.28" size="1.778" layer="95"/>
+</segment>
+</net>
+<net name="SPI1_MISO" class="0">
+<segment>
+<pinref part="IC2" gate="G$1" pin="SO"/>
+<wire x1="160.02" y1="17.78" x2="175.26" y2="17.78" width="0.1524" layer="91"/>
+<label x="172.72" y="17.78" size="1.778" layer="95"/>
+</segment>
+<segment>
+<pinref part="IC1" gate="G$1" pin="PA6"/>
+<wire x1="83.82" y1="71.12" x2="93.98" y2="71.12" width="0.1524" layer="91"/>
+<label x="91.44" y="71.12" size="1.778" layer="95"/>
+</segment>
+</net>
