File: ab-berry/ab-berry-rev2.sch (EAGLE design)
At the start: 72 parts, among them IC1 STM32F303CCT6, IC2 AT45DB161D-SU, U1 LM1117MPX-3.3/NOPB or AP2114H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, U2 PRTR5V0U2X

Commit message: ab-berry-rev 2.1 wip
Parts:
- removed R2, R3, R4: 0, microbuilder:RESISTOR0603
- removed USR: (no value), microbuilder:SWITCH_TACT_SMT
- added C24: 4.7nF, microbuilder:CAP_CERAMIC0603
- added CAN_TERM: (no value), pinhead+:PINHD-2X2SMT
- added R26, R27: 60 1%, microbuilder:RESISTOR0603
- D1: value SN65HVD232 -> SN65HVD230
Connections:
- removed net BTN_USR: IC1.PC13, USR.S
- removed net N$2: D1.RS, R2.1
- removed net N$4: D1.RXD, R3.1
- removed net N$5: D1.TXD, R4.1
- new net N$21: C24.P$2, D1.VREF, R26.2, R27.1
- new net N$22: CAN_TERMG$1.2, R27.2
- new net N$23: CAN_TERMG$2.2, R26.1
- net CAN_H: now also CAN_TERMG$1.1
- net CAN_L: now also CAN_TERMG$2.1
- net CAN_RX: now also D1.RXD; no longer R3.2
- net CAN_TX: now also D1.TXD; no longer R4.2
- net GND: now also C24.P$1, D1.RS; no longer R2.2, USR.P
- net ROT1_A: now also IC1.PB12; no longer IC1.PB14
- net ROT1_B: now also IC1.PB13; no longer IC1.PB15
- net ROT1_SW: now also IC1.PB15; no longer IC1.PB12
- net ROT4_A: now also IC1.PB14; no longer IC1.PB13

Commit message: ab-berry rev2.1 sent to macrofab
Parts:
- removed CAN_TERM: (no value), pinhead+:PINHD-2X2SMT
- removed JP1, JP2: (no value), keves:PINHD-1X4
- added TERM: (no value), pinhead:PINHD-2X2
- added X2, X3: 04-JST-B4B-XH-A, bt_con-jst-xh:04-JST-B4B-XH-A
Connections:
- removed net N$22: CAN_TERMG$1.2, R27.2
- removed net N$23: CAN_TERMG$2.2, R26.1
- new net N$4: R27.2, TERM.2
- new net N$5: R26.1, TERM.4
- net 5.0V: now also X2-1.1, X3-1.1; no longer JP1.1, JP2.1
- net CAN_H: now also TERM.1, X2-3.1, X3-3.1; no longer CAN_TERMG$1.1, JP1.3, JP2.3
- net CAN_L: now also TERM.3, X2-2.1, X3-2.1; no longer CAN_TERMG$2.1, JP1.2, JP2.2
- net GND: now also X2-4.1, X3-4.1; no longer JP1.4, JP2.4
- net N$10: now also ROT2.CH_B; no longer ROT1.CH_B
- net N$11: now also ROT2.CH_A; no longer ROT1.CH_A
- net N$14: now also ROT1.CH_B; no longer ROT2.CH_B
- net N$15: now also ROT1.CH_A; no longer ROT2.CH_A
- net ROT1_A: now also C18.P$1, IC1.PB4, R15.1; no longer C14.P$1, IC1.PB12, R7.1
- net ROT1_B: now also C19.P$1, IC1.PB5, R16.1; no longer C15.P$1, IC1.PB13, R8.1
- net ROT1_SW: now also IC1.PB3; no longer IC1.PB15
- net ROT2_A: now also C14.P$1, IC1.PB12, R7.1; no longer C18.P$1, IC1.PB4, R15.1
- net ROT2_B: now also C15.P$1, IC1.PB13, R8.1; no longer C19.P$1, IC1.PB5, R16.1
- net ROT2_SW: now also IC1.PB15; no longer IC1.PB3
Other:
- moved on the sheet: C24, C7, D1, R26, R27, ROT1, ROT2
