File: midimixer-channel/dac-eval.sch (EAGLE design)
At the start: 18 parts, among them IC1 NE5534AD

Commit message: wip
Parts:
- removed U$1: PCM4104, BurrBrownAudioParts:PCM4104
- added OUT1: NMJ4HFD2, pl-jacks:MONOSWS
- added R7: 100 0.1%, microbuilder:RESISTOR0603
- added R8: 2K 0.1%, microbuilder:RESISTOR0603
- C6, C8: value 10uF -> 4.7uF
Connections:
- removed net N$1: C1.P$1, C2.+
- removed net N$2: C1.P$2, C3.+
- new net N$12: OUT1.T, R7.2
- new net OUT1+: C1.P$2, C3.+, R8.1
- new net OUT1-: C1.P$1, C2.+, R8.2
- net AGND: now also OUT1.S, OUT1.SN
- net N$10: now also R7.1
- net N$8: now also IC1.+IN; no longer IC1.-IN
- net N$9: now also IC1.-IN; no longer IC1.+IN
Other:
- moved on the sheet: C5, C6, C7, C8, IC1

Commit message: dac wip
Parts:
- added C11, C21, C31: 22pF, microbuilder:CAP_CERAMIC0603
- added C12, C13, C22, C23, C32, C33: 100uF EMVE160ADA101MF55G, SparkFun-Capacitors:CAP_POLD
- added C14, C24, C34: 2200pF ECH-U1H222JX5, microbuilder:CAP_CERAMIC0805
- added C15, C17, C25, C27, C35, C37: 0.1uF, microbuilder:CAP_CERAMIC0603
- added C16, C18, C26, C28, C36, C38: 4.7uF, microbuilder:CAP_CERAMIC0603
- added C19, C20, C29, C30, C39, C40: 560pF ECH-U1H561JX5, microbuilder:CAP_CERAMIC0805
- added IC2, IC3, IC4: NE5534AD, linear:NE5534AD
- added OUT2, OUT3, OUT4: NMJ4HFD2, pl-jacks:MONOSWS
- added R10, R17, R18, R25, R26, R9: 604 0.1%, microbuilder:RESISTOR0603
- added R11, R12, R19, R20, R27, R28: 499 0.1%, microbuilder:RESISTOR0603
- added R13, R14, R21, R22, R29, R30: 1K 0.1%, microbuilder:RESISTOR0603
- added R15, R23, R31: 100 0.1%, microbuilder:RESISTOR0603
- added R16, R24, R32: 2K 0.1%, microbuilder:RESISTOR0603
Connections:
- new net N$1: C12.-, R9.1
- new net N$11: C14.P$1, R11.1, R14.1, R9.2
- new net N$13: C19.P$1, IC2.+IN, R12.2
- new net N$14: C20.P$2, IC2.-IN, R11.2
- new net N$15: C20.P$1, IC2.OUT, R14.2, R15.1
- new net N$16: OUT2.T, R15.2
- new net N$17: C22.-, R17.1
- new net N$18: C23.-, R18.1
- new net N$19: C24.P$2, R18.2, R20.1, R21.2
- new net N$2: C13.-, R10.1
- new net N$20: C24.P$1, R17.2, R19.1, R22.1
- new net N$21: C29.P$1, IC3.+IN, R20.2
- new net N$22: C30.P$2, IC3.-IN, R19.2
- new net N$23: C30.P$1, IC3.OUT, R22.2, R23.1
- new net N$24: OUT3.T, R23.2
- new net N$25: C32.-, R25.1
- new net N$26: C33.-, R26.1
- new net N$27: C34.P$2, R26.2, R28.1, R29.2
- new net N$28: C34.P$1, R25.2, R27.1, R30.1
- new net N$29: C39.P$1, IC4.+IN, R28.2
- new net N$30: C40.P$2, IC4.-IN, R27.2
- new net N$31: C40.P$1, IC4.OUT, R30.2, R31.1
- new net N$32: OUT4.T, R31.2
- new net N$7: C14.P$2, R10.2, R12.1, R13.2
- new net OUT2+: C11.P$2, C13.+, R16.1
- new net OUT2-: C11.P$1, C12.+, R16.2
- new net OUT3+: C21.P$2, C23.+, R24.1
- new net OUT3-: C21.P$1, C22.+, R24.2
- new net OUT4+: C31.P$2, C33.+, R32.1
- new net OUT4-: C31.P$1, C32.+, R32.2
- net +12V: now also C15.P$1, C16.P$1, C25.P$1, C26.P$1, C35.P$1, C36.P$1, IC2.V+, IC3.V+, IC4.V+
- net -12V: now also C17.P$2, C18.P$2, C27.P$2, C28.P$2, C37.P$2, C38.P$2, IC2.V-, IC3.V-, IC4.V-
- net AGND: now also C15.P$2, C16.P$2, C17.P$1, C18.P$1, C19.P$2, C25.P$2, C26.P$2, C27.P$1, C28.P$1, C29.P$2, C35.P$2, C36.P$2, C37.P$1, C38.P$1, C39.P$2, OUT2.S, OUT2.SN, OUT3.S, OUT3.SN, OUT4.S, OUT4.SN, R13.1, R21.1, R29.1

Commit message: dac wip
Parts:
- added C41, C42, C49, C50, C52: 0.1uF, microbuilder:CAP_CERAMIC0603
- added C43, C44, C45, C46: 0.01uF, microbuilder:CAP_CERAMIC0603
- added C47, C48, C51: 4.7uF, microbuilder:CAP_CERAMIC0603
- added DAC: PCM4104, BurrBrownAudioParts:PCM4104
- added JP1: (no value), pinhead:PINHD-2X4
- added JP2: (no value), pinhead:PINHD-2X5
- added R33, R34, R35, R36, R37, R38, R39, R40, R41, R42: 10K, microbuilder:RESISTOR0603
- added S1: SWS010, smd-special:SWS010
- added SW1: 76SB10ST, special:SW_DIP-10
Connections:
- new net 3.3V: C51.P$1, C52.P$1, DAC.VDD, R33.2, R34.2, R35.2, R36.2, R37.2, R38.2, R39.2, R40.2, R41.2, R42.2
- new net AVCC: C43.P$1, C44.P$1, C45.P$1, C46.P$1, C47.P$2, C48.P$2, C49.P$2, C50.P$2, DAC.VCC1, DAC.VCC2, DAC.VREF1+, DAC.VREF2+, DAC.VREF3+, DAC.VREF4+
- new net DAC_CLK: JP1.3
- new net DAC_CS: JP1.1
- new net DAC_MISO: JP1.7
- new net DAC_MOSI: JP1.5
- new net DAC_RST: DAC.RST_, R41.1
- new net GND: C51.P$2, C52.P$2, DAC.DGND, DAC.N/C1, DAC.N/C2, DAC.N/C3, DAC.N/C4, DAC.SUB, SW1.11, SW1.12, SW1.13, SW1.14, SW1.15, SW1.16, SW1.17, SW1.18, SW1.19, SW1.20
- new net N$33: C41.P$2, DAC.VCOM1
- new net N$34: C42.P$2, DAC.VCOM2
- new net N$35: DAC.CS_, JP1.2
- new net N$36: DAC.CCLK, JP1.4
- new net N$37: DAC.CDIN, JP1.6
- new net N$38: DAC.CDOUT, JP1.8
- new net N$39: DAC.SCKI, JP2.2
- new net N$40: DAC.BCK, JP2.4
- new net N$41: DAC.LRCK, JP2.6
- new net N$42: DAC.DATA0, JP2.8
- new net N$43: DAC.DATA1, JP2.10
- new net N$44: DAC.FS1, R42.1, SW1.1
- new net N$45: DAC.FS0, R40.1, SW1.2
- new net N$46: DAC.FMT2, R39.1, SW1.3
- new net N$47: DAC.FMT1, R38.1, SW1.4
- new net N$48: DAC.FMT0, R37.1, SW1.5
- new net N$49: DAC.DEM1, R36.1, SW1.6
- new net N$50: DAC.DEM0, R35.1, SW1.7
- new net N$51: DAC.MUTE, R34.1, SW1.8
- new net N$52: DAC.MODE, R33.1, SW1.9
- new net SAI_BCK: JP2.3
- new net SAI_D0: JP2.7
- new net SAI_D1: JP2.9
- new net SAI_LRCK: JP2.5
- new net SAI_SCK: JP2.1
- net AGND: now also C41.P$1, C42.P$1, C43.P$2, C44.P$2, C45.P$2, C46.P$2, C47.P$1, C48.P$1, C49.P$1, C50.P$1, DAC.AGND1, DAC.AGND2, DAC.VREF1-, DAC.VREF2-, DAC.VREF3-, DAC.VREF4-
- net OUT1+: now also DAC.VOUT1+
- net OUT1-: now also DAC.VOUT1-
- net OUT2+: now also DAC.VOUT2+
- net OUT2-: now also DAC.VOUT2-
- net OUT3+: now also DAC.VOUT3+
- net OUT3-: now also DAC.VOUT3-
- net OUT4+: now also DAC.VOUT4+
- net OUT4-: now also DAC.VOUT4-
Other:
- note added: "TODOs: - AVCC Supply - +/-12V Supply - Connect AGND to GND"

Commit message: dac wip
Parts:
- removed S1: SWS010, smd-special:SWS010
- R16, R24, R32, R8: value 2K 0.1% -> 2K 0.1% DNP
Changed lines of the file:
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@@
 <part name="OUT1" library="pl-jacks" deviceset="MONOSW" device="S" value="NMJ4HFD2"/>
 <part name="U$6" library="microbuilder" deviceset="AGND" device=""/>
-<part name="R8" library="microbuilder" deviceset="RESISTOR" device="0603" value="2K 0.1%"/>
+<part name="R8" library="microbuilder" deviceset="RESISTOR" device="0603" value="2K 0.1% DNP"/>
 <part name="C11" library="microbuilder" deviceset="CAP_CERAMIC" device="0603" value="22pF"/>
 <part name="C12" library="SparkFun-Capacitors" deviceset="CAP_POL" device="D" value="100uF EMVE160ADA101MF55G"/>
@@
 <part name="OUT2" library="pl-jacks" deviceset="MONOSW" device="S" value="NMJ4HFD2"/>
 <part name="U$10" library="microbuilder" deviceset="AGND" device=""/>
-<part name="R16" library="microbuilder" deviceset="RESISTOR" device="0603" value="2K 0.1%"/>
+<part name="R16" library="microbuilder" deviceset="RESISTOR" device="0603" value="2K 0.1% DNP"/>
 <part name="C21" library="microbuilder" deviceset="CAP_CERAMIC" device="0603" value="22pF"/>
 <part name="C22" library="SparkFun-Capacitors" deviceset="CAP_POL" device="D" value="100uF EMVE160ADA101MF55G"/>
@@
 <part name="OUT3" library="pl-jacks" deviceset="MONOSW" device="S" value="NMJ4HFD2"/>
 <part name="U$15" library="microbuilder" deviceset="AGND" device=""/>
-<part name="R24" library="microbuilder" deviceset="RESISTOR" device="0603" value="2K 0.1%"/>
+<part name="R24" library="microbuilder" deviceset="RESISTOR" device="0603" value="2K 0.1% DNP"/>
 <part name="C31" library="microbuilder" deviceset="CAP_CERAMIC" device="0603" value="22pF"/>
 <part name="C32" library="SparkFun-Capacitors" deviceset="CAP_POL" device="D" value="100uF EMVE160ADA101MF55G"/>
@@
 <part name="OUT4" library="pl-jacks" deviceset="MONOSW" device="S" value="NMJ4HFD2"/>
 <part name="U$20" library="microbuilder" deviceset="AGND" device=""/>
-<part name="R32" library="microbuilder" deviceset="RESISTOR" device="0603" value="2K 0.1%"/>
+<part name="R32" library="microbuilder" deviceset="RESISTOR" device="0603" value="2K 0.1% DNP"/>
 <part name="DAC" library="BurrBrownAudioParts" deviceset="PCM4104" device=""/>
 <part name="C41" library="microbuilder" deviceset="CAP_CERAMIC" device="0603" value="0.1uF"/>
@@
 <part name="JP1" library="pinhead" deviceset="PINHD-2X4" device=""/>
 <part name="JP2" library="pinhead" deviceset="PINHD-2X5" device=""/>
-<part name="S1" library="smd-special" deviceset="SWS010" device=""/>
 <part name="SW1" library="special" deviceset="SW_DIP-10" device="" value="76SB10ST"/>
 <part name="U$21" library="microbuilder" deviceset="GND" device=""/>
@@
 <part name="R42" library="microbuilder" deviceset="RESISTOR" device="0603" value="10K"/>
 <part name="U$40" library="microbuilder" deviceset="3.3V" device=""/>
+<part name="U$41" library="microbuilder" deviceset="AGND" device=""/>
 </parts>
 <sheets>
@@
 <instance part="JP1" gate="A" x="-27.94" y="45.72"/>
 <instance part="JP2" gate="A" x="-27.94" y="63.5"/>
-<instance part="S1" gate="G$1" x="27.94" y="129.54"/>
 <instance part="SW1" gate="G$1" x="-35.56" y="91.44"/>
 <instance part="U$21" gate="G$1" x="-50.8" y="78.74" rot="R270"/>
@@
 <instance part="R42" gate="G$1" x="-17.78" y="116.84" rot="R90"/>
 <instance part="U$40" gate="G$1" x="5.08" y="127"/>
+<instance part="U$41" gate="G$1" x="76.2" y="88.9"/>
 </instances>
 <busses>
@@
 <segment>
 <pinref part="DAC" gate="G$1" pin="RST_"/>
-<wire x1="5.08" y1="101.6" x2="-12.7" y2="101.6" width="0.1524" layer="91"/>
+<wire x1="5.08" y1="101.6" x2="-25.4" y2="101.6" width="0.1524" layer="91"/>
 <label x="-12.7" y="101.6" size="1.778" layer="95"/>
 <pinref part="R41" gate="G$1" pin="1"/>
