File: midimixer-channel/dac-eval.brd (EAGLE design)
At the start: 100 x 80 mm, 18 parts, among them IC1 NE5534AD

Commit message: wip
Parts:
- removed U$1: PCM4104, BurrBrownAudioParts:SQFP-S-7X7-48
- added OUT1: NMJ4HFD2, pl-jacks:NMJ4HC-S
- added R7: 100 0.1%, microbuilder:0603
- added R8: 2K 0.1%, microbuilder:0603
- C6, C8: value 10uF -> 4.7uF
Connections:
- removed net N$1: C1.1, C2.+
- removed net N$2: C1.2, C3.+
- removed net VDD: U$1.19
- new net N$12: OUT1.T, R7.2
- new net OUT1+: C1.2, C3.+, R8.1
- new net OUT1-: C1.1, C2.+, R8.2
- net AGND: now also OUT1.S, OUT1.SN
- net N$10: now also R7.1
- net N$8: now also IC1.3; no longer IC1.2
- net N$9: now also IC1.2; no longer IC1.3
Changed lines of the file:
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@@
 </autorouter>
 <elements>
-<element name="U$1" library="BurrBrownAudioParts" package="SQFP-S-7X7-48" value="PCM4104" x="-20.32" y="6.35"/>
 <element name="C1" library="microbuilder" package="0603" value="22pF" x="-25.4" y="-1.27"/>
 <element name="C2" library="SparkFun-Capacitors" package="PANASONIC_D" value="100uF EMVE160ADA101MF55G" x="-22.86" y="-6.35"/>
@@
 <element name="IC1" library="linear" package="SO08" value="NE5534AD" x="-33.02" y="-29.21"/>
 <element name="C5" library="microbuilder" package="0603" value="0.1uF" x="-35.56" y="-34.29"/>
-<element name="C6" library="microbuilder" package="0603" value="10uF" x="-35.56" y="-36.83"/>
+<element name="C6" library="microbuilder" package="0603" value="4.7uF" x="-35.56" y="-36.83"/>
 <element name="C7" library="microbuilder" package="0603" value="0.1uF" x="-35.56" y="-39.37"/>
-<element name="C8" library="microbuilder" package="0603" value="10uF" x="-35.56" y="-41.91"/>
+<element name="C8" library="microbuilder" package="0603" value="4.7uF" x="-35.56" y="-41.91"/>
 <element name="C9" library="microbuilder" package="0805" value="560pF ECH-U1H561JX5" x="-34.29" y="-44.45"/>
 <element name="C10" library="microbuilder" package="0805" value="560pF ECH-U1H561JX5" x="-34.29" y="-46.99"/>
 <element name="R6" library="microbuilder" package="0603" value="1K 0.1%" x="-35.56" y="-49.53"/>
+<element name="R7" library="microbuilder" package="0603" value="100 0.1%" x="-35.56" y="-52.07"/>
+<element name="OUT1" library="pl-jacks" package="NMJ4HC-S" value="NMJ4HFD2" x="-21.59" y="-63.5"/>
+<element name="R8" library="microbuilder" package="0603" value="2K 0.1%" x="-35.56" y="-74.93"/>
 </elements>
 <signals>
-<signal name="VDD">
-<contactref element="U$1" pad="19"/>
-</signal>
-<signal name="N$1">
+<signal name="OUT1-">
 <contactref element="C2" pad="+"/>
 <contactref element="C1" pad="1"/>
+<contactref element="R8" pad="2"/>
+<wire x1="-20.46" y1="-6.35" x2="-34.71" y2="-74.93" width="0" layer="19" extent="1-1"/>
 <wire x1="-26.25" y1="-1.27" x2="-20.46" y2="-6.35" width="0" layer="19" extent="1-1"/>
 </signal>
-<signal name="N$2">
+<signal name="OUT1+">
 <contactref element="C3" pad="+"/>
 <contactref element="C1" pad="2"/>
+<contactref element="R8" pad="1"/>
+<wire x1="-20.46" y1="-13.97" x2="-36.41" y2="-74.93" width="0" layer="19" extent="1-1"/>
 <wire x1="-24.55" y1="-1.27" x2="-20.46" y2="-13.97" width="0" layer="19" extent="1-1"/>
 </signal>
@@
 <contactref element="C8" pad="1"/>
 <contactref element="C9" pad="2"/>
+<contactref element="OUT1" pad="SN"/>
+<contactref element="OUT1" pad="S"/>
+<wire x1="-16.51" y1="-55.385" x2="-16.51" y2="-71.615" width="0" layer="19" extent="1-1"/>
+<wire x1="-33.34" y1="-44.45" x2="-16.51" y2="-55.385" width="0" layer="19" extent="1-1"/>
+<wire x1="-36.41" y1="-41.91" x2="-33.34" y2="-44.45" width="0" layer="19" extent="1-1"/>
 <wire x1="-36.41" y1="-39.37" x2="-36.41" y2="-41.91" width="0" layer="19" extent="1-1"/>
 <wire x1="-34.71" y1="-36.83" x2="-36.41" y2="-39.37" width="0" layer="19" extent="1-1"/>
 <wire x1="-34.71" y1="-34.29" x2="-34.71" y2="-36.83" width="0" layer="19" extent="1-1"/>
-<wire x1="-33.34" y1="-44.45" x2="-36.41" y2="-41.91" width="0" layer="19" extent="1-1"/>
 <wire x1="-26.25" y1="-31.75" x2="-34.71" y2="-34.29" width="0" layer="19" extent="1-1"/>
 </signal>
 <signal name="N$8">
 <contactref element="R4" pad="2"/>
-<contactref element="IC1" pad="2"/>
 <contactref element="C9" pad="1"/>
-<wire x1="-33.655" y1="-31.81" x2="-35.24" y2="-44.45" width="0" layer="19" extent="1-1"/>
-<wire x1="-24.55" y1="-29.21" x2="-33.655" y2="-31.81" width="0" layer="19" extent="1-1"/>
+<contactref element="IC1" pad="3"/>
+<wire x1="-32.385" y1="-31.81" x2="-35.24" y2="-44.45" width="0" layer="19" extent="1-1"/>
+<wire x1="-24.55" y1="-29.21" x2="-32.385" y2="-31.81" width="0" layer="19" extent="1-1"/>
 </signal>
 <signal name="N$9">
 <contactref element="R3" pad="2"/>
-<contactref element="IC1" pad="3"/>
 <contactref element="C10" pad="2"/>
-<wire x1="-32.385" y1="-31.81" x2="-33.34" y2="-46.99" width="0" layer="19" extent="1-1"/>
-<wire x1="-24.55" y1="-26.67" x2="-32.385" y2="-31.81" width="0" layer="19" extent="1-1"/>
+<contactref element="IC1" pad="2"/>
+<wire x1="-33.655" y1="-31.81" x2="-33.34" y2="-46.99" width="0" layer="19" extent="1-1"/>
+<wire x1="-24.55" y1="-26.67" x2="-33.655" y2="-31.81" width="0" layer="19" extent="1-1"/>
 </signal>
 <signal name="+12V">
-<contactref element="IC1" pad="7"/>
 <contactref element="C6" pad="1"/>
 <contactref element="C5" pad="1"/>
+<contactref element="IC1" pad="7"/>
 <wire x1="-36.41" y1="-34.29" x2="-36.41" y2="-36.83" width="0" layer="19" extent="1-1"/>
 <wire x1="-33.655" y1="-26.61" x2="-36.41" y2="-34.29" width="0" layer="19" extent="1-1"/>
 </signal>
 <signal name="-12V">
-<contactref element="IC1" pad="4"/>
 <contactref element="C7" pad="2"/>
 <contactref element="C8" pad="2"/>
+<contactref element="IC1" pad="4"/>
 <wire x1="-34.71" y1="-39.37" x2="-34.71" y2="-41.91" width="0" layer="19" extent="1-1"/>
 <wire x1="-31.115" y1="-31.81" x2="-34.71" y2="-39.37" width="0" layer="19" extent="1-1"/>
 </signal>
 <signal name="N$10">
-<contactref element="IC1" pad="6"/>
 <contactref element="C10" pad="1"/>
 <contactref element="R6" pad="2"/>
+<contactref element="R7" pad="1"/>
+<contactref element="IC1" pad="6"/>
+<wire x1="-34.71" y1="-49.53" x2="-36.41" y2="-52.07" width="0" layer="19" extent="1-1"/>
 <wire x1="-35.24" y1="-46.99" x2="-34.71" y2="-49.53" width="0" layer="19" extent="1-1"/>
 <wire x1="-32.385" y1="-26.61" x2="-35.24" y2="-46.99" width="0" layer="19" extent="1-1"/>
 </signal>
+<signal name="N$12">
+<contactref element="R7" pad="2"/>
+<contactref element="OUT1" pad="T"/>
+<wire x1="-29.21" y1="-55.385" x2="-34.71" y2="-52.07" width="0" layer="19" extent="1-1"/>
+</signal>
 </signals>

Commit message: dac wip
Parts:
- moved R8 117.4 mm to (48.5, 6.99), turned to 270 degrees
- moved R7 89.1 mm to (27.2, 11.2), turned to 90 degrees
- moved C9 87.2 mm to (33.0, 11.0), turned to 90 degrees
- moved C8 84.9 mm to (30.0, 12.1)
- moved R6 84.4 mm to (31.0, 2.41), turned to 90 degrees
- moved C10 84.0 mm to (33.0, 3.30), turned to 90 degrees
- moved C7 82.2 mm to (30.0, 10.3)
- moved OUT1 80.0 mm to (11.7, 9.27)
- moved R5 75.1 mm to (35.9, 11.6), turned to 180 degrees
- moved C6 72.5 mm to (25.9, 1.65)
- moved C1 72.5 mm to (46.6, 6.86), turned to 90 degrees
- moved C5 72.1 mm to (25.9, 3.43)
- moved IC1 70.7 mm to (27.8, 6.86), turned to 90 degrees
- moved R4 70.0 mm to (33.9, 8.00), turned to 180 degrees
- moved C4 69.6 mm to (36.8, 7.11), turned to 90 degrees
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Routing:
- net N$12: track 0.00 -> 25.3 mm
- net N$10: track 0.00 -> 13.8 mm
- net N$6: track 0.00 -> 11.5 mm
- net AGND: track 0.00 -> 11.4 mm, vias 0 -> 4
- net +12V: track 0.00 -> 8.45 mm
- net OUT1+: track 0.00 -> 5.76 mm
- net N$5: track 0.00 -> 5.74 mm
- net OUT1-: track 0.00 -> 5.13 mm
- net N$8: track 0.00 -> 4.97 mm
- net N$9: track 0.00 -> 4.63 mm
- net -12V: track 0.00 -> 3.47 mm
- net N$4: track 0.00 -> 3.16 mm
- net N$3: track 0.00 -> 3.06 mm
- added copper zone on layer 16, net AGND

Commit message: dac wip
Parts:
- added C11, C21, C31: 22pF, microbuilder:0603
- added C12, C13, C22, C23, C32, C33: 100uF EMVE160ADA101MF55G, SparkFun-Capacitors:PANASONIC_D
- added C14, C24, C34: 2200pF ECH-U1H222JX5, microbuilder:0805
- added C15, C17, C25, C27, C35, C37: 0.1uF, microbuilder:0603
- added C16, C18, C26, C28, C36, C38: 4.7uF, microbuilder:0603
- added C19, C20, C29, C30, C39, C40: 560pF ECH-U1H561JX5, microbuilder:0805
- added IC2, IC3, IC4: NE5534AD, linear:SO08
- added OUT2, OUT3, OUT4: NMJ4HFD2, pl-jacks:NMJ4HC-S
- added R10, R17, R18, R25, R26, R9: 604 0.1%, microbuilder:0603
- added R11, R12, R19, R20, R27, R28: 499 0.1%, microbuilder:0603
- added R13, R14, R21, R22, R29, R30: 1K 0.1%, microbuilder:0603
- added R15, R23, R31: 100 0.1%, microbuilder:0603
- added R16, R24, R32: 2K 0.1%, microbuilder:0603
Connections:
- new net N$1: C12.-, R9.1
- new net N$11: C14.1, R11.1, R14.1, R9.2
- new net N$13: C19.1, IC2.3, R12.2
- new net N$14: C20.2, IC2.2, R11.2
- new net N$15: C20.1, IC2.6, R14.2, R15.1
- new net N$16: OUT2.T, R15.2
- new net N$17: C22.-, R17.1
- new net N$18: C23.-, R18.1
- new net N$19: C24.2, R18.2, R20.1, R21.2
- new net N$2: C13.-, R10.1
- new net N$20: C24.1, R17.2, R19.1, R22.1
- new net N$21: C29.1, IC3.3, R20.2
- new net N$22: C30.2, IC3.2, R19.2
- new net N$23: C30.1, IC3.6, R22.2, R23.1
- new net N$24: OUT3.T, R23.2
- new net N$25: C32.-, R25.1
- new net N$26: C33.-, R26.1
- new net N$27: C34.2, R26.2, R28.1, R29.2
- new net N$28: C34.1, R25.2, R27.1, R30.1
- new net N$29: C39.1, IC4.3, R28.2
- new net N$30: C40.2, IC4.2, R27.2
- new net N$31: C40.1, IC4.6, R30.2, R31.1
- new net N$32: OUT4.T, R31.2
- new net N$7: C14.2, R10.2, R12.1, R13.2
- new net OUT2+: C11.2, C13.+, R16.1
- new net OUT2-: C11.1, C12.+, R16.2
- new net OUT3+: C21.2, C23.+, R24.1
- new net OUT3-: C21.1, C22.+, R24.2
- new net OUT4+: C31.2, C33.+, R32.1
- new net OUT4-: C31.1, C32.+, R32.2
- net +12V: now also C15.1, C16.1, C25.1, C26.1, C35.1, C36.1, IC2.7, IC3.7, IC4.7
- net -12V: now also C17.2, C18.2, C27.2, C28.2, C37.2, C38.2, IC2.4, IC3.4, IC4.4
- net AGND: now also C15.2, C16.2, C17.1, C18.1, C19.2, C25.2, C26.2, C27.1, C28.1, C29.2, C35.2, C36.2, C37.1, C38.1, C39.2, OUT2.S, OUT2.SN, OUT3.S, OUT3.SN, OUT4.S, OUT4.SN, R13.1, R21.1, R29.1
Routing:
- net -12V: track 3.47 -> 128.8 mm
- net +12V: track 8.45 -> 118.3 mm, vias 0 -> 4
- net AGND: track 11.4 -> 45.7 mm, vias 4 -> 16
- net N$16: track 0.00 -> 25.3 mm, vias 0 -> 1
- net N$32: track 0.00 -> 25.3 mm, vias 0 -> 1
- net N$24: track 0.00 -> 25.3 mm, vias 0 -> 1
- net N$31: track 0.00 -> 13.8 mm
- net N$23: track 0.00 -> 13.8 mm
- net N$15: track 0.00 -> 13.8 mm
- net N$20: track 0.00 -> 11.5 mm
- net N$11: track 0.00 -> 11.5 mm
- net N$28: track 0.00 -> 11.5 mm
- net OUT4+: track 0.00 -> 5.76 mm
- net OUT3+: track 0.00 -> 5.76 mm
- net OUT2+: track 0.00 -> 5.76 mm
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
Commit message: dac wip
Parts:
- added C41, C42, C49, C50, C52: 0.1uF, microbuilder:0603
- added C43, C44, C45, C46: 0.01uF, microbuilder:0603
- added C47, C48, C51: 4.7uF, microbuilder:0603
- added DAC: PCM4104, BurrBrownAudioParts:SQFP-S-7X7-48
- added JP1: (no value), pinhead:2X04
- added JP2: (no value), pinhead:2X05
- added R33, R34, R35, R36, R37, R38, R39, R40, R41, R42: 10K, microbuilder:0603
- added S1: SWS010, smd-special:SMS-010
- added SW1: 76SB10ST, special:EDG-10
Connections:
- new net 3.3V: C51.1, C52.1, DAC.19, R33.2, R34.2, R35.2, R36.2, R37.2, R38.2, R39.2, R40.2, R41.2, R42.2
- new net AVCC: C43.1, C44.1, C45.1, C46.1, C47.2, C48.2, C49.2, C50.2, DAC.32, DAC.40, DAC.41, DAC.44, DAC.45, DAC.5
- new net DAC_CLK: JP1.3
- new net DAC_CS: JP1.1
- new net DAC_MISO: JP1.7
- new net DAC_MOSI: JP1.5
- new net DAC_RST: DAC.9, R41.1
- new net GND: C51.2, C52.2, DAC.13, DAC.20, DAC.30, DAC.31, DAC.6, DAC.7, SW1.11, SW1.12, SW1.13, SW1.14, SW1.15, SW1.16, SW1.17, SW1.18, SW1.19, SW1.20
- new net N$33: C41.2, DAC.48
- new net N$34: C42.2, DAC.37
- new net N$35: DAC.21, JP1.2
- new net N$36: DAC.22, JP1.4
- new net N$37: DAC.23, JP1.6
- new net N$38: DAC.24, JP1.8
- new net N$39: DAC.14, JP2.2
- new net N$40: DAC.15, JP2.4
- new net N$41: DAC.16, JP2.6
- new net N$42: DAC.17, JP2.8
- new net N$43: DAC.18, JP2.10
- new net N$44: DAC.29, R42.1, SW1.1
- new net N$45: DAC.28, R40.1, SW1.2
- new net N$46: DAC.27, R39.1, SW1.3
- new net N$47: DAC.26, R38.1, SW1.4
- new net N$48: DAC.25, R37.1, SW1.5
- new net N$49: DAC.11, R36.1, SW1.6
- new net N$50: DAC.12, R35.1, SW1.7
- new net N$51: DAC.10, R34.1, SW1.8
- new net N$52: DAC.8, R33.1, SW1.9
- new net SAI_BCK: JP2.3
- new net SAI_D0: JP2.7
- new net SAI_D1: JP2.9
- new net SAI_LRCK: JP2.5
- new net SAI_SCK: JP2.1
- net AGND: now also C41.1, C42.1, C43.2, C44.2, C45.2, C46.2, C47.1, C48.1, C49.1, C50.1, DAC.3, DAC.33, DAC.34, DAC.4, DAC.42, DAC.43
- net OUT1+: now also DAC.1
- net OUT1-: now also DAC.2
- net OUT2+: now also DAC.47
- net OUT2-: now also DAC.46
- net OUT3+: now also DAC.38
- net OUT3-: now also DAC.39
- net OUT4+: now also DAC.36
- net OUT4-: now also DAC.35

Commit message: dac wip
Parts:
- removed S1: SWS010, smd-special:SMS-010
- R16, R24, R32, R8: value 2K 0.1% -> 2K 0.1% DNP
- moved R41 209.0 mm to (125.9, 55.1), turned to 270 degrees
- moved R42 206.9 mm to (106.7, 63.2), turned to 270 degrees
- moved R40 204.0 mm to (109.1, 63.2), turned to 270 degrees
- moved R39 203.3 mm to (111.5, 63.2), turned to 270 degrees
- moved R38 202.7 mm to (113.9, 63.2), turned to 270 degrees
- moved R37 202.1 mm to (116.3, 63.2), turned to 270 degrees
- moved R36 201.6 mm to (118.7, 63.2), turned to 270 degrees
- moved R35 201.1 mm to (121.2, 63.2), turned to 270 degrees
- moved R34 200.7 mm to (123.6, 63.2), turned to 270 degrees
- moved R33 200.3 mm to (126.0, 63.2), turned to 270 degrees
- moved SW1 187.7 mm to (117.0, 70.2)
- moved JP1 148.1 mm to (125.9, 42.9), turned to 90 degrees
- moved C52 102.9 mm to (72.3, 39.1), turned to 90 degrees
- moved C51 100.0 mm to (70.5, 39.1), turned to 90 degrees
- moved C50 91.8 mm to (56.5, 43.2)
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Routing:
- net AVCC: track 0.00 -> 58.3 mm
- net AGND: track 45.7 -> 83.6 mm, vias 16 -> 30
- net OUT1-: track 5.13 -> 41.3 mm, vias 0 -> 2
- net OUT1+: track 5.76 -> 40.4 mm, vias 0 -> 2
- net OUT4+: track 5.76 -> 34.0 mm, vias 0 -> 2
- net OUT4-: track 5.13 -> 32.2 mm, vias 0 -> 2
- net OUT2-: track 5.13 -> 23.8 mm, vias 0 -> 2
- net OUT2+: track 5.76 -> 24.0 mm, vias 0 -> 2
- net OUT3-: track 5.13 -> 21.7 mm, vias 0 -> 2
- net OUT3+: track 5.76 -> 22.2 mm, vias 0 -> 2
- net N$34: track 0.00 -> 4.98 mm
- net GND: track 0.00 -> 4.53 mm
- net 3.3V: track 0.00 -> 4.53 mm
- net N$33: track 0.00 -> 4.10 mm
- added copper zone on layer 1, net GND

Commit message: dac wip
Parts:
- moved JP2 145.4 mm to (129.8, 26.2), turned to 90 degrees
- moved C52 4.83 mm to (68.3, 36.3)
- moved C44 4.83 mm to (51.9, 31.6)
- moved C46 4.83 mm to (58.2, 43.2)
- moved C41 4.83 mm to (54.6, 29.5)
- moved C45 4.83 mm to (52.6, 36.8)
- moved C48 4.83 mm to (52.6, 38.6)
- moved C43 4.83 mm to (58.7, 28.4)
- moved C42 4.83 mm to (54.2, 43.2)
- moved C47 4.83 mm to (51.8, 33.3)
- moved C49 4.83 mm to (51.8, 35.1)
- moved C50 4.83 mm to (52.6, 40.4)
- moved C51 4.83 mm to (66.5, 36.3)
- moved DAC 4.83 mm to (59.9, 35.8)
Routing:
- net OUT2+: track 24.0 -> 18.4 mm
- net OUT1+: track 40.4 -> 35.3 mm
- net OUT1-: track 41.3 -> 36.2 mm
- net OUT2-: track 23.8 -> 19.1 mm
- net OUT3-: track 21.7 -> 18.4 mm
- net OUT3+: track 22.2 -> 19.4 mm
- net OUT4-: track 32.2 -> 33.2 mm
- net OUT4+: track 34.0 -> 34.7 mm

Commit message: dac wip
Parts:
- moved R41 71.9 mm to (61.2, 23.6)
- moved R38 68.6 mm to (46.4, 51.3)
- moved JP2 60.6 mm to (69.2, 28.2)
- moved R42 60.1 mm to (48.3, 49.0), turned to 90 degrees
- moved R39 60.1 mm to (53.1, 49.1), turned to 90 degrees
- moved R40 60.0 mm to (50.8, 49.0), turned to 90 degrees
- moved R34 58.6 mm to (66.4, 50.2), turned to 180 degrees
- moved R37 58.6 mm to (59.4, 49.4), turned to 0 degrees
- moved R33 58.4 mm to (69.5, 48.4)
- moved SW1 57.8 mm to (60.8, 56.3)
- moved JP1 57.5 mm to (68.3, 42.2), turned to 180 degrees
- moved R35 56.7 mm to (66.7, 47.5), turned to 0 degrees
- moved R36 54.9 mm to (66.7, 45.7), turned to 0 degrees
- moved C51 1.91 mm to (68.5, 36.4)
- moved C52 1.91 mm to (70.2, 36.4)
Routing:
- net 3.3V: track 4.53 -> 63.1 mm, vias 0 -> 4
- net N$52: track 0.00 -> 34.8 mm, vias 0 -> 1
- net N$47: track 0.00 -> 28.3 mm
- net N$51: track 0.00 -> 26.1 mm, vias 0 -> 1
- net N$49: track 0.00 -> 25.1 mm, vias 0 -> 2
- net N$50: track 0.00 -> 23.6 mm, vias 0 -> 2
- net N$44: track 0.00 -> 22.6 mm
- net N$45: track 0.00 -> 20.9 mm
- net N$46: track 0.00 -> 19.0 mm
- net N$48: track 0.00 -> 14.6 mm
- net N$39: track 0.00 -> 12.7 mm
- net N$40: track 0.00 -> 10.9 mm
- net N$35: track 0.00 -> 10.3 mm
- net N$41: track 0.00 -> 9.07 mm
- net N$36: track 0.00 -> 7.45 mm
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
Commit message: dac wip
Parts:
- moved R41 2.80 mm to (63.0, 25.8), turned to 90 degrees
Routing:
- net DAC_RST: track 7.36 -> 8.00 mm
Changed lines of the file:
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@@
 <element name="R39" library="microbuilder" package="0603" value="10K" x="53.086" y="49.149" rot="R90"/>
 <element name="R40" library="microbuilder" package="0603" value="10K" x="50.8" y="49.022" rot="R90"/>
-<element name="R41" library="microbuilder" package="0603" value="10K" x="61.214" y="23.622" rot="R270"/>
+<element name="R41" library="microbuilder" package="0603" value="10K" x="62.992" y="25.781" rot="R90"/>
 <element name="R42" library="microbuilder" package="0603" value="10K" x="48.26" y="49.022" rot="R90"/>
 </elements>
@@
 <wire x1="67.525" y1="45.72" x2="67.525" y2="47.498" width="0.3048" layer="1"/>
 <wire x1="67.525" y1="45.72" x2="67.988" y2="36.064" width="0" layer="19" extent="1-1"/>
-<wire x1="61.214" y1="22.772" x2="64.044" y2="36.064" width="0" layer="19" extent="1-1"/>
+<wire x1="62.992" y1="26.631" x2="64.044" y2="36.064" width="0" layer="19" extent="1-1"/>
 </signal>
 <signal name="N$35">
@@
 <wire x1="61.194" y1="29.992" x2="61.214" y2="29.972" width="0.3048" layer="1"/>
 <via x="61.214" y="29.972" extent="1-16" drill="0.6"/>
-<wire x1="61.214" y1="29.972" x2="61.214" y2="26.035" width="0.3048" layer="16"/>
-<wire x1="61.214" y1="26.035" x2="61.341" y2="25.908" width="0.3048" layer="16"/>
-<via x="61.341" y="25.908" extent="1-16" drill="0.6"/>
-<wire x1="61.341" y1="25.908" x2="61.341" y2="24.599" width="0.3048" layer="1"/>
-<wire x1="61.341" y1="24.599" x2="61.214" y2="24.472" width="0.3048" layer="1"/>
+<wire x1="61.214" y1="29.972" x2="61.214" y2="25.908" width="0.3048" layer="16"/>
+<via x="61.214" y="25.908" extent="1-16" drill="0.6"/>
+<wire x1="62.992" y1="24.931" x2="62.191" y2="24.931" width="0.3048" layer="1"/>
+<wire x1="62.191" y1="24.931" x2="61.214" y2="25.908" width="0.3048" layer="1"/>
 </signal>
 </signals>
