File: midimixer-channel/dac-eval-simplified.brd (EAGLE design)
At the start: 100 x 80 mm, 98 parts, among them IC1 NE5534AD, IC2 NE5534AD, IC3 NE5534AD, IC4 NE5534AD

Commit message: dac wip
Parts:
- added AC_IN, DC12, DC17: (no value), con-ptr500:AK500/3
- added C53, C54, C55, C56: 220pF 50V (VJ0603Y221KXACW1BC), microbuilder:0603
- added C57, C58: 2200uF 50v UHE1H222MHD6, rcl:E7,5-18
- added C59, C60: 1uF BFC237011105, capacitor-wima:C5B7.2
- added C61, C62, C63, C64, C65, C66: 4.7uF, microbuilder:0603
- added D1, D2, D3, D4: MUR820, diode:C221B1A
- added D5, D6, D7, D8, D9: 1N4004, diode:DO41-10
- added DC9: (no value), con-ptr500:AK500/2
- added IC5: 7912, linear:TO220H
- added IC6: 7812T, linear:TO220H
- added IC7: 7809, linear:TO220H
- added JP11, JP7, JP8: (no value), microbuilder:1X02_ROUND
- added LED1, LED2, LED3, LED4, LED5: (no value), microbuilder:CHIPLED_0603
- added R34, R35: 1K, microbuilder:0603
- added R36, R37: 680, microbuilder:0603
- added R38: 470, microbuilder:0603
- JP1, JP2: device pinhead:2X05 -> microbuilder:2X05
- JP3, JP4: device pinhead:1X02 -> microbuilder:1X02_ROUND
Connections:
- new net +17: C53.2, C54.1, C57.+, C59.1, D1.C, D2.C, DC17.3, JP11.1, JP7.1, R34.2
- new net +9V: C65.2, C66.2, D9.C, DC9.2, IC7.1, IC7.3, JP11.2, R38.2
- new net -17: C55.2, C56.1, C58.-, C60.2, D3.A, D4.A, DC17.1, JP8.2, LED2.C
- new net N$46: AC_IN.1, C53.1, C56.2, D1.A, D3.C
- new net N$47: AC_IN.3, C54.2, C55.1, D2.A, D4.C
- new net N$49: LED2.A, R35.1
- new net N$50: LED1.A, R34.1
- new net N$51: C61.2, D5.C, IC6.1, JP7.2
- new net N$54: DC9.1
- new net N$55: C63.1, D8.A, IC5.2, JP8.1
- new net N$57: LED5.A, R38.1
- new net N$62: LED3.A, R36.1
- new net N$63: LED4.A, R37.1
- net +12V: now also C62.2, D5.A, D6.C, DC12.3, IC6.3, R36.2
- net -12V: now also C64.1, D7.A, D8.C, DC12.1, IC5.3, LED4.C
- net GND: now also AC_IN.2, C57.-, C58.+, C59.2, C60.1, C61.1, C62.1, C63.2, C64.2, C65.1, C66.1, D6.A, D7.C, D9.A, DC12.2, DC17.2, IC5.1, IC6.2, IC7.2, LED1.C, LED3.C, LED5.C, R35.2, R37.2

Commit message: wip
Parts:
- removed AC_IN, DC12, DC17: (no value), con-ptr500:AK500/3
- removed C56: 220pF 50V (VJ0603Y221KXACW1BC), microbuilder:0603
- removed C57, C58: 2200uF 50v UHE1H222MHD6, rcl:E7,5-18
- removed C59, C60: 1uF BFC237011105, capacitor-wima:C5B7.2
- removed C61, C62, C63, C64, C65, C66: 4.7uF, microbuilder:0603
- removed D1, D2, D3, D4: MUR820, diode:C221B1A
- removed D5, D6, D7, D8, D9: 1N4004, diode:DO41-10
- removed DC9: (no value), con-ptr500:AK500/2
- removed IC5: 7912, linear:TO220H
- removed IC6: 7812T, linear:TO220H
- removed IC7: 7809, linear:TO220H
- removed JP11, JP7, JP8: (no value), microbuilder:1X02_ROUND
- removed LED1, LED2, LED3, LED4, LED5: (no value), microbuilder:CHIPLED_0603
- removed R34, R35: 1K, microbuilder:0603
- removed R36, R37: 680, microbuilder:0603
- removed R38: 470, microbuilder:0603
- added DC_12: (no value), con-ptr500:AK500/3
- added U$30: ADP3301ARZ-5, keves:SO08
- added X1: (no value), con-ptr500:AK500/2
- C53: value 220pF 50V (VJ0603Y221KXACW1BC) -> 2.2uF (EMK107BB7225KA-T)
- C54: value 220pF 50V (VJ0603Y221KXACW1BC) -> 0.01uF
- C55: value 220pF 50V (VJ0603Y221KXACW1BC) -> 10uF
- moved C54 61.3 mm to (-21.1, -34.2), turned to 0 degrees
- moved C55 56.4 mm to (-21.1, -36.6), turned to 0 degrees
- moved C53 51.8 mm to (-21.1, -31.8), turned to 0 degrees
Connections:
- removed net +17: C53.2, C54.1, C57.+, C59.1, D1.C, D2.C, DC17.3, JP11.1, JP7.1, R34.2
- removed net -17: C55.2, C56.1, C58.-, C60.2, D3.A, D4.A, DC17.1, JP8.2, LED2.C
- removed net N$46: AC_IN.1, C53.1, C56.2, D1.A, D3.C
- removed net N$49: LED2.A, R35.1
- removed net N$50: LED1.A, R34.1
- removed net N$51: C61.2, D5.C, IC6.1, JP7.2
- removed net N$54: DC9.1
- removed net N$55: C63.1, D8.A, IC5.2, JP8.1
- removed net N$57: LED5.A, R38.1
- removed net N$62: LED3.A, R36.1
- removed net N$63: LED4.A, R37.1
- net +12V: now also DC_12.1; no longer C62.2, D5.A, D6.C, DC12.3, IC6.3, R36.2
- net +9V: now also C53.2, U$30.5, U$30.7, U$30.8, X1.1; no longer C65.2, C66.2, D9.C, DC9.2, IC7.1, IC7.3, JP11.2, R38.2
- net -12V: now also DC_12.3; no longer C64.1, D7.A, D8.C, DC12.1, IC5.3, LED4.C
- net 3.3V: now also C54.2, C55.2, U$30.1, U$30.2
- net GND: now also C53.1, C55.1, DC_12.2, U$30.4, X1.2; no longer AC_IN.2, C57.-, C58.+, C59.2, C60.1, C61.1, C62.1, C63.2, C64.2, C65.1, C66.1, D6.A, D7.C, D9.A, DC12.2, DC17.2, IC5.1, IC6.2, IC7.2, LED1.C, LED3.C, LED5.C, R35.2, R37.2
- net N$47: now also C54.1, U$30.3; no longer AC_IN.3, C54.2, C55.1, D2.A, D4.C

Commit message: wip
Parts:
- added C56: 2.2uF (EMK107BB7225KA-T), microbuilder:0603
- added C57, C59, C62, C65: 0.1uF, microbuilder:0603
- added C58, C63, C64: 10uF, microbuilder:0603
- added C60, C61: 100uF EMVE160ADA101MF55G, SparkFun-Capacitors:PANASONIC_D
- added EN_3.3, EN_DAC_VCC, EN_DAC_VREF: (no value), microbuilder:1X02_OVAL
- added IC5: REG1117-5, burr-brown:SOT223
- added U$43: ADR02, keves:SOIC8
- U$30: value ADP3301ARZ-5 -> ADP3301ARZ-3.3
- renumbered X1 to DC_9
Connections:
- new net N$46: C54.2, C55.2, EN_3.3.1, U$30.1, U$30.2
- new net N$48: C58.2, C59.2, EN_DAC_VREF.1, U$43.6
- new net N$51: C64.1, C65.1, EN_DAC_VCC.1, IC5.2
- net +12V: now also C60.+
- net +9V: now also C56.1, C57.2, C62.1, C63.2, IC5.3, U$43.2
- net -12V: now also C61.-
- net 3.3V: now also EN_3.3.2; no longer C54.2, C55.2, U$30.1, U$30.2
- net DAC_VCC: now also EN_DAC_VCC.2
- net DAC_VREF: now also EN_DAC_VREF.2
- net GND: now also C56.2, C57.1, C58.1, C59.1, C60.-, C61.+, C62.2, C63.1, C64.2, C65.2, IC5.1, U$43.4

Commit message: wip
Parts:
- removed JP3, JP4: (no value), microbuilder:1X02_ROUND
- moved C61 163.9 mm to (61.7, 72.1), turned to 270 degrees
- moved C60 152.5 mm to (61.8, 63.9), turned to 270 degrees
- moved DC_12 114.9 mm to (69.5, 68.3), turned to 90 degrees
- moved JP1 84.9 mm to (68.8, 47.4), turned to 90 degrees
- moved C44 3.45 mm to (52.3, 35.1)
- moved C47 1.78 mm to (51.7, 31.5)
- moved C49 1.78 mm to (51.7, 33.3)
- moved C45 0.25 mm to (52.3, 36.8)
Connections:
- removed net DAC_CLK: JP1.3
- removed net DAC_CS: JP1.1
- removed net DAC_MISO: JP1.7
- removed net DAC_MOSI: JP1.5
- removed net DAC_RST_: DAC.9, JP1.10, R33.1
- removed net N$44: C43.1, C44.1, C45.1, C46.1, DAC.32, DAC.41, DAC.44, DAC.5, JP3.1
- removed net N$45: C47.2, C48.2, C49.2, C50.2, DAC.40, DAC.45, JP4.1
- removed net SAI_BCK: JP2.3
- removed net SAI_D0: JP2.7
- removed net SAI_D1: JP2.9
- removed net SAI_LRCK: JP2.5
- removed net SAI_SCK: JP2.1
- net DAC_RST: now also DAC.9, JP1.10, R33.1; no longer JP1.9
- net DAC_VCC: now also C47.2, C48.2, C49.2, C50.2, DAC.40, DAC.45; no longer JP4.2
- net DAC_VREF: now also C43.1, C44.1, C45.1, C46.1, DAC.32, DAC.41, DAC.44, DAC.5; no longer JP3.2
- net GND: now also JP1.1, JP1.3, JP1.5, JP1.7, JP1.9, JP2.1, JP2.3, JP2.5, JP2.7, JP2.9
Routing:
- net DAC_VREF: track 0.00 -> 63.9 mm
- net +12V: track 118.3 -> 180.0 mm, vias 4 -> 8
- net -12V: track 128.8 -> 179.2 mm
- net DAC_RST: track 0.00 -> 26.5 mm, vias 0 -> 2
- net N$38: track 1.86 -> 12.8 mm
- net DAC_VCC: track 0.00 -> 10.6 mm
- net GND: track 106.7 -> 116.5 mm
- net N$37: track 2.19 -> 11.4 mm
- net 3.3V: track 6.38 -> 14.7 mm
- net N$36: track 5.66 -> 9.51 mm

Commit message: wip
Parts:
- moved C63 165.4 mm to (59.7, 55.6), turned to 90 degrees
- moved EN_DAC_VCC 164.3 mm to (58.8, 51.2)
- moved C62 158.6 mm to (57.7, 55.6), turned to 270 degrees
- moved C65 157.3 mm to (49.8, 51.1), turned to 180 degrees
- moved C64 156.0 mm to (53.5, 51.1)
- moved IC5 147.6 mm to (51.6, 55.4), turned to 90 degrees
- moved EN_3.3 112.1 mm to (59.7, 22.4)
- moved EN_DAC_VREF 108.9 mm to (52.7, 14.0), turned to 180 degrees
- moved C56 108.0 mm to (65.8, 10.9), turned to 90 degrees
- moved C57 107.6 mm to (64.0, 10.9), turned to 270 degrees
- moved C58 104.6 mm to (54.0, 10.3), turned to 90 degrees
- moved C59 104.3 mm to (52.1, 10.4), turned to 90 degrees
- moved C53 99.9 mm to (62.9, 22.4), turned to 270 degrees
- moved U$43 97.2 mm to (58.9, 10.7), turned to 90 degrees
- moved C55 95.9 mm to (55.2, 21.5), turned to 180 degrees
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Routing:
- net +9V: track 0.00 -> 93.0 mm
- net DAC_VCC: track 10.6 -> 62.7 mm, vias 0 -> 9
- net GND: track 116.5 -> 146.2 mm, vias 37 -> 45
- net DAC_VREF: track 63.9 -> 78.8 mm
- net N$51: track 0.00 -> 14.6 mm
- net 3.3V: track 14.7 -> 24.9 mm
- net N$46: track 0.00 -> 8.79 mm
- net N$48: track 0.00 -> 7.12 mm
- net OUT3-: track 18.4 -> 22.6 mm
- net OUT1+: track 37.6 -> 33.6 mm
- net DAC_RST: track 26.5 -> 30.6 mm
- net OUT3+: track 19.4 -> 22.3 mm
- net N$47: track 0.00 -> 2.67 mm
- net OUT1-: track 38.4 -> 36.1 mm
Other:
- board size 100 x 80 mm -> 76.2 x 80 mm

Commit message: wip
Parts:
- moved DC_9 3.81 mm to (69.7, 16.0)
Routing:
- net +9V: track 93.0 -> 88.3 mm
- net DAC_VCC: track 62.7 -> 59.8 mm
Other:
- board size 76.2 x 80 mm -> 73.4 x 76.4 mm
- board text added: "PCM4104 Eval - Rev A Eran Rundstein, Dec 2016"
Changed lines of the file:
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@@
 <board>
 <plain>
-<wire x1="0" y1="0" x2="76.2" y2="0" width="0" layer="20"/>
-<wire x1="76.2" y1="0" x2="76.2" y2="80" width="0" layer="20"/>
-<wire x1="76.2" y1="80" x2="0" y2="80" width="0" layer="20"/>
-<wire x1="0" y1="80" x2="0" y2="0" width="0" layer="20"/>
+<wire x1="0" y1="0" x2="73.152" y2="0" width="0" layer="20"/>
+<wire x1="73.152" y1="0" x2="72.898" y2="76.444" width="0" layer="20"/>
+<wire x1="72.898" y1="76.444" x2="-0.254" y2="76.444" width="0" layer="20"/>
+<wire x1="-0.254" y1="76.444" x2="0" y2="0" width="0" layer="20"/>
+<text x="52.578" y="3.81" size="0.8128" layer="21" font="vector">PCM4104 Eval - Rev A
+Eran Rundstein, Dec 2016</text>
 </plain>
 <attributes>
@@
 <attribute name="OC_FARNELL" value="unknown" x="69.469" y="68.326" size="1.778" layer="27" rot="R90" display="off"/>
 </element>
-<element name="DC_9" library="con-ptr500" package="AK500/2" value="" x="72.009" y="12.954" rot="R90">
-<attribute name="MF" value="" x="72.009" y="12.954" size="1.778" layer="27" rot="R90" display="off"/>
-<attribute name="MPN" value="" x="72.009" y="12.954" size="1.778" layer="27" rot="R90" display="off"/>
-<attribute name="OC_NEWARK" value="unknown" x="72.009" y="12.954" size="1.778" layer="27" rot="R90" display="off"/>
-<attribute name="OC_FARNELL" value="unknown" x="72.009" y="12.954" size="1.778" layer="27" rot="R90" display="off"/>
+<element name="DC_9" library="con-ptr500" package="AK500/2" value="" x="69.723" y="16.002" rot="R90">
+<attribute name="MF" value="" x="69.723" y="16.002" size="1.778" layer="27" rot="R90" display="off"/>
+<attribute name="MPN" value="" x="69.723" y="16.002" size="1.778" layer="27" rot="R90" display="off"/>
+<attribute name="OC_NEWARK" value="unknown" x="69.723" y="16.002" size="1.778" layer="27" rot="R90" display="off"/>
+<attribute name="OC_FARNELL" value="unknown" x="69.723" y="16.002" size="1.778" layer="27" rot="R90" display="off"/>
 </element>
 <element name="U$30" library="keves" package="SO08" value="ADP3301ARZ-3.3" x="59.817" y="17.907" rot="R270"/>
@@
 <wire x1="57.873" y1="42.33" x2="57.023" y2="43.18" width="0.3048" layer="1"/>
 <contactref element="DAC" pad="10"/>
-<via x="71.755" y="37.465" extent="1-16" drill="0.6"/>
-<wire x1="70.231" y1="37.299" x2="71.589" y2="37.299" width="0.3048" layer="1"/>
-<wire x1="71.589" y1="37.299" x2="71.755" y2="37.465" width="0.3048" layer="1"/>
+<via x="70.231" y="39.243" extent="1-16" drill="0.6"/>
 <wire x1="60.194" y1="39.914" x2="60.194" y2="38.358" width="0.3048" layer="1"/>
 <wire x1="60.194" y1="38.358" x2="60.452" y2="38.1" width="0.3048" layer="1"/>
@@
 <via x="56.134" y="23.114" extent="1-16" drill="0.6"/>
 <wire x1="56.134" y1="23.114" x2="56.134" y2="24.003" width="0.6096" layer="16"/>
+<wire x1="70.231" y1="37.299" x2="70.231" y2="39.243" width="0.3048" layer="1"/>
 </signal>
 <signal name="3.3V">
@@
 <wire x1="52.666" y1="33.401" x2="52.539" y2="33.274" width="0.3048" layer="1"/>
 <wire x1="53.428" y1="40.386" x2="53.428" y2="40.806" width="0.4064" layer="1"/>
-<wire x1="53.428" y1="40.806" x2="51.943" y2="42.291" width="0.4064" layer="1"/>
+<wire x1="53.428" y1="40.806" x2="51.943" y2="42.291" width="0.6096" layer="1"/>
 <wire x1="51.943" y1="42.291" x2="51.943" y2="42.418" width="0.4064" layer="1"/>
 <via x="51.943" y="44.45" extent="1-16" drill="0.6"/>
-<wire x1="51.943" y1="42.418" x2="51.943" y2="43.434" width="0.4064" layer="1"/>
-<wire x1="51.943" y1="43.434" x2="51.943" y2="44.45" width="0.4064" layer="1"/>
-<wire x1="51.943" y1="44.45" x2="51.943" y2="43.434" width="0.4064" layer="16"/>
-<wire x1="51.943" y1="43.434" x2="51.943" y2="42.418" width="0.4064" layer="16"/>
-<wire x1="51.943" y1="44.45" x2="51.943" y2="46.482" width="0.4064" layer="16"/>
-<wire x1="51.943" y1="46.482" x2="51.943" y2="47.752" width="0.4064" layer="16"/>
-<wire x1="51.943" y1="47.752" x2="52.324" y2="48.133" width="0.4064" layer="16"/>
-<wire x1="52.324" y1="48.133" x2="52.578" y2="48.133" width="0.4064" layer="16"/>
-<wire x1="52.578" y1="48.133" x2="53.594" y2="48.133" width="0.4064" layer="16"/>
-<via x="53.594" y="48.133" extent="1-16" drill="0.6"/>
-<via x="52.578" y="48.133" extent="1-16" drill="0.6"/>
+<wire x1="51.943" y1="42.418" x2="51.943" y2="43.434" width="0.6096" layer="1"/>
+<wire x1="51.943" y1="43.434" x2="51.943" y2="44.45" width="0.6096" layer="1"/>
+<wire x1="51.943" y1="44.45" x2="51.943" y2="43.434" width="0.6096" layer="16"/>
+<wire x1="51.943" y1="43.434" x2="51.943" y2="42.418" width="0.6096" layer="16"/>
+<wire x1="51.943" y1="44.45" x2="51.943" y2="46.609" width="0.6096" layer="16"/>
 <via x="51.943" y="43.434" extent="1-16" drill="0.6"/>
 <via x="51.943" y="42.418" extent="1-16" drill="0.6"/>
-<wire x1="60.071" y1="50.673" x2="60.071" y2="51.181" width="0.4064" layer="1"/>
-<wire x1="53.594" y1="48.133" x2="52.324" y2="48.133" width="0.4064" layer="1"/>
-<wire x1="52.324" y1="48.133" x2="51.943" y2="47.752" width="0.4064" layer="1"/>
-<wire x1="51.943" y1="47.752" x2="51.943" y2="46.482" width="0.4064" layer="1"/>
-<via x="51.943" y="46.482" extent="1-16" drill="0.6"/>
-<wire x1="53.594" y1="48.133" x2="57.531" y2="48.133" width="0.4064" layer="1"/>
-<wire x1="57.531" y1="48.133" x2="60.071" y2="50.673" width="0.4064" layer="1"/>
+<wire x1="49.53" y1="46.609" x2="50.546" y2="46.609" width="0.6096" layer="1"/>
+<wire x1="50.546" y1="46.609" x2="51.562" y2="46.609" width="0.6096" layer="1"/>
+<wire x1="51.562" y1="46.609" x2="57.531" y2="46.609" width="0.6096" layer="1"/>
 <wire x1="52.539" y1="31.496" x2="51.269" y2="30.226" width="0.6096" layer="1"/>
 <wire x1="51.269" y1="30.226" x2="51.181" y2="30.226" width="0.6096" layer="1"/>
@@
 <wire x1="50.165" y1="30.226" x2="49.149" y2="30.226" width="0.6096" layer="1"/>
 <wire x1="48.387" y1="30.226" x2="47.625" y2="30.988" width="0.6096" layer="16"/>
-<wire x1="47.9425" y1="47.0535" x2="49.022" y2="48.133" width="0.6096" layer="16"/>
-<wire x1="49.022" y1="48.133" x2="52.578" y2="48.133" width="0.6096" layer="16"/>
+<wire x1="49.53" y1="46.609" x2="50.546" y2="46.609" width="0.6096" layer="16"/>
+<wire x1="50.546" y1="46.609" x2="51.562" y2="46.609" width="0.6096" layer="16"/>
+<wire x1="51.562" y1="46.609" x2="51.943" y2="46.609" width="0.6096" layer="16"/>
 <wire x1="48.387" y1="30.226" x2="50.165" y2="30.226" width="0.6096" layer="16"/>
 <wire x1="50.165" y1="30.226" x2="51.181" y2="30.226" width="0.6096" layer="16"/>
@@
 <via x="51.181" y="30.226" extent="1-16" drill="0.6"/>
 <via x="50.165" y="30.226" extent="1-16" drill="0.6"/>
-<wire x1="47.625" y1="30.988" x2="47.625" y2="46.736" width="0.6096" layer="16"/>
-<wire x1="47.625" y1="46.736" x2="47.9425" y2="47.0535" width="0.6096" layer="16"/>
+<wire x1="47.625" y1="30.988" x2="47.625" y2="43.815" width="0.6096" layer="16"/>
+<via x="49.53" y="46.609" extent="1-16" drill="0.6"/>
+<via x="50.546" y="46.609" extent="1-16" drill="0.6"/>
+<via x="51.562" y="46.609" extent="1-16" drill="0.6"/>
+<wire x1="47.625" y1="43.815" x2="47.625" y2="44.196" width="0.6096" layer="16"/>
+<wire x1="49.53" y1="46.609" x2="47.625" y2="44.704" width="0.6096" layer="16"/>
+<wire x1="47.625" y1="44.704" x2="47.625" y2="44.196" width="0.6096" layer="16"/>
+<wire x1="57.531" y1="46.609" x2="60.071" y2="49.149" width="0.6096" layer="1"/>
+<wire x1="60.071" y1="49.149" x2="60.071" y2="51.181" width="0.6096" layer="1"/>
 </signal>
 <signal name="+9V">
@@
 <wire x1="63.969" y1="10.033" x2="64.008" y2="10.072" width="0.6096" layer="1"/>
 <wire x1="64.008" y1="10.072" x2="65.786" y2="10.072" width="0.6096" layer="1"/>
-<wire x1="65.786" y1="10.072" x2="71.6416" y2="10.072" width="0.6096" layer="1"/>
-<wire x1="71.6416" y1="10.072" x2="72.009" y2="10.4394" width="0.6096" layer="1"/>
-<wire x1="62.8904" y1="16.002" x2="66.4464" y2="16.002" width="0.6096" layer="1"/>
-<wire x1="66.4464" y1="16.002" x2="72.009" y2="10.4394" width="0.6096" layer="1"/>
-<wire x1="62.865" y1="21.502" x2="72.048" y2="21.502" width="0.6096" layer="1"/>
-<wire x1="72.048" y1="21.502" x2="73.152" y2="22.606" width="0.6096" layer="1"/>
-<wire x1="73.152" y1="22.606" x2="73.152" y2="53.848" width="0.6096" layer="1"/>
-<wire x1="73.152" y1="53.848" x2="70.485" y2="56.515" width="0.6096" layer="1"/>
+<wire x1="62.8904" y1="16.002" x2="67.2084" y2="16.002" width="0.6096" layer="1"/>
+<wire x1="62.865" y1="21.502" x2="71.286" y2="21.502" width="0.6096" layer="1"/>
+<wire x1="72.39" y1="54.61" x2="70.485" y2="56.515" width="0.6096" layer="1"/>
 <wire x1="70.485" y1="56.515" x2="59.729" y2="56.515" width="0.6096" layer="1"/>
 <wire x1="59.729" y1="56.515" x2="59.69" y2="56.476" width="0.6096" layer="1"/>
+<wire x1="71.286" y1="21.502" x2="72.39" y2="22.606" width="0.6096" layer="1"/>
+<wire x1="72.39" y1="22.606" x2="72.39" y2="54.61" width="0.6096" layer="1"/>
+<wire x1="65.786" y1="10.072" x2="67.984" y2="10.072" width="0.6096" layer="1"/>
+<wire x1="67.984" y1="10.072" x2="69.723" y2="11.811" width="0.6096" layer="1"/>
+<wire x1="69.723" y1="11.811" x2="69.723" y2="13.4874" width="0.6096" layer="1"/>
+<wire x1="69.723" y1="13.4874" x2="67.2084" y2="16.002" width="0.6096" layer="1"/>
 </signal>
 <signal name="N$47">
@@
 </board>
 </drawing>
+<compatibility>
+<note version="6.3" minversion="6.2.2" severity="warning">
+Since Version 6.2.2 text objects can contain more than one line,
+which will not be processed correctly with this version.
+</note>
+</compatibility>
 </eagle>
