File: midimixer-channel/dac-eval-simplified.brd (EAGLE design)
At the start: 73.4 x 76.4 mm, 117 parts, among them IC1 NE5534AD, IC2 NE5534AD, IC3 NE5534AD, IC4 NE5534AD, IC5 REG1117-5

Commit message: wip
Parts:
- moved C60 2.16 mm to (59.7, 63.9)
- moved C61 2.04 mm to (59.7, 72.0)
Connections:
- net N$35 renamed DAC_CS
- net N$36 renamed DAC_CLK
- net N$37 renamed DAC_MOSI
- net N$38 renamed DAC_MISO
- net N$39 renamed DAC_SCK
- net N$40 renamed DAC_BCK
- net N$41 renamed DAC_LRCK
- net N$42 renamed DAC_D0
- net N$43 renamed DAC_D1
Routing:
- net GND: track 146.6 -> 156.3 mm
- net +12V: track 180.0 -> 178.6 mm
Other:
- board size 73.4 x 76.4 mm -> 73.2 x 76.5 mm
- board text added: "+12"
- board text added: "+9V"
- board text added: "-12"
- board text added: "BCK"
- board text added: "CLK"
- board text added: "CS"
- board text added: "D0"
- board text added: "D1"
- board text added: "GND"
- board text added: "LRCK"
- board text added: "MISO"
- board text added: "MOSI"
- board text added: "RST"
- board text added: "SCK"
Changed lines of the file:
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@@
 <plain>
 <wire x1="0" y1="0" x2="73.152" y2="0" width="0" layer="20"/>
-<wire x1="73.152" y1="0" x2="72.898" y2="76.444" width="0" layer="20"/>
-<wire x1="72.898" y1="76.444" x2="-0.254" y2="76.444" width="0" layer="20"/>
-<wire x1="-0.254" y1="76.444" x2="0" y2="0" width="0" layer="20"/>
+<wire x1="73.152" y1="0" x2="73.152" y2="76.454" width="0" layer="20"/>
+<wire x1="73.152" y1="76.454" x2="0" y2="76.454" width="0" layer="20"/>
+<wire x1="0" y1="76.454" x2="0" y2="0" width="0" layer="20"/>
 <text x="52.578" y="3.81" size="0.8128" layer="21" font="vector">PCM4104 Eval - Rev A
 Eran Rundstein, Dec 2016</text>
+<text x="67.056" y="23.622" size="0.8128" layer="21" font="vector" rot="R180">SCK</text>
+<text x="67.056" y="26.035" size="0.8128" layer="21" font="vector" rot="R180">BCK</text>
+<text x="67.31" y="28.575" size="0.8128" layer="21" font="vector" rot="R180">LRCK</text>
+<text x="67.056" y="31.115" size="0.8128" layer="21" font="vector" rot="R180">D0</text>
+<text x="67.056" y="33.655" size="0.8128" layer="21" font="vector" rot="R180">D1</text>
+<text x="63.881" y="52.07" size="0.8128" layer="21" font="vector">RST</text>
+<text x="63.246" y="49.53" size="0.8128" layer="21" font="vector">MISO</text>
+<text x="63.373" y="46.99" size="0.8128" layer="21" font="vector">MOSI</text>
+<text x="63.754" y="44.45" size="0.8128" layer="21" font="vector">CLK</text>
+<text x="64.516" y="41.91" size="0.8128" layer="21" font="vector">CS</text>
+<text x="69.469" y="9.779" size="0.8128" layer="21" font="vector">+9V</text>
+<text x="65.405" y="18.161" size="0.8128" layer="21" font="vector" rot="R90">GND</text>
+<text x="65.278" y="72.009" size="0.8128" layer="21" font="vector" rot="R90">-12</text>
+<text x="64.77" y="61.976" size="0.8128" layer="21" font="vector" rot="R90">+12</text>
+<text x="64.897" y="67.437" size="0.8128" layer="21" font="vector" rot="R90">GND</text>
 </plain>
 <attributes>
@@
 <element name="C59" library="microbuilder" package="0603" value="0.1uF" x="52.07" y="10.414" rot="R90"/>
 <element name="EN_DAC_VREF" library="microbuilder" package="1X02_OVAL" value="" x="52.705" y="13.97" rot="R180"/>
-<element name="C60" library="SparkFun-Capacitors" package="PANASONIC_D" value="100uF EMVE160ADA101MF55G" x="61.849" y="63.881" rot="R270"/>
-<element name="C61" library="SparkFun-Capacitors" package="PANASONIC_D" value="100uF EMVE160ADA101MF55G" x="61.722" y="72.136" rot="R270"/>
+<element name="C60" library="SparkFun-Capacitors" package="PANASONIC_D" value="100uF EMVE160ADA101MF55G" x="59.69" y="63.881" rot="R270"/>
+<element name="C61" library="SparkFun-Capacitors" package="PANASONIC_D" value="100uF EMVE160ADA101MF55G" x="59.69" y="72.009" rot="R270"/>
 <element name="IC5" library="burr-brown" package="SOT223" value="REG1117-5" x="51.562" y="55.372" rot="R90">
 <attribute name="MF" value="" x="51.562" y="55.372" size="1.778" layer="27" rot="R90" display="off"/>
@@
 <contactref element="DC_12" pad="1"/>
 <contactref element="C60" pad="+"/>
-<wire x1="69.469" y1="63.3222" x2="63.6902" y2="63.3222" width="1.016" layer="1"/>
-<wire x1="63.6902" y1="63.3222" x2="61.849" y2="61.481" width="1.016" layer="1"/>
-<wire x1="61.849" y1="61.481" x2="60.058" y2="61.481" width="1.016" layer="1"/>
-<wire x1="60.058" y1="61.481" x2="58.674" y2="62.865" width="1.016" layer="1"/>
 <wire x1="51.689" y1="72.263" x2="51.435" y2="72.263" width="1.016" layer="16"/>
 <wire x1="51.435" y1="72.263" x2="50.419" y2="72.263" width="1.016" layer="16"/>
@@
 <wire x1="48.387" y1="72.263" x2="25.019" y2="72.263" width="1.016" layer="16"/>
 <wire x1="25.019" y1="72.263" x2="22.098" y2="69.342" width="1.016" layer="16"/>
-<wire x1="58.674" y1="62.865" x2="58.674" y2="70.612" width="1.016" layer="1"/>
-<wire x1="58.674" y1="70.612" x2="57.023" y2="72.263" width="1.016" layer="1"/>
-<wire x1="57.023" y1="72.263" x2="51.435" y2="72.263" width="1.016" layer="1"/>
 <wire x1="51.435" y1="72.263" x2="50.419" y2="72.263" width="1.016" layer="1"/>
 <wire x1="50.419" y1="72.263" x2="49.403" y2="72.263" width="1.016" layer="1"/>
@@
 <via x="50.419" y="72.263" extent="1-16" drill="0.6"/>
 <via x="51.435" y="72.263" extent="1-16" drill="0.6"/>
+<wire x1="59.69" y1="61.481" x2="67.6278" y2="61.481" width="1.016" layer="1"/>
+<wire x1="67.6278" y1="61.481" x2="69.469" y2="63.3222" width="1.016" layer="1"/>
+<wire x1="59.69" y1="61.481" x2="58.915" y2="61.481" width="1.016" layer="1"/>
+<wire x1="58.915" y1="61.481" x2="56.515" y2="63.881" width="1.016" layer="1"/>
+<wire x1="56.515" y1="63.881" x2="56.515" y2="69.215" width="1.016" layer="1"/>
+<wire x1="56.515" y1="69.215" x2="53.467" y2="72.263" width="1.016" layer="1"/>
+<wire x1="53.467" y1="72.263" x2="51.435" y2="72.263" width="1.016" layer="1"/>
 </signal>
 <signal name="-12V">
@@
 <contactref element="DC_12" pad="3"/>
 <contactref element="C61" pad="-"/>
-<wire x1="69.469" y1="73.3298" x2="62.9282" y2="73.3298" width="1.016" layer="1"/>
-<wire x1="62.9282" y1="73.3298" x2="61.722" y2="74.536" width="1.016" layer="1"/>
-<wire x1="61.722" y1="74.536" x2="20.434" y2="74.536" width="1.016" layer="1"/>
-<wire x1="20.434" y1="74.536" x2="19.304" y2="73.406" width="1.016" layer="1"/>
+<wire x1="20.066" y1="74.168" x2="19.304" y2="73.406" width="1.016" layer="1"/>
 <wire x1="19.304" y1="73.406" x2="19.304" y2="72.136" width="1.016" layer="1"/>
 <wire x1="19.304" y1="72.136" x2="19.558" y2="71.882" width="1.016" layer="1"/>
+<wire x1="69.469" y1="73.3298" x2="68.3898" y2="74.409" width="1.016" layer="1"/>
+<wire x1="68.3898" y1="74.409" x2="59.69" y2="74.409" width="1.016" layer="1"/>
+<wire x1="59.449" y1="74.168" x2="20.066" y2="74.168" width="1.016" layer="1"/>
+<wire x1="59.449" y1="74.168" x2="59.69" y2="74.409" width="1.016" layer="1"/>
 </signal>
 <signal name="N$10">
@@
 <wire x1="29.122" y1="12.065" x2="29.122" y2="10.287" width="0.508" layer="1"/>
 <polygon width="0.508" layer="16">
-<vertex x="0.381" y="75.565"/>
-<vertex x="99.822" y="75.565"/>
-<vertex x="99.822" y="0.508"/>
+<vertex x="0.381" y="76.2"/>
+<vertex x="72.898" y="76.2"/>
+<vertex x="72.898" y="0.508"/>
 <vertex x="0.254" y="0.508"/>
 <vertex x="0.254" y="18.288"/>
@@
 <contactref element="JP1" pad="7"/>
 <contactref element="JP1" pad="9"/>
-<wire x1="69.469" y1="68.326" x2="63.894" y2="68.326" width="1.016" layer="1"/>
-<wire x1="63.894" y1="68.326" x2="61.849" y2="66.281" width="1.016" layer="1"/>
-<wire x1="63.894" y1="68.326" x2="63.132" y2="68.326" width="1.016" layer="1"/>
-<wire x1="63.132" y1="68.326" x2="61.722" y2="69.736" width="1.016" layer="1"/>
 <wire x1="51.474" y1="35.052" x2="49.657" y2="35.052" width="0.3048" layer="1"/>
 <via x="49.657" y="35.052" extent="1-16" drill="0.6"/>
@@
 <wire x1="56.134" y1="23.114" x2="56.134" y2="24.003" width="0.6096" layer="16"/>
 <wire x1="70.231" y1="37.299" x2="70.231" y2="39.243" width="0.3048" layer="1"/>
+<wire x1="69.469" y1="68.326" x2="68.186" y2="69.609" width="1.016" layer="1"/>
+<wire x1="68.186" y1="69.609" x2="59.69" y2="69.609" width="1.016" layer="1"/>
+<wire x1="59.69" y1="66.281" x2="67.424" y2="66.281" width="1.016" layer="1"/>
+<wire x1="67.424" y1="66.281" x2="69.469" y2="68.326" width="1.016" layer="1"/>
 </signal>
 <signal name="3.3V">
@@
 <wire x1="60.96" y1="28.155" x2="61.888" y2="29.083" width="0.6096" layer="1"/>
 </signal>
-<signal name="N$35">
+<signal name="DAC_CS">
 <contactref element="DAC" pad="21"/>
 <wire x1="64.044" y1="37.064" x2="65.766" y2="37.064" width="0.3048" layer="1"/>
@@
 <wire x1="66.294" y1="41.021" x2="67.564" y2="42.291" width="0.3048" layer="1"/>
 </signal>
-<signal name="N$36">
+<signal name="DAC_CLK">
 <contactref element="DAC" pad="22"/>
 <wire x1="64.044" y1="37.564" x2="65.377" y2="37.564" width="0.3048" layer="1"/>
@@
 <wire x1="65.786" y1="43.053" x2="67.564" y2="44.831" width="0.3048" layer="1"/>
 </signal>
-<signal name="N$37">
+<signal name="DAC_MOSI">
 <contactref element="DAC" pad="23"/>
 <wire x1="64.044" y1="38.064" x2="65.115" y2="38.064" width="0.3048" layer="1"/>
@@
 <wire x1="65.278" y1="45.085" x2="67.564" y2="47.371" width="0.3048" layer="1"/>
 </signal>
-<signal name="N$38">
+<signal name="DAC_MISO">
 <contactref element="DAC" pad="24"/>
 <contactref element="JP1" pad="8"/>
@@
 <wire x1="64.044" y1="46.391" x2="67.564" y2="49.911" width="0.3048" layer="1"/>
 </signal>
-<signal name="N$39">
+<signal name="DAC_SCK">
 <contactref element="DAC" pad="14"/>
 <contactref element="JP2" pad="2"/>
@@
 <wire x1="65.278" y1="25.781" x2="67.945" y2="23.114" width="0.3048" layer="1"/>
 </signal>
-<signal name="N$40">
+<signal name="DAC_BCK">
 <contactref element="DAC" pad="15"/>
 <contactref element="JP2" pad="4"/>
@@
 <wire x1="65.786" y1="27.813" x2="66.167" y2="27.432" width="0.3048" layer="1"/>
 </signal>
-<signal name="N$41">
+<signal name="DAC_LRCK">
 <contactref element="DAC" pad="16"/>
 <contactref element="JP2" pad="6"/>
@@
 <wire x1="66.294" y1="29.845" x2="67.945" y2="28.194" width="0.3048" layer="1"/>
 </signal>
-<signal name="N$42">
+<signal name="DAC_D0">
 <contactref element="DAC" pad="17"/>
 <contactref element="JP2" pad="8"/>
@@
 <wire x1="66.802" y1="31.877" x2="67.945" y2="30.734" width="0.3048" layer="1"/>
 </signal>
-<signal name="N$43">
+<signal name="DAC_D1">
 <contactref element="DAC" pad="18"/>
 <contactref element="JP2" pad="10"/>

Commit message: wip
Parts:
- moved C56 2.16 mm to (64.4, 12.6)
- moved U$43 2.16 mm to (57.5, 12.3)
- moved C57 2.16 mm to (62.6, 12.6)
- moved C58 2.16 mm to (52.6, 11.9)
- moved C59 2.16 mm to (50.7, 12.1)
- moved EN_DAC_VREF 2.16 mm to (51.3, 15.6)
Routing:
- net -12V: track 179.1 -> 169.2 mm
- net +12V: track 178.6 -> 171.0 mm
- net DAC_VREF: track 78.8 -> 77.8 mm
- net GND: track 156.3 -> 155.5 mm
- net OUT1+: track 33.6 -> 34.2 mm
