File: midimixer-channel/dac-eval-simplified.sch (EAGLE design)
At the start: 98 parts, among them IC1 NE5534AD, IC2 NE5534AD, IC3 NE5534AD, IC4 NE5534AD

Commit message: dac wip
Parts:
- added AC_IN, DC12, DC17: (no value), con-ptr500:AK500/3
- added C53, C54, C55, C56: 220pF 50V (VJ0603Y221KXACW1BC), microbuilder:CAP_CERAMIC0603
- added C57, C58: 2200uF 50v UHE1H222MHD6, rcl:CPOL-USE7.5-18
- added C59, C60: 1uF BFC237011105, capacitor-wima:C5/7.2
- added C61, C62, C63, C64, C65, C66: 4.7uF, microbuilder:CAP_CERAMIC0603
- added D1, D2, D3, D4: MUR820, diode:MUR820
- added D5, D6, D7, D8, D9: 1N4004, diode:1N4004
- added DC9: (no value), con-ptr500:AK500/2
- added IC5: 7912, linear:7912T
- added IC6: 7812T, linear:7812T
- added IC7: 7809, linear:7812T
- added JP11, JP7, JP8: (no value), microbuilder:HEADER-1X2ROUND
- added LED1, LED2, LED3, LED4, LED5: (no value), microbuilder:LED0603
- added R34, R35: 1K, microbuilder:RESISTOR0603
- added R36, R37: 680, microbuilder:RESISTOR0603
- added R38: 470, microbuilder:RESISTOR0603
- JP1, JP2: device pinhead:PINHD-2X5 -> microbuilder:HEADER-2X5
- JP3, JP4: device pinhead:PINHD-1X2 -> microbuilder:HEADER-1X2ROUND
Connections:
- new net +17: C53.P$2, C54.P$1, C57.+, C59.1, D1.C, D2.C, DC17-3.KL, JP11.1, JP7.1, R34.2
- new net +9V: C65.P$2, C66.P$2, D9.C, DC9-2.KL, IC7.VI, IC7.VO, JP11.2, R38.2
- new net -17: C55.P$2, C56.P$1, C58.-, C60.2, D3.A, D4.A, DC17-1.KL, JP8.2, LED2.C
- new net N$46: AC_IN-1.KL, C53.P$1, C56.P$2, D1.A, D3.C
- new net N$47: AC_IN-3.KL, C54.P$2, C55.P$1, D2.A, D4.C
- new net N$49: LED2.A, R35.1
- new net N$50: LED1.A, R34.1
- new net N$51: C61.P$2, D5.C, IC6.VI, JP7.2
- new net N$54: DC9-1.KL
- new net N$55: C63.P$1, D8.A, IC5.VI, JP8.1
- new net N$57: LED5.A, R38.1
- new net N$62: LED3.A, R36.1
- new net N$63: LED4.A, R37.1
- net +12V: now also C62.P$2, D5.A, D6.C, DC12-3.KL, IC6.VO, R36.2
- net -12V: now also C64.P$1, D7.A, D8.C, DC12-1.KL, IC5.VO, LED4.C
- net GND: now also AC_IN-2.KL, C57.-, C58.+, C59.2, C60.1, C61.P$1, C62.P$1, C63.P$2, C64.P$2, C65.P$1, C66.P$1, D6.A, D7.C, D9.A, DC12-2.KL, DC17-2.KL, IC5.GND, IC6.GND, IC7.GND, LED1.C, LED3.C, LED5.C, R35.2, R37.2
Other:
- note added: "Input from AC transfomer, +/-12v"

Commit message: wip
Parts:
- removed AC_IN, DC12, DC17: (no value), con-ptr500:AK500/3
- removed C56: 220pF 50V (VJ0603Y221KXACW1BC), microbuilder:CAP_CERAMIC0603
- removed C57, C58: 2200uF 50v UHE1H222MHD6, rcl:CPOL-USE7.5-18
- removed C59, C60: 1uF BFC237011105, capacitor-wima:C5/7.2
- removed C61, C62, C63, C64, C65, C66: 4.7uF, microbuilder:CAP_CERAMIC0603
- removed D1, D2, D3, D4: MUR820, diode:MUR820
- removed D5, D6, D7, D8, D9: 1N4004, diode:1N4004
- removed DC9: (no value), con-ptr500:AK500/2
- removed IC5: 7912, linear:7912T
- removed IC6: 7812T, linear:7812T
- removed IC7: 7809, linear:7812T
- removed JP11, JP7, JP8: (no value), microbuilder:HEADER-1X2ROUND
- removed LED1, LED2, LED3, LED4, LED5: (no value), microbuilder:LED0603
- removed R34, R35: 1K, microbuilder:RESISTOR0603
- removed R36, R37: 680, microbuilder:RESISTOR0603
- removed R38: 470, microbuilder:RESISTOR0603
- added DC_12: (no value), con-ptr500:AK500/3
- added U$30: ADP3301ARZ-5, keves:ADP3301
- added X1: (no value), con-ptr500:AK500/2
- C53: value 220pF 50V (VJ0603Y221KXACW1BC) -> 2.2uF (EMK107BB7225KA-T)
- C54: value 220pF 50V (VJ0603Y221KXACW1BC) -> 0.01uF
- C55: value 220pF 50V (VJ0603Y221KXACW1BC) -> 10uF
Connections:
- removed net +17: C53.P$2, C54.P$1, C57.+, C59.1, D1.C, D2.C, DC17-3.KL, JP11.1, JP7.1, R34.2
- removed net -17: C55.P$2, C56.P$1, C58.-, C60.2, D3.A, D4.A, DC17-1.KL, JP8.2, LED2.C
- removed net N$46: AC_IN-1.KL, C53.P$1, C56.P$2, D1.A, D3.C
- removed net N$49: LED2.A, R35.1
- removed net N$50: LED1.A, R34.1
- removed net N$51: C61.P$2, D5.C, IC6.VI, JP7.2
- removed net N$54: DC9-1.KL
- removed net N$55: C63.P$1, D8.A, IC5.VI, JP8.1
- removed net N$57: LED5.A, R38.1
- removed net N$62: LED3.A, R36.1
- removed net N$63: LED4.A, R37.1
- net +12V: now also DC_12-1.KL; no longer C62.P$2, D5.A, D6.C, DC12-3.KL, IC6.VO, R36.2
- net +9V: now also C53.P$2, U$30.IN1, U$30.IN2, U$30.SD, X1-1.KL; no longer C65.P$2, C66.P$2, D9.C, DC9-2.KL, IC7.VI, IC7.VO, JP11.2, R38.2
- net -12V: now also DC_12-3.KL; no longer C64.P$1, D7.A, D8.C, DC12-1.KL, IC5.VO, LED4.C
- net 3.3V: now also C54.P$2, C55.P$2, U$30.OUT1, U$30.OUT2
- net GND: now also C53.P$1, C55.P$1, DC_12-2.KL, U$30.GND, X1-2.KL; no longer AC_IN-2.KL, C57.-, C58.+, C59.2, C60.1, C61.P$1, C62.P$1, C63.P$2, C64.P$2, C65.P$1, C66.P$1, D6.A, D7.C, D9.A, DC12-2.KL, DC17-2.KL, IC5.GND, IC6.GND, IC7.GND, LED1.C, LED3.C, LED5.C, R35.2, R37.2
- net N$47: now also C54.P$1, U$30.NR; no longer AC_IN-3.KL, C54.P$2, C55.P$1, D2.A, D4.C
Other:
- note removed: "Input from AC transfomer, +/-12v"

Commit message: wip
Parts:
- removed X1: (no value), con-ptr500:AK500/2
- added C56: 2.2uF (EMK107BB7225KA-T), microbuilder:CAP_CERAMIC0603
- added C57, C59, C62, C65: 0.1uF, microbuilder:CAP_CERAMIC0603
- added C58, C63, C64: 10uF, microbuilder:CAP_CERAMIC0603
- added C60, C61: 100uF EMVE160ADA101MF55G, SparkFun-Capacitors:CAP_POLD
- added DC_9: (no value), con-ptr500:AK500/2
- added EN_3.3, EN_DAC_VCC, EN_DAC_VREF: (no value), microbuilder:HEADER-1X2
- added IC5: REG1117-5, burr-brown:REG1117
- added U$43: ADR02, keves:ADR02
- U$30: value ADP3301ARZ-5 -> ADP3301ARZ-3.3
Connections:
- new net N$46: C54.P$2, C55.P$2, EN_3.3.1, U$30.OUT1, U$30.OUT2
- new net N$48: C58.P$2, C59.P$2, EN_DAC_VREF.1, U$43.VOUT
- new net N$51: C64.P$1, C65.P$1, EN_DAC_VCC.1, IC5.VOUT
- net +12V: now also C60.+
- net +9V: now also C56.P$1, C57.P$2, C62.P$1, C63.P$2, DC_9-1.KL, IC5.VIN, U$43.VIN; no longer X1-1.KL
- net -12V: now also C61.-
- net 3.3V: now also EN_3.3.2; no longer C54.P$2, C55.P$2, U$30.OUT1, U$30.OUT2
- net DAC_VCC: now also EN_DAC_VCC.2
- net DAC_VREF: now also EN_DAC_VREF.2
- net GND: now also C56.P$2, C57.P$1, C58.P$1, C59.P$1, C60.-, C61.+, C62.P$2, C63.P$1, C64.P$2, C65.P$2, DC_9-2.KL, IC5.GND, U$43.GND; no longer X1-2.KL
Other:
- note added: "TODOs: - DAC_VREF - DAC_VCC"
- note removed: "TODOs: - AVCC Supply - +/-12V Supply - Connect AGND to GND"
- moved on the sheet: DC_12-1, DC_12-2, DC_12-3

Commit message: wip
Parts:
- removed JP3, JP4: (no value), microbuilder:HEADER-1X2ROUND
Connections:
- removed net DAC_CLK: JP1.3
- removed net DAC_CS: JP1.1
- removed net DAC_MISO: JP1.7
- removed net DAC_MOSI: JP1.5
- removed net DAC_RST_: DAC.RST_, JP1.10, R33.1
- removed net N$44: C43.P$1, C44.P$1, C45.P$1, C46.P$1, DAC.VREF1+, DAC.VREF2+, DAC.VREF3+, DAC.VREF4+, JP3.1
- removed net N$45: C47.P$2, C48.P$2, C49.P$2, C50.P$2, DAC.VCC1, DAC.VCC2, JP4.1
- removed net SAI_BCK: JP2.3
- removed net SAI_D0: JP2.7
- removed net SAI_D1: JP2.9
- removed net SAI_LRCK: JP2.5
- removed net SAI_SCK: JP2.1
- net DAC_RST: now also DAC.RST_, JP1.10, R33.1; no longer JP1.9
- net DAC_VCC: now also C47.P$2, C48.P$2, C49.P$2, C50.P$2, DAC.VCC1, DAC.VCC2; no longer JP4.2
- net DAC_VREF: now also C43.P$1, C44.P$1, C45.P$1, C46.P$1, DAC.VREF1+, DAC.VREF2+, DAC.VREF3+, DAC.VREF4+; no longer JP3.2
- net GND: now also JP1.1, JP1.3, JP1.5, JP1.7, JP1.9, JP2.1, JP2.3, JP2.5, JP2.7, JP2.9
Other:
- moved on the sheet: JP1, JP2

Commit message: wip
Connections:
- net N$35 renamed DAC_CS
- net N$36 renamed DAC_CLK
- net N$37 renamed DAC_MOSI
- net N$38 renamed DAC_MISO
- net N$39 renamed DAC_SCK
- net N$40 renamed DAC_BCK
- net N$41 renamed DAC_LRCK
- net N$42 renamed DAC_D0
- net N$43 renamed DAC_D1
Changed lines of the file:
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@@
 </segment>
 </net>
-<net name="N$35" class="0">
+<net name="DAC_CS" class="0">
 <segment>
 <pinref part="DAC" gate="G$1" pin="CS_"/>
@@
 </segment>
 </net>
-<net name="N$36" class="0">
+<net name="DAC_CLK" class="0">
 <segment>
 <pinref part="DAC" gate="G$1" pin="CCLK"/>
@@
 </segment>
 </net>
-<net name="N$37" class="0">
+<net name="DAC_MOSI" class="0">
 <segment>
 <pinref part="DAC" gate="G$1" pin="CDIN"/>
@@
 </segment>
 </net>
-<net name="N$38" class="0">
+<net name="DAC_MISO" class="0">
 <segment>
 <pinref part="DAC" gate="G$1" pin="CDOUT"/>
@@
 </segment>
 </net>
-<net name="N$39" class="0">
+<net name="DAC_SCK" class="0">
 <segment>
 <pinref part="DAC" gate="G$1" pin="SCKI"/>
@@
 </segment>
 </net>
-<net name="N$40" class="0">
+<net name="DAC_BCK" class="0">
 <segment>
 <pinref part="DAC" gate="G$1" pin="BCK"/>
@@
 </segment>
 </net>
-<net name="N$41" class="0">
+<net name="DAC_LRCK" class="0">
 <segment>
 <pinref part="DAC" gate="G$1" pin="LRCK"/>
@@
 </segment>
 </net>
-<net name="N$42" class="0">
+<net name="DAC_D0" class="0">
 <segment>
 <pinref part="DAC" gate="G$1" pin="DATA0"/>
@@
 </segment>
 </net>
-<net name="N$43" class="0">
+<net name="DAC_D1" class="0">
 <segment>
 <pinref part="DAC" gate="G$1" pin="DATA1"/>

Commit message: wip
Other:
- note removed: "TODOs: - DAC_VREF - DAC_VCC"
Changed lines of the file:
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@@
 <sheet>
 <plain>
-<text x="81.28" y="111.76" size="1.778" layer="91">TODOs:
-- DAC_VREF
-- DAC_VCC</text>
 </plain>
 <instances>
@@
 </schematic>
 </drawing>
-<compatibility>
-<note version="6.3" minversion="6.2.2" severity="warning">
-Since Version 6.2.2 text objects can contain more than one line,
-which will not be processed correctly with this version.
-</note>
-</compatibility>
 </eagle>

Commit message: wip
Parts:
- removed C32, C33: 100uF EMVE160ADA101MF55G, SparkFun-Capacitors:CAP_POLD
- added C67: 22pF VJ0805A220FXBPW1BC, microbuilder:CAP_CERAMIC0805
- C1, C11, C21, C31: value 22pF -> 22pF VJ0603A220JXACW1BC
- C10: value 560pF ECH-U1H561JX5 -> 27pF CC0805FRNPO9BN270
- C39, C40: value 560pF ECH-U1H561JX5 -> 680pF ECH-U1H681JX5
- C4: value 2200pF ECH-U1H222JX5 -> 100pF ECH-U1H101JX5
- C9: value 560pF ECH-U1H561JX5 -> 22pF VJ0805A220FXBPW1BC
- IC1: value NE5534AD -> ISL28110
- IC4: value NE5534AD -> OPA227
- R1, R2: value 604 0.1% -> 12k 0.1%
- R25, R26: value 604 0.1% -> 820 0.1%
- R27, R28: value 499 0.1% -> 910 0.1%
- R29, R30: value 1K 0.1% -> 1.6K 0.1%
- R3, R4: value 499 0.1% -> 10k 0.1%
- R5, R6: value 1K 0.1% -> 20K 0.1%
Connections:
- removed net N$25: C32.-, R25.1
- removed net N$26: C33.-, R26.1
- new net N$35: C67.P$1, IC3.CMP
- new net N$36: C67.P$2, IC3.ON/CMP
- net OUT4+: now also R26.1; no longer C33.+
- net OUT4-: now also R25.1; no longer C32.+
Other:
- note added: "Filter 1 (JFET)"
- note added: "Filter 2 (NE5534 + Cap)"
- note added: "Filter 3 (NE5534)"
- note added: "Filter 4 (OPA227)"
