File: midimixer-channel/compressor.sch (EAGLE design)
At the start: 11 parts, among them J1 STEREOSW, U1 THAT4301P20-I

Commit message: compressor
Parts:
- added C5: 100n MKS4F031002C00KSSD, capacitor-wima:C7.5/4
- added C6: 47u, rcl:CPOL-USB45181D
- added MASTER_OUT: STEREOSW, pl-jacks:STEREOSW
- added R10: 2M, rcl:R-US_0204/7
- added R6: 5.1k 3300ppm (TFPTL15L5001FL2B), rcl:R-US_0204/7
- added R7: 30.1k, rcl:R-US_0204/7
- added R8: 590k, rcl:R-US_0204/7
- added R9: 28.8k, rcl:R-US_0204/7
- added U$9: 10k PTV111-1415A-B1103, keves:PTV111-1
- renumbered J1 to MASTER_IN
Connections:
- new net N$10: R7.2
- new net N$11: R8.2, U$9.S
- new net N$12: C6.+
- new net N$13: C6.-, R9.1
- new net N$14: R9.2, U1-RMS.RMS-IN
- new net N$15: R10.1, U1-RMS.RMS-IT
- new net N$8: C5.1, R6.1, U1-OA2.OUT, U1-VCA.EC-
- new net N$9: C5.2, R6.2, R7.1, R8.1, U1-OA2.-IN
- net +15V: now also U$9.A
- net -15V: now also R10.2, U$9.E
- net GND: now also MASTER_OUT.R, MASTER_OUT.S, U1-OA2.+IN
- net N$5: now also MASTER_OUT.T
Other:
- moved on the sheet: U1-OA2, U1-RMS

Commit message: wip
Parts:
- added C7: 470n MKS2D034701E00JSSD, capacitor-wima:C5/4.5
- added C8: 47n BFC247086473, capacitor-wima:C5/7.2
- added C9: 2n C326C202J1G5CA7301, capacitor-wima:C5/2.5
- added IC1: NE5532N, linear:NE5532N
- added LED1, LED2: (no value), led:LED5MM
- added R11: 150, rcl:R-US_0204/7
- added R12: 2M, rcl:R-US_0204/7
Connections:
- removed net N$12: C6.+
- new net N$16: C7.2, R11.1
- new net N$17: C7.1, C8.1, U1-RMS.RMS-CT
- new net N$18: C9.1, IC1B.OUT, LED1.C, LED2.A, R11.2, R12.2
- new net N$19: C8.2, C9.2, IC1B.-IN, LED1.A, LED2.C, R12.1
- net +15V: now also IC1P.V+
- net -15V: now also IC1P.V-
- net GND: now also IC1B.+IN
- net N$1: now also C6.+
Changed lines of the file:
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@@
 <part name="R10" library="rcl" deviceset="R-US_" device="0204/7" value="2M"/>
 <part name="P-4" library="supply1" deviceset="-15V" device=""/>
+<part name="C7" library="capacitor-wima" deviceset="C" device="5/4.5" value="470n MKS2D034701E00JSSD"/>
+<part name="R11" library="rcl" deviceset="R-US_" device="0204/7" value="150"/>
+<part name="C8" library="capacitor-wima" deviceset="C" device="5/7.2" value="47n BFC247086473"/>
+<part name="R12" library="rcl" deviceset="R-US_" device="0204/7" value="2M"/>
+<part name="C9" library="capacitor-wima" deviceset="C" device="5/2.5" value="2n C326C202J1G5CA7301"/>
+<part name="LED1" library="led" deviceset="LED" device="5MM"/>
+<part name="LED2" library="led" deviceset="LED" device="5MM"/>
+<part name="IC1" library="linear" deviceset="NE5532" device="N"/>
+<part name="P-5" library="supply1" deviceset="-15V" device=""/>
+<part name="P+4" library="supply1" deviceset="+15V" device=""/>
+<part name="U$10" library="microbuilder" deviceset="GND" device=""/>
 </parts>
 <sheets>
@@
 <instance part="R10" gate="G$1" x="55.88" y="-55.88" rot="R270"/>
 <instance part="P-4" gate="1" x="55.88" y="-68.58"/>
+<instance part="C7" gate="G$1" x="96.52" y="-58.42" rot="R90"/>
+<instance part="R11" gate="G$1" x="111.76" y="-58.42"/>
+<instance part="C8" gate="G$1" x="88.9" y="-66.04"/>
+<instance part="R12" gate="G$1" x="111.76" y="-78.74"/>
+<instance part="C9" gate="G$1" x="111.76" y="-86.36" rot="R270"/>
+<instance part="LED1" gate="G$1" x="109.22" y="-96.52" rot="R90"/>
+<instance part="LED2" gate="G$1" x="109.22" y="-106.68" rot="R270"/>
+<instance part="IC1" gate="A" x="-43.18" y="-66.04"/>
+<instance part="IC1" gate="B" x="104.14" y="-134.62" rot="MR180"/>
+<instance part="IC1" gate="P" x="104.14" y="-134.62"/>
+<instance part="P-5" gate="1" x="104.14" y="-147.32"/>
+<instance part="P+4" gate="1" x="104.14" y="-121.92"/>
+<instance part="U$10" gate="G$1" x="88.9" y="-139.7"/>
 </instances>
 <busses>
@@
 <junction x="2.54" y="48.26"/>
 <wire x1="2.54" y1="48.26" x2="-2.54" y2="48.26" width="0.1524" layer="91"/>
-<wire x1="2.54" y1="48.26" x2="2.54" y2="-5.08" width="0.1524" layer="91"/>
+<wire x1="2.54" y1="48.26" x2="2.54" y2="-40.64" width="0.1524" layer="91"/>
+<pinref part="C6" gate="G$1" pin="+"/>
+<wire x1="15.24" y1="-40.64" x2="2.54" y2="-40.64" width="0.1524" layer="91"/>
 </segment>
 </net>
@@
 <wire x1="63.5" y1="-20.32" x2="63.5" y2="-17.78" width="0.1524" layer="91"/>
 </segment>
+<segment>
+<pinref part="IC1" gate="B" pin="+IN"/>
+<pinref part="U$10" gate="G$1" pin="GND"/>
+<wire x1="88.9" y1="-137.16" x2="96.52" y2="-137.16" width="0.1524" layer="91"/>
+</segment>
 </net>
 <net name="N$2" class="0">
@@
 <wire x1="55.88" y1="-66.04" x2="55.88" y2="-60.96" width="0.1524" layer="91"/>
 </segment>
+<segment>
+<pinref part="IC1" gate="P" pin="V-"/>
+<pinref part="P-5" gate="1" pin="-15V"/>
+<wire x1="104.14" y1="-144.78" x2="104.14" y2="-142.24" width="0.1524" layer="91"/>
+</segment>
 </net>
 <net name="+15V" class="0">
@@
 <pinref part="P+3" gate="1" pin="+15V"/>
 <wire x1="88.9" y1="-5.08" x2="88.9" y2="-7.62" width="0.1524" layer="91"/>
+</segment>
+<segment>
+<pinref part="IC1" gate="P" pin="V+"/>
+<pinref part="P+4" gate="1" pin="+15V"/>
+<wire x1="104.14" y1="-124.46" x2="104.14" y2="-127" width="0.1524" layer="91"/>
 </segment>
 </net>
@@
 </segment>
 </net>
-<net name="N$12" class="0">
-<segment>
-<pinref part="C6" gate="G$1" pin="+"/>
-<wire x1="15.24" y1="-40.64" x2="2.54" y2="-40.64" width="0.1524" layer="91"/>
-<wire x1="2.54" y1="-40.64" x2="2.54" y2="-7.62" width="0.1524" layer="91"/>
-</segment>
-</net>
 <net name="N$13" class="0">
 <segment>
@@
 </segment>
 </net>
+<net name="N$16" class="0">
+<segment>
+<pinref part="C7" gate="G$1" pin="2"/>
+<pinref part="R11" gate="G$1" pin="1"/>
+<wire x1="106.68" y1="-58.42" x2="101.6" y2="-58.42" width="0.1524" layer="91"/>
+</segment>
+</net>
+<net name="N$17" class="0">
+<segment>
+<pinref part="U1" gate="-RMS" pin="RMS-CT"/>
+<pinref part="C8" gate="G$1" pin="1"/>
+<wire x1="86.36" y1="-45.72" x2="88.9" y2="-45.72" width="0.1524" layer="91"/>
+<wire x1="88.9" y1="-45.72" x2="88.9" y2="-58.42" width="0.1524" layer="91"/>
+<pinref part="C7" gate="G$1" pin="1"/>
+<wire x1="88.9" y1="-58.42" x2="88.9" y2="-63.5" width="0.1524" layer="91"/>
+<wire x1="93.98" y1="-58.42" x2="88.9" y2="-58.42" width="0.1524" layer="91"/>
+<junction x="88.9" y="-58.42"/>
+</segment>
+</net>
+<net name="N$18" class="0">
+<segment>
+<pinref part="R11" gate="G$1" pin="2"/>
+<wire x1="116.84" y1="-58.42" x2="119.38" y2="-58.42" width="0.1524" layer="91"/>
+<wire x1="119.38" y1="-58.42" x2="119.38" y2="-78.74" width="0.1524" layer="91"/>
+<pinref part="R12" gate="G$1" pin="2"/>
+<wire x1="119.38" y1="-78.74" x2="119.38" y2="-86.36" width="0.1524" layer="91"/>
+<wire x1="119.38" y1="-86.36" x2="119.38" y2="-96.52" width="0.1524" layer="91"/>
+<wire x1="119.38" y1="-96.52" x2="119.38" y2="-106.68" width="0.1524" layer="91"/>
+<wire x1="119.38" y1="-106.68" x2="119.38" y2="-134.62" width="0.1524" layer="91"/>
+<wire x1="119.38" y1="-78.74" x2="116.84" y2="-78.74" width="0.1524" layer="91"/>
+<pinref part="C9" gate="G$1" pin="1"/>
+<wire x1="114.3" y1="-86.36" x2="119.38" y2="-86.36" width="0.1524" layer="91"/>
+<pinref part="LED1" gate="G$1" pin="C"/>
+<wire x1="114.3" y1="-96.52" x2="119.38" y2="-96.52" width="0.1524" layer="91"/>
+<wire x1="111.76" y1="-106.68" x2="119.38" y2="-106.68" width="0.1524" layer="91"/>
+<pinref part="LED2" gate="G$1" pin="A"/>
+<junction x="119.38" y="-106.68"/>
+<junction x="119.38" y="-96.52"/>
+<junction x="119.38" y="-86.36"/>
+<junction x="119.38" y="-78.74"/>
+<pinref part="IC1" gate="B" pin="OUT"/>
+<wire x1="111.76" y1="-134.62" x2="119.38" y2="-134.62" width="0.1524" layer="91"/>
+</segment>
+</net>
+<net name="N$19" class="0">
+<segment>
+<pinref part="C8" gate="G$1" pin="2"/>
+<wire x1="88.9" y1="-71.12" x2="88.9" y2="-78.74" width="0.1524" layer="91"/>
+<pinref part="R12" gate="G$1" pin="1"/>
+<wire x1="88.9" y1="-78.74" x2="88.9" y2="-86.36" width="0.1524" layer="91"/>
+<wire x1="88.9" y1="-86.36" x2="88.9" y2="-96.52" width="0.1524" layer="91"/>
+<wire x1="88.9" y1="-96.52" x2="88.9" y2="-106.68" width="0.1524" layer="91"/>
+<wire x1="88.9" y1="-106.68" x2="88.9" y2="-132.08" width="0.1524" layer="91"/>
+<wire x1="106.68" y1="-78.74" x2="88.9" y2="-78.74" width="0.1524" layer="91"/>
+<pinref part="C9" gate="G$1" pin="2"/>
+<wire x1="106.68" y1="-86.36" x2="88.9" y2="-86.36" width="0.1524" layer="91"/>
+<pinref part="LED1" gate="G$1" pin="A"/>
+<wire x1="106.68" y1="-96.52" x2="88.9" y2="-96.52" width="0.1524" layer="91"/>
+<pinref part="LED2" gate="G$1" pin="C"/>
+<wire x1="104.14" y1="-106.68" x2="88.9" y2="-106.68" width="0.1524" layer="91"/>
+<junction x="88.9" y="-78.74"/>
+<junction x="88.9" y="-86.36"/>
+<junction x="88.9" y="-96.52"/>
+<junction x="88.9" y="-106.68"/>
+<pinref part="IC1" gate="B" pin="-IN"/>
+<wire x1="96.52" y1="-132.08" x2="88.9" y2="-132.08" width="0.1524" layer="91"/>
+</segment>
+</net>

Commit message: wip
Parts:
- removed U$9: 10k PTV111-1415A-B1103, keves:PTV111-1
- added C10: 22p K220J10C0GF5UH5, rcl:C-EU050-035X075
- added D1, D2, D3: 1N4148DO35-7, diode:1N4148DO35-7
- added HARD/SOFT, VARIABLE/AUTO: 108-1MD1T1B1M2QE-EVX, keves:108-1MD1T1B1M2QE-EVX
- added R13: 5.1k 3300ppm (TFPTL15L5001FL2B), rcl:R-US_0204/7
- added R14, R16, R20: 30.1k, rcl:R-US_0204/7
- added R15: 590k, rcl:R-US_0204/7
- added R17: 220k, rcl:R-US_0204/7
- added R18: 1.4k, rcl:R-US_0204/7
- added R19: 15k, rcl:R-US_0204/7
- added U$11, U$13: 10k RK09D1130C2P, keves:ALPS-RK09D
- added U$12: 50k RK09D1130A1L, keves:ALPS-RK09D
Connections:
- new net N$12: R13.1, U1-RMS.RMS-OUT
- new net N$20: C10.2, D1.C, R13.2, R14.1, R15.2, R16.2, U1-OA1.-IN
- new net N$21: R15.1, U$12.S
- new net N$22: HARD/SOFT.P1, R14.2
- new net N$23: C10.1, D1.A, D2.C, HARD/SOFT.S1, U1-OA1.OUT
- new net N$24: D2.A, HARD/SOFT.O1, R18.2, U$13.A
- new net N$25: HARD/SOFT.P, R16.1
- new net N$26: D3.A, HARD/SOFT.S, R17.1
- new net N$28: R18.1, R19.1, U$13.S, VARIABLE/AUTO.P, VARIABLE/AUTO.S1
- new net N$29: R20.2, VARIABLE/AUTO.O1
- new net N$30: VARIABLE/AUTO.O
- net +15V: now also R17.2, U$11.A, U$12.E; no longer U$9.A
- net -15V: now also U$11.E, U$12.A; no longer U$9.E
- net GND: now also D3.C, R19.2, U$13.E, U1-OA1.+IN
- net N$10: now also VARIABLE/AUTO.P1
- net N$11: now also U$11.S; no longer U$9.S
Other:
- moved on the sheet: U1-OA1

Commit message: wip
Parts:
- added ATTACK: 10k RK09D1130C2P, keves:ALPS-RK09D
- added C11: 4.7u 515D475M050JA6AE3, rcl:CPOL-USE2-5
- added D4, D5, D6, D7: 1N4148DO35-7, diode:1N4148DO35-7
- added IC2: LM393N, linear:LM393N
- added Q1, Q2, Q3: 2N3906, transistor-pnp:2N3906
- added R21, R25: 5.1k, rcl:R-US_0204/7
- added R22: 127k, rcl:R-US_0204/7
- added R23: 510, rcl:R-US_0204/7
- added R24: 18M, rcl:R-US_0204/7
- added R26: 10k, rcl:R-US_0204/7
- added R27: 30.1k, rcl:R-US_0204/7
- added R28: 1.8M, rcl:R-US_0204/7
- added R29: 12.7k, rcl:R-US_0204/7
- added R30: 51, rcl:R-US_0204/7
- added RELEASE: 50k RK09D1130A1L, keves:ALPS-RK09D
- added T1, T2, T3: 2N3904, transistor:2N3904
- added U$17: J113, keves:J113
Connections:
- new net N$27: IC2A.-IN, R20.1, R21.1, R26.1, U$17.S
- new net N$31: C11.+, D4.C, D5.A, U$17.G
- new net N$32: D5.C, D7.C, T1.C
- new net N$33: D4.A, D6.A, Q1.C
- new net N$34: R22.2, RELEASE.S
- new net N$35: D6.C, D7.A, IC2A.OUT, R25.2
- new net N$36: Q2.E, R22.1, R23.2
- new net N$37: Q1.B, Q2.B, Q3.E
- new net N$38: Q2.C, Q3.B, R24.1
- new net N$39: T1.B, T2.E, T3.B
- new net N$40: R28.2, T2.B, T3.C
- new net N$44: ATTACK.S, R29.1
- new net N$45: R29.2, R30.2, T3.E
- net +15V: now also ATTACK.E, IC2P.V+, Q1.E, R23.1, R25.1, R28.1, RELEASE.E, T2.C, U$17.D
- net -15V: now also ATTACK.A, C11.-, IC2P.V-, Q3.C, R21.2, R24.2, R30.1, RELEASE.A, T1.E
- net GND: now also R26.2, R27.2
- net N$30: now also IC2A.+IN, R27.1
Other:
- moved on the sheet: R20

Commit message: wip
Parts:
- removed MASTER_IN, MASTER_OUT: STEREOSW, pl-jacks:STEREOSW
- added C12: 220u UFW1H221MPD, rcl:CPOL-USE5-10.5
- added C13, C14: 0.1u MKS4F031002C00KSSD, capacitor-wima:C7.5/4
- added C15: 10n K103K10X7RH5TH5 DNP, rcl:C-EU050-025X075
- added IN, OUT: (no value), con-ptr500:AK500/2
- added R31: 2M DNP?, rcl:R-US_0204/7
- added R32: 100, rcl:R-US_0204/7
- R15: value 590k -> 590k OR 390k
- renumbered U$11 to GAIN, U$12 to THRESHOLD, U$13 to RATIO
Connections:
- new net N$41: C12.+, C13.2, OUT-2.KL
- new net N$42: R32.2, U1-OA1.OUT
- net -15V: now also R31.1
- net GND: now also C15.1, IN-1.KL, OUT-1.KL; no longer MASTER_IN.S, MASTER_OUT.R, MASTER_OUT.S
- net N$1: now also C14.2, IN-2.KL; no longer MASTER_IN.T
- net N$17: now also C15.2
- net N$2: now also C14.1
- net N$20: now also R31.2
- net N$23: now also R32.1; no longer U1-OA1.OUT
- net N$5: now also C12.-, C13.1; no longer MASTER_OUT.T
Other:
- note added: "TODO: - PSU connector - Level meters - Sidechain"

Commit message: wip
Parts:
- added C16, C18, C21: 0.1uF K104K15X7RF53L2, rcl:C-EU025-024X044
- added C17, C19, C20: 22u RNS1D220MDS1, rcl:CPOL-USE2.5-7
- added D8: DC7G3HWA, SparkFun-LED:LED_BARGRAPH_10
- added IC3: LM3914N, linear:LM3914N
- added IC4: TL072P, linear:TL072P
- added IC5: 78L05Z, linear:78L05Z
- added PWR: (no value), con-ptr500:AK500/3
- added R33: 1.2k DNP, rcl:R-US_0204/7
- added R34, R37, R38: 10, rcl:R-US_0204/7
- added R35: 91k, rcl:R-US_0204/7
- added R36: 9.53k (20dB) / 4.75k (10dB) / 2.4k (5dB), rcl:R-US_0204/7
Connections:
- new net GR_METER: IC4A.+IN, R7.2, VARIABLE/AUTO.P1
- new net N$43: D8J.C, IC3.L10
- new net N$46: D8I.C, IC3.L9
- new net N$47: D8H.C, IC3.L8
- new net N$48: D8G.C, IC3.L7
- new net N$49: D8F.C, IC3.L6
- new net N$50: D8E.C, IC3.L5
- new net N$51: D8D.C, IC3.L4
- new net N$52: D8C.C, IC3.L3
- new net N$53: D8B.C, IC3.L2
- new net N$54: D8A.C, IC3.L1
- new net N$55: IC3.RHI, IC3.VR, R33.1
- new net N$56: IC3.ADJ, R33.2
- new net N$58: IC3.SIG, IC4B.OUT, R35.2
- new net N$59: IC4B.-IN, R35.1, R36.2
- new net N$60: IC4A.-IN, IC4A.OUT, R36.1
- new net N$61: C18.2, C19.-, IC4P.V-, R37.2
- new net N$62: C20.+, D8A.A, D8B.A, D8C.A, D8D.A, D8E.A, D8F.A, D8G.A, D8H.A, D8I.A, D8J.A, R38.2
- new net N$63: C16.2, C17.+, C21.2, IC3.MDE, IC3.V+, IC4P.V+, IC5.VI, R34.2
- net +15V: now also PWR-1.KL, R34.1
- net -15V: now also PWR-3.KL, R37.1
- net GND: now also C16.1, C17.-, C18.1, C19.+, C20.-, C21.1, IC3.RLO, IC3.V-, IC4B.+IN, IC5.GND, PWR-2.KL
- net N$10: now also IC5.VO, R38.1; no longer R7.2, VARIABLE/AUTO.P1
Other:
- note added: "J/I/H are RED"
- note added: "TODO: - Sidechain"
- note removed: "TODO: - PSU connector - Level meters - Sidechain"

Commit message: wip
Parts:
- ATTACK, C10, C11, C12, C13, C14, C15, C16, C17, C18, C19, C2, C20, C21, C3, C4, C5, C7, C8, C9, D1, D2, D3, D4, D5, D6, D7, D8, GAIN, HARD/SOFT, IC1, IC2, IC3, IC4, IC5, LED1, LED2, Q1, Q2, Q3, R1, R10, R11, R12, R13, R14, R15, R16, R17, R18, R19, R2, R20, R21, R22, R23, R24, R25, R26, R27, R28, R29, R3, R30, R31, R32, R33, R34, R35, R36, R37, R38, R4, R5, R6, R7, R8, R9, RATIO, RELEASE, T1, T2, T3, THRESHOLD, U$17, U1, VARIABLE/AUTO: OC_NEWARK (none) -> unknown
- C1, C6: MPN (none) -> ERJ-1TRQFR47U; OC_NEWARK (none) -> 01X1464
Connections:
- removed net N$28: R18.1, R19.1, RATIO.S, VARIABLE/AUTO.P, VARIABLE/AUTO.S1
- removed net N$56: IC3.ADJ, R33.2
- net GND: now also IC3.ADJ, R33.2
- net GR_METER: now also R18.1, R19.1, RATIO.S, VARIABLE/AUTO.P, VARIABLE/AUTO.S1
Other:
- moved on the sheet: R33

Commit message: wip
Parts:
- added BYPASS_SW, SC_SW: 108-1MD1T1B1M2QE-EVX, keves:108-1MD1T1B1M2QE-EVX
- added COMP_ON, SC_ON: (no value), led:LED5MM
- added R39, R40: 1k, rcl:R-US_0204/7
- added SC: (no value), con-ptr500:AK500/2
Connections:
- new net N$28: SC_ON.C, SC_SW.O
- new net N$56: R39.2, SC_ON.A
- new net N$57: BYPASS_SW.P, OUT-2.KL
- new net N$64: BYPASS_SW.O1, COMP_ON.C
- new net N$65: COMP_ON.A, R40.2
- new net SC_IN: C6.+, SC_SW.P1
- new net SIG_IN: BYPASS_SW.S, C1.+, C14.2, IN-2.KL, SC_SW.S1
- net +15V: now also R39.1, R40.1
- net GND: now also BYPASS_SW.P1, SC-1.KL, SC_SW.P
- net N$1: now also SC-2.KL, SC_SW.O1; no longer C1.+, C14.2, C6.+, IN-2.KL
- net N$41: now also BYPASS_SW.O; no longer OUT-2.KL
Other:
- note added: "TODO: - Sidechain - Bypass"
- note removed: "TODO: - Sidechain"
- moved on the sheet: IN-1, IN-2, OUT-1, OUT-2
