File: midimixer-channel/midimixer-channel-before-rearrangement.sch (EAGLE design)
At the start: 113 parts, among them IC1 74LS595D, IC2 74LS595D, IC3 74LS595D, IC4 74165D, IC5 74165D, U1 LM1117IMPX-3.3/NOPB

Commit message: midimixer-channel wip
Parts:
- removed U$19: ABM7-8.000MHZ-D2Y-T, keves:ABM7-8.000MHZ-D2Y-T
- added R15, R16: 22, microbuilder:RESISTOR0603
- added USB: (no value), microbuilder:HEADER-1X4ROUND
- added VBUS: (no value), microbuilder:JUMPER2
- added Y1: 8MHz 695-HCM49-8-U, microbuilder:CRYSTALSMD
- LCD: value SSD1306-7PINWITHOUT-HOLES -> SSD1306-7PIN; device keves:SSD1306-7PINWITHOUT-HOLES -> keves:SSD1306-7PIN
Connections:
- new net N$7: R15.2, USB.2
- new net N$8: R16.2, USB.3
- new net USB_DM: CPU1.PA11, R15.1
- new net USB_DP: CPU1.PA12, R16.1
- net 5.0V: now also VBUS.1
- net ADC0: now also POT2.WIPER; no longer FADER1.S
- net ADC7: now also FADER1.S; no longer POT2.WIPER
- net CAN_H: now also BUS1.2, BUS2.2; no longer BUS1.3, BUS2.3
- net CAN_L: now also BUS1.3, BUS2.3; no longer BUS1.2, BUS2.2
- net GND: now also USB.4
- net N$1: now also Y1.1; no longer U$19.1
- net N$2: now also Y1.2; no longer U$19.2
- net USB_VBUS: now also USB.1, VBUS.2
Changed lines of the file:
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@@
 <part name="CPU1" library="SparkFun-DigitalIC" deviceset="STM32F405RG" device=""/>
 <part name="U$2" library="microbuilder" deviceset="3.3V" device=""/>
+<part name="Y1" library="microbuilder" deviceset="CRYSTAL" device="SMD" value="8MHz 695-HCM49-8-U"/>
 <part name="C5" library="microbuilder" deviceset="CAP_CERAMIC" device="0603" value="18pf"/>
 <part name="C6" library="microbuilder" deviceset="CAP_CERAMIC" device="0603" value="18pf"/>
@@
 <part name="R12" library="microbuilder" deviceset="RESISTOR" device="_0603" value="10k"/>
 <part name="U$17" library="microbuilder" deviceset="GND" device=""/>
+<part name="U$19" library="microbuilder" deviceset="GND" device=""/>
+<part name="R15" library="microbuilder" deviceset="RESISTOR" device="0603" value="22"/>
+<part name="R16" library="microbuilder" deviceset="RESISTOR" device="0603" value="22"/>
+<part name="VBUS" library="microbuilder" deviceset="JUMPER2" device=""/>
+<part name="U$20" library="microbuilder" deviceset="5.0V" device=""/>
 <part name="PWR3.3V" library="microbuilder" deviceset="HEADER-1X2" device="ROUND"/>
 <part name="U$24" library="microbuilder" deviceset="GND" device=""/>
@@
 <part name="U$36" library="microbuilder" deviceset="GND" device=""/>
 <part name="BUS2" library="microbuilder" deviceset="HEADER-1X4" device="ROUND"/>
+<part name="USB" library="microbuilder" deviceset="HEADER-1X4" device="ROUND"/>
 <part name="IC5" library="SparkFun-DigitalIC" deviceset="74*165" device="D"/>
 <part name="U$18" library="microbuilder" deviceset="3.3V" device=""/>
@@
 <part name="POT3" library="keves" deviceset="POTENTIOMETER" device="PTV09A_VERTICAL"/>
 <part name="POT1" library="keves" deviceset="POTENTIOMETER" device="PTV09A_VERTICAL"/>
-<part name="LCD" library="keves" deviceset="SSD1306-7PIN" device="WITHOUT-HOLES"/>
+<part name="LCD" library="keves" deviceset="SSD1306-7PIN" device=""/>
 <part name="TC1" library="TagConnect" deviceset="TC2050-IDC" device="-NL"/>
 <part name="U$55" library="microbuilder" deviceset="3.3V" device=""/>
@@
 <part name="U$87" library="microbuilder" deviceset="3.3V" device=""/>
 <part name="U$117" library="microbuilder" deviceset="3.3V" device=""/>
-<part name="U$19" library="keves" deviceset="ABM7-8.000MHZ-D2Y-T" device=""/>
 </parts>
 <sheets>
@@
 <instance part="CPU1" gate="G$1" x="50.8" y="71.12"/>
 <instance part="U$2" gate="G$1" x="22.86" y="119.38"/>
+<instance part="Y1" gate="G$1" x="10.16" y="101.6" rot="R90"/>
 <instance part="C5" gate="G$1" x="2.54" y="104.14" rot="R90"/>
 <instance part="C6" gate="G$1" x="2.54" y="99.06" rot="R90"/>
@@
 <instance part="R12" gate="G$1" x="88.9" y="101.6"/>
 <instance part="U$17" gate="G$1" x="99.06" y="101.6" rot="R90"/>
+<instance part="U$19" gate="G$1" x="137.16" y="96.52"/>
+<instance part="R15" gate="G$1" x="129.54" y="111.76"/>
+<instance part="R16" gate="G$1" x="129.54" y="109.22"/>
+<instance part="VBUS" gate="A" x="129.54" y="124.46"/>
+<instance part="U$20" gate="G$1" x="121.92" y="121.92" rot="R90"/>
 <instance part="PWR3.3V" gate="G$1" x="180.34" y="81.28"/>
 <instance part="U$24" gate="G$1" x="165.1" y="81.28" rot="R270"/>
@@
 <instance part="U$36" gate="G$1" x="5.08" y="0" rot="R90"/>
 <instance part="BUS2" gate="A" x="-2.54" y="-2.54" rot="R180"/>
+<instance part="USB" gate="A" x="142.24" y="109.22"/>
 <instance part="IC5" gate="A" x="-83.82" y="-50.8"/>
 <instance part="U$18" gate="G$1" x="-101.6" y="-38.1" rot="R90"/>
@@
 <instance part="U$63" gate="G$1" x="157.48" y="109.22" rot="R270"/>
 <instance part="U$64" gate="G$1" x="157.48" y="104.14" rot="R270"/>
-<instance part="U$19" gate="G$1" x="10.16" y="101.6" rot="R90"/>
 </instances>
 <busses>
@@
 <wire x1="22.86" y1="99.06" x2="10.16" y2="99.06" width="0.2032" layer="91"/>
 <pinref part="C6" gate="G$1" pin="P$2"/>
-<pinref part="U$19" gate="G$1" pin="1"/>
+<pinref part="Y1" gate="G$1" pin="1"/>
+<junction x="10.16" y="99.06"/>
 <wire x1="10.16" y1="99.06" x2="5.08" y2="99.06" width="0.2032" layer="91"/>
-<junction x="10.16" y="99.06"/>
 </segment>
 </net>
@@
 <wire x1="22.86" y1="101.6" x2="15.24" y2="101.6" width="0.2032" layer="91"/>
 <wire x1="15.24" y1="101.6" x2="15.24" y2="104.14" width="0.2032" layer="91"/>
+<wire x1="15.24" y1="104.14" x2="10.16" y2="104.14" width="0.2032" layer="91"/>
 <pinref part="C5" gate="G$1" pin="P$2"/>
-<wire x1="15.24" y1="104.14" x2="10.16" y2="104.14" width="0.2032" layer="91"/>
-<pinref part="U$19" gate="G$1" pin="2"/>
+<pinref part="Y1" gate="G$1" pin="2"/>
+<junction x="10.16" y="104.14"/>
 <wire x1="10.16" y1="104.14" x2="5.08" y2="104.14" width="0.2032" layer="91"/>
-<junction x="10.16" y="104.14"/>
 </segment>
 </net>
@@
 <pinref part="U$17" gate="G$1" pin="GND"/>
 <wire x1="96.52" y1="101.6" x2="93.98" y2="101.6" width="0.1524" layer="91"/>
+</segment>
+<segment>
+<pinref part="U$19" gate="G$1" pin="GND"/>
+<wire x1="139.7" y1="106.68" x2="137.16" y2="106.68" width="0.2032" layer="91"/>
+<wire x1="137.16" y1="106.68" x2="137.16" y2="99.06" width="0.2032" layer="91"/>
+<pinref part="USB" gate="A" pin="4"/>
 </segment>
 <segment>
@@
 </segment>
 </net>
+<net name="N$7" class="0">
+<segment>
+<pinref part="R15" gate="G$1" pin="2"/>
+<wire x1="139.7" y1="111.76" x2="134.62" y2="111.76" width="0.2032" layer="91"/>
+<pinref part="USB" gate="A" pin="2"/>
+</segment>
+</net>
+<net name="N$8" class="0">
+<segment>
+<pinref part="R16" gate="G$1" pin="2"/>
+<wire x1="139.7" y1="109.22" x2="134.62" y2="109.22" width="0.2032" layer="91"/>
+<pinref part="USB" gate="A" pin="3"/>
+</segment>
+</net>
+<net name="USB_DM" class="0">
+<segment>
+<pinref part="R15" gate="G$1" pin="1"/>
+<wire x1="124.46" y1="111.76" x2="116.84" y2="111.76" width="0.2032" layer="91"/>
+<label x="114.3" y="111.76" size="1.778" layer="95"/>
+</segment>
+<segment>
+<pinref part="CPU1" gate="G$1" pin="PA11"/>
+<wire x1="81.28" y1="60.96" x2="91.44" y2="60.96" width="0.2032" layer="91"/>
+<label x="88.9" y="60.96" size="1.778" layer="95"/>
+</segment>
+</net>
+<net name="USB_DP" class="0">
+<segment>
+<pinref part="R16" gate="G$1" pin="1"/>
+<wire x1="124.46" y1="109.22" x2="116.84" y2="109.22" width="0.2032" layer="91"/>
+<label x="114.3" y="109.22" size="1.778" layer="95"/>
+</segment>
+<segment>
+<pinref part="CPU1" gate="G$1" pin="PA12"/>
+<wire x1="81.28" y1="63.5" x2="91.44" y2="63.5" width="0.2032" layer="91"/>
+<label x="88.9" y="63.5" size="1.778" layer="95"/>
+</segment>
+</net>
 <net name="USB_VBUS" class="0">
+<segment>
+<wire x1="139.7" y1="114.3" x2="132.08" y2="114.3" width="0.2032" layer="91"/>
+<label x="114.3" y="114.3" size="1.778" layer="95"/>
+<pinref part="VBUS" gate="A" pin="2"/>
+<wire x1="132.08" y1="114.3" x2="116.84" y2="114.3" width="0.2032" layer="91"/>
+<wire x1="132.08" y1="121.92" x2="132.08" y2="114.3" width="0.2032" layer="91"/>
+<junction x="132.08" y="114.3"/>
+<pinref part="USB" gate="A" pin="1"/>
+</segment>
 <segment>
 <pinref part="CPU1" gate="G$1" pin="PA9/UART1_TX"/>
@@
 </net>
 <net name="5.0V" class="0">
+<segment>
+<pinref part="U$20" gate="G$1" pin="5.0V"/>
+<pinref part="VBUS" gate="A" pin="1"/>
+<wire x1="124.46" y1="121.92" x2="129.54" y2="121.92" width="0.2032" layer="91"/>
+</segment>
 <segment>
 <pinref part="U1" gate="G$1" pin="IN"/>
@@
 </segment>
 <segment>
-<pinref part="BUS1" gate="A" pin="2"/>
-<wire x1="0" y1="-5.08" x2="15.24" y2="-5.08" width="0.2032" layer="91"/>
-<label x="12.7" y="-5.08" size="1.778" layer="95"/>
-<pinref part="BUS2" gate="A" pin="2"/>
-<junction x="0" y="-5.08"/>
-<wire x1="0" y1="-5.08" x2="-10.16" y2="-5.08" width="0.1524" layer="91"/>
+<pinref part="BUS1" gate="A" pin="3"/>
+<wire x1="0" y1="-2.54" x2="15.24" y2="-2.54" width="0.2032" layer="91"/>
+<label x="12.7" y="-2.54" size="1.778" layer="95"/>
+<pinref part="BUS2" gate="A" pin="3"/>
+<junction x="0" y="-2.54"/>
+<wire x1="0" y1="-2.54" x2="-10.16" y2="-2.54" width="0.1524" layer="91"/>
 </segment>
 </net>
@@
 </segment>
 <segment>
-<pinref part="BUS1" gate="A" pin="3"/>
-<wire x1="0" y1="-2.54" x2="15.24" y2="-2.54" width="0.2032" layer="91"/>
-<label x="12.7" y="-2.54" size="1.778" layer="95"/>
-<pinref part="BUS2" gate="A" pin="3"/>
-<junction x="0" y="-2.54"/>
-<wire x1="0" y1="-2.54" x2="-10.16" y2="-2.54" width="0.1524" layer="91"/>
+<pinref part="BUS1" gate="A" pin="2"/>
+<wire x1="0" y1="-5.08" x2="15.24" y2="-5.08" width="0.2032" layer="91"/>
+<label x="12.7" y="-5.08" size="1.778" layer="95"/>
+<pinref part="BUS2" gate="A" pin="2"/>
+<junction x="0" y="-5.08"/>
+<wire x1="0" y1="-5.08" x2="-10.16" y2="-5.08" width="0.1524" layer="91"/>
 </segment>
 </net>
@@
 </segment>
 </net>
+<net name="ADC7" class="0">
+<segment>
+<pinref part="FADER1" gate="G$1" pin="S"/>
+<wire x1="17.78" y1="7.62" x2="17.78" y2="2.54" width="0.2032" layer="91"/>
+<label x="17.78" y="5.08" size="1.778" layer="95"/>
+</segment>
+</net>
 <net name="ADC1" class="0">
 <segment>
@@
 <net name="ADC0" class="0">
 <segment>
-<pinref part="FADER1" gate="G$1" pin="S"/>
-<wire x1="17.78" y1="7.62" x2="17.78" y2="2.54" width="0.2032" layer="91"/>
-<label x="17.78" y="5.08" size="1.778" layer="95"/>
+<wire x1="45.72" y1="-17.78" x2="45.72" y2="-20.32" width="0.2032" layer="91"/>
+<label x="45.72" y="-17.78" size="1.778" layer="95"/>
+<pinref part="POT2" gate="G$1" pin="WIPER"/>
 </segment>
 </net>
@@
 </segment>
 </net>
-<net name="ADC7" class="0">
-<segment>
-<wire x1="45.72" y1="-17.78" x2="45.72" y2="-20.32" width="0.2032" layer="91"/>
-<label x="45.72" y="-17.78" size="1.778" layer="95"/>
-<pinref part="POT2" gate="G$1" pin="WIPER"/>
-</segment>
-</net>
