File: midimixer-channel/midimixer-channel.brd (EAGLE design)
At the start: 50.8 x 241.3 mm, 117 parts, among them IC1 74LS595D, IC2 74LS595D, IC3 74LS595D, IC4 74165D, IC5 74165D, U1 LM1117IMPX-3.3/NOPB, Y1 8MHz 695-HCM49-8-U

Commit message: midimixer-channel wip
Parts:
- removed R15, R16: 22, microbuilder:0603
- removed USB: (no value), microbuilder:1X04_ROUND
- removed VBUS: (no value), microbuilder:JUMPER2
- removed Y1: 8MHz 695-HCM49-8-U, microbuilder:HC49UP
- added U$19: ABM7-8.000MHZ-D2Y-T, keves:ABM7-8.000MHZ-D2Y-T
- LCD: value SSD1306-7PIN -> SSD1306-7PINWITHOUT-HOLES; device keves:SSD1306-7PIN -> keves:SSD1306-7PIN-NO-HOLES
- moved BUS1 39.8 mm to (49.5, 10.2), flipped to the bottom, turned to 90 degrees
- moved RST 37.3 mm to (14.4, 32.0)
- moved R11 32.9 mm to (47.5, 9.78)
- moved C16 31.3 mm to (23.7, 26.7)
- moved C5 28.2 mm to (20.2, 12.6), flipped to the bottom
- moved C6 28.1 mm to (20.2, 16.3), flipped to the bottom
- moved C13 18.0 mm to (43.1, 13.6), flipped to the bottom, turned to 180 degrees
- moved C12 15.2 mm to (43.1, 11.6), flipped to the bottom, turned to 0 degrees
- moved C9 11.8 mm to (39.1, 25.5), flipped to the bottom, turned to 270 degrees
- moved C11 11.3 mm to (28.3, 9.91), flipped to the bottom, turned to 270 degrees
- moved C19 10.4 mm to (25.0, 20.2)
- moved C18 10.3 mm to (23.1, 20.7)
- moved L1 10.3 mm to (21.3, 20.2)
- moved C15 10.0 mm to (4.57, 13.8), turned to 180 degrees
- moved C17 9.56 mm to (9.65, 20.4), turned to 270 degrees
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Connections:
- removed net N$7: R15.2, USB.2
- removed net N$8: R16.2, USB.3
- removed net USB_DM: CPU1.44, R15.1
- removed net USB_DP: CPU1.45, R16.1
- net 5.0V: no longer VBUS.1
- net ADC0: now also FADER1.P2; no longer POT2.CENTER
- net ADC7: now also POT2.CENTER; no longer FADER1.P2
- net CAN_H: now also BUS1.3, BUS2.3; no longer BUS1.2, BUS2.2
- net CAN_L: now also BUS1.2, BUS2.2; no longer BUS1.3, BUS2.3
- net GND: no longer USB.4
- net N$1: now also U$19.P$1; no longer Y1.1
- net N$2: now also U$19.P$2; no longer Y1.2
- net USB_VBUS: no longer USB.1, VBUS.2
Routing:
- net LCD_CS: track 251.3 -> 0.00 mm, vias 2 -> 0
- net LCD_CLK: track 247.1 -> 0.00 mm, vias 2 -> 0
- net LCD_MOSI: track 246.5 -> 0.00 mm, vias 2 -> 0
- net LCD_DC: track 245.4 -> 0.00 mm, vias 2 -> 0
- net LCD_RST: track 236.3 -> 0.00 mm, vias 3 -> 0
- net SPI2_CLK: track 212.4 -> 0.00 mm, vias 4 -> 0
- net SPI2_RC2: track 210.0 -> 0.00 mm, vias 1 -> 0
- net SPI2_MISO: track 185.0 -> 0.00 mm, vias 1 -> 0
- net ADC3: track 166.3 -> 0.00 mm
- net ADC0: track 159.2 -> 0.00 mm
- net GND: track 151.6 -> 0.00 mm, vias 19 -> 0
- net N$28: track 148.5 -> 0.00 mm, vias 2 -> 0
- net ADC4: track 143.8 -> 0.00 mm
- net ADC1: track 127.9 -> 0.00 mm
- net ADC5: track 121.0 -> 0.00 mm
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- added copper zone on layer 1, net 3.3V
- added copper zone on layer 16, net GND
- removed copper zone on layer 16, net 3.3V
- removed copper zone on layer 1, net GND

Commit message: wip
Parts:
- removed C16: 0.1uF, microbuilder:0603
- removed RST: (no value), microbuilder:EVQ-Q2
- moved R38 120.3 mm to (3.68, 175.9)
- moved R34 39.4 mm to (41.0, 82.4), turned to 0 degrees
- moved LED1 27.7 mm to (11.2, 33.3)
- moved R17 20.8 mm to (14.6, 33.3)
- moved R35 20.6 mm to (20.7, 53.5)
- moved C3 14.0 mm to (23.2, 35.2)
- moved R36 12.8 mm to (27.9, 66.5), turned to 0 degrees
- moved C4 12.0 mm to (24.8, 82.3)
- moved R37 9.80 mm to (29.5, 82.2), turned to 180 degrees
- moved USR 9.47 mm to (46.0, 21.6)
- moved C21 9.27 mm to (29.6, 80.4), turned to 0 degrees
- moved C2 7.25 mm to (24.6, 96.5), turned to 0 degrees
- moved IC3 5.28 mm to (23.2, 102.7), turned to 90 degrees
- moved R21 5.02 mm to (25.4, 70.5), turned to 180 degrees
- moved C11 2.18 mm to (30.1, 8.64)
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Connections:
- removed net BTN_LED1: BTN2.LED1+, IC2.15
- removed net BTN_LED10: BTN6.LED2+, IC1.2
- removed net BTN_LED11: BTN3.LED1+, IC1.4
- removed net BTN_LED12: BTN3.LED2+, IC1.5
- removed net BTN_LED2: BTN2.LED2+, IC2.3
- removed net BTN_LED3: BTN1.LED1+, IC2.5
- removed net BTN_LED4: BTN1.LED2+, IC2.7
- removed net BTN_LED5: BTN4.LED1+, IC2.4
- removed net BTN_LED6: BTN6.LED1+, IC1.3
- removed net BTN_LED7: BTN5.LED1+, IC1.6
- removed net BTN_LED8: BTN5.LED2+, IC1.7
- removed net BTN_LED9: BTN4.LED2+, IC2.6
- removed net BTN_UUSED2: IC1.15
- removed net DIN_10: BTN4.SW3, BTN4.SW4, C20.2, IC5.12, R36.1
- removed net DIN_11: BTN6.SW3, BTN6.SW4, C24.2, IC5.13, R35.1
- removed net DIN_12: BTN5.SW4, C23.2, IC5.14, R34.1
- removed net DIN_13: BTN2.SW3, BTN2.SW4, C22.2, IC5.3, R33.1
- removed net DIN_14: BTN3.SW4, C25.2, IC5.4, R32.1
- removed net DIN_9: BTN1.SW4, C21.2, IC5.11, R37.1
- removed net N$31: D1.1, IC2.2
- removed net N$49: D1.10, IC3.15
- removed net N$50: D1.9, IC3.1
- removed net N$51: D1.8, IC3.2
- removed net N$54: D1.5, IC3.5
- removed net USB_VBUS: CPU1.42
- new net BTN1: BTN1.SW3, BTN1.SW4, C21.2, IC5.11, R37.1
- new net BTN1_LED1: BTN1.LED1+, IC2.1
- new net BTN1_LED2: BTN1.LED2+, IC2.2
- new net BTN2: BTN2.SW3, BTN2.SW4, C22.2, IC5.14, R34.1
- new net BTN2_LED1: BTN2.LED1+, IC1.1
- new net BTN2_LED2: BTN2.LED2+, IC1.2
- new net BTN3: BTN3.SW3, BTN3.SW4, C25.2, IC5.12, R36.1
- new net BTN3_LED1: BTN3.LED1+, IC2.3
- new net BTN3_LED2: BTN3.LED2+, IC2.4
- new net BTN4: BTN4.SW3, BTN4.SW4, C20.2, IC5.4, R32.1
- new net BTN4_LED1: BTN4.LED1+, IC1.3
- new net BTN4_LED2: BTN4.LED2+, IC1.4
- new net BTN5: BTN5.SW3, BTN5.SW4, C23.2, IC5.13, R35.1
- new net BTN5_LED1: BTN5.LED1+, IC2.5
- new net BTN5_LED2: BTN5.LED2+, IC2.15
- new net BTN6: BTN6.SW3, BTN6.SW4, C24.2, IC5.3, R33.1
- new net BTN6_LED1: BTN6.LED1+, IC1.5
- new net BTN6_LED2: BTN6.LED2+, IC1.6
- new net BTN_UNUSED2: IC1.7
- new net N$38: D1.10, IC3.7
- new net N$41: D1.9, IC3.6
- new net N$42: D1.8, IC3.5
- new net N$7: D1.5, IC3.2
- new net N$8: D1.2, IC2.7
- net BTN_UNUSED1: now also IC1.15; no longer IC1.1
- net GND: now also BTN1.SW1, BTN3.SW1, BTN5.SW1; no longer C16.2, RST.A, RST.A'
- net N$11: now also D1.1, IC2.6; no longer D1.2, IC2.1
- net N$26: now also IC4.10; no longer IC5.10
- net N$28: now also IC4.9, IC5.10; no longer IC4.10, IC5.9
- net N$52: now also IC3.4; no longer IC3.3
- net N$53: now also IC3.3; no longer IC3.4
- net N$55: now also IC3.1; no longer IC3.6
- net N$56: now also IC3.15; no longer IC3.7
- net NRST: no longer C16.1, RST.B, RST.B'
- net SPI2_MISO: now also IC5.9; no longer IC4.9
- net SPI2_RC1: now also CPU1.11; no longer CPU1.33
- net SPI2_RC2: now also CPU1.10; no longer CPU1.37
Routing:
- net LCD_CLK: track 0.00 -> 247.5 mm
- net LCD_MOSI: track 0.00 -> 246.1 mm
- net LCD_RST: track 0.00 -> 244.5 mm
- net LCD_DC: track 0.00 -> 242.9 mm
- net LCD_CS: track 0.00 -> 236.4 mm
- net BTN2: track 0.00 -> 67.5 mm, vias 0 -> 1
- net BTN4: track 0.00 -> 61.9 mm, vias 0 -> 1
- net 3.3V: track 45.5 -> 97.0 mm, vias 9 -> 25
- net BTN2_LED1: track 0.00 -> 50.5 mm
- net BTN5_LED2: track 0.00 -> 46.7 mm, vias 0 -> 1
- net BTN6: track 0.00 -> 45.3 mm, vias 0 -> 1
- net BTN2_LED2: track 0.00 -> 42.3 mm
- net BTN5_LED1: track 0.00 -> 41.5 mm, vias 0 -> 1
- net BTN1: track 0.00 -> 39.0 mm, vias 0 -> 1
- net SPI2_RC2: track 0.00 -> 39.0 mm, vias 0 -> 2
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
Commit message: wip
Parts:
- moved R38 5.92 mm to (7.11, 180.7), turned to 0 degrees
- moved R1 1.27 mm to (7.11, 179.1)
- moved R5 0.77 mm to (6.73, 183.9)
- moved R9 0.51 mm to (18.7, 181.4)
- moved C1 0.38 mm to (8.26, 187.1)
Connections:
- net LCD_RST: now also CPU1.54; no longer CPU1.24
Routing:
- net SPI2_RC2: track 39.0 -> 205.2 mm, vias 2 -> 3
- net N$28: track 0.00 -> 146.3 mm, vias 0 -> 2
- net SPI2_CLK: track 19.1 -> 131.8 mm, vias 2 -> 4
- net DIN_5: track 0.00 -> 39.1 mm
- net DIN_7: track 0.00 -> 29.9 mm
- net DIN_3: track 0.00 -> 24.9 mm
- net 3.3V: track 97.0 -> 120.7 mm, vias 25 -> 35
- net DIN_6: track 0.00 -> 20.6 mm
- net DIN_2: track 0.00 -> 18.7 mm
- net LCD_DC: track 242.9 -> 260.9 mm, vias 0 -> 1
- net LCD_CS: track 236.4 -> 253.6 mm, vias 0 -> 1
- net LCD_MOSI: track 246.1 -> 262.6 mm, vias 0 -> 1
- net LCD_CLK: track 247.5 -> 263.4 mm, vias 0 -> 1
- net LCD_RST: track 244.5 -> 259.8 mm, vias 0 -> 1
- net DIN_1: track 0.00 -> 14.0 mm
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
Commit message: wip
Parts:
- moved C3 1.78 mm to (23.4, 33.4), turned to 90 degrees
- moved C2 0.52 mm to (25.1, 96.4)
- moved IC3 0.52 mm to (23.7, 102.6)
- moved C4 0.51 mm to (25.3, 82.3)
- moved IC2 0.51 mm to (23.7, 88.4)
Connections:
- net ADC0 renamed FADER
- net ADC6 renamed POT7
- net ADC7 renamed POT2
- removed net ADC1: CPU1.15, POT4.CENTER
- removed net ADC2: CPU1.16, POT6.CENTER
- removed net ADC3: CPU1.17, POT1.CENTER
- removed net ADC4: CPU1.20, POT3.CENTER
- removed net ADC5: CPU1.21, POT5.CENTER
- new net POT1: CPU1.15, POT1.CENTER
- new net POT3: CPU1.16, POT3.CENTER
- new net POT4: CPU1.21, POT4.CENTER
- new net POT5: CPU1.17, POT5.CENTER
- new net POT6: CPU1.20, POT6.CENTER
Routing:
- net POT1: track 0.00 -> 177.9 mm, vias 0 -> 2
- net POT3: track 0.00 -> 155.0 mm, vias 0 -> 2
- net POT5: track 0.00 -> 127.0 mm, vias 0 -> 4
- net SPI2_MOSI: track 0.00 -> 108.7 mm, vias 0 -> 2
- net N$12: track 0.00 -> 103.3 mm, vias 0 -> 2
- net SPI2_CLK: track 131.8 -> 223.5 mm, vias 4 -> 8
- net SPI2_RC1: track 36.0 -> 108.0 mm, vias 4 -> 6
- net SPI2_MISO: track 0.00 -> 30.5 mm, vias 0 -> 3
- net N$24: track 0.00 -> 4.58 mm
- net N$28: track 146.3 -> 150.6 mm
- net SPI2_RC2: track 205.2 -> 208.0 mm
- net BTN3: track 22.9 -> 25.1 mm
- net BTN5_LED1: track 41.5 -> 43.3 mm
- net 3.3V: track 120.7 -> 119.6 mm
- net N$38: track 6.79 -> 5.86 mm
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
Commit message: wip
Parts:
- moved C7 0.77 mm to (37.0, 25.5)
- moved C8 0.38 mm to (31.2, 26.4)
- moved C9 0.18 mm to (39.0, 25.4)
Connections:
- net POT4: now also CPU1.22; no longer CPU1.21
- net POT7: now also CPU1.21; no longer CPU1.22
Routing:
- net POT2: track 0.00 -> 172.5 mm, vias 0 -> 1
- net POT4: track 0.00 -> 145.8 mm, vias 0 -> 1
- net POT6: track 0.00 -> 114.0 mm, vias 0 -> 1
- net POT7: track 0.00 -> 86.0 mm, vias 0 -> 2
- net SPI2_MISO: track 30.5 -> 53.2 mm, vias 3 -> 6
- net SPI2_CLK: track 223.5 -> 245.5 mm, vias 8 -> 10
- net PB2: track 0.00 -> 17.6 mm, vias 0 -> 2
- net N$12: track 103.3 -> 94.3 mm
- net 3.3V: track 119.6 -> 124.5 mm, vias 35 -> 36
- net N$4: track 0.00 -> 2.18 mm
- net LCD_RST: track 259.8 -> 258.0 mm
- net LCD_MOSI: track 262.6 -> 260.9 mm
- net LCD_DC: track 260.9 -> 259.2 mm
- net LCD_CLK: track 263.4 -> 261.7 mm
- net SPI2_RC2: vias 3 -> 5

Commit message: wip
Parts:
- added LED: (no value), microbuilder:CHIPLED_0603
- added PWR5.0V: (no value), microbuilder:1X02_ROUND
- added R2: 330, microbuilder:0603
- moved C18 0.92 mm to (22.9, 21.6)
- moved C19 0.92 mm to (24.8, 21.1)
- moved L1 0.92 mm to (21.1, 21.1)
- renumbered LED1 to PWR
Connections:
- new net N$31: LED.A, R2.1
- new net N$43: CPU1.25, R2.2
- net 5.0V: now also PWR5.0V.1
- net GND: now also LED.C, PWR5.0V.2
Routing:
- net N$43: track 0.00 -> 10.4 mm
- net FADER: track 25.7 -> 34.1 mm
- net POT4: track 145.8 -> 143.8 mm
- net POT2: track 172.5 -> 170.5 mm
- net 5.0V: track 64.5 -> 66.5 mm
- net N$31: track 0.00 -> 1.96 mm
- net SPI2_RC2: track 208.0 -> 206.2 mm, vias 5 -> 4
- net N$28: track 150.6 -> 151.8 mm

Commit message: wip
Parts:
- H1, H2, H3, H4, H5, H6: value STAND-OFF -> MOUNT-HOLE3.2; device SparkFun-Electromechanical:STAND-OFF -> holes:3,2
- moved PWR5.0V 34.6 mm to (10.7, 1.52), turned to 180 degrees
- moved R10 5.04 mm to (20.2, 8.51), turned to 90 degrees
- moved R11 2.04 mm to (47.6, 11.8)
- moved BUS1 1.65 mm to (49.5, 11.8)
- moved BUS2 1.65 mm to (1.27, 11.8)
- moved C12 1.53 mm to (41.5, 11.7), turned to 90 degrees
- moved C13 1.27 mm to (44.3, 13.6)
- moved LED 0.38 mm to (39.2, 34.4)
- moved R2 0.38 mm to (39.2, 30.9)
Routing:
- net POT1: track 177.9 -> 190.6 mm
- net POT3: track 155.0 -> 164.7 mm
- net SPI2_RC2: track 206.2 -> 215.7 mm
- net N$28: track 151.8 -> 161.0 mm
- net LCD_CS: track 253.6 -> 262.3 mm
- net SPI2_CLK: track 245.1 -> 236.5 mm
- net POT4: track 143.8 -> 136.3 mm
- net LCD_MOSI: track 260.9 -> 267.2 mm
- net LCD_DC: track 259.2 -> 265.0 mm
- net LCD_CLK: track 261.7 -> 267.4 mm
- net LCD_RST: track 258.0 -> 263.6 mm
- net POT2: track 170.5 -> 173.3 mm
- net CAN_L: track 62.4 -> 59.9 mm
- net CAN_H: track 62.6 -> 60.1 mm
- net 3.3V: track 124.1 -> 121.9 mm
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
Commit message: midimixer-channel rev a sent to macrofab
Parts:
- removed PWR3.3V, PWR5.0V: (no value), microbuilder:1X02_ROUND
- removed R11: 120 DNP, microbuilder:_0603
- added C16: 4.7nF, microbuilder:0603
- added R3, R7: 60 1%, microbuilder:0603
- added TERM: (no value), pinhead:2X02
- BUS1, BUS2: value (none) -> 04-JST-B4B-XH-A; device microbuilder:1X04_ROUND -> bt_con-jst-xh:B4B-XH
- D2: value SN65HVD232 -> SN65HVD230
- moved BUS1 47.0 mm to (2.54, 12.7)
- moved BUS2 45.9 mm to (47.1, 12.7)
- moved C15 7.11 mm to (4.70, 21.0)
- moved U1 7.11 mm to (4.57, 25.8)
- moved C17 6.35 mm to (9.78, 26.8)
- moved USR 3.74 mm to (45.3, 25.3), turned to 180 degrees
- moved C10 2.80 mm to (25.8, 6.86), turned to 180 degrees
- moved R10 2.41 mm to (17.8, 8.51)
- moved C13 1.65 mm to (42.7, 13.6)
- moved C12 1.33 mm to (41.1, 10.4)
Connections:
- new net CAN_VREF: C16.2, D2.5, R3.2, R7.1
- new net N$46: R7.2, TERM.2
- new net N$47: R3.1, TERM.4
- net 3.3V: no longer PWR3.3V.1
- net 5.0V: now also BUS1.P$1, BUS2.P$1; no longer BUS1.1, BUS2.1, PWR5.0V.1
- net CAN_H: now also BUS1.P$3, BUS2.P$3, TERM.3; no longer BUS1.3, BUS2.3, R11.1
- net CAN_L: now also BUS1.P$2, BUS2.P$2, TERM.1; no longer BUS1.2, BUS2.2, R11.2
- net GND: now also BUS1.P$4, BUS2.P$4, C16.1; no longer BUS1.4, BUS2.4, PWR3.3V.2, PWR5.0V.2
Routing:
- net N$46: track 0.00 -> 13.2 mm, vias 0 -> 1
- net N$47: track 0.00 -> 12.3 mm, vias 0 -> 1
- net CAN_VREF: track 0.00 -> 7.68 mm
- net CAN_L: track 59.9 -> 63.0 mm
- net 5.0V: track 66.8 -> 69.6 mm
- net 3.3V: track 121.9 -> 119.4 mm
- net CAN_H: track 60.1 -> 62.6 mm
- net N$3: track 3.35 -> 1.70 mm
- net PB2: track 17.6 -> 16.0 mm
- net N$73: track 2.54 -> 3.54 mm
- net LCD_RST: track 263.6 -> 263.0 mm
- net LCD_MOSI: track 267.2 -> 266.6 mm
- net LCD_CLK: track 267.4 -> 266.8 mm
- net SPI2_MOSI: track 108.9 -> 108.3 mm
- net LCD_DC: track 265.0 -> 264.5 mm
Other:
- board text added: "Eran Rundstein, 2017"
- board text removed: "Eran Rundstein, 2016"
