File: midimixer-channel/midimixer-channel.sch (EAGLE design)
At the start: 113 parts, among them IC1 74LS595D, IC2 74LS595D, IC3 74LS595D, IC4 74165D, IC5 74165D, U1 LM1117IMPX-3.3/NOPB

Commit message: wip
Parts:
- removed C16: 0.1uF, microbuilder:CAP_CERAMIC0603
- removed RST: (no value), microbuilder:SWITCH_TACT_SMT
Connections:
- removed net BTN_LED1: BTN2.LED1+, IC2.QA
- removed net BTN_LED10: BTN6.LED2+, IC1.QC
- removed net BTN_LED11: BTN3.LED1+, IC1.QE
- removed net BTN_LED12: BTN3.LED2+, IC1.QF
- removed net BTN_LED2: BTN2.LED2+, IC2.QD
- removed net BTN_LED3: BTN1.LED1+, IC2.QF
- removed net BTN_LED4: BTN1.LED2+, IC2.QH
- removed net BTN_LED5: BTN4.LED1+, IC2.QE
- removed net BTN_LED6: BTN6.LED1+, IC1.QD
- removed net BTN_LED7: BTN5.LED1+, IC1.QG
- removed net BTN_LED8: BTN5.LED2+, IC1.QH
- removed net BTN_LED9: BTN4.LED2+, IC2.QG
- removed net BTN_UUSED2: IC1.QA
- removed net DIN_10: BTN4.SW2_A, BTN4.SW2_B, C20.P$2, IC5.B, R36.1
- removed net DIN_11: BTN6.SW2_A, BTN6.SW2_B, C24.P$2, IC5.C, R35.1
- removed net DIN_12: BTN5.SW2_B, C23.P$2, IC5.D, R34.1
- removed net DIN_13: BTN2.SW2_A, BTN2.SW2_B, C22.P$2, IC5.E, R33.1
- removed net DIN_14: BTN3.SW2_B, C25.P$2, IC5.F, R32.1
- removed net DIN_9: BTN1.SW2_B, C21.P$2, IC5.A, R37.1
- removed net N$31: D1A.A, IC2.QC
- removed net N$49: D1J.A, IC3.QA
- removed net N$50: D1I.A, IC3.QB
- removed net N$51: D1H.A, IC3.QC
- removed net N$54: D1E.A, IC3.QF
- removed net USB_VBUS: CPU1.PA9/UART1_TX
- new net BTN1: BTN1.SW2_A, BTN1.SW2_B, C21.P$2, IC5.A, R37.1
- new net BTN1_LED1: BTN1.LED1+, IC2.QB
- new net BTN1_LED2: BTN1.LED2+, IC2.QC
- new net BTN2: BTN2.SW2_A, BTN2.SW2_B, C22.P$2, IC5.D, R34.1
- new net BTN2_LED1: BTN2.LED1+, IC1.QB
- new net BTN2_LED2: BTN2.LED2+, IC1.QC
- new net BTN3: BTN3.SW2_A, BTN3.SW2_B, C25.P$2, IC5.B, R36.1
- new net BTN3_LED1: BTN3.LED1+, IC2.QD
- new net BTN3_LED2: BTN3.LED2+, IC2.QE
- new net BTN4: BTN4.SW2_A, BTN4.SW2_B, C20.P$2, IC5.F, R32.1
- new net BTN4_LED1: BTN4.LED1+, IC1.QD
- new net BTN4_LED2: BTN4.LED2+, IC1.QE
- new net BTN5: BTN5.SW2_A, BTN5.SW2_B, C23.P$2, IC5.C, R35.1
- new net BTN5_LED1: BTN5.LED1+, IC2.QF
- new net BTN5_LED2: BTN5.LED2+, IC2.QA
- new net BTN6: BTN6.SW2_A, BTN6.SW2_B, C24.P$2, IC5.E, R33.1
- new net BTN6_LED1: BTN6.LED1+, IC1.QF
- new net BTN6_LED2: BTN6.LED2+, IC1.QG
- new net BTN_UNUSED2: IC1.QH
- new net N$38: D1J.A, IC3.QH
- new net N$41: D1I.A, IC3.QG
- new net N$42: D1H.A, IC3.QF
- new net N$7: D1E.A, IC3.QC
- new net N$8: D1B.A, IC2.QH
- net BTN_UNUSED1: now also IC1.QA; no longer IC1.QB
- net GND: now also BTN1.SW1_A, BTN3.SW1_A, BTN5.SW1_A; no longer C16.P$2, RST.P, RST.P1
- net N$11: now also D1A.A, IC2.QG; no longer D1B.A, IC2.QB
- net N$26: now also IC4.SER; no longer IC5.SER
- net N$28: now also IC4.QH, IC5.SER; no longer IC4.SER, IC5.QH
- net N$52: now also IC3.QE; no longer IC3.QD
- net N$53: now also IC3.QD; no longer IC3.QE
- net N$55: now also IC3.QB; no longer IC3.QG
- net N$56: now also IC3.QA; no longer IC3.QH
- net NRST: no longer C16.P$1, RST.S, RST.S1
- net SPI2_MISO: now also IC5.QH; no longer IC4.QH
- net SPI2_RC1: now also CPU1.PC3; no longer CPU1.PB12/I2S2_WS
- net SPI2_RC2: now also CPU1.PC2; no longer CPU1.PC6/I2S2_MCK
Other:
- note removed: "PD10 in Midibox!!"
- moved on the sheet: C1, C2, C26, IC3, IC4, IC5, R30, R31, R32, R33, R34, R35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

Commit message: wip
Connections:
- net LCD_RST: now also CPU1.PD2/SDIO_CMD; no longer CPU1.PC4
Changed lines of the file:
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@@
 </segment>
 <segment>
-<pinref part="CPU1" gate="G$1" pin="PC4"/>
-<wire x1="22.86" y1="53.34" x2="2.54" y2="53.34" width="0.1524" layer="91"/>
-<label x="0" y="53.34" size="1.778" layer="95"/>
+<pinref part="CPU1" gate="G$1" pin="PD2/SDIO_CMD"/>
+<wire x1="81.28" y1="86.36" x2="96.52" y2="86.36" width="0.1524" layer="91"/>
+<label x="88.9" y="86.36" size="1.778" layer="95"/>
 </segment>
 </net>

Commit message: wip
Connections:
- net ADC0 renamed FADER
- net ADC6 renamed POT7
- net ADC7 renamed POT2
- removed net ADC1: CPU1.PA1, POT4.WIPER
- removed net ADC2: CPU1.PA2/UART2_TX, POT6.WIPER
- removed net ADC3: CPU1.PA3/UART2_RX, POT1.WIPER
- removed net ADC4: CPU1.PA4/SPI1_NSS, POT3.WIPER
- removed net ADC5: CPU1.PA5/SPI1_SCK, POT5.WIPER
- new net POT1: CPU1.PA1, POT1.WIPER
- new net POT3: CPU1.PA2/UART2_TX, POT3.WIPER
- new net POT4: CPU1.PA5/SPI1_SCK, POT4.WIPER
- new net POT5: CPU1.PA3/UART2_RX, POT5.WIPER
- new net POT6: CPU1.PA4/SPI1_NSS, POT6.WIPER
Changed lines of the file:
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@@
 </segment>
 </net>
-<net name="ADC0" class="0">
+<net name="FADER" class="0">
 <segment>
 <pinref part="CPU1" gate="G$1" pin="PA0"/>
@@
 </segment>
 </net>
-<net name="ADC1" class="0">
+<net name="POT6" class="0">
+<segment>
+<pinref part="CPU1" gate="G$1" pin="PA4/SPI1_NSS"/>
+<wire x1="22.86" y1="63.5" x2="2.54" y2="63.5" width="0.2032" layer="91"/>
+<label x="0" y="63.5" size="1.778" layer="95"/>
+</segment>
+</net>
+<net name="POT1" class="0">
 <segment>
 <pinref part="CPU1" gate="G$1" pin="PA1"/>
@@
 </segment>
 </net>
-<net name="ADC2" class="0">
-<segment>
-<pinref part="CPU1" gate="G$1" pin="PA2/UART2_TX"/>
-<wire x1="22.86" y1="73.66" x2="2.54" y2="73.66" width="0.2032" layer="91"/>
-<label x="0" y="73.66" size="1.778" layer="95"/>
-</segment>
-</net>
-<net name="ADC3" class="0">
+<net name="POT5" class="0">
 <segment>
 <pinref part="CPU1" gate="G$1" pin="PA3/UART2_RX"/>
@@
 </segment>
 </net>
-<net name="ADC4" class="0">
-<segment>
-<pinref part="CPU1" gate="G$1" pin="PA4/SPI1_NSS"/>
-<wire x1="22.86" y1="63.5" x2="2.54" y2="63.5" width="0.2032" layer="91"/>
-<label x="0" y="63.5" size="1.778" layer="95"/>
-</segment>
-</net>
-<net name="ADC5" class="0">
-<segment>
-<pinref part="CPU1" gate="G$1" pin="PA5/SPI1_SCK"/>
-<wire x1="22.86" y1="60.96" x2="2.54" y2="60.96" width="0.2032" layer="91"/>
-<label x="0" y="60.96" size="1.778" layer="95"/>
-</segment>
-</net>
-<net name="ADC6" class="0">
+<net name="POT7" class="0">
 <segment>
 <pinref part="CPU1" gate="G$1" pin="PA6/SPI1_MISO"/>
@@
 </segment>
 </net>
-<net name="ADC7" class="0">
+<net name="POT2" class="0">
 <segment>
 <pinref part="CPU1" gate="G$1" pin="PA7/SPI1_MOSI"/>
@@
 <wire x1="-60.96" y1="12.7" x2="-60.96" y2="2.54" width="0.2032" layer="91"/>
 <junction x="-60.96" y="2.54"/>
+</segment>
+</net>
+<net name="POT3" class="0">
+<segment>
+<pinref part="CPU1" gate="G$1" pin="PA2/UART2_TX"/>
+<wire x1="22.86" y1="73.66" x2="2.54" y2="73.66" width="0.2032" layer="91"/>
+<label x="0" y="73.66" size="1.778" layer="95"/>
+</segment>
+</net>
+<net name="POT4" class="0">
+<segment>
+<pinref part="CPU1" gate="G$1" pin="PA5/SPI1_SCK"/>
+<wire x1="22.86" y1="60.96" x2="2.54" y2="60.96" width="0.2032" layer="91"/>
+<label x="0" y="60.96" size="1.778" layer="95"/>
 </segment>
 </net>
@@
 </segment>
 </net>
-<net name="ADC1" class="0">
+<net name="POT4" class="0">
 <segment>
 <wire x1="45.72" y1="-35.56" x2="45.72" y2="-38.1" width="0.2032" layer="91"/>
@@
 </segment>
 </net>
-<net name="ADC5" class="0">
+<net name="POT5" class="0">
 <segment>
 <wire x1="7.62" y1="-35.56" x2="7.62" y2="-38.1" width="0.2032" layer="91"/>
@@
 </segment>
 </net>
-<net name="ADC6" class="0">
+<net name="POT7" class="0">
 <segment>
 <wire x1="7.62" y1="-17.78" x2="7.62" y2="-20.32" width="0.2032" layer="91"/>
@@
 </segment>
 </net>
-<net name="ADC2" class="0">
+<net name="POT6" class="0">
 <segment>
 <wire x1="45.72" y1="-53.34" x2="45.72" y2="-55.88" width="0.2032" layer="91"/>
@@
 </segment>
 </net>
-<net name="ADC0" class="0">
+<net name="FADER" class="0">
 <segment>
 <pinref part="FADER1" gate="G$1" pin="S"/>
@@
 </segment>
 </net>
-<net name="ADC3" class="0">
+<net name="POT1" class="0">
 <segment>
 <wire x1="7.62" y1="-76.2" x2="7.62" y2="-78.74" width="0.2032" layer="91"/>
@@
 </segment>
 </net>
-<net name="ADC4" class="0">
+<net name="POT3" class="0">
 <segment>
 <wire x1="7.62" y1="-55.88" x2="7.62" y2="-58.42" width="0.2032" layer="91"/>
@@
 </segment>
 </net>
-<net name="ADC7" class="0">
+<net name="POT2" class="0">
 <segment>
 <wire x1="45.72" y1="-17.78" x2="45.72" y2="-20.32" width="0.2032" layer="91"/>

Commit message: wip
Connections:
- net POT4: now also CPU1.PA6/SPI1_MISO; no longer CPU1.PA5/SPI1_SCK
- net POT7: now also CPU1.PA5/SPI1_SCK; no longer CPU1.PA6/SPI1_MISO
Changed lines of the file:
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@@
-</segment>
-</net>
-<net name="POT7" class="0">
-<segment>
-<pinref part="CPU1" gate="G$1" pin="PA6/SPI1_MISO"/>
-<wire x1="22.86" y1="58.42" x2="2.54" y2="58.42" width="0.2032" layer="91"/>
-<label x="0" y="58.42" size="1.778" layer="95"/>
 </segment>
 </net>
@@
 <net name="POT4" class="0">
 <segment>
+<pinref part="CPU1" gate="G$1" pin="PA6/SPI1_MISO"/>
+<wire x1="22.86" y1="58.42" x2="2.54" y2="58.42" width="0.2032" layer="91"/>
+<label x="0" y="58.42" size="1.778" layer="95"/>
+</segment>
+</net>
+<net name="POT7" class="0">
+<segment>
 <pinref part="CPU1" gate="G$1" pin="PA5/SPI1_SCK"/>

Commit message: wip
Parts:
- added LED: (no value), microbuilder:LED0603
- added PWR5.0V: (no value), microbuilder:HEADER-1X2ROUND
- added R2: 330, microbuilder:RESISTOR0603
- renumbered LED1 to PWR
Connections:
- new net N$31: LED.A, R2.1
- new net N$43: CPU1.PC5, R2.2
- net 5.0V: now also PWR5.0V.1
- net GND: now also LED.C, PWR5.0V.2
Changed lines of the file:
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@@
 <part name="U$28" library="microbuilder" deviceset="3.3V" device=""/>
 <part name="U$29" library="microbuilder" deviceset="GND" device=""/>
-<part name="LED1" library="microbuilder" deviceset="LED" device="0603"/>
+<part name="PWR" library="microbuilder" deviceset="LED" device="0603"/>
 <part name="U$30" library="microbuilder" deviceset="GND" device=""/>
 <part name="L1" library="SparkFun-Passives" deviceset="INDUCTOR" device="0805"/>
@@
 <part name="U$19" library="keves" deviceset="ABM7-8.000MHZ-D2Y-T" device=""/>
 <part name="U$20" library="microbuilder" deviceset="3.3V" device=""/>
+<part name="R2" library="microbuilder" deviceset="RESISTOR" device="0603" value="330"/>
+<part name="LED" library="microbuilder" deviceset="LED" device="0603"/>
+<part name="U$32" library="microbuilder" deviceset="GND" device=""/>
+<part name="PWR5.0V" library="microbuilder" deviceset="HEADER-1X2" device="ROUND"/>
+<part name="U$113" library="microbuilder" deviceset="GND" device=""/>
+<part name="U$114" library="microbuilder" deviceset="5.0V" device=""/>
 </parts>
 <sheets>
@@
 <instance part="U$28" gate="G$1" x="177.8" y="66.04"/>
 <instance part="U$29" gate="G$1" x="137.16" y="48.26"/>
-<instance part="LED1" gate="G$1" x="177.8" y="40.64" rot="R270"/>
+<instance part="PWR" gate="G$1" x="177.8" y="40.64" rot="R270"/>
 <instance part="U$30" gate="G$1" x="177.8" y="30.48"/>
 <instance part="L1" gate="G$1" x="190.5" y="60.96" rot="R90"/>
@@
 <instance part="U$19" gate="G$1" x="10.16" y="101.6" rot="R90"/>
 <instance part="U$20" gate="G$1" x="-71.12" y="68.58"/>
+<instance part="R2" gate="G$1" x="10.16" y="50.8"/>
+<instance part="LED" gate="G$1" x="-2.54" y="50.8" rot="R180"/>
+<instance part="U$32" gate="G$1" x="-10.16" y="50.8" rot="R270"/>
+<instance part="PWR5.0V" gate="G$1" x="203.2" y="81.28"/>
+<instance part="U$113" gate="G$1" x="193.04" y="81.28" rot="R270"/>
+<instance part="U$114" gate="G$1" x="190.5" y="83.82" rot="R90"/>
 </instances>
 <busses>
@@
 </segment>
 <segment>
-<pinref part="LED1" gate="G$1" pin="C"/>
+<pinref part="PWR" gate="G$1" pin="C"/>
 <pinref part="U$30" gate="G$1" pin="GND"/>
 <wire x1="177.8" y1="33.02" x2="177.8" y2="35.56" width="0.1524" layer="91"/>
@@
 <wire x1="160.02" y1="104.14" x2="162.56" y2="104.14" width="0.1524" layer="91"/>
 </segment>
+<segment>
+<pinref part="LED" gate="G$1" pin="C"/>
+<pinref part="U$32" gate="G$1" pin="GND"/>
+<wire x1="-7.62" y1="50.8" x2="-5.08" y2="50.8" width="0.1524" layer="91"/>
+</segment>
+<segment>
+<pinref part="PWR5.0V" gate="G$1" pin="2"/>
+<pinref part="U$113" gate="G$1" pin="GND"/>
+<wire x1="195.58" y1="81.28" x2="200.66" y2="81.28" width="0.1524" layer="91"/>
+</segment>
 </net>
 <net name="NRST" class="0">
@@
 <wire x1="0" y1="-7.62" x2="-10.16" y2="-7.62" width="0.1524" layer="91"/>
 </segment>
+<segment>
+<pinref part="PWR5.0V" gate="G$1" pin="1"/>
+<pinref part="U$114" gate="G$1" pin="5.0V"/>
+<wire x1="193.04" y1="83.82" x2="200.66" y2="83.82" width="0.1524" layer="91"/>
+</segment>
 </net>
 <net name="N$5" class="0">
 <segment>
 <pinref part="R17" gate="G$1" pin="1"/>
-<pinref part="LED1" gate="G$1" pin="A"/>
+<pinref part="PWR" gate="G$1" pin="A"/>
 <wire x1="177.8" y1="45.72" x2="177.8" y2="50.8" width="0.1524" layer="91"/>
 </segment>
@@
 </segment>
 </net>
+<net name="N$31" class="0">
+<segment>
+<pinref part="R2" gate="G$1" pin="1"/>
+<pinref part="LED" gate="G$1" pin="A"/>
+<wire x1="2.54" y1="50.8" x2="5.08" y2="50.8" width="0.1524" layer="91"/>
+</segment>
+</net>
+<net name="N$43" class="0">
+<segment>
+<pinref part="CPU1" gate="G$1" pin="PC5"/>
+<pinref part="R2" gate="G$1" pin="2"/>
+<wire x1="22.86" y1="50.8" x2="15.24" y2="50.8" width="0.1524" layer="91"/>
+</segment>
+</net>

Commit message: wip
Parts:
- H1, H2, H3, H4, H5, H6: value STAND-OFF -> MOUNT-HOLE3.2; device SparkFun-Electromechanical:STAND-OFF -> holes:MOUNT-HOLE3.2
Changed lines of the file:
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@@
 <part name="U$76" library="microbuilder" deviceset="GND" device=""/>
 <part name="U$77" library="microbuilder" deviceset="3.3V" device=""/>
-<part name="H3" library="SparkFun-Electromechanical" deviceset="STAND-OFF" device=""/>
-<part name="H4" library="SparkFun-Electromechanical" deviceset="STAND-OFF" device=""/>
-<part name="H1" library="SparkFun-Electromechanical" deviceset="STAND-OFF" device=""/>
-<part name="H2" library="SparkFun-Electromechanical" deviceset="STAND-OFF" device=""/>
+<part name="H3" library="holes" deviceset="MOUNT-HOLE" device="3.2"/>
+<part name="H4" library="holes" deviceset="MOUNT-HOLE" device="3.2"/>
+<part name="H1" library="holes" deviceset="MOUNT-HOLE" device="3.2"/>
+<part name="H2" library="holes" deviceset="MOUNT-HOLE" device="3.2"/>
 <part name="U$78" library="microbuilder" deviceset="GND" device=""/>
 <part name="U$79" library="microbuilder" deviceset="GND" device=""/>
@@
 <part name="R38" library="microbuilder" deviceset="RESISTOR" device="_0603" value="10k"/>
 <part name="U$47" library="microbuilder" deviceset="3.3V" device=""/>
-<part name="H5" library="SparkFun-Electromechanical" deviceset="STAND-OFF" device=""/>
-<part name="H6" library="SparkFun-Electromechanical" deviceset="STAND-OFF" device=""/>
+<part name="H5" library="holes" deviceset="MOUNT-HOLE" device="3.2"/>
+<part name="H6" library="holes" deviceset="MOUNT-HOLE" device="3.2"/>
 <part name="POT2" library="keves" deviceset="POTENTIOMETER" device="PTV09A_VERTICAL"/>
 <part name="POT7" library="keves" deviceset="POTENTIOMETER" device="PTV09A_VERTICAL"/>

Commit message: midimixer-channel rev a sent to macrofab
Parts:
- removed PWR3.3V, PWR5.0V: (no value), microbuilder:HEADER-1X2ROUND
- removed R11: 120 DNP, microbuilder:RESISTOR_0603
- added C16: 4.7nF, microbuilder:CAP_CERAMIC0603
- added R3, R7: 60 1%, microbuilder:RESISTOR0603
- added TERM: (no value), pinhead:PINHD-2X2
- BUS1, BUS2: value (none) -> 04-JST-B4B-XH-A; device microbuilder:HEADER-1X4ROUND -> bt_con-jst-xh:04-JST-B4B-XH-A
- D2: value SN65HVD232 -> SN65HVD230
Connections:
- new net CAN_VREF: C16.P$2, D2.VREF, R3.2, R7.1
- new net N$46: R7.2, TERM.2
- new net N$47: R3.1, TERM.4
- net 3.3V: no longer PWR3.3V.1
- net 5.0V: now also BUS1-1.1, BUS2-1.1; no longer BUS1.1, BUS2.1, PWR5.0V.1
- net CAN_H: now also BUS1-3.1, BUS2-3.1, TERM.3; no longer BUS1.3, BUS2.3, R11.1
- net CAN_L: now also BUS1-2.1, BUS2-2.1, TERM.1; no longer BUS1.2, BUS2.2, R11.2
- net GND: now also BUS1-4.1, BUS2-4.1, C16.P$1; no longer BUS1.4, BUS2.4, PWR3.3V.2, PWR5.0V.2
