File: midimixer-channel/midimixer-channel-rev2.brd (EAGLE design)
At the start: 50.8 x 241.3 mm, 114 parts, among them IC1 74LS595D, IC2 74LS595D, IC3 74LS595D, IC4 74165D, IC5 74165D, U1 LM1117IMPX-3.3/NOPB

Commit message: wip
Parts:
- moved PWR 32.5 mm to (19.9, 231.3)
- moved R17 32.5 mm to (19.9, 227.8)
- moved R2 29.3 mm to (21.7, 227.8), turned to 270 degrees
- moved LED 28.8 mm to (21.7, 231.3), turned to 0 degrees
- moved C12 2.01 mm to (15.7, 221.7), turned to 180 degrees
- moved TC1 0.51 mm to (2.79, 216.9)
- moved C13 0.38 mm to (15.5, 219.7)
Connections:
- net DIN_1 renamed ROT2_A
- net DIN_2 renamed ROT2_B
- net DIN_3 renamed ROT2_SW
- net DIN_5 renamed ROT1_SW
- net DIN_6 renamed ROT1_A
- net DIN_7 renamed ROT1_B
- net N$26: now also IC5.9
- net N$28: no longer IC4.9
- net N$43: now also CPU1.53; no longer CPU1.25
- net SPI2_MISO: now also IC4.9; no longer IC5.9
Routing:
- net UART_RX: track 0.00 -> 24.1 mm, vias 0 -> 2
- net UART_TX: track 0.00 -> 23.8 mm, vias 0 -> 2
- net SWCK: track 0.00 -> 22.3 mm, vias 0 -> 2
- net SWDIO: track 0.00 -> 17.1 mm, vias 0 -> 2
- net 3.3V: track 35.7 -> 51.8 mm, vias 9 -> 14
- net AVDD: track 0.00 -> 7.93 mm
- net 5.0V: track 78.9 -> 85.0 mm, vias 5 -> 0
- net N$43: track 0.00 -> 5.16 mm
- net N$4: track 0.00 -> 2.18 mm
- net N$3: track 0.00 -> 2.08 mm
- net N$5: track 0.00 -> 1.83 mm
- net N$31: track 0.00 -> 1.83 mm
Other:
- board text added: "Switched between the two HC165 parallel->serial registers"
- board text added: "USER LED MOVED FROM PC5 TO PC12"

Commit message: wip
Parts:
- moved R1 123.1 mm to (19.1, 56.5), turned to 90 degrees
- moved R43 6.45 mm to (9.27, 192.7), turned to 180 degrees
- moved R45 6.38 mm to (9.27, 194.4), turned to 180 degrees
- moved FADER1 6.35 mm to (12.7, 50.8)
- moved C29 6.20 mm to (6.60, 193.4)
- moved C30 5.12 mm to (18.8, 193.3)
- moved R44 5.08 mm to (16.1, 192.4), turned to 0 degrees
- moved R46 5.00 mm to (16.1, 194.2), turned to 0 degrees
- moved R5 1.65 mm to (7.37, 185.4)
- moved C1 1.35 mm to (7.24, 188.0), turned to 180 degrees
- moved R9 0.36 mm to (18.4, 181.6)
Connections:
- net FADER: now also CPU1.22; no longer CPU1.14
- net POT1: now also CPU1.14; no longer CPU1.15
- net POT2: now also CPU1.17; no longer CPU1.23
- net POT3: now also CPU1.15; no longer CPU1.16
- net POT4: now also CPU1.16; no longer CPU1.22
- net POT5: now also CPU1.23; no longer CPU1.17
Routing:
- net FADER: track 0.00 -> 210.2 mm, vias 0 -> 1
- net POT7: track 0.00 -> 126.8 mm, vias 0 -> 1
- net POT5: track 0.00 -> 101.4 mm, vias 0 -> 1
- net POT6: track 0.00 -> 100.9 mm, vias 0 -> 1
- net POT3: track 0.00 -> 86.8 mm, vias 0 -> 1
- net POT4: track 0.00 -> 84.8 mm, vias 0 -> 1
- net POT1: track 0.00 -> 62.9 mm, vias 0 -> 1
- net SPI2_MOSI: track 0.00 -> 62.8 mm, vias 0 -> 1
- net SPI2_CLK: track 0.00 -> 60.7 mm, vias 0 -> 2
- net POT2: track 0.00 -> 55.3 mm, vias 0 -> 1
- net SPI2_MISO: track 0.00 -> 53.4 mm, vias 0 -> 2
- net ROT2_SW: track 0.00 -> 24.5 mm
- net 3.3V: track 51.8 -> 72.4 mm, vias 14 -> 24
- net ROT2_A: track 0.00 -> 18.9 mm
- net ROT2_B: track 0.00 -> 16.7 mm
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
Commit message: wip
Parts:
- added BTN7, BTN8: B3W-9000-RG2N, keves:B3W-9000-X2X
- added C31, C32: 0.1uF, microbuilder:0603
- added R11, R16: 1k, microbuilder:0603
- added R15, R8: 120, microbuilder:0603
- added T1, T2: MMBT2222A, transistor:SOT23-BEC
- BTN1, BTN2: value B3W-9000-RG2N -> B3W-9000-B1N; device keves:B3W-9000-X2X -> keves:B3W-9000-X1X
- moved BTN2 177.9 mm to (-110.7, -21.2)
- moved BTN1 153.2 mm to (-110.7, 5.97)
- moved IC1 32.6 mm to (29.1, 4.45)
- moved C3 24.4 mm to (22.1, 9.02)
- moved BTN3 14.0 mm to (25.4, 76.2)
- moved BTN4 14.0 mm to (38.1, 76.2)
- moved BTN5 14.0 mm to (25.4, 62.2)
- moved BTN6 14.0 mm to (38.1, 62.2)
Connections:
- removed net BTN1_LED1: BTN1.LED1+, IC2.1
- removed net BTN1_LED2: BTN1.LED2+, IC2.2
- removed net BTN2_LED1: BTN2.LED1+, IC1.1
- removed net BTN2_LED2: BTN2.LED2+, IC1.2
- removed net BTN_UNUSED1: IC1.15
- removed net BTN_UNUSED2: IC1.7
- removed net DIN_15: IC5.5, R31.1
- removed net DIN_16: IC5.6, R30.1
- new net BTN1_LED: IC1.7, R11.1
- new net BTN2_LED: IC1.15, R16.1
- new net BTN7: BTN7.SW3, BTN7.SW4, C23.2, IC5.13, R35.1
- new net BTN7_LED1: BTN7.LED1+, IC2.5
- new net BTN7_LED2: BTN7.LED2+, IC2.15
- new net BTN8: BTN8.SW3, BTN8.SW4, C24.2, IC5.3, R33.1
- new net BTN8_LED1: BTN8.LED1+, IC1.5
- new net BTN8_LED2: BTN8.LED2+, IC1.6
- new net N$48: BTN2.LED1-, R15.1
- new net N$49: BTN1.LED1-, R8.1
- new net N$50: R8.2, T1.C
- new net N$51: R11.2, T1.B
- new net N$54: R15.2, T2.C
- new net N$58: R16.2, T2.B
- net 5.0V: now also BTN1.LED1+, BTN2.LED1+
- net BTN1: now also C31.2, IC5.5, R31.1; no longer C21.2, IC5.11, R37.1
- net BTN2: now also C32.2, IC5.6, R30.1; no longer C22.2, IC5.14, R34.1
- net BTN3: now also C21.2, IC5.11, R37.1; no longer C25.2, IC5.12, R36.1
- net BTN3_LED1: now also IC2.1; no longer IC2.3
- net BTN3_LED2: now also IC2.2; no longer IC2.4
- net BTN4: now also C22.2, IC5.14, R34.1; no longer C20.2, IC5.4, R32.1
- net BTN4_LED1: now also IC1.1; no longer IC1.3
- net BTN4_LED2: now also IC1.2; no longer IC1.4
- net BTN5: now also C25.2, IC5.12, R36.1; no longer C23.2, IC5.13, R35.1
- net BTN5_LED1: now also IC2.3; no longer IC2.5
- net BTN5_LED2: now also IC2.4; no longer IC2.15
- net BTN6: now also C20.2, IC5.4, R32.1; no longer C24.2, IC5.3, R33.1
- net BTN6_LED1: now also IC1.3; no longer IC1.5
- net BTN6_LED2: now also IC1.4; no longer IC1.6
- net GND: now also BTN7.SW1, BTN7.SW2, BTN8.SW1, BTN8.SW2, C31.1, C32.1, T1.E, T2.E
- net N$10: now also BTN6.LED2-; no longer BTN4.LED2-
- net N$24: now also BTN3.LED1-; no longer BTN1.LED1-
- net N$25: now also BTN3.LED2-; no longer BTN1.LED2-
- net N$29: now also BTN7.LED1-; no longer BTN5.LED1-
- net N$30: now also BTN7.LED2-; no longer BTN5.LED2-
- net N$34: now also BTN8.LED1-; no longer BTN6.LED1-
- net N$35: now also BTN8.LED2-; no longer BTN6.LED2-
- net N$39: now also BTN4.LED1-; no longer BTN2.LED1-
- net N$40: now also BTN4.LED2-; no longer BTN2.LED2-
- net N$44: now also BTN5.LED1-; no longer BTN3.LED1-
- net N$45: now also BTN5.LED2-; no longer BTN3.LED2-
- net N$9: now also BTN6.LED1-; no longer BTN4.LED1-
Routing:
- net SPI2_RC2: track 0.00 -> 36.4 mm, vias 0 -> 2

Commit message: wip
Parts:
- removed RN1, RN2: 4606X-101-101LF, resistor-sil:SIL6
- added R47, R48, R49, R50, R51, R52, R53, R54, R55, R56: 100, microbuilder:_0603
- moved C32 192.0 mm to (41.0, 75.9), flipped to the bottom, turned to 180 degrees
- moved R15 182.8 mm to (39.5, 70.9), flipped to the bottom, turned to 270 degrees
- moved R16 182.1 mm to (33.4, 67.2), flipped to the bottom, turned to 180 degrees
- moved T2 181.4 mm to (37.7, 68.1), flipped to the bottom, turned to 90 degrees
- moved BTN2 175.5 mm to (38.1, 71.8)
- moved C31 163.0 mm to (28.6, 76.2), flipped to the bottom, turned to 180 degrees
- moved R8 160.2 mm to (27.1, 70.9), flipped to the bottom, turned to 270 degrees
- moved T1 159.2 mm to (25.3, 68.3), flipped to the bottom, turned to 90 degrees
- moved R11 158.4 mm to (21.3, 67.3), flipped to the bottom, turned to 180 degrees
- moved BTN1 151.2 mm to (25.4, 71.8)
- moved R31 40.3 mm to (41.1, 77.7)
- moved R34 32.4 mm to (41.0, 50.0)
- moved R30 30.3 mm to (28.8, 78.1)
- moved R33 29.6 mm to (33.8, 33.9)
- moved R32 25.3 mm to (34.0, 47.9)
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Connections:
- net BTN1: now also IC5.6, R30.1; no longer IC5.5, R31.1
- net BTN2: now also IC5.5, R31.1; no longer IC5.6, R30.1
- net BTN4: now also IC5.12, R36.1; no longer IC5.14, R34.1
- net BTN5: now also IC5.13, R35.1; no longer IC5.12, R36.1
- net BTN6: now also IC5.14, R34.1; no longer IC5.4, R32.1
- net BTN7: now also IC5.4, R32.1; no longer IC5.13, R35.1
- net GND: now also R47.1, R48.1, R49.1, R50.1, R51.1, R52.1, R53.1, R54.1, R55.1, R56.1; no longer RN1.1, RN2.1
- net N$14: now also D1.11, R47.2; no longer D1.20, RN1.2
- net N$15: now also D1.12, R48.2; no longer D1.19, RN1.3
- net N$16: now also D1.13, R49.2; no longer D1.18, RN1.4
- net N$17: now also D1.14, R50.2; no longer D1.17, RN1.5
- net N$18: now also D1.15, R51.2; no longer D1.16, RN1.6
- net N$19: now also D1.16, R52.2; no longer D1.15, RN2.2
- net N$20: now also D1.17, R53.2; no longer D1.14, RN2.3
- net N$21: now also D1.18, R54.2; no longer D1.13, RN2.4
- net N$22: now also D1.19, R55.2; no longer D1.12, RN2.5
- net N$23: now also D1.20, R56.2; no longer D1.11, RN2.6
Routing:
- net BTN8: track 0.00 -> 56.1 mm, vias 0 -> 1
- net BTN2: track 0.00 -> 48.7 mm, vias 0 -> 1
- net BTN7: track 0.00 -> 42.3 mm, vias 0 -> 1
- net BTN6: track 0.00 -> 38.2 mm, vias 0 -> 1
- net BTN1: track 0.00 -> 35.8 mm, vias 0 -> 1
- net BTN4: track 0.00 -> 32.2 mm, vias 0 -> 1
- net BTN5: track 0.00 -> 25.8 mm, vias 0 -> 1
- net BTN3: track 0.00 -> 18.5 mm, vias 0 -> 1
- net 3.3V: track 72.4 -> 84.9 mm, vias 24 -> 30
- net N$24: track 0.00 -> 2.73 mm
- net N$17: track 0.00 -> 2.67 mm
- net N$15: track 0.00 -> 2.59 mm
- net N$22: track 0.00 -> 2.54 mm
- net N$21: track 0.00 -> 2.54 mm
- net N$20: track 0.00 -> 2.54 mm
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Other:
- board text added: "Button input order changed"

Commit message: wip
Parts:
- moved C3 81.9 mm to (92.7, 50.4)
- moved IC1 22.0 mm to (12.4, 18.8), turned to 270 degrees
- moved R16 17.8 mm to (33.4, 49.4)
- moved BTN7 17.8 mm to (25.4, 12.1)
- moved BTN8 17.8 mm to (38.1, 12.1)
- moved BUS1 17.8 mm to (2.54, 210.8)
- moved BUS2 17.8 mm to (47.1, 210.8)
- moved C1 17.8 mm to (7.24, 170.2)
- moved C10 17.8 mm to (29.7, 212.5)
- moved C11 17.8 mm to (28.4, 206.9)
- moved C12 17.8 mm to (15.7, 204.0)
- moved C13 17.8 mm to (15.5, 201.9)
- moved C14 17.8 mm to (20.3, 217.3)
- moved C15 17.8 mm to (7.62, 217.8)
- moved C16 17.8 mm to (39.9, 206.9)
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Connections:
- net BTN1_LED: now also IC2.15; no longer IC1.7
- net BTN2_LED: now also IC2.1; no longer IC1.15
- net BTN3_LED1: now also IC2.4; no longer IC2.1
- net BTN3_LED2: now also IC2.5; no longer IC2.2
- net BTN4_LED1: now also IC2.2; no longer IC1.1
- net BTN4_LED2: now also IC2.3; no longer IC1.2
- net BTN5_LED1: now also IC1.1; no longer IC2.3
- net BTN5_LED2: now also IC1.2; no longer IC2.4
- net BTN7_LED1: now also IC1.7; no longer IC2.5
- net BTN7_LED2: now also IC1.15; no longer IC2.15
Routing:
- net BTN4_LED2: track 0.00 -> 47.3 mm
- net BTN3_LED2: track 0.00 -> 40.5 mm
- net BTN4_LED1: track 0.00 -> 39.5 mm
- net BTN3_LED1: track 0.00 -> 32.3 mm
- net BTN2_LED: track 0.00 -> 28.3 mm
- net BTN1_LED: track 0.00 -> 9.94 mm
- net N$11: track 0.00 -> 6.07 mm
- net N$8: track 0.00 -> 5.54 mm
- net 3.3V: track 84.9 -> 88.3 mm, vias 30 -> 31
- net N$50: track 0.00 -> 2.46 mm
- net FADER: track 210.2 -> 212.5 mm
- net N$49: track 0.00 -> 1.97 mm
Other:
- board size 50.8 x 241.3 mm -> 50.8 x 223.5 mm

Commit message: wip
Parts:
- moved C3 85.7 mm to (9.02, 31.8), turned to 0 degrees
- moved R35 17.0 mm to (29.5, 31.9), turned to 180 degrees
- moved R32 12.9 mm to (29.3, 18.0), turned to 180 degrees
- moved R33 7.96 mm to (41.4, 18.4)
- moved C23 6.95 mm to (29.5, 16.1), turned to 0 degrees
- moved IC1 6.90 mm to (10.9, 25.5)
- moved C25 6.86 mm to (29.6, 30.1)
- moved R24 6.53 mm to (26.7, 11.2), turned to 270 degrees
- moved C24 3.75 mm to (41.3, 16.5), turned to 180 degrees
- moved R28 3.69 mm to (26.7, 25.0), turned to 270 degrees
- moved R26 1.31 mm to (39.4, 11.3), turned to 270 degrees
- moved R29 1.09 mm to (24.1, 25.1), turned to 270 degrees
- moved R27 1.09 mm to (36.8, 11.2), turned to 270 degrees
- moved R25 0.76 mm to (24.4, 11.3), turned to 270 degrees
- moved C2 0.51 mm to (25.7, 78.6)
Connections:
- net BTN5_LED1: now also IC1.2; no longer IC1.1
- net BTN5_LED2: now also IC1.3; no longer IC1.2
- net BTN6_LED1: now also IC1.1; no longer IC1.3
- net BTN7_LED1: now also IC1.6; no longer IC1.7
- net BTN7_LED2: now also IC1.7; no longer IC1.15
- net BTN8_LED2: now also IC1.15; no longer IC1.6
Routing:
- net SPI2_CLK: track 60.7 -> 222.1 mm, vias 2 -> 7
- net SPI2_MOSI: track 62.8 -> 138.2 mm, vias 1 -> 4
- net N$12: track 0.00 -> 67.6 mm, vias 0 -> 2
- net SPI2_RC1: track 0.00 -> 67.1 mm, vias 0 -> 2
- net BTN8_LED2: track 0.00 -> 45.9 mm, vias 0 -> 1
- net BTN8_LED1: track 0.00 -> 28.2 mm, vias 0 -> 1
- net BTN6_LED2: track 0.00 -> 27.7 mm
- net N$57: track 0.00 -> 26.6 mm, vias 0 -> 2
- net BTN6_LED1: track 0.00 -> 25.3 mm, vias 0 -> 1
- net BTN7_LED2: track 0.00 -> 22.4 mm
- net 3.3V: track 88.3 -> 106.0 mm, vias 31 -> 40
- net BTN7_LED1: track 0.00 -> 15.1 mm
- net BTN5_LED2: track 0.00 -> 14.6 mm
- net N$56: track 0.00 -> 13.4 mm
- net BTN5_LED1: track 0.00 -> 12.1 mm
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
Commit message: wip
Routing:
- net 5.0V: track 85.0 -> 262.1 mm
- net SPI2_RC1: track 67.1 -> 231.4 mm, vias 2 -> 8
- net SPI2_RC2: track 36.4 -> 188.0 mm, vias 2 -> 6
- net N$26: track 2.18 -> 137.5 mm, vias 0 -> 6
- net ROT1_SW: track 1.83 -> 40.0 mm, vias 0 -> 2
- net ROT1_B: track 1.91 -> 30.3 mm, vias 0 -> 2
- net NRST: track 0.00 -> 27.9 mm, vias 0 -> 2
- net ROT1_A: track 2.03 -> 20.6 mm, vias 0 -> 2
- net SPI2_CLK: track 222.1 -> 240.2 mm, vias 7 -> 9
- net N$51: track 0.00 -> 3.92 mm
- net N$58: track 0.00 -> 2.39 mm
- net N$54: track 0.00 -> 2.22 mm
- net N$48: track 0.00 -> 2.22 mm
- net 3.3V: track 106.0 -> 107.6 mm
- net N$55: track 7.45 -> 6.17 mm
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
Commit message: wip
Connections:
- removed net PB2: CPU1.28
Routing:
- net SPI2_CLK: track 240.2 -> 249.0 mm
Other:
- board text added: "Designed by:"
- board text added: "Pulsar Heavy Industries"
- board text added: "midimixer-channel rev 2.0"
- board text removed: "midimixer-channel rev A"
