File: midimixer-channel/midimixer-channel-rev2.brd (EAGLE design)
At the start: 50.8 x 223.5 mm, 132 parts, among them IC1 74LS595D, IC2 74LS595D, IC3 74LS595D, IC4 74165D, IC5 74165D, T1 MMBT2222A, T2 MMBT2222A, U1 LM1117IMPX-3.3/NOPB

Commit message: wip
Parts:
- added C33, C34, C35, C36, C37, C38, C39, C40: 0.01uF, microbuilder:0603
Connections:
- net 3.3V: now also C33.2, C34.2, C35.2, C36.2, C37.2, C38.2, C39.2, C40.2
- net GND: now also C33.1, C34.1, C35.1, C36.1, C37.1, C38.1, C39.1, C40.1
Routing:
- net 3.3V: track 107.6 -> 127.8 mm
- net GND: track 0.00 -> 18.8 mm
- net SPI2_CLK: track 249.0 -> 240.2 mm
Changed lines of the file:
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@@
 <element name="R55" library="microbuilder" package="_0603" value="100" x="5.588" y="71.12" rot="MR180"/>
 <element name="R56" library="microbuilder" package="_0603" value="100" x="5.715" y="68.58" rot="MR180"/>
+<element name="C33" library="microbuilder" package="0603" value="0.01uF" x="38.3032" y="145.9738" rot="MR180"/>
+<element name="C34" library="microbuilder" package="0603" value="0.01uF" x="12.7508" y="146.05" rot="MR180"/>
+<element name="C35" library="microbuilder" package="0603" value="0.01uF" x="38.481" y="120.6246" rot="MR180"/>
+<element name="C36" library="microbuilder" package="0603" value="0.01uF" x="12.5476" y="120.7008" rot="MR180"/>
+<element name="C37" library="microbuilder" package="0603" value="0.01uF" x="12.5984" y="95.25" rot="MR180"/>
+<element name="C38" library="microbuilder" package="0603" value="0.01uF" x="38.3032" y="95.0722" rot="MR180"/>
+<element name="C39" library="microbuilder" package="0603" value="0.01uF" x="38.2524" y="69.723" rot="MR180"/>
+<element name="C40" library="microbuilder" package="0603" value="0.01uF" x="13.9446" y="62.23" rot="MR0"/>
 </elements>
 <signals>
@@
 <wire x1="8.167" y1="31.75" x2="8.167" y2="30.017" width="0.254" layer="16"/>
 <wire x1="8.167" y1="30.017" x2="8.122" y2="29.972" width="0.254" layer="16"/>
+<contactref element="C33" pad="2"/>
+<contactref element="C34" pad="2"/>
+<contactref element="C35" pad="2"/>
+<contactref element="C36" pad="2"/>
+<contactref element="C37" pad="2"/>
+<contactref element="C38" pad="2"/>
+<contactref element="C39" pad="2"/>
+<contactref element="C40" pad="2"/>
+<wire x1="13.0946" y1="62.23" x2="10.9601" y2="62.23" width="0.4064" layer="16"/>
+<wire x1="39.1024" y1="69.723" x2="39.1024" y2="70.2424" width="0.254" layer="16"/>
+<wire x1="39.1024" y1="70.2424" x2="40.6" y2="71.74" width="0.254" layer="16"/>
+<wire x1="39.1532" y1="95.0722" x2="39.1532" y2="95.6932" width="0.254" layer="16"/>
+<wire x1="39.1532" y1="95.6932" x2="40.6" y2="97.14" width="0.254" layer="16"/>
+<wire x1="13.4484" y1="95.25" x2="13.4484" y2="95.3884" width="0.254" layer="16"/>
+<wire x1="13.4484" y1="95.3884" x2="15.2" y2="97.14" width="0.254" layer="16"/>
+<wire x1="39.331" y1="120.6246" x2="39.331" y2="121.271" width="0.254" layer="16"/>
+<wire x1="39.331" y1="121.271" x2="40.6" y2="122.54" width="0.254" layer="16"/>
+<wire x1="13.3976" y1="120.7008" x2="13.3976" y2="120.7376" width="0.254" layer="16"/>
+<wire x1="13.3976" y1="120.7376" x2="15.2" y2="122.54" width="0.254" layer="16"/>
+<wire x1="13.6008" y1="146.05" x2="13.6008" y2="146.3408" width="0.254" layer="16"/>
+<wire x1="13.6008" y1="146.3408" x2="15.2" y2="147.94" width="0.254" layer="16"/>
+<wire x1="39.1532" y1="145.9738" x2="39.1532" y2="146.4932" width="0.254" layer="16"/>
+<wire x1="39.1532" y1="146.4932" x2="40.6" y2="147.94" width="0.254" layer="16"/>
 </signal>
 <signal name="N$1">
@@
 <contactref element="R55" pad="1"/>
 <contactref element="R56" pad="1"/>
+<contactref element="C33" pad="1"/>
+<contactref element="C34" pad="1"/>
+<contactref element="C35" pad="1"/>
+<contactref element="C36" pad="1"/>
+<contactref element="C37" pad="1"/>
+<contactref element="C38" pad="1"/>
+<contactref element="C39" pad="1"/>
+<contactref element="C40" pad="1"/>
+<wire x1="37.4024" y1="69.723" x2="37.4024" y2="69.9376" width="0.254" layer="16"/>
+<wire x1="37.4024" y1="69.9376" x2="35.6" y2="71.74" width="0.254" layer="16"/>
+<wire x1="37.4532" y1="95.0722" x2="37.4532" y2="95.2868" width="0.254" layer="16"/>
+<wire x1="37.4532" y1="95.2868" x2="35.6" y2="97.14" width="0.254" layer="16"/>
+<wire x1="11.7484" y1="95.25" x2="11.7484" y2="95.5916" width="0.254" layer="16"/>
+<wire x1="11.7484" y1="95.5916" x2="10.2" y2="97.14" width="0.254" layer="16"/>
+<wire x1="37.631" y1="120.6246" x2="37.5154" y2="120.6246" width="0.254" layer="16"/>
+<wire x1="37.5154" y1="120.6246" x2="35.6" y2="122.54" width="0.254" layer="16"/>
+<wire x1="11.6976" y1="120.7008" x2="11.6976" y2="121.0424" width="0.254" layer="16"/>
+<wire x1="11.6976" y1="121.0424" x2="10.2" y2="122.54" width="0.254" layer="16"/>
+<wire x1="11.9008" y1="146.05" x2="11.9008" y2="146.2392" width="0.254" layer="16"/>
+<wire x1="11.9008" y1="146.2392" x2="10.2" y2="147.94" width="0.254" layer="16"/>
+<wire x1="35.6" y1="147.94" x2="35.6466" y2="147.94" width="0.254" layer="16"/>
+<wire x1="35.6466" y1="147.94" x2="35.6616" y2="147.955" width="0.254" layer="16"/>
+<wire x1="35.6616" y1="147.955" x2="35.6616" y2="147.7654" width="0.254" layer="16"/>
+<wire x1="35.6616" y1="147.7654" x2="37.4532" y2="145.9738" width="0.254" layer="16"/>
 </signal>
 <signal name="NRST">
@@
 <wire x1="1.651" y1="127.889" x2="15.113" y2="114.427" width="0.254" layer="1"/>
 <wire x1="15.113" y1="114.427" x2="16.002" y2="114.427" width="0.254" layer="1"/>
-<wire x1="16.002" y1="114.427" x2="17.145" y2="104.902" width="0.254" layer="1"/>
-<via x="17.145" y="104.902" extent="1-16" drill="0.6"/>
-<wire x1="17.145" y1="104.902" x2="20.828" y2="109.601" width="0.254" layer="16"/>
+<wire x1="16.002" y1="114.427" x2="17.7546" y2="112.6744" width="0.254" layer="1"/>
+<via x="17.7546" y="112.6744" extent="1-16" drill="0.6"/>
+<wire x1="17.7546" y1="112.6744" x2="20.828" y2="109.601" width="0.254" layer="16"/>
 <via x="20.828" y="109.601" extent="1-16" drill="0.6"/>
 <wire x1="20.828" y1="109.601" x2="21.209" y2="109.22" width="0.254" layer="1"/>

Commit message: wip
Parts:
- added C42, C43, C44, C45, C46, C47, C48, C49: 0.01uF, microbuilder:0603
Connections:
- net FADER: now also C42.2
- net GND: now also C42.1, C43.1, C44.1, C45.1, C46.1, C47.1, C48.1, C49.1
- net POT1: now also C46.2
- net POT2: now also C49.2
- net POT3: now also C45.2
- net POT4: now also C48.2
- net POT5: now also C44.2
- net POT6: now also C47.2
- net POT7: now also C43.2
Routing:
- net POT5: track 101.4 -> 103.4 mm
- net POT3: track 86.8 -> 88.7 mm
- net POT6: track 100.9 -> 102.8 mm
- net FADER: track 212.5 -> 214.4 mm
- net POT1: track 62.9 -> 64.8 mm
- net POT4: track 84.8 -> 86.6 mm
- net POT2: track 55.3 -> 57.1 mm
- net POT7: track 126.8 -> 128.5 mm
Changed lines of the file:
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@@
 <layer number="24" name="bOrigins" color="15" fill="1" visible="yes" active="yes"/>
 <layer number="25" name="tNames" color="7" fill="1" visible="yes" active="yes"/>
-<layer number="26" name="bNames" color="7" fill="1" visible="no" active="yes"/>
+<layer number="26" name="bNames" color="7" fill="1" visible="yes" active="yes"/>
 <layer number="27" name="tValues" color="7" fill="1" visible="no" active="yes"/>
 <layer number="28" name="bValues" color="7" fill="1" visible="no" active="yes"/>
@@
 <element name="POT2" library="keves" package="PTV09A-4" value="" x="38.1" y="154.94"/>
 <element name="POT7" library="keves" package="PTV09A-4" value="" x="38.1" y="78.74"/>
-<element name="POT4" library="keves" package="PTV09A-4" value="" x="38.1" y="129.54"/>
+<element name="POT4" library="keves" package="PTV09A-4" value="" x="38.1" y="129.54" smashed="yes">
+<attribute name="NAME" x="36.068" y="119.634" size="1.27" layer="21"/>
+</element>
 <element name="POT5" library="keves" package="PTV09A-4" value="" x="12.7" y="104.14"/>
 <element name="POT6" library="keves" package="PTV09A-4" value="" x="38.1" y="104.14"/>
-<element name="POT3" library="keves" package="PTV09A-4" value="" x="12.7" y="129.54"/>
+<element name="POT3" library="keves" package="PTV09A-4" value="" x="12.7" y="129.54" smashed="yes">
+<attribute name="NAME" x="10.668" y="119.634" size="1.27" layer="21"/>
+</element>
 <element name="POT1" library="keves" package="PTV09A-4" value="" x="12.7" y="154.94"/>
 <element name="LCD" library="keves" package="SSD1306-7PIN-NO-HOLES" value="SSD1306-7PINWITHOUT-HOLES" x="25.4" y="195.58"/>
@@
 <element name="C39" library="microbuilder" package="0603" value="0.01uF" x="38.2524" y="69.723" rot="MR180"/>
 <element name="C40" library="microbuilder" package="0603" value="0.01uF" x="13.9446" y="62.23" rot="MR0"/>
+<element name="C42" library="microbuilder" package="0603" value="0.01uF" x="14.4018" y="6.5278" smashed="yes" rot="MR270">
+<attribute name="NAME" x="13.462" y="7.5692" size="0.8128" layer="26" font="vector" ratio="18" rot="MR270"/>
+<attribute name="VALUE" x="15.1638" y="4.7498" size="0.4064" layer="28" font="vector" ratio="10" rot="MR270"/>
+</element>
+<element name="C43" library="microbuilder" package="0603" value="0.01uF" x="38.1" y="74.3458" smashed="yes" rot="MR270">
+<attribute name="NAME" x="39.9796" y="75.311" size="0.8128" layer="26" font="vector" ratio="18" rot="MR270"/>
+<attribute name="VALUE" x="38.862" y="72.5678" size="0.4064" layer="28" font="vector" ratio="10" rot="MR270"/>
+</element>
+<element name="C44" library="microbuilder" package="0603" value="0.01uF" x="12.7254" y="99.9744" smashed="yes" rot="MR270">
+<attribute name="NAME" x="14.5542" y="101.0158" size="0.8128" layer="26" font="vector" ratio="18" rot="MR270"/>
+<attribute name="VALUE" x="13.4874" y="98.1964" size="0.4064" layer="28" font="vector" ratio="10" rot="MR270"/>
+</element>
+<element name="C45" library="microbuilder" package="0603" value="0.01uF" x="12.6746" y="125.222" smashed="yes" rot="MR270">
+<attribute name="NAME" x="14.5288" y="125.8316" size="0.8128" layer="26" font="vector" ratio="18" rot="MR270"/>
+<attribute name="VALUE" x="13.4366" y="123.444" size="0.4064" layer="28" font="vector" ratio="10" rot="MR270"/>
+</element>
+<element name="C46" library="microbuilder" package="0603" value="0.01uF" x="12.7" y="150.6728" smashed="yes" rot="MR270">
+<attribute name="NAME" x="14.5288" y="151.3586" size="0.8128" layer="26" font="vector" ratio="18" rot="MR270"/>
+<attribute name="VALUE" x="13.462" y="148.8948" size="0.4064" layer="28" font="vector" ratio="10" rot="MR270"/>
+</element>
+<element name="C47" library="microbuilder" package="0603" value="0.01uF" x="38.0238" y="99.8474" smashed="yes" rot="MR270">
+<attribute name="NAME" x="39.7764" y="100.4062" size="0.8128" layer="26" font="vector" ratio="18" rot="MR270"/>
+<attribute name="VALUE" x="38.7858" y="98.0694" size="0.4064" layer="28" font="vector" ratio="10" rot="MR270"/>
+</element>
+<element name="C48" library="microbuilder" package="0603" value="0.01uF" x="38.0238" y="125.1966" smashed="yes" rot="MR270">
+<attribute name="NAME" x="39.8018" y="125.7808" size="0.8128" layer="26" font="vector" ratio="18" rot="MR270"/>
+<attribute name="VALUE" x="38.7858" y="123.4186" size="0.4064" layer="28" font="vector" ratio="10" rot="MR270"/>
+</element>
+<element name="C49" library="microbuilder" package="0603" value="0.01uF" x="38.1254" y="150.5966" smashed="yes" rot="MR270">
+<attribute name="NAME" x="39.9288" y="151.3586" size="0.8128" layer="26" font="vector" ratio="18" rot="MR270"/>
+<attribute name="VALUE" x="38.8874" y="148.8186" size="0.4064" layer="28" font="vector" ratio="10" rot="MR270"/>
+</element>
 </elements>
 <signals>
@@
 <wire x1="35.6616" y1="147.955" x2="35.6616" y2="147.7654" width="0.254" layer="16"/>
 <wire x1="35.6616" y1="147.7654" x2="37.4532" y2="145.9738" width="0.254" layer="16"/>
+<contactref element="C42" pad="1"/>
+<contactref element="C43" pad="1"/>
+<contactref element="C44" pad="1"/>
+<contactref element="C45" pad="1"/>
+<contactref element="C46" pad="1"/>
+<contactref element="C47" pad="1"/>
+<contactref element="C48" pad="1"/>
+<contactref element="C49" pad="1"/>
 </signal>
 <signal name="NRST">
@@
 <wire x1="27.813" y1="191.516" x2="27.305" y2="191.008" width="0.254" layer="1"/>
 <wire x1="27.305" y1="191.008" x2="27.305" y2="150.114" width="0.254" layer="1"/>
+<contactref element="C49" pad="2"/>
+<wire x1="38.1254" y1="149.7466" x2="38.1254" y2="148.6916" width="0.254" layer="16"/>
+<wire x1="38.1254" y1="148.6916" x2="38.1" y2="148.6662" width="0.254" layer="16"/>
+<wire x1="38.1" y1="148.6662" x2="38.1" y2="147.94" width="0.254" layer="16"/>
 </signal>
 <signal name="N$11">
@@
 <wire x1="1.524" y1="42.418" x2="2.032" y2="41.91" width="0.254" layer="1"/>
 <wire x1="2.032" y1="41.91" x2="2.032" y2="11.811" width="0.254" layer="1"/>
+<contactref element="C42" pad="2"/>
+<wire x1="14.4018" y1="5.6778" x2="14.4018" y2="3.8481" width="0.254" layer="16"/>
+<wire x1="14.4018" y1="3.8481" x2="14.4399" y2="3.81" width="0.254" layer="16"/>
 </signal>
 <signal name="POT4">
@@
 <wire x1="27.492" y1="194.878" x2="27.051" y2="194.437" width="0.254" layer="16"/>
 <via x="27.051" y="194.437" extent="1-16" drill="0.6"/>
+<contactref element="C48" pad="2"/>
+<wire x1="38.0238" y1="124.3466" x2="38.0238" y2="122.6162" width="0.254" layer="16"/>
+<wire x1="38.0238" y1="122.6162" x2="38.1" y2="122.54" width="0.254" layer="16"/>
 </signal>
 <signal name="POT6">
@@
 <wire x1="26.162" y1="186.436" x2="26.035" y2="186.309" width="0.254" layer="16"/>
 <wire x1="26.289" y1="186.055" x2="26.035" y2="186.309" width="0.254" layer="1"/>
+<contactref element="C47" pad="2"/>
+<wire x1="38.0238" y1="98.9974" x2="38.0238" y2="97.2162" width="0.254" layer="16"/>
+<wire x1="38.0238" y1="97.2162" x2="38.1" y2="97.14" width="0.254" layer="16"/>
 </signal>
 <signal name="POT1">
@@
 <wire x1="23.114" y1="181.483" x2="23.749" y2="180.848" width="0.254" layer="1"/>
 <wire x1="23.749" y1="180.848" x2="23.749" y2="152.019" width="0.254" layer="1"/>
+<contactref element="C46" pad="2"/>
+<wire x1="12.7" y1="149.8228" x2="12.7" y2="147.94" width="0.254" layer="16"/>
 </signal>
 <signal name="POT3">
 <contactref element="POT3" pad="CENTER"/>
-<wire x1="12.7" y1="122.54" x2="12.7" y2="123.952" width="0.254" layer="1"/>
+<wire x1="12.7" y1="122.54" x2="12.7" y2="122.555" width="0.254" layer="1"/>
 <wire x1="12.7" y1="123.952" x2="13.843" y2="125.095" width="0.254" layer="1"/>
 <wire x1="13.843" y1="125.095" x2="20.955" y2="125.095" width="0.254" layer="1"/>
@@
 <via x="26.035" y="194.945" extent="1-16" drill="0.6"/>
 <wire x1="26.035" y1="194.945" x2="26.035" y2="187.706" width="0.254" layer="1"/>
+<contactref element="C45" pad="2"/>
+<wire x1="12.7" y1="123.952" x2="12.7" y2="122.555" width="0.254" layer="1"/>
+<wire x1="12.7" y1="122.555" x2="12.6746" y2="122.5296" width="0.254" layer="1"/>
+<wire x1="12.6746" y1="122.5296" x2="12.6492" y2="122.5296" width="0.254" layer="1"/>
+<wire x1="12.6746" y1="124.372" x2="12.6746" y2="122.5654" width="0.254" layer="16"/>
+<wire x1="12.6746" y1="122.5654" x2="12.7" y2="122.54" width="0.254" layer="16"/>
 </signal>
 <signal name="POT5">
@@
 <wire x1="25.007" y1="191.758" x2="24.638" y2="191.389" width="0.254" layer="16"/>
 <wire x1="24.638" y1="191.389" x2="24.638" y2="187.96" width="0.254" layer="16"/>
+<contactref element="C44" pad="2"/>
+<wire x1="12.7254" y1="99.1244" x2="12.7254" y2="97.1654" width="0.254" layer="16"/>
+<wire x1="12.7254" y1="97.1654" x2="12.7" y2="97.14" width="0.254" layer="16"/>
 </signal>
 <signal name="POT7">
@@
 <wire x1="25.273" y1="186.944" x2="25.273" y2="185.293" width="0.254" layer="16"/>
 <wire x1="25.273" y1="185.293" x2="25.527" y2="185.039" width="0.254" layer="16"/>
+<contactref element="C43" pad="2"/>
+<wire x1="38.1" y1="73.4958" x2="38.1" y2="71.74" width="0.254" layer="16"/>
 </signal>
 <signal name="LCD_MISO_UNUSED">

Commit message: midimixer-channel-rev2: illustrator file, change r8 and r15 to 200 ohm (blue leds too bright)
Parts:
- R15, R8: value 120 -> 200
Changed lines of the file:
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@@
 <element name="BTN1" library="keves" package="B3W-9000-X1X" value="B3W-9000-B1N" x="25.4" y="53.975"/>
 <element name="C31" library="microbuilder" package="0603" value="0.1uF" x="28.575" y="58.42" rot="MR180"/>
-<element name="R8" library="microbuilder" package="0603" value="120" x="27.051" y="53.086" rot="MR270"/>
+<element name="R8" library="microbuilder" package="0603" value="200" x="27.051" y="53.086" rot="MR270"/>
 <element name="T1" library="transistor" package="SOT23-BEC" value="MMBT2222A" x="24.638" y="53.213" rot="MR180"/>
 <element name="R11" library="microbuilder" package="0603" value="1k" x="23.622" y="59.055" rot="MR270"/>
 <element name="BTN2" library="keves" package="B3W-9000-X1X" value="B3W-9000-B1N" x="38.1" y="53.975"/>
 <element name="C32" library="microbuilder" package="0603" value="0.1uF" x="41.021" y="58.166" rot="MR180"/>
-<element name="R15" library="microbuilder" package="0603" value="120" x="39.497" y="53.086" smashed="yes" rot="MR270">
+<element name="R15" library="microbuilder" package="0603" value="200" x="39.497" y="53.086" smashed="yes" rot="MR270">
 <attribute name="NAME" x="38.481" y="55.118" size="0.8128" layer="26" font="vector" ratio="18" rot="MR270"/>
 <attribute name="VALUE" x="40.259" y="51.308" size="0.4064" layer="28" font="vector" ratio="10" rot="MR270"/>
