File: midimixer-channel/midimixer-channel-rev2.sch (EAGLE design)
At the start: 114 parts, among them IC1 74LS595D, IC2 74LS595D, IC3 74LS595D, IC4 74165D, IC5 74165D, U1 LM1117IMPX-3.3/NOPB

Commit message: wip
Connections:
- net DIN_1 renamed ROT2_A
- net DIN_2 renamed ROT2_B
- net DIN_3 renamed ROT2_SW
- net DIN_5 renamed ROT1_SW
- net DIN_6 renamed ROT1_A
- net DIN_7 renamed ROT1_B
- net N$26: now also IC5.QH
- net N$28: no longer IC4.QH
- net N$43: now also CPU1.PC12/SDIO_CLK; no longer CPU1.PC5
- net SPI2_MISO: now also IC4.QH; no longer IC5.QH
Other:
- moved on the sheet: LED, R2
Changed lines of the file:
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@@
 <instance part="U$19" gate="G$1" x="10.16" y="101.6" rot="R90"/>
 <instance part="U$20" gate="G$1" x="-71.12" y="68.58"/>
-<instance part="R2" gate="G$1" x="10.16" y="50.8"/>
-<instance part="LED" gate="G$1" x="-2.54" y="50.8" rot="R180"/>
-<instance part="U$32" gate="G$1" x="-10.16" y="50.8" rot="R270"/>
+<instance part="R2" gate="G$1" x="111.76" y="83.82" rot="R180"/>
+<instance part="LED" gate="G$1" x="124.46" y="83.82"/>
+<instance part="U$32" gate="G$1" x="132.08" y="83.82" rot="R90"/>
 <instance part="R3" gate="G$1" x="88.9" y="-50.8" rot="R90"/>
 <instance part="R7" gate="G$1" x="88.9" y="-40.64" rot="R90"/>
@@
 <pinref part="LED" gate="G$1" pin="C"/>
 <pinref part="U$32" gate="G$1" pin="GND"/>
-<wire x1="-7.62" y1="50.8" x2="-5.08" y2="50.8" width="0.1524" layer="91"/>
+<wire x1="129.54" y1="83.82" x2="127" y2="83.82" width="0.1524" layer="91"/>
 </segment>
 <segment>
@@
 <pinref part="IC4" gate="A" pin="CLK"/>
 <pinref part="IC5" gate="A" pin="CLK"/>
+<label x="-104.14" y="-30.48" size="1.778" layer="95" rot="R90"/>
 </segment>
 <segment>
@@
 <net name="SPI2_MISO" class="0">
 <segment>
-<wire x1="-101.6" y1="-2.54" x2="-114.3" y2="-2.54" width="0.2032" layer="91"/>
 <wire x1="-114.3" y1="-2.54" x2="-114.3" y2="139.7" width="0.2032" layer="91"/>
 <label x="-111.76" y="137.16" size="1.778" layer="95" rot="R90"/>
-<pinref part="IC5" gate="A" pin="QH"/>
+<wire x1="-114.3" y1="-2.54" x2="-114.3" y2="-53.34" width="0.1524" layer="91"/>
+<pinref part="IC4" gate="A" pin="QH"/>
+<wire x1="-114.3" y1="-53.34" x2="-101.6" y2="-53.34" width="0.1524" layer="91"/>
+<label x="-114.3" y="-30.48" size="1.778" layer="95" rot="R90"/>
 </segment>
 <segment>
@@
 <wire x1="-101.6" y1="0" x2="-121.92" y2="0" width="0.2032" layer="91"/>
 <wire x1="-121.92" y1="0" x2="-121.92" y2="2.54" width="0.2032" layer="91"/>
-<wire x1="-101.6" y1="-53.34" x2="-127" y2="-53.34" width="0.2032" layer="91"/>
-<wire x1="-127" y1="-53.34" x2="-127" y2="0" width="0.2032" layer="91"/>
-<wire x1="-127" y1="0" x2="-121.92" y2="0" width="0.2032" layer="91"/>
-<junction x="-121.92" y="0"/>
-<pinref part="IC4" gate="A" pin="QH"/>
 <pinref part="IC5" gate="A" pin="SER"/>
 </segment>
 </net>
-<net name="DIN_1" class="0">
+<net name="ROT2_A" class="0">
 <segment>
 <pinref part="IC4" gate="A" pin="A"/>
@@
 </segment>
 </net>
-<net name="DIN_2" class="0">
+<net name="ROT2_B" class="0">
 <segment>
 <pinref part="IC4" gate="A" pin="B"/>
@@
 </segment>
 </net>
-<net name="DIN_3" class="0">
+<net name="ROT2_SW" class="0">
 <segment>
 <pinref part="IC4" gate="A" pin="C"/>
@@
 </segment>
 </net>
-<net name="DIN_5" class="0">
+<net name="ROT1_SW" class="0">
 <segment>
 <pinref part="IC4" gate="A" pin="E"/>
@@
 </segment>
 </net>
-<net name="DIN_6" class="0">
+<net name="ROT1_A" class="0">
 <segment>
 <pinref part="IC4" gate="A" pin="F"/>
@@
 </segment>
 </net>
-<net name="DIN_7" class="0">
+<net name="ROT1_B" class="0">
 <segment>
 <pinref part="IC4" gate="A" pin="G"/>
@@
 <pinref part="IC4" gate="A" pin="SH/!LD"/>
 <pinref part="IC5" gate="A" pin="SH/!LD"/>
+<label x="-116.84" y="-30.48" size="1.778" layer="95" rot="R90"/>
 </segment>
 <segment>
@@
 <segment>
 <pinref part="R38" gate="G$1" pin="1"/>
-<wire x1="-101.6" y1="-50.8" x2="-121.92" y2="-50.8" width="0.2032" layer="91"/>
+<wire x1="-101.6" y1="-50.8" x2="-109.22" y2="-50.8" width="0.2032" layer="91"/>
+<wire x1="-109.22" y1="-50.8" x2="-121.92" y2="-50.8" width="0.2032" layer="91"/>
 <wire x1="-121.92" y1="-50.8" x2="-121.92" y2="-48.26" width="0.2032" layer="91"/>
 <pinref part="IC4" gate="A" pin="SER"/>
+<pinref part="IC5" gate="A" pin="QH"/>
+<wire x1="-101.6" y1="-2.54" x2="-109.22" y2="-2.54" width="0.1524" layer="91"/>
+<wire x1="-109.22" y1="-2.54" x2="-109.22" y2="-50.8" width="0.1524" layer="91"/>
+<junction x="-109.22" y="-50.8"/>
 </segment>
 </net>
@@
 <pinref part="R2" gate="G$1" pin="1"/>
 <pinref part="LED" gate="G$1" pin="A"/>
-<wire x1="2.54" y1="50.8" x2="5.08" y2="50.8" width="0.1524" layer="91"/>
-</segment>
-</net>
-<net name="N$43" class="0">
-<segment>
-<pinref part="CPU1" gate="G$1" pin="PC5"/>
-<pinref part="R2" gate="G$1" pin="2"/>
-<wire x1="22.86" y1="50.8" x2="15.24" y2="50.8" width="0.1524" layer="91"/>
+<wire x1="119.38" y1="83.82" x2="116.84" y2="83.82" width="0.1524" layer="91"/>
 </segment>
 </net>
@@
 <wire x1="83.82" y1="-45.72" x2="88.9" y2="-45.72" width="0.1524" layer="91"/>
 <label x="78.74" y="-45.72" size="1.778" layer="95"/>
+</segment>
+</net>
+<net name="N$43" class="0">
+<segment>
+<pinref part="CPU1" gate="G$1" pin="PC12/SDIO_CLK"/>
+<pinref part="R2" gate="G$1" pin="2"/>
+<wire x1="81.28" y1="83.82" x2="106.68" y2="83.82" width="0.1524" layer="91"/>
 </segment>
 </net>
@@
 </segment>
 </net>
-<net name="DIN_7" class="0">
+<net name="ROT1_B" class="0">
 <segment>
 <pinref part="R40" gate="G$1" pin="1"/>
@@
 </segment>
 </net>
-<net name="DIN_6" class="0">
+<net name="ROT1_A" class="0">
 <segment>
 <pinref part="R39" gate="G$1" pin="1"/>
@@
 </segment>
 </net>
-<net name="DIN_1" class="0">
+<net name="ROT2_A" class="0">
 <segment>
 <pinref part="R43" gate="G$1" pin="1"/>
@@
 </segment>
 </net>
-<net name="DIN_2" class="0">
+<net name="ROT2_B" class="0">
 <segment>
 <pinref part="R44" gate="G$1" pin="1"/>
@@
 </segment>
 </net>
-<net name="DIN_3" class="0">
+<net name="ROT2_SW" class="0">
 <segment>
 <pinref part="ROT2" gate="G$1" pin="SW2"/>
 <wire x1="83.82" y1="55.88" x2="81.28" y2="55.88" width="0.1524" layer="91"/>
 <label x="81.28" y="55.88" size="1.778" layer="95" rot="R180"/>
-</segment>
-</net>
-<net name="DIN_5" class="0">
-<segment>
-<pinref part="ROT1" gate="G$1" pin="SW2"/>
-<wire x1="-2.54" y1="50.8" x2="-5.08" y2="50.8" width="0.1524" layer="91"/>
-<label x="-5.08" y="50.8" size="1.778" layer="95" rot="R180"/>
 </segment>
 </net>
@@
 </segment>
 </net>
+<net name="ROT1_SW" class="0">
+<segment>
+<pinref part="ROT1" gate="G$1" pin="SW2"/>
+<wire x1="-2.54" y1="50.8" x2="-5.08" y2="50.8" width="0.1524" layer="91"/>
+<label x="-5.08" y="50.8" size="1.778" layer="95" rot="R180"/>
+</segment>
+</net>

Commit message: wip
Connections:
- net FADER: now also CPU1.PA6/SPI1_MISO; no longer CPU1.PA0
- net POT1: now also CPU1.PA0; no longer CPU1.PA1
- net POT2: now also CPU1.PA3/UART2_RX; no longer CPU1.PA7/SPI1_MOSI
- net POT3: now also CPU1.PA1; no longer CPU1.PA2/UART2_TX
- net POT4: now also CPU1.PA2/UART2_TX; no longer CPU1.PA6/SPI1_MISO
- net POT5: now also CPU1.PA7/SPI1_MOSI; no longer CPU1.PA3/UART2_RX
Changed lines of the file:
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@@
 <net name="FADER" class="0">
 <segment>
-<pinref part="CPU1" gate="G$1" pin="PA0"/>
-<wire x1="22.86" y1="78.74" x2="2.54" y2="78.74" width="0.2032" layer="91"/>
-<label x="0" y="78.74" size="1.778" layer="95"/>
+<pinref part="CPU1" gate="G$1" pin="PA6/SPI1_MISO"/>
+<wire x1="22.86" y1="58.42" x2="2.54" y2="58.42" width="0.2032" layer="91"/>
+<label x="0" y="58.42" size="1.778" layer="95"/>
 </segment>
 </net>
@@
 </segment>
 </net>
-<net name="POT1" class="0">
-<segment>
-<pinref part="CPU1" gate="G$1" pin="PA1"/>
-<wire x1="22.86" y1="76.2" x2="2.54" y2="76.2" width="0.2032" layer="91"/>
-<label x="0" y="76.2" size="1.778" layer="95"/>
-</segment>
-</net>
-<net name="POT5" class="0">
+<net name="POT2" class="0">
 <segment>
 <pinref part="CPU1" gate="G$1" pin="PA3/UART2_RX"/>
 <wire x1="22.86" y1="71.12" x2="2.54" y2="71.12" width="0.2032" layer="91"/>
 <label x="0" y="71.12" size="1.778" layer="95"/>
-</segment>
-</net>
-<net name="POT2" class="0">
-<segment>
-<pinref part="CPU1" gate="G$1" pin="PA7/SPI1_MOSI"/>
-<wire x1="22.86" y1="55.88" x2="2.54" y2="55.88" width="0.2032" layer="91"/>
-<label x="0" y="55.88" size="1.778" layer="95"/>
 </segment>
 </net>
@@
 </segment>
 </net>
-<net name="POT3" class="0">
+<net name="POT4" class="0">
 <segment>
 <pinref part="CPU1" gate="G$1" pin="PA2/UART2_TX"/>
 <wire x1="22.86" y1="73.66" x2="2.54" y2="73.66" width="0.2032" layer="91"/>
 <label x="0" y="73.66" size="1.778" layer="95"/>
-</segment>
-</net>
-<net name="POT4" class="0">
-<segment>
-<pinref part="CPU1" gate="G$1" pin="PA6/SPI1_MISO"/>
-<wire x1="22.86" y1="58.42" x2="2.54" y2="58.42" width="0.2032" layer="91"/>
-<label x="0" y="58.42" size="1.778" layer="95"/>
 </segment>
 </net>
@@
 </segment>
 </net>
+<net name="POT5" class="0">
+<segment>
+<pinref part="CPU1" gate="G$1" pin="PA7/SPI1_MOSI"/>
+<wire x1="22.86" y1="55.88" x2="2.54" y2="55.88" width="0.2032" layer="91"/>
+<label x="0" y="55.88" size="1.778" layer="95"/>
+</segment>
+</net>
+<net name="POT3" class="0">
+<segment>
+<pinref part="CPU1" gate="G$1" pin="PA1"/>
+<wire x1="22.86" y1="76.2" x2="2.54" y2="76.2" width="0.2032" layer="91"/>
+<label x="0" y="76.2" size="1.778" layer="95"/>
+</segment>
+</net>
+<net name="POT1" class="0">
+<segment>
+<pinref part="CPU1" gate="G$1" pin="PA0"/>
+<wire x1="22.86" y1="78.74" x2="2.54" y2="78.74" width="0.2032" layer="91"/>
+<label x="0" y="78.74" size="1.778" layer="95"/>
+</segment>
+</net>

Commit message: wip
Parts:
- added BTN7, BTN8: B3W-9000-RG2N, keves:B3W-9000-RG2N
- added C31, C32: 0.1uF, microbuilder:CAP_CERAMIC0603
- added R11, R16: 1k, microbuilder:RESISTOR0603
- added R15, R8: 120, microbuilder:RESISTOR0603
- added T1, T2: MMBT2222A, transistor:MMBT2222ALT1-NPN-SOT23-BEC
- BTN1, BTN2: value B3W-9000-RG2N -> B3W-9000-B1N; device keves:B3W-9000-RG2N -> keves:B3W-9000-B1N
Connections:
- removed net BTN1_LED1: BTN1.LED1+, IC2.QB
- removed net BTN1_LED2: BTN1.LED2+, IC2.QC
- removed net BTN2_LED1: BTN2.LED1+, IC1.QB
- removed net BTN2_LED2: BTN2.LED2+, IC1.QC
- removed net BTN_UNUSED1: IC1.QA
- removed net BTN_UNUSED2: IC1.QH
- removed net DIN_15: IC5.G, R31.1
- removed net DIN_16: IC5.H, R30.1
- new net BTN1_LED: IC1.QH, R11.1
- new net BTN2_LED: IC1.QA, R16.1
- new net BTN7: BTN7.SW2_A, BTN7.SW2_B, C23.P$2, IC5.C, R35.1
- new net BTN7_LED1: BTN7.LED1+, IC2.QF
- new net BTN7_LED2: BTN7.LED2+, IC2.QA
- new net BTN8: BTN8.SW2_A, BTN8.SW2_B, C24.P$2, IC5.E, R33.1
- new net BTN8_LED1: BTN8.LED1+, IC1.QF
- new net BTN8_LED2: BTN8.LED2+, IC1.QG
- new net N$48: BTN2.LED1-, R15.1
- new net N$49: BTN1.LED1-, R8.1
- new net N$50: R8.2, T1.C
- new net N$51: R11.2, T1.B
- new net N$54: R15.2, T2.C
- new net N$58: R16.2, T2.B
- net 5.0V: now also BTN1.LED1+, BTN2.LED1+
- net BTN1: now also C31.P$2, IC5.G, R31.1; no longer C21.P$2, IC5.A, R37.1
- net BTN2: now also C32.P$2, IC5.H, R30.1; no longer C22.P$2, IC5.D, R34.1
- net BTN3: now also C21.P$2, IC5.A, R37.1; no longer C25.P$2, IC5.B, R36.1
- net BTN3_LED1: now also IC2.QB; no longer IC2.QD
- net BTN3_LED2: now also IC2.QC; no longer IC2.QE
- net BTN4: now also C22.P$2, IC5.D, R34.1; no longer C20.P$2, IC5.F, R32.1
- net BTN4_LED1: now also IC1.QB; no longer IC1.QD
- net BTN4_LED2: now also IC1.QC; no longer IC1.QE
- net BTN5: now also C25.P$2, IC5.B, R36.1; no longer C23.P$2, IC5.C, R35.1
- net BTN5_LED1: now also IC2.QD; no longer IC2.QF
- net BTN5_LED2: now also IC2.QE; no longer IC2.QA
- net BTN6: now also C20.P$2, IC5.F, R32.1; no longer C24.P$2, IC5.E, R33.1
- net BTN6_LED1: now also IC1.QD; no longer IC1.QF
- net BTN6_LED2: now also IC1.QE; no longer IC1.QG
- net GND: now also BTN7.SW1_A, BTN7.SW1_B, BTN8.SW1_A, BTN8.SW1_B, C31.P$1, C32.P$1, T1.E, T2.E
- net N$10: now also BTN6.LED2-; no longer BTN4.LED2-
- net N$24: now also BTN3.LED1-; no longer BTN1.LED1-
- net N$25: now also BTN3.LED2-; no longer BTN1.LED2-
- net N$29: now also BTN7.LED1-; no longer BTN5.LED1-
- net N$30: now also BTN7.LED2-; no longer BTN5.LED2-
- net N$34: now also BTN8.LED1-; no longer BTN6.LED1-
- net N$35: now also BTN8.LED2-; no longer BTN6.LED2-
- net N$39: now also BTN4.LED1-; no longer BTN2.LED1-
- net N$40: now also BTN4.LED2-; no longer BTN2.LED2-
- net N$44: now also BTN5.LED1-; no longer BTN3.LED1-
- net N$45: now also BTN5.LED2-; no longer BTN3.LED2-
- net N$9: now also BTN6.LED1-; no longer BTN4.LED1-
Other:
- moved on the sheet: BTN3, BTN4, BTN5, BTN6

Commit message: wip
Parts:
- removed RN1, RN2: 4606X-101-101LF, resistor-sil:G05R
- added R47, R48, R49, R50, R51, R52, R53, R54, R55, R56: 100, microbuilder:RESISTOR_0603
Connections:
- net BTN1: now also IC5.H, R30.1; no longer IC5.G, R31.1
- net BTN2: now also IC5.G, R31.1; no longer IC5.H, R30.1
- net BTN4: now also IC5.B, R36.1; no longer IC5.D, R34.1
- net BTN5: now also IC5.C, R35.1; no longer IC5.B, R36.1
- net BTN6: now also IC5.D, R34.1; no longer IC5.F, R32.1
- net BTN7: now also IC5.F, R32.1; no longer IC5.C, R35.1
- net GND: now also R47.1, R48.1, R49.1, R50.1, R51.1, R52.1, R53.1, R54.1, R55.1, R56.1; no longer RN1.1, RN2.1
- net N$14: now also D1J.C, R47.2; no longer D1A.C, RN1.2
- net N$15: now also D1I.C, R48.2; no longer D1B.C, RN1.3
- net N$16: now also D1H.C, R49.2; no longer D1C.C, RN1.4
- net N$17: now also D1G.C, R50.2; no longer D1D.C, RN1.5
- net N$18: now also D1F.C, R51.2; no longer D1E.C, RN1.6
- net N$19: now also D1E.C, R52.2; no longer D1F.C, RN2.2
- net N$20: now also D1D.C, R53.2; no longer D1G.C, RN2.3
- net N$21: now also D1C.C, R54.2; no longer D1H.C, RN2.4
- net N$22: now also D1B.C, R55.2; no longer D1I.C, RN2.5
- net N$23: now also D1A.C, R56.2; no longer D1J.C, RN2.6

Commit message: wip
Connections:
- net BTN1_LED: now also IC2.QA; no longer IC1.QH
- net BTN2_LED: now also IC2.QB; no longer IC1.QA
- net BTN3_LED1: now also IC2.QE; no longer IC2.QB
- net BTN3_LED2: now also IC2.QF; no longer IC2.QC
- net BTN4_LED1: now also IC2.QC; no longer IC1.QB
- net BTN4_LED2: now also IC2.QD; no longer IC1.QC
- net BTN5_LED1: now also IC1.QB; no longer IC2.QD
- net BTN5_LED2: now also IC1.QC; no longer IC2.QE
- net BTN7_LED1: now also IC1.QH; no longer IC2.QF
- net BTN7_LED2: now also IC1.QA; no longer IC2.QA
Changed lines of the file:
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@@
-</segment>
-</net>
-<net name="BTN2_LED" class="0">
-<segment>
-<pinref part="IC1" gate="A" pin="QA"/>
-<wire x1="-71.12" y1="114.3" x2="-58.42" y2="114.3" width="0.2032" layer="91"/>
-<label x="-60.96" y="114.3" size="1.778" layer="95"/>
 </segment>
 </net>
@@
 </segment>
 </net>
-<net name="BTN1_LED" class="0">
+<net name="BTN8_LED2" class="0">
+<segment>
+<pinref part="IC1" gate="A" pin="QG"/>
+<wire x1="-71.12" y1="129.54" x2="-58.42" y2="129.54" width="0.2032" layer="91"/>
+<label x="-60.96" y="129.54" size="1.778" layer="95"/>
+</segment>
+</net>
+<net name="BTN8_LED1" class="0">
+<segment>
+<pinref part="IC1" gate="A" pin="QF"/>
+<wire x1="-71.12" y1="127" x2="-58.42" y2="127" width="0.2032" layer="91"/>
+<label x="-60.96" y="127" size="1.778" layer="95"/>
+</segment>
+</net>
+<net name="BTN6_LED2" class="0">
+<segment>
+<pinref part="IC1" gate="A" pin="QE"/>
+<wire x1="-71.12" y1="124.46" x2="-58.42" y2="124.46" width="0.2032" layer="91"/>
+<label x="-60.96" y="124.46" size="1.778" layer="95"/>
+</segment>
+</net>
+<net name="BTN6_LED1" class="0">
+<segment>
+<pinref part="IC1" gate="A" pin="QD"/>
+<wire x1="-71.12" y1="121.92" x2="-58.42" y2="121.92" width="0.2032" layer="91"/>
+<label x="-60.96" y="121.92" size="1.778" layer="95"/>
+</segment>
+</net>
+<net name="BTN7_LED1" class="0">
 <segment>
 <pinref part="IC1" gate="A" pin="QH"/>
@@
 </segment>
 </net>
-<net name="BTN8_LED2" class="0">
-<segment>
-<pinref part="IC1" gate="A" pin="QG"/>
-<wire x1="-71.12" y1="129.54" x2="-58.42" y2="129.54" width="0.2032" layer="91"/>
-<label x="-60.96" y="129.54" size="1.778" layer="95"/>
-</segment>
-</net>
-<net name="BTN8_LED1" class="0">
-<segment>
-<pinref part="IC1" gate="A" pin="QF"/>
-<wire x1="-71.12" y1="127" x2="-58.42" y2="127" width="0.2032" layer="91"/>
-<label x="-60.96" y="127" size="1.778" layer="95"/>
-</segment>
-</net>
-<net name="BTN6_LED2" class="0">
-<segment>
-<pinref part="IC1" gate="A" pin="QE"/>
-<wire x1="-71.12" y1="124.46" x2="-58.42" y2="124.46" width="0.2032" layer="91"/>
-<label x="-60.96" y="124.46" size="1.778" layer="95"/>
-</segment>
-</net>
-<net name="BTN6_LED1" class="0">
-<segment>
-<pinref part="IC1" gate="A" pin="QD"/>
-<wire x1="-71.12" y1="121.92" x2="-58.42" y2="121.92" width="0.2032" layer="91"/>
-<label x="-60.96" y="121.92" size="1.778" layer="95"/>
-</segment>
-</net>
-<net name="BTN7_LED1" class="0">
-<segment>
-<pinref part="IC2" gate="A" pin="QF"/>
-<wire x1="-71.12" y1="91.44" x2="-60.96" y2="91.44" width="0.2032" layer="91"/>
-<label x="-68.58" y="91.44" size="1.778" layer="95"/>
-</segment>
-</net>
-<net name="BTN5_LED2" class="0">
-<segment>
-<pinref part="IC2" gate="A" pin="QE"/>
-<wire x1="-71.12" y1="88.9" x2="-60.96" y2="88.9" width="0.2032" layer="91"/>
-<label x="-68.58" y="88.9" size="1.778" layer="95"/>
-</segment>
-</net>
-<net name="BTN5_LED1" class="0">
-<segment>
-<pinref part="IC2" gate="A" pin="QD"/>
-<wire x1="-71.12" y1="86.36" x2="-60.96" y2="86.36" width="0.2032" layer="91"/>
-<label x="-68.58" y="86.36" size="1.778" layer="95"/>
-</segment>
-</net>
-<net name="BTN3_LED2" class="0">
-<segment>
-<pinref part="IC2" gate="A" pin="QC"/>
-<wire x1="-71.12" y1="83.82" x2="-60.96" y2="83.82" width="0.1524" layer="91"/>
-<label x="-68.58" y="83.82" size="1.778" layer="95"/>
-</segment>
-</net>
-<net name="BTN3_LED1" class="0">
-<segment>
-<pinref part="IC2" gate="A" pin="QB"/>
-<wire x1="-71.12" y1="81.28" x2="-60.96" y2="81.28" width="0.1524" layer="91"/>
-<label x="-68.58" y="81.28" size="1.778" layer="95"/>
-</segment>
-</net>
 <net name="BTN7_LED2" class="0">
 <segment>
-<pinref part="IC2" gate="A" pin="QA"/>
-<wire x1="-71.12" y1="78.74" x2="-60.96" y2="78.74" width="0.2032" layer="91"/>
-<label x="-68.58" y="78.74" size="1.778" layer="95"/>
-</segment>
-</net>
-<net name="BTN4_LED1" class="0">
-<segment>
-<pinref part="IC1" gate="A" pin="QB"/>
-<wire x1="-71.12" y1="116.84" x2="-58.42" y2="116.84" width="0.2032" layer="91"/>
-<label x="-60.96" y="116.84" size="1.778" layer="95"/>
-</segment>
-</net>
-<net name="BTN4_LED2" class="0">
-<segment>
-<pinref part="IC1" gate="A" pin="QC"/>
-<wire x1="-71.12" y1="119.38" x2="-58.42" y2="119.38" width="0.2032" layer="91"/>
-<label x="-60.96" y="119.38" size="1.778" layer="95"/>
+<pinref part="IC1" gate="A" pin="QA"/>
+<wire x1="-71.12" y1="114.3" x2="-58.42" y2="114.3" width="0.2032" layer="91"/>
+<label x="-60.96" y="114.3" size="1.778" layer="95"/>
 </segment>
 </net>
@@
 </segment>
 </net>
+<net name="BTN2_LED" class="0">
+<segment>
+<pinref part="IC2" gate="A" pin="QB"/>
+<wire x1="-71.12" y1="81.28" x2="-60.96" y2="81.28" width="0.1524" layer="91"/>
+<label x="-68.58" y="81.28" size="1.778" layer="95"/>
+</segment>
+</net>
+<net name="BTN5_LED1" class="0">
+<segment>
+<pinref part="IC1" gate="A" pin="QB"/>
+<wire x1="-71.12" y1="116.84" x2="-58.42" y2="116.84" width="0.2032" layer="91"/>
+<label x="-60.96" y="116.84" size="1.778" layer="95"/>
+</segment>
+</net>
+<net name="BTN5_LED2" class="0">
+<segment>
+<pinref part="IC1" gate="A" pin="QC"/>
+<wire x1="-71.12" y1="119.38" x2="-58.42" y2="119.38" width="0.2032" layer="91"/>
+<label x="-60.96" y="119.38" size="1.778" layer="95"/>
+</segment>
+</net>
+<net name="BTN1_LED" class="0">
+<segment>
+<pinref part="IC2" gate="A" pin="QA"/>
+<wire x1="-71.12" y1="78.74" x2="-60.96" y2="78.74" width="0.2032" layer="91"/>
+<label x="-68.58" y="78.74" size="1.778" layer="95"/>
+</segment>
+</net>
+<net name="BTN3_LED1" class="0">
+<segment>
+<pinref part="IC2" gate="A" pin="QE"/>
+<wire x1="-71.12" y1="88.9" x2="-60.96" y2="88.9" width="0.2032" layer="91"/>
+<label x="-68.58" y="88.9" size="1.778" layer="95"/>
+</segment>
+</net>
+<net name="BTN4_LED1" class="0">
+<segment>
+<pinref part="IC2" gate="A" pin="QC"/>
+<wire x1="-71.12" y1="83.82" x2="-60.96" y2="83.82" width="0.1524" layer="91"/>
+<label x="-68.58" y="83.82" size="1.778" layer="95"/>
+</segment>
+</net>
+<net name="BTN4_LED2" class="0">
+<segment>
+<pinref part="IC2" gate="A" pin="QD"/>
+<wire x1="-71.12" y1="86.36" x2="-60.96" y2="86.36" width="0.2032" layer="91"/>
+<label x="-68.58" y="86.36" size="1.778" layer="95"/>
+</segment>
+</net>
+<net name="BTN3_LED2" class="0">
+<segment>
+<pinref part="IC2" gate="A" pin="QF"/>
+<wire x1="-71.12" y1="91.44" x2="-60.96" y2="91.44" width="0.2032" layer="91"/>
+<label x="-68.58" y="91.44" size="1.778" layer="95"/>
+</segment>
+</net>
