File: midimixer-channel/midimixer-channel-rev2.sch (EAGLE design)
At the start: 132 parts, among them IC1 74LS595D, IC2 74LS595D, IC3 74LS595D, IC4 74165D, IC5 74165D, T1 MMBT2222A, T2 MMBT2222A, U1 LM1117IMPX-3.3/NOPB

Commit message: wip
Connections:
- net BTN5_LED1: now also IC1.QC; no longer IC1.QB
- net BTN5_LED2: now also IC1.QD; no longer IC1.QC
- net BTN6_LED1: now also IC1.QB; no longer IC1.QD
- net BTN7_LED1: now also IC1.QG; no longer IC1.QH
- net BTN7_LED2: now also IC1.QH; no longer IC1.QA
- net BTN8_LED2: now also IC1.QA; no longer IC1.QG
Changed lines of the file:
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@@
 </segment>
 </net>
-<net name="BTN8_LED2" class="0">
+<net name="BTN8_LED1" class="0">
+<segment>
+<pinref part="IC1" gate="A" pin="QF"/>
+<wire x1="-71.12" y1="127" x2="-58.42" y2="127" width="0.2032" layer="91"/>
+<label x="-60.96" y="127" size="1.778" layer="95"/>
+</segment>
+</net>
+<net name="BTN6_LED2" class="0">
+<segment>
+<pinref part="IC1" gate="A" pin="QE"/>
+<wire x1="-71.12" y1="124.46" x2="-58.42" y2="124.46" width="0.2032" layer="91"/>
+<label x="-60.96" y="124.46" size="1.778" layer="95"/>
+</segment>
+</net>
+<net name="BTN7_LED1" class="0">
 <segment>
 <pinref part="IC1" gate="A" pin="QG"/>
 <wire x1="-71.12" y1="129.54" x2="-58.42" y2="129.54" width="0.2032" layer="91"/>
 <label x="-60.96" y="129.54" size="1.778" layer="95"/>
-</segment>
-</net>
-<net name="BTN8_LED1" class="0">
-<segment>
-<pinref part="IC1" gate="A" pin="QF"/>
-<wire x1="-71.12" y1="127" x2="-58.42" y2="127" width="0.2032" layer="91"/>
-<label x="-60.96" y="127" size="1.778" layer="95"/>
-</segment>
-</net>
-<net name="BTN6_LED2" class="0">
-<segment>
-<pinref part="IC1" gate="A" pin="QE"/>
-<wire x1="-71.12" y1="124.46" x2="-58.42" y2="124.46" width="0.2032" layer="91"/>
-<label x="-60.96" y="124.46" size="1.778" layer="95"/>
-</segment>
-</net>
-<net name="BTN6_LED1" class="0">
-<segment>
-<pinref part="IC1" gate="A" pin="QD"/>
-<wire x1="-71.12" y1="121.92" x2="-58.42" y2="121.92" width="0.2032" layer="91"/>
-<label x="-60.96" y="121.92" size="1.778" layer="95"/>
-</segment>
-</net>
-<net name="BTN7_LED1" class="0">
-<segment>
-<pinref part="IC1" gate="A" pin="QH"/>
-<wire x1="-71.12" y1="132.08" x2="-58.42" y2="132.08" width="0.2032" layer="91"/>
-<label x="-60.96" y="132.08" size="1.778" layer="95"/>
-</segment>
-</net>
-<net name="BTN7_LED2" class="0">
-<segment>
-<pinref part="IC1" gate="A" pin="QA"/>
-<wire x1="-71.12" y1="114.3" x2="-58.42" y2="114.3" width="0.2032" layer="91"/>
-<label x="-60.96" y="114.3" size="1.778" layer="95"/>
 </segment>
 </net>
@@
 <net name="BTN5_LED1" class="0">
 <segment>
+<pinref part="IC1" gate="A" pin="QC"/>
+<wire x1="-71.12" y1="119.38" x2="-58.42" y2="119.38" width="0.2032" layer="91"/>
+<label x="-60.96" y="119.38" size="1.778" layer="95"/>
+</segment>
+</net>
+<net name="BTN1_LED" class="0">
+<segment>
+<pinref part="IC2" gate="A" pin="QA"/>
+<wire x1="-71.12" y1="78.74" x2="-60.96" y2="78.74" width="0.2032" layer="91"/>
+<label x="-68.58" y="78.74" size="1.778" layer="95"/>
+</segment>
+</net>
+<net name="BTN3_LED1" class="0">
+<segment>
+<pinref part="IC2" gate="A" pin="QE"/>
+<wire x1="-71.12" y1="88.9" x2="-60.96" y2="88.9" width="0.2032" layer="91"/>
+<label x="-68.58" y="88.9" size="1.778" layer="95"/>
+</segment>
+</net>
+<net name="BTN4_LED1" class="0">
+<segment>
+<pinref part="IC2" gate="A" pin="QC"/>
+<wire x1="-71.12" y1="83.82" x2="-60.96" y2="83.82" width="0.1524" layer="91"/>
+<label x="-68.58" y="83.82" size="1.778" layer="95"/>
+</segment>
+</net>
+<net name="BTN4_LED2" class="0">
+<segment>
+<pinref part="IC2" gate="A" pin="QD"/>
+<wire x1="-71.12" y1="86.36" x2="-60.96" y2="86.36" width="0.2032" layer="91"/>
+<label x="-68.58" y="86.36" size="1.778" layer="95"/>
+</segment>
+</net>
+<net name="BTN3_LED2" class="0">
+<segment>
+<pinref part="IC2" gate="A" pin="QF"/>
+<wire x1="-71.12" y1="91.44" x2="-60.96" y2="91.44" width="0.2032" layer="91"/>
+<label x="-68.58" y="91.44" size="1.778" layer="95"/>
+</segment>
+</net>
+<net name="BTN6_LED1" class="0">
+<segment>
 <pinref part="IC1" gate="A" pin="QB"/>
 <wire x1="-71.12" y1="116.84" x2="-58.42" y2="116.84" width="0.2032" layer="91"/>
@@
 <net name="BTN5_LED2" class="0">
 <segment>
-<pinref part="IC1" gate="A" pin="QC"/>
-<wire x1="-71.12" y1="119.38" x2="-58.42" y2="119.38" width="0.2032" layer="91"/>
-<label x="-60.96" y="119.38" size="1.778" layer="95"/>
-</segment>
-</net>
-<net name="BTN1_LED" class="0">
-<segment>
-<pinref part="IC2" gate="A" pin="QA"/>
-<wire x1="-71.12" y1="78.74" x2="-60.96" y2="78.74" width="0.2032" layer="91"/>
-<label x="-68.58" y="78.74" size="1.778" layer="95"/>
-</segment>
-</net>
-<net name="BTN3_LED1" class="0">
-<segment>
-<pinref part="IC2" gate="A" pin="QE"/>
-<wire x1="-71.12" y1="88.9" x2="-60.96" y2="88.9" width="0.2032" layer="91"/>
-<label x="-68.58" y="88.9" size="1.778" layer="95"/>
-</segment>
-</net>
-<net name="BTN4_LED1" class="0">
-<segment>
-<pinref part="IC2" gate="A" pin="QC"/>
-<wire x1="-71.12" y1="83.82" x2="-60.96" y2="83.82" width="0.1524" layer="91"/>
-<label x="-68.58" y="83.82" size="1.778" layer="95"/>
-</segment>
-</net>
-<net name="BTN4_LED2" class="0">
-<segment>
-<pinref part="IC2" gate="A" pin="QD"/>
-<wire x1="-71.12" y1="86.36" x2="-60.96" y2="86.36" width="0.2032" layer="91"/>
-<label x="-68.58" y="86.36" size="1.778" layer="95"/>
-</segment>
-</net>
-<net name="BTN3_LED2" class="0">
-<segment>
-<pinref part="IC2" gate="A" pin="QF"/>
-<wire x1="-71.12" y1="91.44" x2="-60.96" y2="91.44" width="0.2032" layer="91"/>
-<label x="-68.58" y="91.44" size="1.778" layer="95"/>
-</segment>
-</net>
+<pinref part="IC1" gate="A" pin="QD"/>
+<wire x1="-71.12" y1="121.92" x2="-58.42" y2="121.92" width="0.2032" layer="91"/>
+<label x="-60.96" y="121.92" size="1.778" layer="95"/>
+</segment>
+</net>
+<net name="BTN8_LED2" class="0">
+<segment>
+<pinref part="IC1" gate="A" pin="QA"/>
+<wire x1="-71.12" y1="114.3" x2="-58.42" y2="114.3" width="0.2032" layer="91"/>
+<label x="-60.96" y="114.3" size="1.778" layer="95"/>
+</segment>
+</net>
+<net name="BTN7_LED2" class="0">
+<segment>
+<pinref part="IC1" gate="A" pin="QH"/>
+<wire x1="-71.12" y1="132.08" x2="-58.42" y2="132.08" width="0.2032" layer="91"/>
+<label x="-60.96" y="132.08" size="1.778" layer="95"/>
+</segment>
+</net>

Commit message: wip
Connections:
- removed net PB2: CPU1.PB2-BOOT1
Changed lines of the file:
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@@
 <instance part="U$13" gate="G$1" x="96.52" y="71.12" rot="R270"/>
 <instance part="C12" gate="G$1" x="91.44" y="73.66"/>
-<instance part="U$14" gate="G$1" x="91.44" y="83.82" rot="R180"/>
+<instance part="U$14" gate="G$1" x="91.44" y="81.28" rot="R180"/>
 <instance part="U$15" gate="G$1" x="91.44" y="109.22" rot="R90"/>
 <instance part="C11" gate="G$1" x="86.36" y="111.76"/>
@@
 <pinref part="C12" gate="G$1" pin="P$1"/>
 <pinref part="U$14" gate="G$1" pin="GND"/>
-<wire x1="91.44" y1="81.28" x2="91.44" y2="78.74" width="0.1524" layer="91"/>
 </segment>
 <segment>
@@
 <pinref part="PWR" gate="G$1" pin="A"/>
 <wire x1="177.8" y1="45.72" x2="177.8" y2="50.8" width="0.1524" layer="91"/>
-</segment>
-</net>
-<net name="PB2" class="0">
-<segment>
-<pinref part="CPU1" gate="G$1" pin="PB2-BOOT1"/>
-<wire x1="22.86" y1="43.18" x2="12.7" y2="43.18" width="0.2032" layer="91"/>
-<label x="12.7" y="43.18" size="1.778" layer="95"/>
 </segment>
 </net>
@@
 <wire x1="177.8" y1="81.28" x2="185.42" y2="81.28" width="0.1524" layer="91"/>
 <label x="182.88" y="81.28" size="1.778" layer="95"/>
+<junction x="175.26" y="81.28"/>
 </segment>
 </net>
@@
 <wire x1="177.8" y1="45.72" x2="185.42" y2="45.72" width="0.1524" layer="91"/>
 <label x="182.88" y="45.72" size="1.778" layer="95"/>
-</segment>
-</net>
+<junction x="175.26" y="45.72"/>
+</segment>
+</net>

Commit message: wip
Parts:
- added C33, C34, C35, C36, C37, C38, C39, C40: 0.01uF, microbuilder:CAP_CERAMIC0603
Connections:
- net 3.3V: now also C33.P$2, C34.P$2, C35.P$2, C36.P$2, C37.P$2, C38.P$2, C39.P$2, C40.P$2
- net GND: now also C33.P$1, C34.P$1, C35.P$1, C36.P$1, C37.P$1, C38.P$1, C39.P$1, C40.P$1
Other:
- moved on the sheet: POT1, POT3, POT4, POT5, POT6
