File: cdf-modular-bridge/cdf-modular-bridge.sch (EAGLE design)
At the start: 9 parts

Commit message: wip
Parts:
- added X1: (no value), con-ptr500:AK500/2
Connections:
- net N$1: now also X1-1.KL
- net N$2: now also X1-2.KL
Other:
- note added: "TODO: - Holes for DC+/DC-/OUT - DC Reservoir capacitors? - VERIFY FOOTPRINTS"
Changed lines of the file:
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@@
 <part name="R1" library="microbuilder" deviceset="RESISTOR" device="1206" value="15"/>
 <part name="R2" library="microbuilder" deviceset="RESISTOR" device="1206" value="15"/>
+<part name="X1" library="con-ptr500" deviceset="AK500/2" device=""/>
 </parts>
 <sheets>
 <sheet>
 <plain>
-<text x="-12.7" y="68.58" size="1.778" layer="91">CONNECT ME</text>
-<text x="-12.7" y="55.88" size="1.778" layer="91">CONNECT ME</text>
 <text x="73.66" y="104.14" size="1.778" layer="91">CONNECT ME</text>
 <text x="96.52" y="58.42" size="1.778" layer="91">CONNECT ME</text>
 <text x="73.66" y="2.54" size="1.778" layer="91">CONNECT ME</text>
+<text x="2.54" y="93.98" size="1.778" layer="91">TODO:
+- Holes for DC+/DC-/OUT
+- DC Reservoir capacitors?
+- VERIFY FOOTPRINTS</text>
 </plain>
 <instances>
@@
 <instance part="R1" gate="G$1" x="48.26" y="81.28"/>
 <instance part="R2" gate="G$1" x="48.26" y="45.72"/>
+<instance part="X1" gate="-1" x="-2.54" y="66.04"/>
+<instance part="X1" gate="-2" x="-2.54" y="60.96"/>
 </instances>
 <busses>
 </busses>
 <nets>
-<net name="N$1" class="0">
-<segment>
-<pinref part="U$5" gate="G$1" pin="PRI_NEG"/>
-<wire x1="10.16" y1="68.58" x2="-5.08" y2="68.58" width="0.1524" layer="91"/>
-</segment>
-</net>
-<net name="N$2" class="0">
-<segment>
-<pinref part="U$5" gate="G$1" pin="PRI_POS"/>
-<wire x1="10.16" y1="55.88" x2="-5.08" y2="55.88" width="0.1524" layer="91"/>
-</segment>
-</net>
 <net name="N$3" class="0">
 <segment>
@@
 </segment>
 </net>
+<net name="N$1" class="0">
+<segment>
+<pinref part="X1" gate="-1" pin="KL"/>
+<pinref part="U$5" gate="G$1" pin="PRI_NEG"/>
+<wire x1="2.54" y1="66.04" x2="10.16" y2="66.04" width="0.1524" layer="91"/>
+<wire x1="10.16" y1="66.04" x2="10.16" y2="68.58" width="0.1524" layer="91"/>
+</segment>
+</net>
+<net name="N$2" class="0">
+<segment>
+<pinref part="X1" gate="-2" pin="KL"/>
+<pinref part="U$5" gate="G$1" pin="PRI_POS"/>
+<wire x1="2.54" y1="60.96" x2="10.16" y2="60.96" width="0.1524" layer="91"/>
+<wire x1="10.16" y1="60.96" x2="10.16" y2="55.88" width="0.1524" layer="91"/>
+</segment>
+</net>
 </nets>
 </sheet>
@@
 </schematic>
 </drawing>
+<compatibility>
+<note version="6.3" minversion="6.2.2" severity="warning">
+Since Version 6.2.2 text objects can contain more than one line,
+which will not be processed correctly with this version.
+</note>
+</compatibility>
 </eagle>

Commit message: wip
Parts:
- added DC+, DC-, OUT: BIG-ASS-HOLE, keves:BIG-ASS-HOLE
- added TP1, TP2: PTR1PAD1-17, testpad:PTR1PAD1-17
- added X2: (no value), con-ptr500:AK500/2
Connections:
- removed net N$10: U$1.C
- removed net N$4: U$1.E, U$2.C, U$3.P$2, U$5.SEC1_POS
- removed net N$6: U$2.E, U$4.P$2, U$5.SEC2_NEG
- new net DC+: DC+.P$1, TP1.TP, U$1.C
- new net DC-: DC-.P$1, TP2.TP, U$2.E, U$4.P$2, U$5.SEC2_POS
- new net OUT: OUT.P$1, U$1.E, U$2.C, U$3.P$2, U$5.SEC1_NEG
- net N$1: now also X2-1.KL
- net N$2: now also X2-2.KL
- net N$7: now also U$5.SEC2_NEG; no longer U$5.SEC2_POS
- net N$8: now also U$5.SEC1_POS; no longer U$5.SEC1_NEG
Other:
- note added: "For capacitor: 940C30S68K-F"
- note removed: "CONNECT ME"
- moved on the sheet: X1-1, X1-2
Changed lines of the file:
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@@
 <part name="R2" library="microbuilder" deviceset="RESISTOR" device="1206" value="15"/>
 <part name="X1" library="con-ptr500" deviceset="AK500/2" device=""/>
+<part name="OUT" library="keves" deviceset="BIG-ASS-HOLE" device=""/>
+<part name="DC+" library="keves" deviceset="BIG-ASS-HOLE" device=""/>
+<part name="DC-" library="keves" deviceset="BIG-ASS-HOLE" device=""/>
+<part name="X2" library="con-ptr500" deviceset="AK500/2" device=""/>
+<part name="TP1" library="testpad" deviceset="PTR1" device="PAD1-17"/>
+<part name="TP2" library="testpad" deviceset="PTR1" device="PAD1-17"/>
 </parts>
 <sheets>
 <sheet>
 <plain>
-<text x="73.66" y="104.14" size="1.778" layer="91">CONNECT ME</text>
-<text x="96.52" y="58.42" size="1.778" layer="91">CONNECT ME</text>
-<text x="73.66" y="2.54" size="1.778" layer="91">CONNECT ME</text>
 <text x="2.54" y="93.98" size="1.778" layer="91">TODO:
 - Holes for DC+/DC-/OUT
 - DC Reservoir capacitors?
 - VERIFY FOOTPRINTS</text>
+<text x="93.98" y="93.98" size="1.778" layer="97">For capacitor: 940C30S68K-F</text>
 </plain>
 <instances>
@@
 <instance part="R1" gate="G$1" x="48.26" y="81.28"/>
 <instance part="R2" gate="G$1" x="48.26" y="45.72"/>
-<instance part="X1" gate="-1" x="-2.54" y="66.04"/>
-<instance part="X1" gate="-2" x="-2.54" y="60.96"/>
+<instance part="X1" gate="-1" x="-12.7" y="66.04"/>
+<instance part="X1" gate="-2" x="-12.7" y="60.96"/>
+<instance part="OUT" gate="G$1" x="109.22" y="58.42"/>
+<instance part="DC+" gate="G$1" x="76.2" y="106.68"/>
+<instance part="DC-" gate="G$1" x="76.2" y="2.54"/>
+<instance part="X2" gate="-1" x="-12.7" y="53.34"/>
+<instance part="X2" gate="-2" x="-12.7" y="48.26"/>
+<instance part="TP1" gate="G$1" x="91.44" y="91.44" rot="R90"/>
+<instance part="TP2" gate="G$1" x="91.44" y="20.32" rot="R90"/>
 </instances>
 <busses>
@@
 </segment>
 </net>
-<net name="N$4" class="0">
+<net name="OUT" class="0">
 <segment>
 <pinref part="U$3" gate="G$1" pin="P$2"/>
@@
 <pinref part="U$2" gate="G$1" pin="C"/>
 <wire x1="73.66" y1="50.8" x2="73.66" y2="58.42" width="0.1524" layer="91"/>
-<pinref part="U$5" gate="G$1" pin="SEC1_POS"/>
-<wire x1="22.86" y1="63.5" x2="53.34" y2="63.5" width="0.1524" layer="91"/>
-<wire x1="53.34" y1="63.5" x2="53.34" y2="58.42" width="0.1524" layer="91"/>
-<wire x1="53.34" y1="58.42" x2="60.96" y2="58.42" width="0.1524" layer="91"/>
 <junction x="73.66" y="58.42"/>
 <junction x="60.96" y="58.42"/>
 <wire x1="73.66" y1="58.42" x2="106.68" y2="58.42" width="0.1524" layer="91"/>
+<pinref part="OUT" gate="G$1" pin="P$1"/>
+<wire x1="60.96" y1="58.42" x2="27.94" y2="58.42" width="0.1524" layer="91"/>
+<wire x1="27.94" y1="58.42" x2="27.94" y2="68.58" width="0.1524" layer="91"/>
+<pinref part="U$5" gate="G$1" pin="SEC1_NEG"/>
+<wire x1="27.94" y1="68.58" x2="22.86" y2="68.58" width="0.1524" layer="91"/>
 </segment>
 </net>
@@
 </segment>
 </net>
-<net name="N$6" class="0">
+<net name="DC-" class="0">
 <segment>
 <pinref part="U$4" gate="G$1" pin="P$2"/>
@@
 <wire x1="60.96" y1="20.32" x2="73.66" y2="20.32" width="0.1524" layer="91"/>
 <wire x1="73.66" y1="20.32" x2="73.66" y2="30.48" width="0.1524" layer="91"/>
-<wire x1="60.96" y1="20.32" x2="27.94" y2="20.32" width="0.1524" layer="91"/>
-<wire x1="27.94" y1="20.32" x2="27.94" y2="60.96" width="0.1524" layer="91"/>
-<pinref part="U$5" gate="G$1" pin="SEC2_NEG"/>
-<wire x1="27.94" y1="60.96" x2="22.86" y2="60.96" width="0.1524" layer="91"/>
+<wire x1="60.96" y1="20.32" x2="22.86" y2="20.32" width="0.1524" layer="91"/>
 <junction x="60.96" y="20.32"/>
 <wire x1="73.66" y1="20.32" x2="73.66" y2="2.54" width="0.1524" layer="91"/>
 <junction x="73.66" y="20.32"/>
+<pinref part="DC-" gate="G$1" pin="P$1"/>
+<wire x1="88.9" y1="20.32" x2="73.66" y2="20.32" width="0.1524" layer="91"/>
+<pinref part="U$5" gate="G$1" pin="SEC2_POS"/>
+<wire x1="22.86" y1="55.88" x2="22.86" y2="20.32" width="0.1524" layer="91"/>
+<pinref part="TP2" gate="G$1" pin="TP"/>
 </segment>
 </net>
@@
 <wire x1="38.1" y1="45.72" x2="38.1" y2="55.88" width="0.1524" layer="91"/>
 <wire x1="43.18" y1="45.72" x2="38.1" y2="45.72" width="0.1524" layer="91"/>
-<pinref part="U$5" gate="G$1" pin="SEC2_POS"/>
-<wire x1="38.1" y1="55.88" x2="22.86" y2="55.88" width="0.1524" layer="91"/>
 <junction x="38.1" y="45.72"/>
+<pinref part="U$5" gate="G$1" pin="SEC2_NEG"/>
+<wire x1="22.86" y1="60.96" x2="25.4" y2="60.96" width="0.1524" layer="91"/>
+<wire x1="25.4" y1="60.96" x2="25.4" y2="55.88" width="0.1524" layer="91"/>
+<wire x1="25.4" y1="55.88" x2="38.1" y2="55.88" width="0.1524" layer="91"/>
 </segment>
 </net>
@@
 <wire x1="38.1" y1="81.28" x2="38.1" y2="73.66" width="0.1524" layer="91"/>
 <pinref part="D1" gate="G$1" pin="C"/>
-<wire x1="38.1" y1="73.66" x2="38.1" y2="68.58" width="0.1524" layer="91"/>
 <wire x1="48.26" y1="73.66" x2="38.1" y2="73.66" width="0.1524" layer="91"/>
-<pinref part="U$5" gate="G$1" pin="SEC1_NEG"/>
-<wire x1="38.1" y1="68.58" x2="22.86" y2="68.58" width="0.1524" layer="91"/>
 <junction x="38.1" y="73.66"/>
+<pinref part="U$5" gate="G$1" pin="SEC1_POS"/>
+<wire x1="22.86" y1="63.5" x2="38.1" y2="63.5" width="0.1524" layer="91"/>
+<wire x1="38.1" y1="63.5" x2="38.1" y2="73.66" width="0.1524" layer="91"/>
 </segment>
 </net>
-<net name="N$10" class="0">
+<net name="DC+" class="0">
 <segment>
 <pinref part="U$1" gate="G$1" pin="C"/>
-<wire x1="73.66" y1="86.36" x2="73.66" y2="106.68" width="0.1524" layer="91"/>
+<wire x1="73.66" y1="86.36" x2="73.66" y2="91.44" width="0.1524" layer="91"/>
+<pinref part="DC+" gate="G$1" pin="P$1"/>
+<wire x1="73.66" y1="91.44" x2="73.66" y2="106.68" width="0.1524" layer="91"/>
+<wire x1="88.9" y1="91.44" x2="73.66" y2="91.44" width="0.1524" layer="91"/>
+<junction x="73.66" y="91.44"/>
+<pinref part="TP1" gate="G$1" pin="TP"/>
 </segment>
 </net>
@@
 <pinref part="X1" gate="-1" pin="KL"/>
 <pinref part="U$5" gate="G$1" pin="PRI_NEG"/>
-<wire x1="2.54" y1="66.04" x2="10.16" y2="66.04" width="0.1524" layer="91"/>
+<wire x1="-7.62" y1="66.04" x2="-2.54" y2="66.04" width="0.1524" layer="91"/>
+<wire x1="-2.54" y1="66.04" x2="10.16" y2="66.04" width="0.1524" layer="91"/>
 <wire x1="10.16" y1="66.04" x2="10.16" y2="68.58" width="0.1524" layer="91"/>
+<pinref part="X2" gate="-1" pin="KL"/>
+<wire x1="-7.62" y1="53.34" x2="-2.54" y2="53.34" width="0.1524" layer="91"/>
+<wire x1="-2.54" y1="53.34" x2="-2.54" y2="66.04" width="0.1524" layer="91"/>
+<junction x="-2.54" y="66.04"/>
 </segment>
 </net>
@@
 <pinref part="X1" gate="-2" pin="KL"/>
 <pinref part="U$5" gate="G$1" pin="PRI_POS"/>
-<wire x1="2.54" y1="60.96" x2="10.16" y2="60.96" width="0.1524" layer="91"/>
+<wire x1="-7.62" y1="60.96" x2="0" y2="60.96" width="0.1524" layer="91"/>
+<wire x1="0" y1="60.96" x2="10.16" y2="60.96" width="0.1524" layer="91"/>
 <wire x1="10.16" y1="60.96" x2="10.16" y2="55.88" width="0.1524" layer="91"/>
+<pinref part="X2" gate="-2" pin="KL"/>
+<wire x1="-7.62" y1="48.26" x2="0" y2="48.26" width="0.1524" layer="91"/>
+<wire x1="0" y1="48.26" x2="0" y2="60.96" width="0.1524" layer="91"/>
+<junction x="0" y="60.96"/>
 </segment>
 </net>

Commit message: wip
Other:
- note removed: "TODO: - Holes for DC+/DC-/OUT - DC Reservoir capacitors? - VERIFY FOOTPRINTS"
Changed lines of the file:
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@@
 <sheet>
 <plain>
-<text x="2.54" y="93.98" size="1.778" layer="91">TODO:
-- Holes for DC+/DC-/OUT
-- DC Reservoir capacitors?
-- VERIFY FOOTPRINTS</text>
 <text x="93.98" y="93.98" size="1.778" layer="97">For capacitor: 940C30S68K-F</text>
 </plain>
@@
 </schematic>
 </drawing>
-<compatibility>
-<note version="6.3" minversion="6.2.2" severity="warning">
-Since Version 6.2.2 text objects can contain more than one line,
-which will not be processed correctly with this version.
-</note>
-</compatibility>
 </eagle>
