File: cdf-modular-bridge/cdf-modular-bridge.brd (EAGLE design)
At the start: 160 x 100 mm, 9 parts

Commit message: wip
Parts:
- added X1: (no value), con-ptr500:AK500/2
- moved R2 6.48 mm to (-40.6, 54.6)
Connections:
- net N$1: now also X1.1
- net N$2: now also X1.2
Changed lines of the file:
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@@
 </element>
 <element name="R1" library="microbuilder" package="1206" value="15" x="-33.02" y="54.61"/>
-<element name="R2" library="microbuilder" package="1206" value="15" x="-41.91" y="60.96"/>
+<element name="R2" library="microbuilder" package="1206" value="15" x="-40.64" y="54.61"/>
 <element name="U$1" library="keves" package="IXGH40N60A" value="Ixgh48n60a3" x="-19.05" y="8.89"/>
 <element name="U$2" library="keves" package="IXGH40N60A" value="Ixgh48n60a3" x="-19.05" y="26.67"/>
@@
 <element name="U$4" library="keves" package="TPSMB15CA" value="TPSMB15CA" x="-30.48" y="63.5"/>
 <element name="U$5" library="keves" package="PULSE-P0584NL" value="PULSE-P0584NL" x="-20.32" y="44.45"/>
+<element name="X1" library="con-ptr500" package="AK500/2" value="" x="-74.93" y="6.35">
+<attribute name="MPN" value="" x="-74.93" y="6.35" size="1.778" layer="27" display="off"/>
+<attribute name="OC_NEWARK" value="unknown" x="-74.93" y="6.35" size="1.778" layer="27" display="off"/>
+<attribute name="OC_FARNELL" value="unknown" x="-74.93" y="6.35" size="1.778" layer="27" display="off"/>
+<attribute name="MF" value="" x="-74.93" y="6.35" size="1.778" layer="27" display="off"/>
+</element>
 </elements>
 <signals>
-<signal name="N$1">
-<contactref element="U$5" pad="10"/>
-</signal>
-<signal name="N$2">
-<contactref element="U$5" pad="1"/>
-</signal>
 <signal name="N$3">
 <contactref element="U$1" pad="G"/>
@@
 <contactref element="R2" pad="2"/>
 <wire x1="-51.34" y1="39.37" x2="-63.26" y2="32.16" width="0" layer="19" extent="1-1"/>
-<wire x1="-40.51" y1="60.96" x2="-51.34" y2="39.37" width="0" layer="19" extent="1-1"/>
-<wire x1="-32.9184" y1="63.5" x2="-40.51" y2="60.96" width="0" layer="19" extent="1-1"/>
+<wire x1="-39.24" y1="54.61" x2="-51.34" y2="39.37" width="0" layer="19" extent="1-1"/>
+<wire x1="-32.9184" y1="63.5" x2="-39.24" y2="54.61" width="0" layer="19" extent="1-1"/>
 </signal>
 <signal name="N$6">
@@
 <contactref element="R2" pad="1"/>
 <contactref element="U$5" pad="8"/>
-<wire x1="-43.31" y1="60.96" x2="-20.32" y2="48.895" width="0" layer="19" extent="1-1"/>
-<wire x1="-55.34" y1="39.37" x2="-43.31" y2="60.96" width="0" layer="19" extent="1-1"/>
+<wire x1="-42.04" y1="54.61" x2="-20.32" y2="48.895" width="0" layer="19" extent="1-1"/>
+<wire x1="-55.34" y1="39.37" x2="-42.04" y2="54.61" width="0" layer="19" extent="1-1"/>
 </signal>
 <signal name="N$8">
@@
 <contactref element="U$1" pad="C"/>
 </signal>
+<signal name="N$1">
+<contactref element="X1" pad="1"/>
+<contactref element="U$5" pad="10"/>
+<wire x1="-33.02" y1="48.895" x2="-77.4446" y2="6.35" width="0" layer="19" extent="1-1"/>
+</signal>
+<signal name="N$2">
+<contactref element="X1" pad="2"/>
+<contactref element="U$5" pad="1"/>
+<wire x1="-33.02" y1="40.005" x2="-72.4154" y2="6.35" width="0" layer="19" extent="1-1"/>
+</signal>
 </signals>

Commit message: wip
Parts:
- added DC+, DC-, OUT: BIG-ASS-HOLE, keves:BIG-ASS-HOLE
- added TP1, TP2: PTR1PAD1-17, testpad:P1-17
- added X2: (no value), con-ptr500:AK500/2
- moved D2 94.4 mm to (39.9, 24.8), flipped to the bottom, turned to 90 degrees
- moved X1 87.7 mm to (12.7, 2.44)
- moved U$4 84.7 mm to (45.5, 26.1), flipped to the bottom, turned to 180 degrees
- moved R2 82.6 mm to (36.1, 24.0), flipped to the bottom, turned to 90 degrees
- moved U$2 79.3 mm to (41.9, 77.4), turned to 90 degrees
- moved U$1 74.0 mm to (8.89, 77.4), turned to 90 degrees
- moved U$5 52.7 mm to (25.4, 18.2), turned to 90 degrees
- moved D1 50.6 mm to (6.35, 24.0), flipped to the bottom, turned to 90 degrees
- moved R1 47.3 mm to (3.30, 24.3), flipped to the bottom, turned to 90 degrees
- moved U$3 41.6 mm to (12.3, 25.9), flipped to the bottom, turned to 180 degrees
Connections:
- removed net N$10: U$1.C
- removed net N$4: U$1.E, U$2.C, U$3.P$2, U$5.3
- removed net N$6: U$2.E, U$4.P$2, U$5.7
- new net DC+: DC+.X, DC+.X@1, DC+.X@10, DC+.X@11, DC+.X@12, DC+.X@120, DC+.X@13, DC+.X@14, DC+.X@15, DC+.X@16, DC+.X@17, DC+.X@18, DC+.X@19, DC+.X@2, DC+.X@20, DC+.X@21, DC+.X@22, DC+.X@23, DC+.X@24, DC+.X@25, DC+.X@26, DC+.X@27, DC+.X@28, DC+.X@29, DC+.X@3, DC+.X@30, DC+.X@31, DC+.X@32, DC+.X@34, DC+.X@4, DC+.X@5, DC+.X@6, DC+.X@7, DC+.X@8, DC+.X@9, TP1.TP, U$1.C
- new net DC-: DC-.X, DC-.X@1, DC-.X@10, DC-.X@11, DC-.X@12, DC-.X@120, DC-.X@13, DC-.X@14, DC-.X@15, DC-.X@16, DC-.X@17, DC-.X@18, DC-.X@19, DC-.X@2, DC-.X@20, DC-.X@21, DC-.X@22, DC-.X@23, DC-.X@24, DC-.X@25, DC-.X@26, DC-.X@27, DC-.X@28, DC-.X@29, DC-.X@3, DC-.X@30, DC-.X@31, DC-.X@32, DC-.X@34, DC-.X@4, DC-.X@5, DC-.X@6, DC-.X@7, DC-.X@8, DC-.X@9, TP2.TP, U$2.E, U$4.P$2, U$5.8
- new net OUT: OUT.X, OUT.X@1, OUT.X@10, OUT.X@11, OUT.X@12, OUT.X@120, OUT.X@13, OUT.X@14, OUT.X@15, OUT.X@16, OUT.X@17, OUT.X@18, OUT.X@19, OUT.X@2, OUT.X@20, OUT.X@21, OUT.X@22, OUT.X@23, OUT.X@24, OUT.X@25, OUT.X@26, OUT.X@27, OUT.X@28, OUT.X@29, OUT.X@3, OUT.X@30, OUT.X@31, OUT.X@32, OUT.X@34, OUT.X@4, OUT.X@5, OUT.X@6, OUT.X@7, OUT.X@8, OUT.X@9, U$1.E, U$2.C, U$3.P$2, U$5.4
- net N$1: now also X2.1
- net N$2: now also X2.2
- net N$7: now also U$5.7; no longer U$5.8
- net N$8: now also U$5.3; no longer U$5.4
Routing:
- net DC-: track 0.00 -> 69.6 mm
- net DC+: track 0.00 -> 32.1 mm
- net N$2: track 0.00 -> 30.7 mm
- net N$1: track 0.00 -> 29.1 mm
- net N$8: track 0.00 -> 28.5 mm
- net N$7: track 0.00 -> 21.0 mm
- net OUT: track 0.00 -> 17.6 mm
- net N$5: track 0.00 -> 15.6 mm
- net N$3: track 0.00 -> 14.3 mm
- added copper zone on layer 1, net DC+
- added copper zone on layer 1, net DC-
- added copper zone on layer 1, net OUT
Other:
- board size 160 x 100 mm -> 50.8 x 38.1 mm
- board text added: "+"
- board text added: "-"
- board text added: "CDF MoBridge rev A"

Commit message: wip
Routing:
- net DC-: track 69.6 -> 50.3 mm
- added copper zone on layer 1, net N$5
Changed lines of the file:
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@@
 </class>
 </classes>
-<designrules name="oshpark">
+<designrules name="oshpark *">
 <description language="de">&lt;b&gt;EAGLE Design Rules&lt;/b&gt;
 &lt;p&gt;
@@
 <param name="dpGapFactor" value="2.5"/>
 <param name="checkGrid" value="0"/>
-<param name="checkAngle" value="0"/>
+<param name="checkAngle" value="1"/>
 <param name="checkFont" value="1"/>
 <param name="checkRestrict" value="1"/>
@@
 <contactref element="U$2" pad="C"/>
 <contactref element="OUT" pad="X"/>
-<polygon width="0.254" layer="1" isolate="0.381" thermals="no">
+<polygon width="0.254" layer="1" isolate="0.381" thermals="no" rank="2">
 <vertex x="44.196" y="38.5064"/>
 <vertex x="12.446" y="38.5064"/>
@@
 <wire x1="36.46" y1="33.1584" x2="36.46" y2="30.2084" width="1.778" layer="16"/>
 <wire x1="36.46" y1="30.2084" x2="39.878" y2="26.7904" width="1.778" layer="16"/>
+<polygon width="0.254" layer="1">
+<vertex x="33.528" y="37.719"/>
+<vertex x="38.862" y="37.719"/>
+<vertex x="38.862" y="29.337"/>
+<vertex x="33.528" y="29.337"/>
+</polygon>
 </signal>
 <signal name="DC-">
@@
 <contactref element="U$2" pad="E"/>
 <contactref element="DC-" pad="X"/>
-<wire x1="47.36" y1="20.5884" x2="38.854609375" y2="15.582528125" width="4.572" layer="1"/>
-<wire x1="38.854609375" y1="15.582528125" x2="38.1" y2="15.1384" width="4.572" layer="1"/>
 <wire x1="47.36" y1="20.5884" x2="47.36" y2="33.1584" width="4.318" layer="1"/>
 <wire x1="47.36" y1="33.1584" x2="47.36" y2="35.3424" width="4.318" layer="1"/>
-<wire x1="47.36" y1="35.3424" x2="47.244" y2="35.0774" width="4.318" layer="1"/>
 <wire x1="47.244" y1="35.0774" x2="47.244" y2="33.2744" width="4.318" layer="1"/>
 <wire x1="47.244" y1="33.2744" x2="47.36" y2="33.1584" width="4.318" layer="1"/>
-<polygon width="0.254" layer="1" isolate="0.381" thermals="no" rank="2">
+<polygon width="0.254" layer="1" isolate="0.381" thermals="no" rank="3">
 <vertex x="50.038" y="38.5064"/>
 <vertex x="33.02" y="38.7604"/>
@@
 <wire x1="37.846" y1="15.3924" x2="38.1" y2="15.1384" width="1.778" layer="1"/>
 <contactref element="TP2" pad="TP"/>
-<wire x1="48.26" y1="9.8044" x2="42.418" y2="15.6464" width="1.016" layer="1"/>
 <wire x1="48.26" y1="2.4384" x2="48.26" y2="9.8044" width="2.54" layer="1"/>
 <contactref element="DC-" pad="X@1"/>
@@
 <wire x1="8.89" y1="18.9484" x2="8.89" y2="33.1584" width="4.318" layer="1"/>
 <wire x1="8.89" y1="35.4584" x2="8.89" y2="33.1584" width="4.318" layer="1"/>
-<polygon width="0.254" layer="1" isolate="0.381" thermals="no" rank="2">
+<polygon width="0.254" layer="1" isolate="0.381" thermals="no" rank="3">
 <vertex x="18.288" y="38.2524"/>
 <vertex x="5.588" y="38.2524"/>

Commit message: cdf-modular-bridge rev B
Routing:
- net DC+: track 32.1 -> 31.0 mm
Other:
- board text added: "CDF MoBridge rev B"
- board text removed: "CDF MoBridge rev A"
Changed lines of the file:
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@@
 <setting verticaltext="up"/>
 </settings>
-<grid distance="15" unitdist="mil" unit="mil" style="lines" multiple="1" display="yes" altdistance="0.025" altunitdist="inch" altunit="inch"/>
+<grid distance="5" unitdist="mil" unit="mil" style="lines" multiple="1" display="yes" altdistance="0.025" altunitdist="inch" altunit="inch"/>
 <layers>
 <layer number="1" name="Top" color="4" fill="1" visible="yes" active="yes"/>
@@
 <text x="46.736" y="0.254" size="5.08" layer="21" font="vector">-</text>
 <text x="31.115" y="3.4544" size="1.016" layer="21" font="vector" rot="R180">CDF MoBridge
-rev A</text>
+rev B</text>
 <polygon width="0.254" layer="29">
 <vertex x="5.08" y="38.5064"/>
@@
 <contactref element="U$2" pad="C"/>
 <contactref element="OUT" pad="X"/>
-<polygon width="0.254" layer="1" isolate="0.381" thermals="no" rank="2">
-<vertex x="44.196" y="38.5064"/>
+<polygon width="0.254" layer="1" isolate="1.778" thermals="no" rank="2">
+<vertex x="43.815" y="38.5064"/>
 <vertex x="12.446" y="38.5064"/>
 <vertex x="12.446" y="25.0444"/>
-<vertex x="44.196" y="25.0444"/>
+<vertex x="43.815" y="25.0444"/>
 </polygon>
 <wire x1="14.34" y1="33.1584" x2="14.34" y2="26.3508" width="1.778" layer="16"/>
@@
 <wire x1="36.46" y1="30.2084" x2="39.878" y2="26.7904" width="1.778" layer="16"/>
 <polygon width="0.254" layer="1">
-<vertex x="33.528" y="37.719"/>
-<vertex x="38.862" y="37.719"/>
+<vertex x="33.528" y="36.576"/>
+<vertex x="38.862" y="36.576"/>
 <vertex x="38.862" y="29.337"/>
 <vertex x="33.528" y="29.337"/>
@@
 <wire x1="47.244" y1="35.0774" x2="47.244" y2="33.2744" width="4.318" layer="1"/>
 <wire x1="47.244" y1="33.2744" x2="47.36" y2="33.1584" width="4.318" layer="1"/>
-<polygon width="0.254" layer="1" isolate="0.381" thermals="no" rank="3">
-<vertex x="50.038" y="38.5064"/>
-<vertex x="33.02" y="38.7604"/>
+<polygon width="0.254" layer="1" isolate="1.27" thermals="no" rank="3">
+<vertex x="50.165" y="36.3474"/>
+<vertex x="33.147" y="36.3474"/>
 <vertex x="33.02" y="8.5344"/>
 <vertex x="50.038" y="8.5344"/>
@@
 <contactref element="U$1" pad="C"/>
 <contactref element="DC+" pad="X"/>
-<wire x1="8.89" y1="18.9484" x2="12.7" y2="15.1384" width="4.572" layer="1"/>
 <wire x1="8.89" y1="18.9484" x2="8.89" y2="33.1584" width="4.318" layer="1"/>
 <wire x1="8.89" y1="35.4584" x2="8.89" y2="33.1584" width="4.318" layer="1"/>
-<polygon width="0.254" layer="1" isolate="0.381" thermals="no" rank="3">
-<vertex x="18.288" y="38.2524"/>
-<vertex x="5.588" y="38.2524"/>
-<vertex x="5.588" y="9.0424"/>
+<polygon width="0.254" layer="1" isolate="1.1938" thermals="no" rank="3">
+<vertex x="18.161" y="36.7284"/>
+<vertex x="6.985" y="36.2204"/>
+<vertex x="6.985" y="8.9154"/>
 <vertex x="18.288" y="9.0424"/>
 </polygon>
@@
 <contactref element="DC+" pad="X@34"/>
 <contactref element="DC+" pad="X@120"/>
+<wire x1="6.858" y1="10.8204" x2="8.636" y2="10.8204" width="0.4064" layer="1"/>
+<wire x1="8.636" y1="10.8204" x2="8.636" y2="13.3604" width="0.4064" layer="1"/>
 </signal>
 <signal name="N$1">
