File: cdf-modular-bridge/cdf-modular-bridge-rev2.brd (EAGLE design)
At the start: 50.8 x 53.3 mm, 20 parts, among them Q1 Ixgh48n60a3, Q2 Ixgh48n60a3, T1 PULSE-P0584NL

Commit message: wip
Parts:
- added C1: PEH534YDC3220M2, rcl:EB35D
Connections:
- net DC+: now also C1.+
- net DC-: now also C1.-
Other:
- board size 50.8 x 53.3 mm -> 50.8 x 94 mm
Changed lines of the file:
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@@
 <setting verticaltext="up"/>
 </settings>
-<grid distance="25" unitdist="mil" unit="mil" style="lines" multiple="1" display="yes" altdistance="0.025" altunitdist="inch" altunit="inch"/>
+<grid distance="100" unitdist="mil" unit="mil" style="lines" multiple="1" display="yes" altdistance="0.025" altunitdist="inch" altunit="inch"/>
 <layers>
 <layer number="1" name="Top" color="4" fill="1" visible="yes" active="yes"/>
@@
 <board>
 <plain>
-<wire x1="0" y1="0" x2="50.8" y2="0" width="0" layer="20"/>
-<wire x1="50.8" y1="0" x2="50.8" y2="53.34" width="0" layer="20"/>
+<wire x1="0" y1="-40.64" x2="50.8" y2="-40.64" width="0" layer="20"/>
+<wire x1="50.8" y1="-40.64" x2="50.8" y2="53.34" width="0" layer="20"/>
 <wire x1="50.8" y1="53.34" x2="0" y2="53.34" width="0" layer="20"/>
-<wire x1="0" y1="53.34" x2="0" y2="0" width="0" layer="20"/>
+<wire x1="0" y1="53.34" x2="0" y2="-40.64" width="0" layer="20"/>
 <text x="0.762" y="9.5504" size="5.08" layer="21" font="vector">+</text>
 <text x="46.736" y="0.254" size="5.08" layer="21" font="vector">-</text>
@@
 <element name="D6" library="keves" package="TO220ABS" value="FMN-2206S" x="39.624" y="29.591"/>
 <element name="D8" library="keves" package="TO220ABS" value="FMN-2206S" x="39.624" y="30.607" rot="R180"/>
+<element name="C1" library="rcl" package="EB35D" value="PEH534YDC3220M2" x="24.765" y="-20.955"/>
 </elements>
 <signals>
@@
 <wire x1="47.9044" y1="41.9354" x2="47.9044" y2="47.854" width="1.778" layer="16"/>
 <wire x1="47.9044" y1="47.854" x2="47.36" y2="48.3984" width="1.778" layer="16"/>
+<contactref element="C1" pad="-"/>
+<wire x1="42.164" y1="27.051" x2="47.36" y2="28.8434" width="0" layer="19" extent="1-1"/>
+<wire x1="37.084" y1="33.147" x2="42.164" y2="33.147" width="0" layer="19" extent="1-1"/>
+<wire x1="37.973" y1="19.5834" x2="37.084" y2="27.051" width="0" layer="19" extent="1-1"/>
+<wire x1="39.37" y1="19.2024" x2="37.973" y2="19.5834" width="0" layer="19" extent="1-1"/>
+<wire x1="40.64" y1="18.8214" x2="39.37" y2="19.2024" width="0" layer="19" extent="1-1"/>
+<wire x1="41.021" y1="17.6784" x2="40.64" y2="18.8214" width="0" layer="19" extent="1-1"/>
+<wire x1="40.767" y1="16.4084" x2="41.021" y2="17.6784" width="0" layer="19" extent="1-1"/>
+<wire x1="41.148" y1="15.2654" x2="40.767" y2="16.4084" width="0" layer="19" extent="1-1"/>
+<wire x1="42.291" y1="15.5194" x2="41.148" y2="15.2654" width="0" layer="19" extent="1-1"/>
+<wire x1="42.037" y1="16.6624" x2="42.291" y2="15.5194" width="0" layer="19" extent="1-1"/>
+<wire x1="42.037" y1="14.3764" x2="42.291" y2="15.5194" width="0" layer="19" extent="1-1"/>
+<wire x1="40.767" y1="14.1224" x2="41.148" y2="15.2654" width="0" layer="19" extent="1-1"/>
+<wire x1="40.767" y1="12.9794" x2="40.767" y2="14.1224" width="0" layer="19" extent="1-1"/>
+<wire x1="40.767" y1="11.8364" x2="40.767" y2="12.9794" width="0" layer="19" extent="1-1"/>
+<wire x1="39.751" y1="11.2014" x2="40.767" y2="11.8364" width="0" layer="19" extent="1-1"/>
+<wire x1="39.624" y1="12.4714" x2="40.767" y2="12.9794" width="0" layer="19" extent="1-1"/>
+<wire x1="42.037" y1="12.9794" x2="40.767" y2="12.9794" width="0" layer="19" extent="1-1"/>
+<wire x1="38.354" y1="12.0904" x2="39.624" y2="12.4714" width="0" layer="19" extent="1-1"/>
+<wire x1="38.481" y1="10.6934" x2="39.751" y2="11.2014" width="0" layer="19" extent="1-1"/>
+<wire x1="39.624" y1="17.5514" x2="41.021" y2="17.6784" width="0" layer="19" extent="1-1"/>
+<wire x1="38.227" y1="17.9324" x2="39.624" y2="17.5514" width="0" layer="19" extent="1-1"/>
+<wire x1="36.83" y1="17.6784" x2="38.227" y2="17.9324" width="0" layer="19" extent="1-1"/>
+<wire x1="36.957" y1="12.4714" x2="38.354" y2="12.0904" width="0" layer="19" extent="1-1"/>
+<wire x1="36.703" y1="11.0744" x2="36.957" y2="12.4714" width="0" layer="19" extent="1-1"/>
+<wire x1="35.433" y1="11.3284" x2="36.703" y2="11.0744" width="0" layer="19" extent="1-1"/>
+<wire x1="35.306" y1="12.4714" x2="35.433" y2="11.3284" width="0" layer="19" extent="1-1"/>
+<wire x1="35.306" y1="13.6144" x2="35.306" y2="12.4714" width="0" layer="19" extent="1-1"/>
+<wire x1="35.306" y1="14.7574" x2="35.306" y2="13.6144" width="0" layer="19" extent="1-1"/>
+<wire x1="35.306" y1="15.9004" x2="35.306" y2="14.7574" width="0" layer="19" extent="1-1"/>
+<wire x1="35.306" y1="17.0434" x2="35.306" y2="15.9004" width="0" layer="19" extent="1-1"/>
+<wire x1="35.306" y1="18.1864" x2="35.306" y2="17.0434" width="0" layer="19" extent="1-1"/>
+<wire x1="34.036" y1="17.0434" x2="35.306" y2="17.0434" width="0" layer="19" extent="1-1"/>
+<wire x1="34.036" y1="15.6464" x2="35.306" y2="15.9004" width="0" layer="19" extent="1-1"/>
+<wire x1="34.036" y1="14.5034" x2="34.036" y2="15.6464" width="0" layer="19" extent="1-1"/>
+<wire x1="34.036" y1="13.3604" x2="34.036" y2="14.5034" width="0" layer="19" extent="1-1"/>
+<wire x1="36.322" y1="19.0754" x2="35.306" y2="18.1864" width="0" layer="19" extent="1-1"/>
+<wire x1="37.846" y1="15.3924" x2="36.83" y2="17.6784" width="0" layer="19" extent="1-1"/>
+<wire x1="48.26" y1="9.8044" x2="42.037" y2="12.9794" width="0" layer="19" extent="1-1"/>
+<wire x1="29.845" y1="-20.955" x2="35.433" y2="11.3284" width="0" layer="19" extent="1-1"/>
 </signal>
 <signal name="N$7">
@@
 <wire x1="13.97" y1="35.179" x2="9.271" y2="35.179" width="1.778" layer="1"/>
 <wire x1="9.271" y1="35.179" x2="8.89" y2="35.56" width="1.778" layer="1"/>
+<contactref element="C1" pad="+"/>
+<wire x1="15.621" y1="17.6784" x2="15.24" y2="18.8214" width="0" layer="19" extent="1-1"/>
+<wire x1="15.367" y1="16.4084" x2="15.621" y2="17.6784" width="0" layer="19" extent="1-1"/>
+<wire x1="15.748" y1="15.2654" x2="15.367" y2="16.4084" width="0" layer="19" extent="1-1"/>
+<wire x1="16.891" y1="15.5194" x2="15.748" y2="15.2654" width="0" layer="19" extent="1-1"/>
+<wire x1="16.637" y1="16.6624" x2="16.891" y2="15.5194" width="0" layer="19" extent="1-1"/>
+<wire x1="16.637" y1="14.3764" x2="16.891" y2="15.5194" width="0" layer="19" extent="1-1"/>
+<wire x1="15.367" y1="14.1224" x2="15.748" y2="15.2654" width="0" layer="19" extent="1-1"/>
+<wire x1="15.367" y1="12.9794" x2="15.367" y2="14.1224" width="0" layer="19" extent="1-1"/>
+<wire x1="15.367" y1="11.8364" x2="15.367" y2="12.9794" width="0" layer="19" extent="1-1"/>
+<wire x1="14.351" y1="11.2014" x2="15.367" y2="11.8364" width="0" layer="19" extent="1-1"/>
+<wire x1="14.224" y1="12.4714" x2="15.367" y2="12.9794" width="0" layer="19" extent="1-1"/>
+<wire x1="16.637" y1="12.9794" x2="15.367" y2="12.9794" width="0" layer="19" extent="1-1"/>
+<wire x1="13.97" y1="19.2024" x2="15.24" y2="18.8214" width="0" layer="19" extent="1-1"/>
+<wire x1="12.954" y1="12.0904" x2="14.224" y2="12.4714" width="0" layer="19" extent="1-1"/>
+<wire x1="13.081" y1="10.6934" x2="14.351" y2="11.2014" width="0" layer="19" extent="1-1"/>
+<wire x1="14.224" y1="17.5514" x2="15.621" y2="17.6784" width="0" layer="19" extent="1-1"/>
+<wire x1="12.827" y1="17.9324" x2="14.224" y2="17.5514" width="0" layer="19" extent="1-1"/>
+<wire x1="11.43" y1="17.6784" x2="12.827" y2="17.9324" width="0" layer="19" extent="1-1"/>
+<wire x1="12.573" y1="19.5834" x2="13.97" y2="19.2024" width="0" layer="19" extent="1-1"/>
+<wire x1="11.557" y1="12.4714" x2="12.954" y2="12.0904" width="0" layer="19" extent="1-1"/>
+<wire x1="11.303" y1="11.0744" x2="11.557" y2="12.4714" width="0" layer="19" extent="1-1"/>
+<wire x1="10.033" y1="11.3284" x2="11.303" y2="11.0744" width="0" layer="19" extent="1-1"/>
+<wire x1="9.906" y1="12.4714" x2="10.033" y2="11.3284" width="0" layer="19" extent="1-1"/>
+<wire x1="9.906" y1="13.6144" x2="9.906" y2="12.4714" width="0" layer="19" extent="1-1"/>
+<wire x1="9.906" y1="14.7574" x2="9.906" y2="13.6144" width="0" layer="19" extent="1-1"/>
+<wire x1="9.906" y1="15.9004" x2="9.906" y2="14.7574" width="0" layer="19" extent="1-1"/>
+<wire x1="9.906" y1="17.0434" x2="9.906" y2="15.9004" width="0" layer="19" extent="1-1"/>
+<wire x1="9.906" y1="18.1864" x2="9.906" y2="17.0434" width="0" layer="19" extent="1-1"/>
+<wire x1="8.89" y1="18.9484" x2="9.906" y2="18.1864" width="0" layer="19" extent="1-1"/>
+<wire x1="8.636" y1="17.0434" x2="9.906" y2="17.0434" width="0" layer="19" extent="1-1"/>
+<wire x1="8.636" y1="15.6464" x2="9.906" y2="15.9004" width="0" layer="19" extent="1-1"/>
+<wire x1="8.636" y1="14.5034" x2="8.636" y2="15.6464" width="0" layer="19" extent="1-1"/>
+<wire x1="8.636" y1="13.3604" x2="8.636" y2="14.5034" width="0" layer="19" extent="1-1"/>
+<wire x1="10.922" y1="19.0754" x2="9.906" y2="18.1864" width="0" layer="19" extent="1-1"/>
+<wire x1="12.7" y1="15.1384" x2="12.827" y2="17.9324" width="0" layer="19" extent="1-1"/>
+<wire x1="19.685" y1="-20.955" x2="2.54" y2="2.4384" width="0" layer="19" extent="1-1"/>
 </signal>
 <signal name="N$1">
