File: cdf-single-driver/cdf-single-driver.sch (EAGLE design)
At the start: 29 parts, among them IC1 R-789.0-0.5

Commit message: wi
Parts:
- removed U$3: FDD8424H, keves:FDD8424H
- added D3: (no value), diode:DIODE-SOD123
- added IC2: UCC27423, keves:UCC27423
- U$1: value UCC27423 -> FDD8424H; device keves:UCC27423 -> keves:FDD8424H
Connections:
- net +24V: now also D3.C, U$1.VCC; no longer U$3.VCC
- net +9V: now also D3.A, IC2.ENA, IC2.ENB, IC2.VCC; no longer U$1.ENA, U$1.ENB, U$1.VCC
- net GND: now also IC2.GND; no longer U$3.GND
- net N$1: now also IC2.INA; no longer U$1.INA
- net N$10: now also U$2.TAB; no longer U$3.TAB
- net N$2: now also IC2.INB; no longer U$1.INB
- net N$3: now also IC2.OUTA, U$1.LSG; no longer U$1.OUTA, U$2.LSG
- net N$4: now also U$1.HSG; no longer U$2.HSG
- net N$5: now also U$1.TAB; no longer U$2.TAB
- net N$8: now also IC2.OUTB, U$2.LSG; no longer U$1.OUTB, U$3.LSG
- net N$9: now also U$2.HSG; no longer U$3.HSG
Other:
- moved on the sheet: U$2
Changed lines of the file:
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@@
 </classes>
 <parts>
-<part name="U$1" library="keves" deviceset="UCC27423" device=""/>
+<part name="IC2" library="keves" deviceset="UCC27423" device=""/>
 <part name="C1" library="microbuilder" deviceset="CAP_CERAMIC" device="0805" value="1u"/>
 <part name="SUPPLY1" library="supply2" deviceset="+9V" device=""/>
@@
 <part name="GATE_IN" library="con-ptr500" deviceset="AK500/3" device=""/>
 <part name="GND3" library="microbuilder" deviceset="GND" device=""/>
-<part name="U$2" library="keves" deviceset="FDD8424H" device=""/>
+<part name="U$1" library="keves" deviceset="FDD8424H" device=""/>
 <part name="GND4" library="microbuilder" deviceset="GND" device=""/>
 <part name="C2" library="microbuilder" deviceset="CAP_CERAMIC" device="0805" value="0.1u"/>
@@
 <part name="R2" library="microbuilder" deviceset="RESISTOR" device="0805" value="15"/>
 <part name="D1" library="diode" deviceset="DIODE-" device="MICROMELF-W" value="MCL4148-TR"/>
-<part name="U$3" library="keves" deviceset="FDD8424H" device=""/>
+<part name="U$2" library="keves" deviceset="FDD8424H" device=""/>
 <part name="GND6" library="microbuilder" deviceset="GND" device=""/>
 <part name="C6" library="microbuilder" deviceset="CAP_CERAMIC" device="0805" value="0.1u"/>
@@
 <part name="C12" library="microbuilder" deviceset="CAP_CERAMIC" device="0805" value="0.1u"/>
 <part name="SUPPLY2" library="supply2" deviceset="+9V" device=""/>
+<part name="D3" library="diode" deviceset="DIODE-" device="SOD123"/>
 </parts>
 <sheets>
@@
 </plain>
 <instances>
-<instance part="U$1" gate="G$1" x="68.58" y="45.72"/>
+<instance part="IC2" gate="G$1" x="68.58" y="45.72"/>
 <instance part="C1" gate="G$1" x="45.72" y="63.5" rot="R90"/>
 <instance part="SUPPLY1" gate="G$1" x="50.8" y="68.58"/>
@@
 <instance part="GATE_IN" gate="-3" x="12.7" y="40.64"/>
 <instance part="GND3" gate="G$1" x="22.86" y="45.72" rot="R90"/>
-<instance part="U$2" gate="G$1" x="147.32" y="81.28"/>
+<instance part="U$1" gate="G$1" x="147.32" y="81.28"/>
 <instance part="GND4" gate="G$1" x="147.32" y="60.96"/>
 <instance part="C2" gate="G$1" x="119.38" y="71.12"/>
@@
 <instance part="R2" gate="G$1" x="172.72" y="73.66" rot="R180"/>
 <instance part="D1" gate="G$1" x="119.38" y="86.36" rot="R90"/>
-<instance part="U$3" gate="G$1" x="144.78" y="27.94"/>
+<instance part="U$2" gate="G$1" x="144.78" y="27.94"/>
 <instance part="GND6" gate="G$1" x="144.78" y="7.62"/>
 <instance part="C6" gate="G$1" x="116.84" y="17.78"/>
@@
 <instance part="C12" gate="G$1" x="-25.4" y="60.96"/>
 <instance part="SUPPLY2" gate="G$1" x="-10.16" y="73.66" rot="R270"/>
+<instance part="D3" gate="G$1" x="-55.88" y="83.82" rot="R180"/>
 </instances>
 <busses>
@@
 <wire x1="48.26" y1="63.5" x2="50.8" y2="63.5" width="0.1524" layer="91"/>
 <wire x1="50.8" y1="63.5" x2="50.8" y2="66.04" width="0.1524" layer="91"/>
-<pinref part="U$1" gate="G$1" pin="ENA"/>
+<pinref part="IC2" gate="G$1" pin="ENA"/>
 <wire x1="50.8" y1="63.5" x2="50.8" y2="55.88" width="0.1524" layer="91"/>
 <wire x1="50.8" y1="63.5" x2="91.44" y2="63.5" width="0.1524" layer="91"/>
 <wire x1="91.44" y1="63.5" x2="91.44" y2="55.88" width="0.1524" layer="91"/>
-<pinref part="U$1" gate="G$1" pin="VCC"/>
+<pinref part="IC2" gate="G$1" pin="VCC"/>
 <wire x1="91.44" y1="55.88" x2="91.44" y2="45.72" width="0.1524" layer="91"/>
 <wire x1="91.44" y1="45.72" x2="83.82" y2="45.72" width="0.1524" layer="91"/>
-<pinref part="U$1" gate="G$1" pin="ENB"/>
+<pinref part="IC2" gate="G$1" pin="ENB"/>
 <wire x1="83.82" y1="55.88" x2="91.44" y2="55.88" width="0.1524" layer="91"/>
 <junction x="91.44" y="55.88"/>
@@
 <pinref part="SUPPLY2" gate="G$1" pin="+9V"/>
 <junction x="-35.56" y="73.66"/>
+<pinref part="D3" gate="G$1" pin="A"/>
+<wire x1="-53.34" y1="83.82" x2="-35.56" y2="83.82" width="0.1524" layer="91"/>
+<wire x1="-35.56" y1="83.82" x2="-35.56" y2="73.66" width="0.1524" layer="91"/>
 </segment>
 </net>
@@
 <segment>
 <pinref part="GND2" gate="G$1" pin="GND"/>
-<pinref part="U$1" gate="G$1" pin="GND"/>
+<pinref part="IC2" gate="G$1" pin="GND"/>
 <wire x1="48.26" y1="45.72" x2="50.8" y2="45.72" width="0.1524" layer="91"/>
 </segment>
@@
 </segment>
 <segment>
-<pinref part="U$2" gate="G$1" pin="GND"/>
+<pinref part="U$1" gate="G$1" pin="GND"/>
 <pinref part="GND4" gate="G$1" pin="GND"/>
 <wire x1="147.32" y1="63.5" x2="147.32" y2="66.04" width="0.1524" layer="91"/>
@@
 </segment>
 <segment>
-<pinref part="U$3" gate="G$1" pin="GND"/>
+<pinref part="U$2" gate="G$1" pin="GND"/>
 <pinref part="GND6" gate="G$1" pin="GND"/>
 <wire x1="144.78" y1="10.16" x2="144.78" y2="12.7" width="0.1524" layer="91"/>
@@
 <segment>
 <pinref part="GATE_IN" gate="-1" pin="KL"/>
-<pinref part="U$1" gate="G$1" pin="INA"/>
+<pinref part="IC2" gate="G$1" pin="INA"/>
 <wire x1="17.78" y1="50.8" x2="50.8" y2="50.8" width="0.1524" layer="91"/>
 </segment>
@@
 <segment>
 <pinref part="GATE_IN" gate="-3" pin="KL"/>
-<pinref part="U$1" gate="G$1" pin="INB"/>
+<pinref part="IC2" gate="G$1" pin="INB"/>
 <wire x1="17.78" y1="40.64" x2="50.8" y2="40.64" width="0.1524" layer="91"/>
 </segment>
@@
 <net name="N$3" class="0">
 <segment>
-<pinref part="U$2" gate="G$1" pin="LSG"/>
+<pinref part="U$1" gate="G$1" pin="LSG"/>
 <wire x1="134.62" y1="76.2" x2="132.08" y2="76.2" width="0.1524" layer="91"/>
 <wire x1="132.08" y1="76.2" x2="132.08" y2="68.58" width="0.1524" layer="91"/>
@@
 <junction x="119.38" y="68.58"/>
 <wire x1="119.38" y1="68.58" x2="106.68" y2="68.58" width="0.1524" layer="91"/>
-<pinref part="U$1" gate="G$1" pin="OUTA"/>
+<pinref part="IC2" gate="G$1" pin="OUTA"/>
 <wire x1="83.82" y1="50.8" x2="106.68" y2="50.8" width="0.1524" layer="91"/>
 <wire x1="106.68" y1="50.8" x2="106.68" y2="68.58" width="0.1524" layer="91"/>
@@
 <net name="N$4" class="0">
 <segment>
-<pinref part="U$2" gate="G$1" pin="HSG"/>
+<pinref part="U$1" gate="G$1" pin="HSG"/>
 <pinref part="C2" gate="G$1" pin="P$1"/>
 <wire x1="134.62" y1="81.28" x2="129.54" y2="81.28" width="0.1524" layer="91"/>
@@
 <wire x1="154.94" y1="93.98" x2="147.32" y2="93.98" width="0.1524" layer="91"/>
 <wire x1="147.32" y1="93.98" x2="147.32" y2="99.06" width="0.1524" layer="91"/>
-<pinref part="U$2" gate="G$1" pin="VCC"/>
+<pinref part="U$1" gate="G$1" pin="VCC"/>
 <wire x1="147.32" y1="93.98" x2="147.32" y2="91.44" width="0.1524" layer="91"/>
 <junction x="147.32" y="93.98"/>
@@
 <wire x1="152.4" y1="40.64" x2="144.78" y2="40.64" width="0.1524" layer="91"/>
 <wire x1="144.78" y1="40.64" x2="144.78" y2="45.72" width="0.1524" layer="91"/>
-<pinref part="U$3" gate="G$1" pin="VCC"/>
+<pinref part="U$2" gate="G$1" pin="VCC"/>
 <wire x1="144.78" y1="40.64" x2="144.78" y2="38.1" width="0.1524" layer="91"/>
 <junction x="144.78" y="40.64"/>
@@
 <junction x="-86.36" y="73.66"/>
 <junction x="-99.06" y="73.66"/>
+<pinref part="D3" gate="G$1" pin="C"/>
+<wire x1="-58.42" y1="83.82" x2="-68.58" y2="83.82" width="0.1524" layer="91"/>
+<wire x1="-68.58" y1="83.82" x2="-68.58" y2="73.66" width="0.1524" layer="91"/>
 </segment>
 </net>
 <net name="N$5" class="0">
 <segment>
-<pinref part="U$2" gate="G$1" pin="TAB"/>
+<pinref part="U$1" gate="G$1" pin="TAB"/>
 <pinref part="C4" gate="G$1" pin="P$2"/>
 <wire x1="160.02" y1="78.74" x2="167.64" y2="78.74" width="0.1524" layer="91"/>
@@
 <net name="N$8" class="0">
 <segment>
-<pinref part="U$3" gate="G$1" pin="LSG"/>
+<pinref part="U$2" gate="G$1" pin="LSG"/>
 <wire x1="132.08" y1="22.86" x2="129.54" y2="22.86" width="0.1524" layer="91"/>
 <wire x1="129.54" y1="22.86" x2="129.54" y2="15.24" width="0.1524" layer="91"/>
@@
 <pinref part="C6" gate="G$1" pin="P$2"/>
 <junction x="116.84" y="15.24"/>
-<pinref part="U$1" gate="G$1" pin="OUTB"/>
+<pinref part="IC2" gate="G$1" pin="OUTB"/>
 <wire x1="116.84" y1="15.24" x2="83.82" y2="15.24" width="0.1524" layer="91"/>
 <wire x1="83.82" y1="15.24" x2="83.82" y2="40.64" width="0.1524" layer="91"/>
@@
 <net name="N$9" class="0">
 <segment>
-<pinref part="U$3" gate="G$1" pin="HSG"/>
+<pinref part="U$2" gate="G$1" pin="HSG"/>
 <pinref part="C6" gate="G$1" pin="P$1"/>
 <wire x1="132.08" y1="27.94" x2="127" y2="27.94" width="0.1524" layer="91"/>
@@
 <net name="N$10" class="0">
 <segment>
-<pinref part="U$3" gate="G$1" pin="TAB"/>
+<pinref part="U$2" gate="G$1" pin="TAB"/>
 <pinref part="OUT" gate="-1" pin="KL"/>
 <wire x1="157.48" y1="25.4" x2="182.88" y2="25.4" width="0.1524" layer="91"/>

Commit message: cdf-single-driver wip
Other:
- note removed: "TODO 24->9v supply"
Changed lines of the file:
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@@
 <part name="H4" library="holes" deviceset="MOUNT-HOLE" device="3.3"/>
 <part name="24V" library="con-ptr500" deviceset="AK500/2" device=""/>
-<part name="P+3" library="supply1" deviceset="+24V" device=""/>
-<part name="GND8" library="microbuilder" deviceset="GND" device=""/>
 <part name="IC1" library="r-78xx_10" deviceset="R-78*-0.5" device="" technology="9.0"/>
 <part name="C8" library="rcl" deviceset="CPOL-US" device="E3.5-8" value="220u"/>
@@
 <part name="SUPPLY2" library="supply2" deviceset="+9V" device=""/>
 <part name="D3" library="diode" deviceset="DIODE-" device="SOD123"/>
+<part name="P+3" library="supply1" deviceset="+24V" device=""/>
+<part name="GND8" library="microbuilder" deviceset="GND" device=""/>
 </parts>
 <sheets>
 <sheet>
 <plain>
-<text x="0" y="88.9" size="1.778" layer="91">TODO 24-&gt;9v supply</text>
 </plain>
 <instances>
@@
 <instance part="24V" gate="-1" x="-45.72" y="101.6"/>
 <instance part="24V" gate="-2" x="-45.72" y="96.52"/>
-<instance part="P+3" gate="1" x="-33.02" y="101.6" rot="R270"/>
-<instance part="GND8" gate="G$1" x="-33.02" y="96.52" rot="R90"/>
 <instance part="IC1" gate="G$1" x="-55.88" y="73.66"/>
 <instance part="C8" gate="G$1" x="-86.36" y="68.58"/>
@@
 <instance part="SUPPLY2" gate="G$1" x="-10.16" y="73.66" rot="R270"/>
 <instance part="D3" gate="G$1" x="-55.88" y="83.82" rot="R180"/>
+<instance part="P+3" gate="1" x="-33.02" y="101.6" rot="R270"/>
+<instance part="GND8" gate="G$1" x="-33.02" y="96.52" rot="R90"/>
 </instances>
 <busses>
@@
 <pinref part="GND7" gate="G$1" pin="GND"/>
 <wire x1="162.56" y1="40.64" x2="160.02" y2="40.64" width="0.1524" layer="91"/>
-</segment>
-<segment>
-<pinref part="24V" gate="-2" pin="KL"/>
-<pinref part="GND8" gate="G$1" pin="GND"/>
-<wire x1="-35.56" y1="96.52" x2="-40.64" y2="96.52" width="0.1524" layer="91"/>
 </segment>
 <segment>
@@
 <wire x1="-35.56" y1="58.42" x2="-35.56" y2="53.34" width="0.1524" layer="91"/>
 </segment>
+<segment>
+<pinref part="24V" gate="-2" pin="KL"/>
+<wire x1="-35.56" y1="96.52" x2="-40.64" y2="96.52" width="0.1524" layer="91"/>
+<pinref part="GND8" gate="G$1" pin="GND"/>
+</segment>
 </net>
 <net name="N$1" class="0">
@@
 <wire x1="116.84" y1="40.64" x2="116.84" y2="35.56" width="0.1524" layer="91"/>
 <junction x="127" y="40.64"/>
-</segment>
-<segment>
-<pinref part="24V" gate="-1" pin="KL"/>
-<pinref part="P+3" gate="1" pin="+24V"/>
-<wire x1="-35.56" y1="101.6" x2="-40.64" y2="101.6" width="0.1524" layer="91"/>
 </segment>
 <segment>
@@
 <wire x1="-68.58" y1="83.82" x2="-68.58" y2="73.66" width="0.1524" layer="91"/>
 </segment>
-</net>
+<segment>
+<pinref part="24V" gate="-1" pin="KL"/>
+<wire x1="-35.56" y1="101.6" x2="-40.64" y2="101.6" width="0.1524" layer="91"/>
+<pinref part="P+3" gate="1" pin="+24V"/>
+</segment>
+</net>
