File: led-keychain/LedKeychain-v2.brd (EAGLE design)
At the start: 57.2 x 26.5 mm, 22 parts, among them IC1 ATMEGA32U4-AU, Q1 CJ2302, Q2 16MHZ

Commit message: wip
Parts:
- removed C4, C5: 8pF, microbuilder:0603-MINI
- removed K1, K2, K3, K4: (no value), Seeed-Switch-2016:SW4-SMD-6.0X6.0X5.0MM
- removed Q1: CJ2302, Seeed-Transistor-2016:SOT-23
- added C8, C9: 20pF, microbuilder:0603-MINI
- added Q3: 16MHz ECS-160-20-5PX-TR, adafruit:HC49UP
- added S1, S2, S3, S4: DTSM-6, switch-tact:DTSM-6
- C3, C6: device microbuilder:0603-MINI -> microbuilder:1206
- Q2: value 16MHZ -> FDN327N; device Seeed-Crystal Oscillator-2016:X2-SMD-5.0X3.2X1.3MM -> microbuilder:SOT23-WIDE
- moved Q2 33.0 mm to (41.4, 13.5), flipped to the bottom, turned to 90 degrees
- moved C3 25.5 mm to (16.8, 13.5), flipped to the bottom, turned to 90 degrees
- moved R1 3.09 mm to (39.1, 11.2), flipped to the bottom
- moved R3 3.07 mm to (17.0, 9.40), turned to 180 degrees
- moved C6 1.70 mm to (17.3, 13.0)
- moved R2 1.63 mm to (17.0, 7.87), turned to 180 degrees
- moved C1 0.76 mm to (9.65, 13.5)
- moved C7 0.76 mm to (9.65, 3.05)
- moved IC1 0.76 mm to (8.13, 10.7)
- moved C2 0.76 mm to (5.08, 7.62)
- renumbered JP1 to LED_HW, JP2 to LED_SW, JP3 to USB
Connections:
- removed net N$1: C5.2, IC1.16, Q2.1
- removed net N$2: C4.2, IC1.17, Q2.2
- new net N$7: C9.2, IC1.16, Q3.1
- new net N$8: C8.2, IC1.17, Q3.2
- net GND: now also C8.1, C9.1, Q2.2, S1.1, S2.1, S3.1, S4.1; no longer C4.1, C5.1, K1.1, K2.1, K3.1, K4.1, Q1.2
- net LED_EN: now also Q2.1; no longer Q1.1
- net LED_GND: now also Q2.3; no longer Q1.3
- net PB1: now also S1.3; no longer K1.2
- net PB2: now also S2.3; no longer K2.2
- net PB3: now also S3.3; no longer K3.2
- net PB4: now also S4.3; no longer K4.2
Routing:
- net N$7: track 0.00 -> 11.0 mm
- net N$8: track 0.00 -> 10.0 mm
- net N$2: track 7.69 -> 0.00 mm
- net N$1: track 7.36 -> 0.00 mm
- net GND: track 12.0 -> 17.1 mm, vias 5 -> 8
- net D+: track 1.78 -> 4.66 mm
- net N$4: track 5.03 -> 2.48 mm
- net LED_EN: track 49.0 -> 46.5 mm, vias 4 -> 3
- net N$5: track 1.83 -> 3.71 mm
- net VCC: track 16.2 -> 14.3 mm, vias 7 -> 6
- net D-: track 2.10 -> 3.50 mm
- net N$3: track 3.65 -> 2.50 mm
- net MOSI: track 34.3 -> 33.1 mm
- net PB2: track 41.2 -> 42.1 mm
- net PB1: track 29.0 -> 29.9 mm
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Other:
- board text added: "Led-Keychain v2"
