File: led-keychain/LedKeychain-v2.sch (EAGLE design)
At the start: 22 parts, among them IC1 ATMEGA32U4-AU, Q1 CJ2302, Q2 16MHZ

Commit message: wip
Parts:
- removed C4, C5: 8pF, microbuilder:CAP_CERAMIC0603MINI
- removed K1, K2, K3, K4: (no value), Seeed-Switch-2016:SMD-SWITCH-TACTILE-SPST-NO(4P-D6.0MM)
- removed Q1: CJ2302, Seeed-Transistor-2016:SMD-MOSFET-N-CH-20V-2.1A-CJ2302(SOT-23)
- added C8, C9: 20pF, microbuilder:CAP_CERAMIC0603MINI
- added Q3: 16MHz ECS-160-20-5PX-TR, adafruit:CRYSTALHC49UP
- added S1, S2, S3, S4: DTSM-6, switch-tact:DTSM-6
- C3, C6: device microbuilder:CAP_CERAMIC0603MINI -> microbuilder:CAP_CERAMIC1206
- Q2: value 16MHZ -> FDN327N; device Seeed-Crystal Oscillator-2016:SMD-CRYSTAL-16MHZ-8PF-20PPM-40R(2P-5.0X3.2MM) -> microbuilder:MOSFET-NWIDE
- renumbered JP1 to LED_HW, JP2 to LED_SW, JP3 to USB
Connections:
- removed net N$1: C5.P$2, IC1.XTAL2, Q2.1
- removed net N$2: C4.P$2, IC1.XTAL1, Q2.2
- new net N$7: C9.P$2, IC1.XTAL2, Q3.1
- new net N$8: C8.P$2, IC1.XTAL1, Q3.2
- net GND: now also C8.P$1, C9.P$1, Q2.S, S1.1, S2.1, S3.1, S4.1; no longer C4.P$1, C5.P$1, K1.A0, K2.A0, K3.A0, K4.A0, Q1.S
- net LED_EN: now also Q2.G; no longer Q1.G
- net LED_GND: now also Q2.D; no longer Q1.D
- net PB1: now also S1.3; no longer K1.B0
- net PB2: now also S2.3; no longer K2.B0
- net PB3: now also S3.3; no longer K3.B0
- net PB4: now also S4.3; no longer K4.B0
Other:
- moved on the sheet: R1
