File: cdf-teensy-interrupter/cdf-teensy-interrupter-v2.brd (EAGLE design)
At the start: 76.2 x 80 mm, 41 parts, among them T1 BC337, T2 BC337, T3 BC337

Commit message: wip
Other:
- board text added: "CDF Interrupter v2 )'( 2017"
Changed lines of the file:
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@@
 <wire x1="0" y1="0" x2="76.2" y2="0" width="0" layer="20"/>
 <wire x1="76.2" y1="0" x2="76.2" y2="80.01" width="0" layer="20"/>
+<text x="25.019" y="74.93" size="1.778" layer="22" font="vector" rot="MR180">CDF Interrupter v2
+)'( 2017</text>
 </plain>
 <attributes>
@@
 </board>
 </drawing>
+<compatibility>
+<note version="6.3" minversion="6.2.2" severity="warning">
+Since Version 6.2.2 text objects can contain more than one line,
+which will not be processed correctly with this version.
+</note>
+</compatibility>
 </eagle>
