File: phi-brain4ch/phi-dac.brd (EAGLE design)
At the start: 119.4 x 101.6 mm, 147 parts, among them IC1 PCM1792A, IC10 LM317, IC11 LM337, IC2 OPA1632D, IC3 OPA1632D, IC4 OPA1632D, IC6 OPA1632D, IC7 REG1117-5, IC8 ADP3301ARZ-3.3, IC9 MGJ2D121515SC, J1 CUI-RCJ-2123, J5 DC21P

Commit message: wip
Parts:
- moved C15 108.1 mm to (55.6, 17.1), flipped to the bottom, turned to 270 degrees
- moved C8 98.1 mm to (58.8, 31.6), flipped to the bottom
- moved C7 77.3 mm to (47.6, 30.6), flipped to the bottom
- moved C16 71.1 mm to (48.9, 15.7), flipped to the bottom, turned to 90 degrees
- moved R38 24.7 mm to (94.7, 43.6)
- moved R36 23.6 mm to (93.2, 46.0)
- moved R37 19.7 mm to (98.9, 44.7)
- moved R35 15.0 mm to (97.3, 47.0), turned to 180 degrees
- moved R32 2.87 mm to (58.8, 2.16), turned to 0 degrees
- moved C47 2.74 mm to (62.7, 14.7), turned to 0 degrees
- moved C17 1.30 mm to (88.9, 44.1)
- moved C48 1.05 mm to (61.1, 8.26), turned to 0 degrees
- moved R23 0.51 mm to (65.4, 17.1)
Routing:
- net DAC_VCC: track 5.79 -> 54.6 mm
- net IN_L_PP: track 2.31 -> 40.7 mm
- net SPI_CLK: track 0.00 -> 36.1 mm, vias 0 -> 2
- net SPI_MISO: track 0.00 -> 35.9 mm, vias 0 -> 1
- net SPI_MOSI: track 0.00 -> 33.1 mm, vias 0 -> 1
- net I2S_BCK: track 0.00 -> 32.3 mm, vias 0 -> 1
- net SPI_CS: track 0.00 -> 31.0 mm, vias 0 -> 1
- net I2S_MCK: track 0.00 -> 30.3 mm, vias 0 -> 1
- net I2S_LRCK: track 0.00 -> 28.3 mm, vias 0 -> 1
- net I2S_DATA: track 0.00 -> 25.0 mm, vias 0 -> 1
- net IN_L_NN: track 2.42 -> 27.1 mm
- net IN_R_PP: track 2.31 -> 23.7 mm
- net AVDD: track 54.6 -> 71.3 mm, vias 0 -> 2
- net N$23: track 12.9 -> 28.5 mm
- net AVCC: track 60.5 -> 74.8 mm, vias 0 -> 3
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
Commit message: wip
Parts:
- moved C7 37.1 mm to (81.3, 15.1), turned to 270 degrees
- moved C8 34.6 mm to (81.2, 5.21), turned to 90 degrees
- moved C43 3.50 mm to (89.9, 14.6), turned to 0 degrees
- moved C44 1.73 mm to (88.9, 6.99)
- moved R32 1.42 mm to (57.5, 1.52)
- moved R7 1.42 mm to (92.1, 17.3)
- moved C48 1.30 mm to (59.8, 8.00)
- moved C10 1.27 mm to (69.5, 16.9)
- moved C13 1.27 mm to (72.5, 12.6)
- moved C14 1.27 mm to (72.5, 8.00)
- moved C2 1.27 mm to (97.4, 16.9)
- moved C3 1.27 mm to (102.5, 8.00)
- moved C4 1.27 mm to (102.5, 12.6)
- moved C5 1.27 mm to (90.8, 11.8)
- moved C6 1.27 mm to (90.8, 8.26)
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Routing:
- net AVCC: track 74.8 -> 90.8 mm, vias 3 -> 6
- net AVDD: track 71.3 -> 85.2 mm, vias 2 -> 6
- net N$28: track 2.17 -> 0.00 mm
- net N$14: track 16.1 -> 17.9 mm
- net GND: track 169.9 -> 168.6 mm
- net IN_L_NN: track 27.1 -> 28.4 mm
- net SPI_MOSI: track 33.1 -> 34.4 mm
- net SPI_MISO: track 35.9 -> 37.2 mm
- net SPI_CS: track 31.0 -> 32.3 mm
- net SPI_CLK: track 36.1 -> 37.4 mm
- net IN_L_PP: track 40.7 -> 41.9 mm
- net I2S_MCK: track 30.3 -> 31.6 mm
- net I2S_LRCK: track 28.3 -> 29.5 mm
- net I2S_DATA: track 25.0 -> 26.3 mm
- net I2S_BCK: track 32.3 -> 33.6 mm
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
Commit message: wip
Parts:
- moved R32 0.25 mm to (57.5, 1.78)
Routing:
- net AVDD: track 85.2 -> 127.9 mm
- net AVCC: track 90.8 -> 118.5 mm
- net N$28: track 0.00 -> 2.55 mm
- net GND: track 168.6 -> 169.4 mm
Changed lines of the file:
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@@
 <element name="R30" library="microbuilder" package="_0805" value="22 0.1%" x="61.722" y="2.159" rot="R180"/>
 <element name="R31" library="microbuilder" package="_0805" value="22 0.1%" x="60.96" y="18.161" rot="R270"/>
-<element name="R32" library="microbuilder" package="_0805" value="0" x="57.531" y="1.524"/>
+<element name="R32" library="microbuilder" package="_0805" value="0" x="57.531" y="1.778"/>
 <element name="R4" library="microbuilder" package="_0805" value="390 0.1%" x="98.171" y="7.493" rot="R90"/>
 <element name="R5" library="microbuilder" package="_0805" value="390 0.1%" x="101.727" y="16.637" rot="R90"/>
@@
 <wire x1="62.738" y1="14.351" x2="62.738" y2="12.788" width="0.4064" layer="1"/>
 <wire x1="62.738" y1="12.788" x2="62.865" y2="12.661" width="0.4064" layer="1"/>
-<wire x1="56.515" y1="1.524" x2="55.372" y2="1.524" width="0.4064" layer="1"/>
-<via x="55.372" y="1.524" extent="1-16" drill="0.3302"/>
-<wire x1="55.372" y1="1.524" x2="55.245" y2="1.524" width="0.4064" layer="16"/>
 <wire x1="90.932" y1="14.605" x2="90.932" y2="15.113" width="0.4064" layer="1"/>
 <wire x1="90.932" y1="15.113" x2="90.043" y2="16.002" width="0.4064" layer="1"/>
@@
 <wire x1="89.535" y1="4.699" x2="89.535" y2="4.572" width="0.4064" layer="16"/>
 <wire x1="89.535" y1="4.572" x2="89.662" y2="4.445" width="0.4064" layer="16"/>
+<wire x1="56.515" y1="1.778" x2="55.753" y2="1.778" width="0.4064" layer="1"/>
+<wire x1="55.753" y1="1.778" x2="55.118" y2="2.413" width="0.4064" layer="1"/>
+<via x="55.118" y="2.413" extent="1-16" drill="0.3302"/>
+<wire x1="55.118" y1="2.413" x2="54.864" y2="2.413" width="0.4064" layer="16"/>
+<wire x1="54.864" y1="2.413" x2="54.737" y2="2.54" width="0.4064" layer="16"/>
 <wire x1="79.886" y1="31.242" x2="72.771" y2="39.243" width="0" layer="19" extent="1-1"/>
 <wire x1="82.55" y1="31.75" x2="79.886" y2="31.242" width="0" layer="19" extent="1-16"/>
@@
 <wire x1="88.9" y1="11.43" x2="88.9" y2="13.335" width="0.4064" layer="1"/>
 <via x="88.9" y="13.335" extent="1-16" drill="0.3302"/>
-<wire x1="88.9" y1="12.446" x2="88.9" y2="11.938" width="0.4064" layer="16"/>
+<wire x1="88.9" y1="12.446" x2="88.9" y2="11.557" width="0.4064" layer="16"/>
 <wire x1="88.9" y1="11.557" x2="88.9" y2="11.303" width="0.4064" layer="16"/>
 <wire x1="88.9" y1="11.303" x2="88.646" y2="11.049" width="0.4064" layer="16"/>
@@
 <via x="88.9" y="11.557" extent="1-16" drill="0.3302"/>
 <wire x1="88.9" y1="13.335" x2="88.9" y2="12.446" width="0.4064" layer="16"/>
-<wire x1="88.9" y1="11.557" x2="88.9" y2="11.938" width="0.4064" layer="16"/>
 <wire x1="90.717" y1="11.049" x2="90.17" y2="11.049" width="0.4064" layer="1"/>
 <wire x1="90.17" y1="11.049" x2="89.789" y2="11.43" width="0.4064" layer="1"/>
 <wire x1="89.789" y1="11.43" x2="89.789" y2="13.716" width="0.4064" layer="1"/>
 <wire x1="89.789" y1="13.716" x2="88.9" y2="14.605" width="0.4064" layer="1"/>
+<wire x1="81.28" y1="12.459" x2="80.378" y2="12.459" width="0.889" layer="16"/>
+<wire x1="80.378" y1="12.459" x2="79.629" y2="13.208" width="0.889" layer="16"/>
+<wire x1="79.629" y1="13.208" x2="64.389" y2="13.208" width="0.889" layer="16"/>
+<wire x1="64.389" y1="13.208" x2="63.246" y2="14.351" width="0.889" layer="16"/>
+<wire x1="63.246" y1="14.351" x2="54.496" y2="14.351" width="0.889" layer="16"/>
+<wire x1="54.496" y1="14.351" x2="54.356" y2="14.491" width="0.889" layer="16"/>
 <wire x1="51.689" y1="76.581" x2="51.523" y2="78.613" width="0" layer="19" extent="1-1"/>
 <wire x1="54.356" y1="14.491" x2="52.451" y2="76.581" width="0" layer="19" extent="1-16"/>
-<wire x1="81.28" y1="12.459" x2="77.724" y2="12.446" width="0" layer="19" extent="1-16"/>
 <wire x1="37.846" y1="15.24" x2="54.356" y2="14.491" width="0" layer="19" extent="16-16"/>
 </signal>
@@
 <wire x1="88.9" y1="8.001" x2="89.701" y2="8.001" width="0.4064" layer="1"/>
 <wire x1="89.701" y1="8.001" x2="90.805" y2="9.105" width="0.4064" layer="1"/>
+<wire x1="81.166" y1="2.54" x2="81.166" y2="2.045" width="0.889" layer="16"/>
+<wire x1="80.01" y1="0.889" x2="54.483" y2="0.889" width="0.889" layer="16"/>
+<wire x1="53.086" y1="2.286" x2="53.086" y2="7.633" width="0.889" layer="16"/>
+<wire x1="53.086" y1="7.633" x2="47.625" y2="13.094" width="0.889" layer="16"/>
+<wire x1="80.01" y1="0.889" x2="81.166" y2="2.045" width="0.889" layer="16"/>
+<wire x1="54.483" y1="0.889" x2="53.086" y2="2.286" width="0.889" layer="16"/>
 <wire x1="37.846" y1="17.78" x2="55.559" y2="83.82" width="0" layer="19" extent="1-1"/>
 <wire x1="47.625" y1="13.094" x2="37.846" y2="17.78" width="0" layer="19" extent="16-16"/>
-<wire x1="81.166" y1="2.54" x2="77.724" y2="7.2136" width="0" layer="19" extent="1-16"/>
 <wire x1="85.725" y1="8.001" x2="85.471" y2="8.001" width="0" layer="19" extent="1-1"/>
 <wire x1="86.614" y1="8.001" x2="87.503" y2="8.001" width="0" layer="19" extent="1-1"/>
@@
 <contactref element="R32" pad="2"/>
 <contactref element="BAL_RIGHT" pad="S"/>
-<wire x1="58.547" y1="1.524" x2="59.195" y2="4.064" width="0" layer="19" extent="1-1"/>
+<wire x1="59.195" y1="4.064" x2="59.195" y2="2.426" width="0.4064" layer="1"/>
+<wire x1="59.195" y1="2.426" x2="58.547" y2="1.778" width="0.4064" layer="1"/>
 </signal>
 <signal name="N$29">

Commit message: wip
Parts:
- moved C40 71.4 mm to (46.2, 16.4), turned to 180 degrees
- moved R25 70.1 mm to (40.6, 18.2), turned to 90 degrees
- moved R11 70.0 mm to (55.4, 17.1), turned to 270 degrees
- moved R9 69.5 mm to (53.1, 17.1), turned to 90 degrees
- moved R10 69.3 mm to (50.5, 17.1), turned to 90 degrees
- moved R26 69.0 mm to (42.9, 18.2), turned to 90 degrees
- moved C42 67.3 mm to (46.2, 18.4), turned to 180 degrees
- moved R27 61.9 mm to (40.6, 22.5), turned to 90 degrees
- moved R12 60.9 mm to (53.1, 21.5), turned to 90 degrees
- moved R28 60.6 mm to (42.9, 22.5), turned to 90 degrees
- moved IC5 60.4 mm to (48.0, 21.7), turned to 270 degrees
- moved C41 53.6 mm to (50.3, 25.0), turned to 0 degrees
- moved C53 52.6 mm to (88.1, 70.9)
- moved C55 52.6 mm to (93.2, 62.0)
- moved LED1 52.6 mm to (87.8, 66.3)
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Connections:
- net N$12: now also J1.P$1; no longer J1.P$3
- net N$27: now also J1.P$3; no longer J1.P$1
Routing:
- net N$26: track 2.53 -> 23.7 mm
- net N$11: track 2.53 -> 22.5 mm
- net OUT_R_PP: track 8.50 -> 28.4 mm, vias 0 -> 2
- net AVCC: track 118.5 -> 136.9 mm, vias 6 -> 7
- net AVDD: track 127.9 -> 143.1 mm, vias 6 -> 7
- net N$27: track 0.00 -> 4.27 mm
- net N$12: track 0.00 -> 3.02 mm
- net OUT_R_NN: track 9.91 -> 7.42 mm
- net N$28: track 2.55 -> 3.19 mm
- net GND: track 169.4 -> 169.3 mm, vias 87 -> 86

Commit message: wip
Parts:
- moved R32 11.7 mm to (45.8, 1.65)
- moved R16 1.55 mm to (85.1, 3.56)
- moved R25 0.52 mm to (40.1, 18.0)
Routing:
- net OUT_L_PP: track 9.07 -> 69.2 mm, vias 0 -> 2
- net OUT_L_NN: track 10.3 -> 55.9 mm, vias 0 -> 4
- net OUT_R_NN: track 7.42 -> 33.5 mm, vias 0 -> 2
- net N$28: track 3.19 -> 14.4 mm
- net OUT_R_PP: track 28.4 -> 38.1 mm
- net N$11: track 22.5 -> 20.9 mm
- net GND: track 169.3 -> 169.7 mm, vias 86 -> 87

Commit message: wip
Parts:
- moved H4 126.6 mm to (116.8, 48.3)
- moved LED3 58.6 mm to (70.5, 37.5), turned to 90 degrees
- moved R45 55.1 mm to (71.1, 40.5), turned to 90 degrees
- moved C65 51.9 mm to (69.1, 42.0), turned to 270 degrees
- moved C64 50.9 mm to (67.2, 42.0), turned to 270 degrees
- moved C53 50.7 mm to (62.1, 27.3), turned to 180 degrees
- moved EN_DAC_VCC 49.6 mm to (70.9, 44.7), turned to 90 degrees
- moved IC7 47.6 mm to (61.8, 42.8), turned to 90 degrees
- moved IC8 47.5 mm to (63.8, 30.7), turned to 90 degrees
- moved C63 46.9 mm to (69.1, 46.0), turned to 270 degrees
- moved C62 45.7 mm to (67.2, 46.0), turned to 90 degrees
- moved LED1 44.7 mm to (66.7, 26.9), turned to 90 degrees
- moved C54 40.0 mm to (69.0, 31.5), turned to 90 degrees
- moved R43 39.0 mm to (70.9, 26.9), turned to 0 degrees
- moved EN_3.3 38.4 mm to (70.7, 28.8), turned to 0 degrees
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Routing:
- net DAC_VCC: track 54.6 -> 77.3 mm
- net 3.3V: track 1.96 -> 23.4 mm
- net N$35: track 0.00 -> 7.14 mm
- net N$42: track 0.00 -> 4.96 mm
- net GND: track 169.7 -> 174.2 mm, vias 87 -> 89
- net N$37: track 2.62 -> 6.27 mm
- net N$36: track 2.27 -> 4.83 mm
Other:
- board size 119.4 x 101.6 mm -> 119.4 x 50.8 mm

Commit message: routed
Parts:
- removed H5, H6: MOUNT-HOLE3.2, holes:3,2
Routing:
- net +12V: track 63.0 -> 162.2 mm
- net N$49: track 6.89 -> 9.83 mm
Changed lines of the file:
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@@
 <setting verticaltext="up"/>
 </settings>
-<grid distance="50" unitdist="mil" unit="mil" style="lines" multiple="1" display="no" altdistance="0.025" altunitdist="inch" altunit="inch"/>
+<grid distance="10" unitdist="mil" unit="mil" style="lines" multiple="1" display="no" altdistance="0.025" altunitdist="inch" altunit="inch"/>
 <layers>
 <layer number="1" name="Top" color="4" fill="1" visible="yes" active="yes"/>
@@
 <element name="H2" library="holes" package="3,2" value="MOUNT-HOLE3.2" x="116.84" y="2.54">
 <attribute name="POPULATE" value="0" x="107.95" y="-24.13" size="1.778" layer="27" display="off"/>
-</element>
-<element name="H5" library="holes" package="3,2" value="MOUNT-HOLE3.2" x="-18.288" y="29.718">
-<attribute name="POPULATE" value="0" x="-18.288" y="11.938" size="1.778" layer="27" display="off"/>
-</element>
-<element name="H6" library="holes" package="3,2" value="MOUNT-HOLE3.2" x="-9.398" y="29.718">
-<attribute name="POPULATE" value="0" x="-18.288" y="3.048" size="1.778" layer="27" display="off"/>
 </element>
 <element name="JP1" library="jumper" package="JP4Q" value="" x="81.407" y="23.749"/>
@@
 <wire x1="3.81" y1="12.446" x2="2.54" y2="12.446" width="1.143" layer="1"/>
 <wire x1="2.54" y1="12.446" x2="1.651" y2="13.335" width="1.143" layer="1"/>
-<wire x1="1.651" y1="13.335" x2="1.651" y2="33.782" width="1.143" layer="1"/>
-<wire x1="1.651" y1="33.782" x2="3.429" y2="35.56" width="1.143" layer="1"/>
-<wire x1="3.429" y1="35.56" x2="11.811" y2="35.56" width="1.143" layer="1"/>
+<wire x1="1.651" y1="13.335" x2="1.651" y2="36.068" width="1.143" layer="1"/>
+<wire x1="1.651" y1="36.068" x2="1.651" y2="37.211" width="1.143" layer="1"/>
+<wire x1="2.159" y1="35.56" x2="11.811" y2="35.56" width="1.143" layer="1"/>
 <wire x1="11.811" y1="35.56" x2="12.319" y2="35.052" width="1.143" layer="1"/>
 <wire x1="12.319" y1="35.052" x2="12.319" y2="34.023" width="1.143" layer="1"/>
@@
 <wire x1="3.937" y1="10.668" x2="3.937" y2="12.319" width="1.143" layer="1"/>
 <wire x1="3.937" y1="12.319" x2="3.81" y2="12.446" width="1.143" layer="1"/>
-<wire x1="64.9986" y1="45.1104" x2="61.722" y2="32.639" width="0" layer="19" extent="1-1"/>
-<wire x1="12.319" y1="34.023" x2="60.6806" y2="32.639" width="0" layer="19" extent="1-1"/>
+<wire x1="64.9986" y1="45.1104" x2="64.9986" y2="48.0314" width="1.143" layer="1"/>
+<wire x1="64.9986" y1="48.0314" x2="64.77" y2="48.26" width="1.143" layer="1"/>
+<wire x1="64.77" y1="48.26" x2="50.292" y2="48.26" width="1.143" layer="1"/>
+<wire x1="50.292" y1="48.26" x2="12.7" y2="48.26" width="1.143" layer="1"/>
+<wire x1="12.7" y1="48.26" x2="1.651" y2="37.211" width="1.143" layer="1"/>
+<wire x1="2.159" y1="35.56" x2="1.651" y2="36.068" width="1.143" layer="1"/>
+<wire x1="61.722" y1="32.639" x2="53.213" y2="32.639" width="1.143" layer="1"/>
+<wire x1="53.213" y1="32.639" x2="50.8" y2="35.052" width="1.143" layer="1"/>
+<wire x1="50.8" y1="35.052" x2="50.8" y2="47.752" width="1.143" layer="1"/>
+<wire x1="50.8" y1="47.752" x2="50.292" y2="48.26" width="1.143" layer="1"/>
 </signal>
 <signal name="N$49">
@@
 <wire x1="11.43" y1="21.206" x2="14.602" y2="21.206" width="1.27" layer="1"/>
 <wire x1="14.602" y1="21.206" x2="14.605" y2="21.209" width="1.27" layer="1"/>
-<wire x1="8.509" y1="21.168" x2="11.43" y2="21.206" width="0" layer="19" extent="1-1"/>
+<wire x1="8.509" y1="21.168" x2="11.392" y2="21.168" width="1.143" layer="1"/>
+<wire x1="11.392" y1="21.168" x2="11.43" y2="21.206" width="1.143" layer="1"/>
 </signal>
 <signal name="N$50">
@@
 <vertex x="69.596" y="43.561"/>
 <vertex x="63.119" y="43.561"/>
-<vertex x="63.119" y="48.895"/>
-<vertex x="55.245" y="48.895"/>
+<vertex x="63.119" y="46.355"/>
+<vertex x="55.245" y="46.355"/>
 <vertex x="55.245" y="36.703"/>
 <vertex x="63.119" y="36.703"/>

Commit message: routed
Parts:
- added C52: 0.1uF, microbuilder:0603
- added OSC1: (no value), microbuilder:OSC_7X5MM
- added R48: 0, microbuilder:_0805
Connections:
- new net N$32: OSC1.3, R48.1
- net 3.3V: now also C52.1, OSC1.4
- net GND: now also C52.2, OSC1.2
- net I2S_MCK: now also R48.2
