File: phi-brain4ch/phi-dac.sch (EAGLE design)
At the start: 146 parts, among them IC1 PCM1792A, IC10 LM317, IC11 LM337, IC2 OPA1632D, IC3 OPA1632D, IC4 OPA1632D, IC6 OPA1632D, IC7 REG1117-5, IC8 ADP3301ARZ-3.3, IC9 MGJ2D121515SC, J1 CUI-RCJ-2123, J5 DC21P

Commit message: wip
Parts:
- added C51: 1uF 12065C105M4Z2A, microbuilder:CAP_CERAMIC1206
Connections:
- net GND: now also C51.P$1
- net N$57: now also C51.P$2
Other:
- moved on the sheet: C38, D4, R42
Changed lines of the file:
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@@
 <part name="C49" library="microbuilder" deviceset="CAP_CERAMIC" device="0603" value="0.1u"/>
 <part name="C50" library="microbuilder" deviceset="CAP_CERAMIC" device="0603" value="0.1u"/>
+<part name="C51" library="microbuilder" deviceset="CAP_CERAMIC" device="1206" value="1uF 12065C105M4Z2A"/>
 </parts>
 <sheets>
@@
 <instance part="C37" gate="G$1" x="190.5" y="147.32"/>
 <instance part="R41" gate="G$1" x="218.44" y="165.1" rot="R90"/>
-<instance part="R42" gate="G$1" x="231.14" y="149.86" rot="R90"/>
+<instance part="R42" gate="G$1" x="228.6" y="149.86" rot="R90"/>
 <instance part="U$29" gate="G$1" x="218.44" y="175.26" rot="R180"/>
-<instance part="C38" gate="G$1" x="241.3" y="165.1"/>
-<instance part="D4" gate="G$1" x="241.3" y="152.4" rot="R90"/>
+<instance part="C38" gate="G$1" x="236.22" y="165.1"/>
+<instance part="D4" gate="G$1" x="236.22" y="152.4" rot="R90"/>
 <instance part="L6" gate="G$1" x="254" y="144.78" rot="R90"/>
 <instance part="U$30" gate="G$1" x="281.94" y="144.78" rot="R270"/>
@@
 <instance part="C49" gate="G$1" x="149.86" y="-22.86"/>
 <instance part="C50" gate="G$1" x="149.86" y="-12.7"/>
+<instance part="C51" gate="G$1" x="243.84" y="154.94"/>
 </instances>
 <busses>
@@
 <junction x="218.44" y="170.18"/>
 <pinref part="C38" gate="G$1" pin="P$1"/>
-<wire x1="218.44" y1="170.18" x2="241.3" y2="170.18" width="0.1524" layer="91"/>
+<wire x1="218.44" y1="170.18" x2="236.22" y2="170.18" width="0.1524" layer="91"/>
+<pinref part="C51" gate="G$1" pin="P$1"/>
+<wire x1="236.22" y1="170.18" x2="243.84" y2="170.18" width="0.1524" layer="91"/>
+<wire x1="243.84" y1="170.18" x2="243.84" y2="160.02" width="0.1524" layer="91"/>
+<junction x="236.22" y="170.18"/>
 </segment>
 <segment>
@@
 <pinref part="D3" gate="G$1" pin="C"/>
 <pinref part="R42" gate="G$1" pin="1"/>
-<wire x1="215.9" y1="132.08" x2="231.14" y2="132.08" width="0.1524" layer="91"/>
-<wire x1="231.14" y1="132.08" x2="231.14" y2="144.78" width="0.1524" layer="91"/>
+<wire x1="215.9" y1="132.08" x2="228.6" y2="132.08" width="0.1524" layer="91"/>
+<wire x1="228.6" y1="132.08" x2="228.6" y2="144.78" width="0.1524" layer="91"/>
 <pinref part="IC11" gate="G$1" pin="OUT"/>
-<wire x1="231.14" y1="144.78" x2="226.06" y2="144.78" width="0.1524" layer="91"/>
-<junction x="231.14" y="144.78"/>
-<wire x1="231.14" y1="144.78" x2="241.3" y2="144.78" width="0.1524" layer="91"/>
-<wire x1="241.3" y1="144.78" x2="241.3" y2="149.86" width="0.1524" layer="91"/>
+<wire x1="228.6" y1="144.78" x2="226.06" y2="144.78" width="0.1524" layer="91"/>
+<junction x="228.6" y="144.78"/>
+<wire x1="228.6" y1="144.78" x2="236.22" y2="144.78" width="0.1524" layer="91"/>
+<wire x1="236.22" y1="144.78" x2="236.22" y2="149.86" width="0.1524" layer="91"/>
 <pinref part="D4" gate="G$1" pin="A"/>
 <pinref part="L6" gate="G$1" pin="1"/>
-<wire x1="246.38" y1="144.78" x2="241.3" y2="144.78" width="0.1524" layer="91"/>
-<junction x="241.3" y="144.78"/>
+<wire x1="246.38" y1="144.78" x2="243.84" y2="144.78" width="0.1524" layer="91"/>
+<junction x="236.22" y="144.78"/>
+<junction x="243.84" y="144.78"/>
+<wire x1="243.84" y1="144.78" x2="236.22" y2="144.78" width="0.1524" layer="91"/>
+<pinref part="C51" gate="G$1" pin="P$2"/>
+<wire x1="243.84" y1="152.4" x2="243.84" y2="144.78" width="0.1524" layer="91"/>
 </segment>
 </net>
@@
 <wire x1="218.44" y1="157.48" x2="218.44" y2="160.02" width="0.1524" layer="91"/>
 <pinref part="R42" gate="G$1" pin="2"/>
-<wire x1="231.14" y1="154.94" x2="231.14" y2="157.48" width="0.1524" layer="91"/>
-<wire x1="231.14" y1="157.48" x2="218.44" y2="157.48" width="0.1524" layer="91"/>
+<wire x1="228.6" y1="154.94" x2="228.6" y2="157.48" width="0.1524" layer="91"/>
+<wire x1="228.6" y1="157.48" x2="218.44" y2="157.48" width="0.1524" layer="91"/>
 <junction x="218.44" y="157.48"/>
-<wire x1="231.14" y1="157.48" x2="241.3" y2="157.48" width="0.1524" layer="91"/>
-<wire x1="241.3" y1="157.48" x2="241.3" y2="154.94" width="0.1524" layer="91"/>
+<wire x1="228.6" y1="157.48" x2="236.22" y2="157.48" width="0.1524" layer="91"/>
+<wire x1="236.22" y1="157.48" x2="236.22" y2="154.94" width="0.1524" layer="91"/>
 <pinref part="C38" gate="G$1" pin="P$2"/>
-<wire x1="241.3" y1="157.48" x2="241.3" y2="162.56" width="0.1524" layer="91"/>
-<junction x="241.3" y="157.48"/>
+<wire x1="236.22" y1="157.48" x2="236.22" y2="162.56" width="0.1524" layer="91"/>
+<junction x="236.22" y="157.48"/>
 <pinref part="D4" gate="G$1" pin="C"/>
-<junction x="231.14" y="157.48"/>
-</segment>
-</net>
+<junction x="228.6" y="157.48"/>
+</segment>
+</net>

Commit message: wip
Parts:
- C24, C25: value 100uF (EEE-1EA101XP) -> 47uF (EEE-HA1C470WR); device microbuilder:CAP_ELECTROLYTICPANASONIC_D -> microbuilder:CAP_ELECTROLYTICPANASONIC_C
Connections:
- removed net N$31: IC1.IOUT_RIGHT_N, JP1.2
- removed net N$32: IC1.IOUT_RIGHT_P, JP1.4
- removed net N$33: IC1.IOUT_LEFT_N, JP1.6
- removed net N$34: IC1.IOUT_LEFT_P, JP1.8
- new net N$22: IC1.IOUT_LEFT_N, JP1.8
- new net N$23: IC1.IOUT_LEFT_P, JP1.6
- new net N$7: IC1.IOUT_RIGHT_P, JP1.2
- new net N$8: IC1.IOUT_RIGHT_N, JP1.4
- net IN_L_NN: now also JP1.7; no longer JP1.5
- net IN_L_PP: now also JP1.5; no longer JP1.7
- net IN_R_NN: now also JP1.3; no longer JP1.1
- net IN_R_PP: now also JP1.1; no longer JP1.3
Other:
- moved on the sheet: JP1
Changed lines of the file:
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@@
 <part name="C23" library="microbuilder" deviceset="CAP_CERAMIC" device="1206" value="10uF"/>
 <part name="U$22" library="microbuilder" deviceset="GND" device=""/>
-<part name="C24" library="microbuilder" deviceset="CAP_ELECTROLYTIC" device="PANASONIC_D" value="100uF (EEE-1EA101XP)"/>
-<part name="C25" library="microbuilder" deviceset="CAP_ELECTROLYTIC" device="PANASONIC_D" value="100uF (EEE-1EA101XP)"/>
+<part name="C24" library="microbuilder" deviceset="CAP_ELECTROLYTIC" device="PANASONIC_C" value="47uF (EEE-HA1C470WR)"/>
+<part name="C25" library="microbuilder" deviceset="CAP_ELECTROLYTIC" device="PANASONIC_C" value="47uF (EEE-HA1C470WR)"/>
 <part name="R34" library="microbuilder" deviceset="RESISTOR" device="_0805" value="1k"/>
 <part name="U$23" library="microbuilder" deviceset="3.3V" device=""/>
@@
 <instance part="H5" gate="G$1" x="10.16" y="210.82"/>
 <instance part="H6" gate="G$1" x="15.24" y="213.36"/>
-<instance part="JP1" gate="B" x="111.76" y="137.16" rot="R90"/>
+<instance part="JP1" gate="B" x="114.3" y="137.16" rot="R90"/>
 <instance part="R33" gate="G$1" x="144.78" y="132.08"/>
 <instance part="GND21" gate="G$1" x="157.48" y="132.08" rot="R90"/>
@@
 </segment>
 </net>
-<net name="N$31" class="0">
-<segment>
-<pinref part="IC1" gate="G$1" pin="IOUT_RIGHT_N"/>
-<pinref part="JP1" gate="B" pin="2"/>
-<wire x1="104.14" y1="134.62" x2="101.6" y2="134.62" width="0.1524" layer="91"/>
-</segment>
-</net>
-<net name="N$32" class="0">
-<segment>
-<pinref part="IC1" gate="G$1" pin="IOUT_RIGHT_P"/>
-<pinref part="JP1" gate="B" pin="4"/>
-<wire x1="104.14" y1="137.16" x2="101.6" y2="137.16" width="0.1524" layer="91"/>
-</segment>
-</net>
-<net name="N$33" class="0">
-<segment>
-<pinref part="IC1" gate="G$1" pin="IOUT_LEFT_N"/>
-<pinref part="JP1" gate="B" pin="6"/>
-<wire x1="104.14" y1="139.7" x2="101.6" y2="139.7" width="0.1524" layer="91"/>
-</segment>
-</net>
-<net name="N$34" class="0">
-<segment>
-<pinref part="IC1" gate="G$1" pin="IOUT_LEFT_P"/>
-<pinref part="JP1" gate="B" pin="8"/>
-<wire x1="104.14" y1="142.24" x2="101.6" y2="142.24" width="0.1524" layer="91"/>
-</segment>
-</net>
 <net name="N$35" class="0">
 <segment>
@@
 </segment>
 <segment>
-<pinref part="JP1" gate="B" pin="7"/>
-<wire x1="119.38" y1="142.24" x2="129.54" y2="142.24" width="0.1524" layer="91"/>
-<label x="127" y="142.24" size="1.778" layer="95"/>
+<pinref part="JP1" gate="B" pin="5"/>
+<wire x1="121.92" y1="139.7" x2="129.54" y2="139.7" width="0.1524" layer="91"/>
+<label x="127" y="139.7" size="1.778" layer="95"/>
 </segment>
 </net>
@@
 </segment>
 <segment>
-<pinref part="JP1" gate="B" pin="5"/>
-<wire x1="119.38" y1="139.7" x2="129.54" y2="139.7" width="0.1524" layer="91"/>
-<label x="127" y="139.7" size="1.778" layer="95"/>
+<pinref part="JP1" gate="B" pin="7"/>
+<wire x1="121.92" y1="142.24" x2="129.54" y2="142.24" width="0.1524" layer="91"/>
+<label x="127" y="142.24" size="1.778" layer="95"/>
 </segment>
 </net>
@@
 </segment>
 <segment>
-<pinref part="JP1" gate="B" pin="3"/>
-<wire x1="119.38" y1="137.16" x2="129.54" y2="137.16" width="0.1524" layer="91"/>
-<label x="127" y="137.16" size="1.778" layer="95"/>
+<pinref part="JP1" gate="B" pin="1"/>
+<wire x1="121.92" y1="134.62" x2="129.54" y2="134.62" width="0.1524" layer="91"/>
+<label x="127" y="134.62" size="1.778" layer="95"/>
 </segment>
 </net>
@@
 </segment>
 <segment>
-<pinref part="JP1" gate="B" pin="1"/>
-<wire x1="119.38" y1="134.62" x2="129.54" y2="134.62" width="0.1524" layer="91"/>
-<label x="127" y="134.62" size="1.778" layer="95"/>
-</segment>
-</net>
+<pinref part="JP1" gate="B" pin="3"/>
+<wire x1="121.92" y1="137.16" x2="129.54" y2="137.16" width="0.1524" layer="91"/>
+<label x="127" y="137.16" size="1.778" layer="95"/>
+</segment>
+</net>
+<net name="N$7" class="0">
+<segment>
+<pinref part="IC1" gate="G$1" pin="IOUT_RIGHT_P"/>
+<pinref part="JP1" gate="B" pin="2"/>
+<wire x1="101.6" y1="137.16" x2="106.68" y2="134.62" width="0.1524" layer="91"/>
+</segment>
+</net>
+<net name="N$8" class="0">
+<segment>
+<pinref part="IC1" gate="G$1" pin="IOUT_RIGHT_N"/>
+<pinref part="JP1" gate="B" pin="4"/>
+<wire x1="101.6" y1="134.62" x2="106.68" y2="137.16" width="0.1524" layer="91"/>
+</segment>
+</net>
+<net name="N$22" class="0">
+<segment>
+<pinref part="IC1" gate="G$1" pin="IOUT_LEFT_N"/>
+<pinref part="JP1" gate="B" pin="8"/>
+<wire x1="101.6" y1="139.7" x2="106.68" y2="142.24" width="0.1524" layer="91"/>
+</segment>
+</net>
+<net name="N$23" class="0">
+<segment>
+<pinref part="IC1" gate="G$1" pin="IOUT_LEFT_P"/>
+<pinref part="JP1" gate="B" pin="6"/>
+<wire x1="101.6" y1="142.24" x2="106.68" y2="139.7" width="0.1524" layer="91"/>
+</segment>
+</net>

Commit message: wip
Connections:
- net N$12: now also J1.1-TIP; no longer J1.2-TIP
- net N$27: now also J1.2-TIP; no longer J1.1-TIP
Other:
- moved on the sheet: J1
Changed lines of the file:
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@@
 <instance part="C7" gate="G$1" x="53.34" y="71.12"/>
 <instance part="C8" gate="G$1" x="53.34" y="58.42"/>
-<instance part="J1" gate="G$1" x="243.84" y="-20.32" rot="MR180"/>
-<instance part="GND10" gate="G$1" x="236.22" y="-22.86" rot="R270"/>
-<instance part="GND11" gate="G$1" x="236.22" y="-17.78" rot="R270"/>
+<instance part="J1" gate="G$1" x="246.38" y="-20.32"/>
+<instance part="GND10" gate="G$1" x="236.22" y="-17.78" rot="R270"/>
+<instance part="GND11" gate="G$1" x="236.22" y="-22.86" rot="R270"/>
 <instance part="IC4" gate="G$1" x="78.74" y="-53.34"/>
 <instance part="GND12" gate="G$1" x="63.5" y="-53.34" rot="R270"/>
@@
 <pinref part="J1" gate="G$1" pin="1-RING"/>
 <pinref part="GND10" gate="G$1" pin="GND"/>
-<wire x1="238.76" y1="-22.86" x2="243.84" y2="-22.86" width="0.1524" layer="91"/>
+<wire x1="238.76" y1="-17.78" x2="246.38" y2="-17.78" width="0.1524" layer="91"/>
 </segment>
 <segment>
 <pinref part="J1" gate="G$1" pin="2-RING"/>
 <pinref part="GND11" gate="G$1" pin="GND"/>
-<wire x1="238.76" y1="-17.78" x2="243.84" y2="-17.78" width="0.1524" layer="91"/>
+<wire x1="238.76" y1="-22.86" x2="246.38" y2="-22.86" width="0.1524" layer="91"/>
 </segment>
 <segment>
@@
 <pinref part="R13" gate="G$1" pin="2"/>
 <wire x1="210.82" y1="30.48" x2="218.44" y2="30.48" width="0.1524" layer="91"/>
-<wire x1="218.44" y1="30.48" x2="218.44" y2="-20.32" width="0.1524" layer="91"/>
-<pinref part="J1" gate="G$1" pin="2-TIP"/>
-<wire x1="243.84" y1="-20.32" x2="218.44" y2="-20.32" width="0.1524" layer="91"/>
+<wire x1="218.44" y1="30.48" x2="218.44" y2="-15.24" width="0.1524" layer="91"/>
+<pinref part="J1" gate="G$1" pin="1-TIP"/>
+<wire x1="246.38" y1="-15.24" x2="218.44" y2="-15.24" width="0.1524" layer="91"/>
 </segment>
 </net>
@@
 <pinref part="R29" gate="G$1" pin="2"/>
 <wire x1="210.82" y1="-53.34" x2="218.44" y2="-53.34" width="0.1524" layer="91"/>
-<wire x1="218.44" y1="-53.34" x2="218.44" y2="-25.4" width="0.1524" layer="91"/>
-<pinref part="J1" gate="G$1" pin="1-TIP"/>
-<wire x1="243.84" y1="-25.4" x2="218.44" y2="-25.4" width="0.1524" layer="91"/>
-</segment>
-</net>
+<wire x1="218.44" y1="-53.34" x2="218.44" y2="-20.32" width="0.1524" layer="91"/>
+<pinref part="J1" gate="G$1" pin="2-TIP"/>
+<wire x1="246.38" y1="-20.32" x2="218.44" y2="-20.32" width="0.1524" layer="91"/>
+</segment>
+</net>

Commit message: routed
Parts:
- removed H5, H6: MOUNT-HOLE3.2, holes:MOUNT-HOLE3.2
Changed lines of the file:
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@@
 <part name="H1" library="holes" deviceset="MOUNT-HOLE" device="3.2"/>
 <part name="H2" library="holes" deviceset="MOUNT-HOLE" device="3.2"/>
-<part name="H5" library="holes" deviceset="MOUNT-HOLE" device="3.2"/>
-<part name="H6" library="holes" deviceset="MOUNT-HOLE" device="3.2"/>
 <part name="JP1" library="jumper" deviceset="JP4Q" device=""/>
 <part name="R33" library="microbuilder" deviceset="RESISTOR" device="_0805" value="10K 0.1% or better (ERA-3AEB103V)"/>
@@
 <instance part="H1" gate="G$1" x="10.16" y="220.98"/>
 <instance part="H2" gate="G$1" x="10.16" y="215.9"/>
-<instance part="H5" gate="G$1" x="10.16" y="210.82"/>
-<instance part="H6" gate="G$1" x="15.24" y="213.36"/>
 <instance part="JP1" gate="B" x="114.3" y="137.16" rot="R90"/>
 <instance part="R33" gate="G$1" x="144.78" y="132.08"/>

Commit message: routed
Parts:
- added C52: 0.1uF, microbuilder:CAP_CERAMIC0603
- added OSC1: (no value), microbuilder:OSCILLATOR
- added R48: 0, microbuilder:RESISTOR_0805
Connections:
- new net N$32: OSC1.OUT, R48.1
- net 3.3V: now also C52.P$1, OSC1.VCC
- net GND: now also C52.P$2, OSC1.GND
- net I2S_MCK: now also R48.2
Changed lines of the file:
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@@
 <part name="C50" library="microbuilder" deviceset="CAP_CERAMIC" device="0603" value="0.1u"/>
 <part name="C51" library="microbuilder" deviceset="CAP_CERAMIC" device="1206" value="1uF 12065C105M4Z2A"/>
+<part name="OSC1" library="microbuilder" deviceset="OSCILLATOR" device=""/>
+<part name="C52" library="microbuilder" deviceset="CAP_CERAMIC" device="0603" value="0.1uF"/>
+<part name="U$45" library="microbuilder" deviceset="3.3V" device=""/>
+<part name="U$47" library="microbuilder" deviceset="GND" device=""/>
+<part name="R48" library="microbuilder" deviceset="RESISTOR" device="_0805" value="0"/>
 </parts>
 <sheets>
@@
 <instance part="C50" gate="G$1" x="149.86" y="-12.7"/>
 <instance part="C51" gate="G$1" x="243.84" y="154.94"/>
+<instance part="OSC1" gate="G$1" x="-12.7" y="83.82"/>
+<instance part="C52" gate="G$1" x="-33.02" y="83.82"/>
+<instance part="U$45" gate="G$1" x="-38.1" y="88.9" rot="R90"/>
+<instance part="U$47" gate="G$1" x="-38.1" y="78.74" rot="R270"/>
+<instance part="R48" gate="G$1" x="5.08" y="83.82"/>
 </instances>
 <busses>
@@
 <pinref part="C10" gate="G$1" pin="P$1"/>
 </segment>
+<segment>
+<pinref part="OSC1" gate="G$1" pin="GND"/>
+<pinref part="U$47" gate="G$1" pin="GND"/>
+<wire x1="-22.86" y1="78.74" x2="-33.02" y2="78.74" width="0.1524" layer="91"/>
+<junction x="-33.02" y="78.74"/>
+<wire x1="-33.02" y1="78.74" x2="-35.56" y2="78.74" width="0.1524" layer="91"/>
+<pinref part="C52" gate="G$1" pin="P$2"/>
+<wire x1="-33.02" y1="81.28" x2="-33.02" y2="78.74" width="0.1524" layer="91"/>
+</segment>
 </net>
 <net name="N$1" class="0">
@@
 <wire x1="-5.08" y1="162.56" x2="2.54" y2="162.56" width="0.1524" layer="91"/>
 </segment>
+<segment>
+<pinref part="OSC1" gate="G$1" pin="VCC"/>
+<wire x1="-22.86" y1="88.9" x2="-33.02" y2="88.9" width="0.1524" layer="91"/>
+<pinref part="U$45" gate="G$1" pin="3.3V"/>
+<pinref part="C52" gate="G$1" pin="P$1"/>
+<junction x="-33.02" y="88.9"/>
+<wire x1="-33.02" y1="88.9" x2="-35.56" y2="88.9" width="0.1524" layer="91"/>
+</segment>
 </net>
 <net name="DAC_VCC" class="0">
@@
 <label x="0" y="129.54" size="1.778" layer="95"/>
 <pinref part="SV1" gate="1" pin="9"/>
+</segment>
+<segment>
+<pinref part="R48" gate="G$1" pin="2"/>
+<wire x1="10.16" y1="83.82" x2="20.32" y2="83.82" width="0.1524" layer="91"/>
+<label x="15.24" y="83.82" size="1.778" layer="95"/>
 </segment>
 </net>
@@
 </segment>
 </net>
+<net name="N$32" class="0">
+<segment>
+<pinref part="R48" gate="G$1" pin="1"/>
+<pinref part="OSC1" gate="G$1" pin="OUT"/>
+<wire x1="0" y1="83.82" x2="-2.54" y2="83.82" width="0.1524" layer="91"/>
+</segment>
+</net>

Commit message: routed
Parts:
- OSC1: value (none) -> 12.288MHz C3391-12.288
Other:
- note added: "TODO: PCM5102? HEADPHONE AMP? 2xCAN CONNECTORS"
Changed lines of the file:
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@@
 <part name="C50" library="microbuilder" deviceset="CAP_CERAMIC" device="0603" value="0.1u"/>
 <part name="C51" library="microbuilder" deviceset="CAP_CERAMIC" device="1206" value="1uF 12065C105M4Z2A"/>
-<part name="OSC1" library="microbuilder" deviceset="OSCILLATOR" device=""/>
+<part name="OSC1" library="microbuilder" deviceset="OSCILLATOR" device="" value="12.288MHz C3391-12.288"/>
 <part name="C52" library="microbuilder" deviceset="CAP_CERAMIC" device="0603" value="0.1uF"/>
 <part name="U$45" library="microbuilder" deviceset="3.3V" device=""/>
@@
 NEED TO VERIFY TIP/RING</text>
 <text x="241.3" y="-2.54" size="1.778" layer="91">NEED TO VERIFY LEFT/RIGHT</text>
+<text x="-17.78" y="96.52" size="1.778" layer="91">TODO:
+PCM5102?
+HEADPHONE AMP?
+2xCAN CONNECTORS</text>
 </plain>
 <instances>
