File: phi-brain4ch/phi-dac.sch (EAGLE design)
At the start: 148 parts, among them IC1 PCM1792A, IC10 LM317, IC11 LM337, IC2 OPA1632D, IC3 OPA1632D, IC4 OPA1632D, IC6 OPA1632D, IC7 REG1117-5, IC8 ADP3301ARZ-3.3, IC9 MGJ2D121515SC, J1 CUI-RCJ-2123, J5 DC21P

Commit message: wip
Parts:
- added C56: 10uF, microbuilder:CAP_CERAMIC1206
- added C57: 0.1uF, microbuilder:CAP_CERAMIC0603
- added C58: 22uF GRM21BR61E226ME44L, microbuilder:CAP_CERAMIC_0805
- added IC12: (no value), keves:MURATA_OKR-T/10-W12-C
- added L7: ILHB1206ER601V, SparkFun-Passives:INDUCTOR1206H*
- added R49: 270 270ohms 25ppm 0.5% (ERA-6AED271V), microbuilder:RESISTOR_0805
- added X1, X2: 04-JST-B4B-XH-A, bt_con-jst-xh:04-JST-B4B-XH-A
- L1, L2, L3, L4, L5, L6: value BLM31PG601SN1L -> ILHB1206ER601V
Connections:
- new net CAN_H: X1-3.1, X2-3.1
- new net CAN_L: X1-2.1, X2-2.1
- new net N$31: L7.2, X1-1.1, X2-1.1
- new net N$33: IC12.TRIM, R49.1
- new net N$34: C56.P$1, C57.P$1, IC12.OUT, L7.1
- net +12V: now also C58.P$1, IC12.IN
- net GND: now also C56.P$2, C57.P$2, C58.P$2, IC12.GND, R49.2, X1-4.1, X2-4.1
Other:
- note added: "TODO: PCM5102? HEADPHONE AMP? 2xCAN CONNECTORS REVERSE POLARITY? FUSE?"
- note removed: "TODO: PCM5102? HEADPHONE AMP? 2xCAN CONNECTORS"
Changed lines of the file:
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@@
 <part name="C17" library="microbuilder" deviceset="CAP_CERAMIC" device="0603" value="0.1uF"/>
 <part name="U$16" library="microbuilder" deviceset="GND" device=""/>
-<part name="L1" library="SparkFun-Passives" deviceset="INDUCTOR" device="H*" technology="1206" value="BLM31PG601SN1L"/>
+<part name="L1" library="SparkFun-Passives" deviceset="INDUCTOR" device="H*" technology="1206" value="ILHB1206ER601V"/>
 <part name="U$15" library="microbuilder" deviceset="3.3V" device=""/>
 <part name="GND22" library="microbuilder" deviceset="GND" device=""/>
@@
 <part name="GND25" library="microbuilder" deviceset="GND" device=""/>
 <part name="C18" library="microbuilder" deviceset="CAP_CERAMIC" device="0603" value="0.1uF"/>
-<part name="L2" library="SparkFun-Passives" deviceset="INDUCTOR" device="H*" technology="1206" value="BLM31PG601SN1L"/>
+<part name="L2" library="SparkFun-Passives" deviceset="INDUCTOR" device="H*" technology="1206" value="ILHB1206ER601V"/>
 <part name="U$17" library="microbuilder" deviceset="GND" device=""/>
 <part name="C19" library="microbuilder" deviceset="CAP_CERAMIC" device="1206" value="10uF"/>
 <part name="U$18" library="microbuilder" deviceset="GND" device=""/>
 <part name="C20" library="microbuilder" deviceset="CAP_CERAMIC" device="0603" value="0.1uF"/>
-<part name="L3" library="SparkFun-Passives" deviceset="INDUCTOR" device="H*" technology="1206" value="BLM31PG601SN1L"/>
+<part name="L3" library="SparkFun-Passives" deviceset="INDUCTOR" device="H*" technology="1206" value="ILHB1206ER601V"/>
 <part name="U$19" library="microbuilder" deviceset="GND" device=""/>
 <part name="C21" library="microbuilder" deviceset="CAP_CERAMIC" device="1206" value="10uF"/>
 <part name="U$20" library="microbuilder" deviceset="GND" device=""/>
 <part name="C22" library="microbuilder" deviceset="CAP_CERAMIC" device="0603" value="0.1uF"/>
-<part name="L4" library="SparkFun-Passives" deviceset="INDUCTOR" device="H*" technology="1206" value="BLM31PG601SN1L"/>
+<part name="L4" library="SparkFun-Passives" deviceset="INDUCTOR" device="H*" technology="1206" value="ILHB1206ER601V"/>
 <part name="U$21" library="microbuilder" deviceset="GND" device=""/>
 <part name="C23" library="microbuilder" deviceset="CAP_CERAMIC" device="1206" value="10uF"/>
@@
 <part name="D2" library="microbuilder" deviceset="DIODE" device="SOD-323"/>
 <part name="U$27" library="microbuilder" deviceset="GND" device=""/>
-<part name="L5" library="SparkFun-Passives" deviceset="INDUCTOR" device="H*" technology="1206" value="BLM31PG601SN1L"/>
+<part name="L5" library="SparkFun-Passives" deviceset="INDUCTOR" device="H*" technology="1206" value="ILHB1206ER601V"/>
 <part name="APWR_EN" library="jumper" deviceset="JP2QE" device=""/>
 <part name="U$28" library="microbuilder" deviceset="AVCC" device=""/>
@@
 <part name="C38" library="microbuilder" deviceset="CAP_CERAMIC" device="0603" value="10uF"/>
 <part name="D4" library="microbuilder" deviceset="DIODE" device="SOD-323"/>
-<part name="L6" library="SparkFun-Passives" deviceset="INDUCTOR" device="H*" technology="1206" value="BLM31PG601SN1L"/>
+<part name="L6" library="SparkFun-Passives" deviceset="INDUCTOR" device="H*" technology="1206" value="ILHB1206ER601V"/>
 <part name="U$30" library="microbuilder" deviceset="AVDD" device=""/>
 <part name="J5" library="keves" deviceset="DC21P" device=""/>
@@
 <part name="U$47" library="microbuilder" deviceset="GND" device=""/>
 <part name="R48" library="microbuilder" deviceset="RESISTOR" device="_0805" value="0"/>
+<part name="IC12" library="keves" deviceset="MURATA_OKR-T/10-W12-C" device=""/>
+<part name="X2" library="bt_con-jst-xh" deviceset="04-JST" device="-B4B-XH-A"/>
+<part name="X1" library="bt_con-jst-xh" deviceset="04-JST" device="-B4B-XH-A"/>
+<part name="U$48" library="microbuilder" deviceset="GND" device=""/>
+<part name="R49" library="microbuilder" deviceset="RESISTOR" device="_0805" value="270 270ohms 25ppm 0.5%  (ERA-6AED271V)"/>
+<part name="L7" library="SparkFun-Passives" deviceset="INDUCTOR" device="H*" technology="1206" value="ILHB1206ER601V"/>
+<part name="C56" library="microbuilder" deviceset="CAP_CERAMIC" device="1206" value="10uF"/>
+<part name="C57" library="microbuilder" deviceset="CAP_CERAMIC" device="0603" value="0.1uF"/>
+<part name="C58" library="microbuilder" deviceset="CAP_CERAMIC" device="_0805" value="22uF GRM21BR61E226ME44L"/>
 </parts>
 <sheets>
@@
 NEED TO VERIFY TIP/RING</text>
 <text x="241.3" y="-2.54" size="1.778" layer="91">NEED TO VERIFY LEFT/RIGHT</text>
-<text x="-17.78" y="96.52" size="1.778" layer="91">TODO:
+<text x="-60.96" y="124.46" size="1.778" layer="91">TODO:
 PCM5102?
 HEADPHONE AMP?
-2xCAN CONNECTORS</text>
+2xCAN CONNECTORS
+REVERSE POLARITY? FUSE?</text>
 </plain>
 <instances>
@@
 <instance part="U$47" gate="G$1" x="-38.1" y="78.74" rot="R270"/>
 <instance part="R48" gate="G$1" x="5.08" y="83.82"/>
+<instance part="IC12" gate="G$1" x="101.6" y="271.78"/>
+<instance part="X2" gate="-1" x="180.34" y="271.78"/>
+<instance part="X2" gate="-2" x="180.34" y="269.24"/>
+<instance part="X2" gate="-3" x="180.34" y="266.7"/>
+<instance part="X2" gate="-4" x="180.34" y="264.16"/>
+<instance part="X1" gate="-1" x="165.1" y="271.78"/>
+<instance part="X1" gate="-2" x="165.1" y="269.24"/>
+<instance part="X1" gate="-3" x="165.1" y="266.7"/>
+<instance part="X1" gate="-4" x="165.1" y="264.16"/>
+<instance part="U$48" gate="G$1" x="101.6" y="254"/>
+<instance part="R49" gate="G$1" x="114.3" y="261.62"/>
+<instance part="L7" gate="G$1" x="152.4" y="271.78" rot="R90"/>
+<instance part="C56" gate="G$1" x="129.54" y="266.7"/>
+<instance part="C57" gate="G$1" x="139.7" y="266.7"/>
+<instance part="C58" gate="G$1" x="63.5" y="264.16"/>
 </instances>
 <busses>
@@
 <wire x1="-33.02" y1="81.28" x2="-33.02" y2="78.74" width="0.1524" layer="91"/>
 </segment>
+<segment>
+<wire x1="154.94" y1="264.16" x2="160.02" y2="264.16" width="0.1524" layer="91"/>
+<pinref part="X2" gate="-4" pin="1"/>
+<wire x1="160.02" y1="264.16" x2="175.26" y2="264.16" width="0.1524" layer="91"/>
+<pinref part="X1" gate="-4" pin="1"/>
+<junction x="160.02" y="264.16"/>
+<wire x1="154.94" y1="264.16" x2="154.94" y2="256.54" width="0.1524" layer="91"/>
+<pinref part="U$48" gate="G$1" pin="GND"/>
+<wire x1="154.94" y1="256.54" x2="139.7" y2="256.54" width="0.1524" layer="91"/>
+<pinref part="IC12" gate="G$1" pin="GND"/>
+<wire x1="139.7" y1="256.54" x2="129.54" y2="256.54" width="0.1524" layer="91"/>
+<wire x1="129.54" y1="256.54" x2="119.38" y2="256.54" width="0.1524" layer="91"/>
+<wire x1="119.38" y1="256.54" x2="101.6" y2="256.54" width="0.1524" layer="91"/>
+<wire x1="101.6" y1="261.62" x2="101.6" y2="256.54" width="0.1524" layer="91"/>
+<junction x="101.6" y="256.54"/>
+<pinref part="R49" gate="G$1" pin="2"/>
+<wire x1="119.38" y1="261.62" x2="119.38" y2="256.54" width="0.1524" layer="91"/>
+<pinref part="C57" gate="G$1" pin="P$2"/>
+<wire x1="139.7" y1="264.16" x2="139.7" y2="256.54" width="0.1524" layer="91"/>
+<junction x="139.7" y="256.54"/>
+<pinref part="C56" gate="G$1" pin="P$2"/>
+<wire x1="129.54" y1="264.16" x2="129.54" y2="256.54" width="0.1524" layer="91"/>
+<junction x="129.54" y="256.54"/>
+<junction x="119.38" y="256.54"/>
+<pinref part="C58" gate="G$1" pin="P$2"/>
+<wire x1="63.5" y1="261.62" x2="63.5" y2="256.54" width="0.1524" layer="91"/>
+<wire x1="63.5" y1="256.54" x2="101.6" y2="256.54" width="0.1524" layer="91"/>
+</segment>
 </net>
 <net name="N$1" class="0">
@@
 <label x="2.54" y="180.34" size="1.778" layer="95" rot="R180"/>
 </segment>
+<segment>
+<pinref part="IC12" gate="G$1" pin="IN"/>
+<wire x1="83.82" y1="271.78" x2="63.5" y2="271.78" width="0.1524" layer="91"/>
+<label x="66.04" y="271.78" size="1.778" layer="95"/>
+<pinref part="C58" gate="G$1" pin="P$1"/>
+<wire x1="63.5" y1="271.78" x2="55.88" y2="271.78" width="0.1524" layer="91"/>
+<wire x1="63.5" y1="269.24" x2="63.5" y2="271.78" width="0.1524" layer="91"/>
+<junction x="63.5" y="271.78"/>
+</segment>
 </net>
 <net name="N$49" class="0">
@@
 </segment>
 </net>
+<net name="N$31" class="0">
+<segment>
+<pinref part="X2" gate="-1" pin="1"/>
+<wire x1="160.02" y1="271.78" x2="175.26" y2="271.78" width="0.1524" layer="91"/>
+<pinref part="X1" gate="-1" pin="1"/>
+<pinref part="L7" gate="G$1" pin="2"/>
+<junction x="160.02" y="271.78"/>
+</segment>
+</net>
+<net name="CAN_H" class="0">
+<segment>
+<wire x1="175.26" y1="266.7" x2="160.02" y2="266.7" width="0.1524" layer="91"/>
+<pinref part="X2" gate="-3" pin="1"/>
+<pinref part="X1" gate="-3" pin="1"/>
+</segment>
+</net>
+<net name="CAN_L" class="0">
+<segment>
+<wire x1="175.26" y1="269.24" x2="160.02" y2="269.24" width="0.1524" layer="91"/>
+<pinref part="X2" gate="-2" pin="1"/>
+<pinref part="X1" gate="-2" pin="1"/>
+</segment>
+</net>
+<net name="N$33" class="0">
+<segment>
+<pinref part="R49" gate="G$1" pin="1"/>
+<pinref part="IC12" gate="G$1" pin="TRIM"/>
+<wire x1="109.22" y1="261.62" x2="106.68" y2="261.62" width="0.1524" layer="91"/>
+</segment>
+</net>
+<net name="N$34" class="0">
+<segment>
+<pinref part="L7" gate="G$1" pin="1"/>
+<wire x1="144.78" y1="271.78" x2="139.7" y2="271.78" width="0.1524" layer="91"/>
+<pinref part="IC12" gate="G$1" pin="OUT"/>
+<pinref part="C56" gate="G$1" pin="P$1"/>
+<wire x1="139.7" y1="271.78" x2="129.54" y2="271.78" width="0.1524" layer="91"/>
+<wire x1="129.54" y1="271.78" x2="121.92" y2="271.78" width="0.1524" layer="91"/>
+<junction x="129.54" y="271.78"/>
+<pinref part="C57" gate="G$1" pin="P$1"/>
+<junction x="139.7" y="271.78"/>
+</segment>
+</net>

Commit message: wip
Parts:
- removed R35, R36, R37, R38: 50, microbuilder:RESISTOR_0805
Connections:
- removed net N$43: IC1.BCK, R36.2
- removed net N$44: IC1.DATA, R37.2
- removed net N$45: IC1.LRCK, R38.2
- removed net N$48: IC1.SCK, R35.2
- net I2S_BCK: now also IC1.BCK; no longer R36.1
- net I2S_DATA: now also IC1.DATA; no longer R37.1
- net I2S_LRCK: now also IC1.LRCK; no longer R38.1
- net I2S_MCK: now also IC1.SCK; no longer R35.1
Changed lines of the file:
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@@
 <part name="U$23" library="microbuilder" deviceset="3.3V" device=""/>
 <part name="U$24" library="microbuilder" deviceset="GND" device=""/>
-<part name="R35" library="microbuilder" deviceset="RESISTOR" device="_0805" value="50"/>
-<part name="R36" library="microbuilder" deviceset="RESISTOR" device="_0805" value="50"/>
-<part name="R37" library="microbuilder" deviceset="RESISTOR" device="_0805" value="50"/>
-<part name="R38" library="microbuilder" deviceset="RESISTOR" device="_0805" value="50"/>
 <part name="IC9" library="keves" deviceset="MURATA-MGJ2" device="" value="MGJ2D121515SC"/>
 <part name="U$25" library="microbuilder" deviceset="GND" device=""/>
@@
 <instance part="U$23" gate="G$1" x="40.64" y="142.24" rot="R90"/>
 <instance part="U$24" gate="G$1" x="55.88" y="129.54" rot="R270"/>
-<instance part="R35" gate="G$1" x="50.8" y="109.22"/>
-<instance part="R36" gate="G$1" x="50.8" y="106.68"/>
-<instance part="R37" gate="G$1" x="50.8" y="104.14"/>
-<instance part="R38" gate="G$1" x="50.8" y="101.6"/>
 <instance part="IC9" gate="G$1" x="104.14" y="172.72"/>
 <instance part="U$25" gate="G$1" x="71.12" y="162.56" rot="R270"/>
@@
 </segment>
 </net>
-<net name="N$43" class="0">
-<segment>
-<pinref part="IC1" gate="G$1" pin="BCK"/>
-<pinref part="R36" gate="G$1" pin="2"/>
-<wire x1="55.88" y1="106.68" x2="60.96" y2="106.68" width="0.1524" layer="91"/>
-</segment>
-</net>
-<net name="N$44" class="0">
-<segment>
-<pinref part="IC1" gate="G$1" pin="DATA"/>
-<pinref part="R37" gate="G$1" pin="2"/>
-<wire x1="55.88" y1="104.14" x2="60.96" y2="104.14" width="0.1524" layer="91"/>
-</segment>
-</net>
-<net name="N$45" class="0">
-<segment>
-<pinref part="IC1" gate="G$1" pin="LRCK"/>
-<pinref part="R38" gate="G$1" pin="2"/>
-<wire x1="55.88" y1="101.6" x2="60.96" y2="101.6" width="0.1524" layer="91"/>
-</segment>
-</net>
-<net name="N$48" class="0">
-<segment>
-<pinref part="IC1" gate="G$1" pin="SCK"/>
-<pinref part="R35" gate="G$1" pin="2"/>
-<wire x1="55.88" y1="109.22" x2="60.96" y2="109.22" width="0.1524" layer="91"/>
-</segment>
-</net>
 <net name="I2S_MCK" class="0">
 <segment>
-<pinref part="R35" gate="G$1" pin="1"/>
-<wire x1="45.72" y1="109.22" x2="20.32" y2="109.22" width="0.1524" layer="91"/>
+<wire x1="60.96" y1="109.22" x2="20.32" y2="109.22" width="0.1524" layer="91"/>
 <wire x1="20.32" y1="109.22" x2="20.32" y2="129.54" width="0.1524" layer="91"/>
 <wire x1="20.32" y1="129.54" x2="-10.16" y2="129.54" width="0.1524" layer="91"/>
 <label x="0" y="129.54" size="1.778" layer="95"/>
 <pinref part="SV1" gate="1" pin="9"/>
+<pinref part="IC1" gate="G$1" pin="SCK"/>
 </segment>
 <segment>
@@
 <net name="I2S_BCK" class="0">
 <segment>
-<pinref part="R36" gate="G$1" pin="1"/>
-<wire x1="45.72" y1="106.68" x2="17.78" y2="106.68" width="0.1524" layer="91"/>
+<wire x1="60.96" y1="106.68" x2="17.78" y2="106.68" width="0.1524" layer="91"/>
 <wire x1="17.78" y1="106.68" x2="17.78" y2="127" width="0.1524" layer="91"/>
 <wire x1="17.78" y1="127" x2="-10.16" y2="127" width="0.1524" layer="91"/>
 <label x="0" y="127" size="1.778" layer="95"/>
 <pinref part="SV1" gate="1" pin="7"/>
+<pinref part="IC1" gate="G$1" pin="BCK"/>
 </segment>
 </net>
 <net name="I2S_DATA" class="0">
 <segment>
-<pinref part="R37" gate="G$1" pin="1"/>
-<wire x1="45.72" y1="104.14" x2="15.24" y2="104.14" width="0.1524" layer="91"/>
+<wire x1="60.96" y1="104.14" x2="15.24" y2="104.14" width="0.1524" layer="91"/>
 <wire x1="15.24" y1="104.14" x2="15.24" y2="124.46" width="0.1524" layer="91"/>
 <wire x1="15.24" y1="124.46" x2="-10.16" y2="124.46" width="0.1524" layer="91"/>
 <label x="0" y="124.46" size="1.778" layer="95"/>
 <pinref part="SV1" gate="1" pin="5"/>
+<pinref part="IC1" gate="G$1" pin="DATA"/>
 </segment>
 </net>
 <net name="I2S_LRCK" class="0">
 <segment>
-<pinref part="R38" gate="G$1" pin="1"/>
-<wire x1="45.72" y1="101.6" x2="12.7" y2="101.6" width="0.1524" layer="91"/>
+<wire x1="60.96" y1="101.6" x2="12.7" y2="101.6" width="0.1524" layer="91"/>
 <wire x1="12.7" y1="101.6" x2="12.7" y2="121.92" width="0.1524" layer="91"/>
 <wire x1="12.7" y1="121.92" x2="-10.16" y2="121.92" width="0.1524" layer="91"/>
 <label x="0" y="121.92" size="1.778" layer="95"/>
 <pinref part="SV1" gate="1" pin="3"/>
-</segment>
-</net>
+<pinref part="IC1" gate="G$1" pin="LRCK"/>
+</segment>
+</net>
