File: phi-brain4ch/phi-dac.sch (EAGLE design)
At the start: 152 parts, among them IC1 PCM1792A, IC10 LM317, IC11 LM337, IC2 OPA1632D, IC3 OPA1632D, IC4 OPA1632D, IC6 OPA1632D, IC7 REG1117-5, IC8 ADP3301ARZ-3.3, IC9 MGJ2D121515SC, J1 CUI-RCJ-2123, J5 DC21P, X1 04-JST-B4B-XH-A, X2 04-JST-B4B-XH-A

Commit message: wip
Parts:
- added C59, C61, C68, C69: 0.1u, microbuilder:CAP_CERAMIC0603
- added C60, C66, C67, C70: 10uF, microbuilder:CAP_CERAMIC1206
- added C71, C72: 2.2uF, microbuilder:CAP_CERAMIC_0805
- added C73, C74: 2.2nF, microbuilder:CAP_CERAMIC_0805
- added IC13: PCM5102, PCM5102:PCM5102
- added L8, L9: ILHB1206ER601V, SparkFun-Passives:INDUCTOR1206H*
- added R35, R36: 470, microbuilder:RESISTOR_0805
Connections:
- new net HP_VCC: C69.P$1, C70.P$1, IC13.CPVDD, IC13.XSMT, L8.1, L9.2
- new net I2S_DATA2: IC13.DIN, SV1.1
- new net N$43: C59.P$1, C60.P$1, IC13.AVDD, L8.2
- new net N$44: C67.P$2, C68.P$2, IC13.LDOO
- new net N$45: C71.P$1, IC13.CAPP
- new net N$48: C61.P$1, C66.P$1, IC13.DVDD, L9.1
- new net N$64: C71.P$2, IC13.CAPM
- new net N$65: C72.P$2, IC13.VNEG
- new net N$67: IC13.OUTL, R35.2
- new net N$68: IC13.OUTR, R36.2
- new net N$69: C74.P$2, R36.1
- new net N$70: C73.P$1, R35.1
- net GND: now also C59.P$2, C60.P$2, C61.P$2, C66.P$2, C67.P$1, C68.P$1, C69.P$2, C70.P$2, C72.P$1, C73.P$2, C74.P$1, IC13.AGND, IC13.CPGND, IC13.DEMP, IC13.DGND, IC13.FLT, IC13.FMT; no longer SV1.1
- net I2S_BCK: now also IC13.BCK
- net I2S_LRCK: now also IC13.LRCK
- net I2S_MCK: now also IC13.SCK

Commit message: wip
Parts:
- added C75: 2.2uF (EMK107BB7225KA-T), microbuilder:CAP_CERAMIC0603
- added C76: 0.01uF, microbuilder:CAP_CERAMIC0603
- added C77: 10uF, microbuilder:CAP_CERAMIC1206
- added HP_EN: (no value), microbuilder:HEADER-1X2
- added IC14: ADP3301ARZ-3.3, keves:ADP3301
- added X3: 04-JST-B4B-XH-A, bt_con-jst-xh:04-JST-B4B-XH-A
Connections:
- new net N$66: C76.P$1, IC14.NR
- new net N$71: C76.P$2, C77.P$2, HP_EN.1, IC14.OUT1, IC14.OUT2
- net +12V: now also C75.P$2, IC14.IN1, IC14.IN2, IC14.SD, X3-1.1
- net GND: now also C75.P$1, C77.P$1, IC14.GND, X3-2.1
- net HP_VCC: now also HP_EN.2
- net N$69: now also X3-4.1
- net N$70: now also X3-3.1
Changed lines of the file:
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@@
 <part name="U$55" library="microbuilder" deviceset="GND" device=""/>
 <part name="U$56" library="microbuilder" deviceset="GND" device=""/>
+<part name="X3" library="bt_con-jst-xh" deviceset="04-JST" device="-B4B-XH-A"/>
+<part name="U$57" library="microbuilder" deviceset="GND" device=""/>
+<part name="IC14" library="keves" deviceset="ADP3301" device="" value="ADP3301ARZ-3.3"/>
+<part name="U$58" library="microbuilder" deviceset="GND" device=""/>
+<part name="C75" library="microbuilder" deviceset="CAP_CERAMIC" device="0603" value="2.2uF (EMK107BB7225KA-T)"/>
+<part name="U$59" library="microbuilder" deviceset="GND" device=""/>
+<part name="C76" library="microbuilder" deviceset="CAP_CERAMIC" device="0603" value="0.01uF"/>
+<part name="C77" library="microbuilder" deviceset="CAP_CERAMIC" device="1206" value="10uF"/>
+<part name="U$61" library="microbuilder" deviceset="GND" device=""/>
+<part name="HP_EN" library="microbuilder" deviceset="HEADER-1X2" device=""/>
 </parts>
 <sheets>
@@
 <instance part="U$55" gate="G$1" x="-129.54" y="152.4"/>
 <instance part="U$56" gate="G$1" x="-129.54" y="175.26" rot="R180"/>
+<instance part="X3" gate="-1" x="-157.48" y="170.18" rot="MR0"/>
+<instance part="X3" gate="-2" x="-157.48" y="167.64" rot="MR0"/>
+<instance part="X3" gate="-3" x="-157.48" y="165.1" rot="MR0"/>
+<instance part="X3" gate="-4" x="-157.48" y="162.56" rot="MR0"/>
+<instance part="U$57" gate="G$1" x="-147.32" y="167.64" rot="R90"/>
+<instance part="IC14" gate="G$1" x="-139.7" y="185.42"/>
+<instance part="U$58" gate="G$1" x="-167.64" y="203.2" rot="R270"/>
+<instance part="C75" gate="G$1" x="-170.18" y="195.58" rot="R180"/>
+<instance part="U$59" gate="G$1" x="-170.18" y="185.42"/>
+<instance part="C76" gate="G$1" x="-129.54" y="203.2" rot="R90"/>
+<instance part="C77" gate="G$1" x="-127" y="195.58" rot="R180"/>
+<instance part="U$61" gate="G$1" x="-127" y="187.96"/>
+<instance part="HP_EN" gate="G$1" x="-101.6" y="200.66" rot="R90"/>
 </instances>
 <busses>
@@
 <pinref part="U$56" gate="G$1" pin="GND"/>
 </segment>
+<segment>
+<pinref part="X3" gate="-2" pin="1"/>
+<pinref part="U$57" gate="G$1" pin="GND"/>
+<wire x1="-149.86" y1="167.64" x2="-152.4" y2="167.64" width="0.1524" layer="91"/>
+</segment>
+<segment>
+<pinref part="IC14" gate="G$1" pin="GND"/>
+<pinref part="U$58" gate="G$1" pin="GND"/>
+<wire x1="-165.1" y1="203.2" x2="-162.56" y2="203.2" width="0.1524" layer="91"/>
+</segment>
+<segment>
+<pinref part="C75" gate="G$1" pin="P$1"/>
+<pinref part="U$59" gate="G$1" pin="GND"/>
+<wire x1="-170.18" y1="187.96" x2="-170.18" y2="190.5" width="0.1524" layer="91"/>
+</segment>
+<segment>
+<pinref part="C77" gate="G$1" pin="P$1"/>
+<pinref part="U$61" gate="G$1" pin="GND"/>
+</segment>
 </net>
 <net name="N$1" class="0">
@@
 <junction x="63.5" y="271.78"/>
 </segment>
+<segment>
+<pinref part="X3" gate="-1" pin="1"/>
+<wire x1="-152.4" y1="170.18" x2="-144.78" y2="170.18" width="0.1524" layer="91"/>
+<label x="-147.32" y="170.18" size="1.778" layer="95"/>
+</segment>
+<segment>
+<pinref part="IC14" gate="G$1" pin="IN2"/>
+<pinref part="IC14" gate="G$1" pin="IN1"/>
+<wire x1="-162.56" y1="195.58" x2="-162.56" y2="198.12" width="0.1524" layer="91"/>
+<wire x1="-162.56" y1="198.12" x2="-170.18" y2="198.12" width="0.1524" layer="91"/>
+<pinref part="C75" gate="G$1" pin="P$2"/>
+<wire x1="-170.18" y1="198.12" x2="-172.72" y2="198.12" width="0.1524" layer="91"/>
+<junction x="-170.18" y="198.12"/>
+<pinref part="IC14" gate="G$1" pin="SD"/>
+<wire x1="-162.56" y1="190.5" x2="-162.56" y2="195.58" width="0.1524" layer="91"/>
+<label x="-175.26" y="198.12" size="1.778" layer="95"/>
+<junction x="-162.56" y="195.58"/>
+<junction x="-162.56" y="198.12"/>
+</segment>
 </net>
 <net name="N$49" class="0">
@@
 <wire x1="-88.9" y1="180.34" x2="-88.9" y2="170.18" width="0.1524" layer="91"/>
 </segment>
+<segment>
+<pinref part="HP_EN" gate="G$1" pin="2"/>
+<wire x1="-101.6" y1="198.12" x2="-86.36" y2="198.12" width="0.1524" layer="91"/>
+<label x="-91.44" y="198.12" size="1.778" layer="95"/>
+</segment>
 </net>
 <net name="N$43" class="0">
@@
 <wire x1="-124.46" y1="162.56" x2="-129.54" y2="162.56" width="0.1524" layer="91"/>
 <pinref part="C74" gate="G$1" pin="P$2"/>
-<wire x1="-129.54" y1="162.56" x2="-134.62" y2="162.56" width="0.1524" layer="91"/>
+<wire x1="-129.54" y1="162.56" x2="-152.4" y2="162.56" width="0.1524" layer="91"/>
 <junction x="-129.54" y="162.56"/>
+<pinref part="X3" gate="-4" pin="1"/>
 </segment>
 </net>
@@
 <wire x1="-121.92" y1="165.1" x2="-129.54" y2="165.1" width="0.1524" layer="91"/>
 <pinref part="C73" gate="G$1" pin="P$1"/>
-<wire x1="-129.54" y1="165.1" x2="-134.62" y2="165.1" width="0.1524" layer="91"/>
+<wire x1="-129.54" y1="165.1" x2="-152.4" y2="165.1" width="0.1524" layer="91"/>
 <junction x="-129.54" y="165.1"/>
-</segment>
-</net>
+<pinref part="X3" gate="-3" pin="1"/>
+</segment>
+</net>
+<net name="N$66" class="0">
+<segment>
+<pinref part="C76" gate="G$1" pin="P$1"/>
+<pinref part="IC14" gate="G$1" pin="NR"/>
+<wire x1="-134.62" y1="203.2" x2="-137.16" y2="203.2" width="0.1524" layer="91"/>
+</segment>
+</net>
+<net name="N$71" class="0">
+<segment>
+<pinref part="IC14" gate="G$1" pin="OUT1"/>
+<junction x="-137.16" y="198.12"/>
+<pinref part="IC14" gate="G$1" pin="OUT2"/>
+<wire x1="-137.16" y1="195.58" x2="-137.16" y2="198.12" width="0.1524" layer="91"/>
+<pinref part="C76" gate="G$1" pin="P$2"/>
+<wire x1="-127" y1="198.12" x2="-137.16" y2="198.12" width="0.1524" layer="91"/>
+<wire x1="-127" y1="203.2" x2="-127" y2="198.12" width="0.1524" layer="91"/>
+<junction x="-127" y="198.12"/>
+<pinref part="C77" gate="G$1" pin="P$2"/>
+<pinref part="HP_EN" gate="G$1" pin="1"/>
+<wire x1="-127" y1="198.12" x2="-104.14" y2="198.12" width="0.1524" layer="91"/>
+</segment>
+</net>

Commit message: with headphone wip
Parts:
- renumbered X3 to HP
Connections:
- net N$69: now also HP-3.1; no longer HP-4.1
- net N$70: now also HP-4.1; no longer HP-3.1
Changed lines of the file:
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@@
 <part name="U$55" library="microbuilder" deviceset="GND" device=""/>
 <part name="U$56" library="microbuilder" deviceset="GND" device=""/>
-<part name="X3" library="bt_con-jst-xh" deviceset="04-JST" device="-B4B-XH-A"/>
+<part name="HP" library="bt_con-jst-xh" deviceset="04-JST" device="-B4B-XH-A"/>
 <part name="U$57" library="microbuilder" deviceset="GND" device=""/>
 <part name="IC14" library="keves" deviceset="ADP3301" device="" value="ADP3301ARZ-3.3"/>
@@
 <instance part="U$55" gate="G$1" x="-129.54" y="152.4"/>
 <instance part="U$56" gate="G$1" x="-129.54" y="175.26" rot="R180"/>
-<instance part="X3" gate="-1" x="-157.48" y="170.18" rot="MR0"/>
-<instance part="X3" gate="-2" x="-157.48" y="167.64" rot="MR0"/>
-<instance part="X3" gate="-3" x="-157.48" y="165.1" rot="MR0"/>
-<instance part="X3" gate="-4" x="-157.48" y="162.56" rot="MR0"/>
+<instance part="HP" gate="-1" x="-157.48" y="170.18" rot="MR0"/>
+<instance part="HP" gate="-2" x="-157.48" y="167.64" rot="MR0"/>
+<instance part="HP" gate="-3" x="-157.48" y="165.1" rot="MR0"/>
+<instance part="HP" gate="-4" x="-157.48" y="162.56" rot="MR0"/>
 <instance part="U$57" gate="G$1" x="-147.32" y="167.64" rot="R90"/>
 <instance part="IC14" gate="G$1" x="-139.7" y="185.42"/>
@@
 </segment>
 <segment>
-<pinref part="X3" gate="-2" pin="1"/>
+<pinref part="HP" gate="-2" pin="1"/>
 <pinref part="U$57" gate="G$1" pin="GND"/>
 <wire x1="-149.86" y1="167.64" x2="-152.4" y2="167.64" width="0.1524" layer="91"/>
@@
 </segment>
 <segment>
-<pinref part="X3" gate="-1" pin="1"/>
+<pinref part="HP" gate="-1" pin="1"/>
 <wire x1="-152.4" y1="170.18" x2="-144.78" y2="170.18" width="0.1524" layer="91"/>
 <label x="-147.32" y="170.18" size="1.778" layer="95"/>
@@
 <wire x1="-124.46" y1="162.56" x2="-129.54" y2="162.56" width="0.1524" layer="91"/>
 <pinref part="C74" gate="G$1" pin="P$2"/>
-<wire x1="-129.54" y1="162.56" x2="-152.4" y2="162.56" width="0.1524" layer="91"/>
-<junction x="-129.54" y="162.56"/>
-<pinref part="X3" gate="-4" pin="1"/>
+<pinref part="HP" gate="-3" pin="1"/>
+<wire x1="-152.4" y1="165.1" x2="-139.7" y2="165.1" width="0.1524" layer="91"/>
+<wire x1="-139.7" y1="165.1" x2="-137.16" y2="162.56" width="0.1524" layer="91"/>
+<wire x1="-137.16" y1="162.56" x2="-129.54" y2="162.56" width="0.1524" layer="91"/>
 </segment>
 </net>
@@
 <wire x1="-121.92" y1="165.1" x2="-129.54" y2="165.1" width="0.1524" layer="91"/>
 <pinref part="C73" gate="G$1" pin="P$1"/>
-<wire x1="-129.54" y1="165.1" x2="-152.4" y2="165.1" width="0.1524" layer="91"/>
-<junction x="-129.54" y="165.1"/>
-<pinref part="X3" gate="-3" pin="1"/>
-</segment>
-</net>
+<wire x1="-129.54" y1="165.1" x2="-137.16" y2="165.1" width="0.1524" layer="91"/>
+<wire x1="-137.16" y1="165.1" x2="-139.7" y2="162.56" width="0.1524" layer="91"/>
+<pinref part="HP" gate="-4" pin="1"/>
+<wire x1="-139.7" y1="162.56" x2="-152.4" y2="162.56" width="0.1524" layer="91"/>
+</segment>
+</net>

Commit message: with headphone wip
Parts:
- removed L9: ILHB1206ER601V, SparkFun-Passives:INDUCTOR1206H*
Connections:
- removed net N$48: C61.P$1, C66.P$1, IC13.DVDD, L9.1
- net HP_VCC: now also C61.P$1, C66.P$1, IC13.DVDD; no longer L9.2
Changed lines of the file:
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@@
 <part name="C61" library="microbuilder" deviceset="CAP_CERAMIC" device="0603" value="0.1u"/>
 <part name="C66" library="microbuilder" deviceset="CAP_CERAMIC" device="1206" value="10uF"/>
-<part name="L9" library="SparkFun-Passives" deviceset="INDUCTOR" device="H*" technology="1206" value="ILHB1206ER601V"/>
 <part name="U$52" library="microbuilder" deviceset="GND" device=""/>
 <part name="C67" library="microbuilder" deviceset="CAP_CERAMIC" device="1206" value="10uF"/>
@@
 <instance part="C61" gate="G$1" x="-53.34" y="177.8" rot="R90"/>
 <instance part="C66" gate="G$1" x="-53.34" y="185.42" rot="R90"/>
-<instance part="L9" gate="G$1" x="-58.42" y="200.66" rot="R180"/>
 <instance part="U$52" gate="G$1" x="-50.8" y="198.12" rot="R180"/>
 <instance part="C67" gate="G$1" x="-45.72" y="185.42" rot="R90"/>
@@
 </segment>
 <segment>
-<pinref part="L9" gate="G$1" pin="2"/>
-<wire x1="-58.42" y1="208.28" x2="-58.42" y2="213.36" width="0.1524" layer="91"/>
-<label x="-58.42" y="210.82" size="1.778" layer="95" rot="R90"/>
+<label x="-58.42" y="190.5" size="1.778" layer="95" rot="R90"/>
+<pinref part="C66" gate="G$1" pin="P$1"/>
+<junction x="-58.42" y="185.42"/>
+<wire x1="-58.42" y1="177.8" x2="-58.42" y2="185.42" width="0.1524" layer="91"/>
+<pinref part="C61" gate="G$1" pin="P$1"/>
+<junction x="-58.42" y="177.8"/>
+<pinref part="IC13" gate="G$1" pin="DVDD"/>
+<wire x1="-58.42" y1="177.8" x2="-58.42" y2="170.18" width="0.1524" layer="91"/>
+<wire x1="-58.42" y1="195.58" x2="-58.42" y2="185.42" width="0.1524" layer="91"/>
 </segment>
 <segment>
@@
 </segment>
 </net>
-<net name="N$48" class="0">
-<segment>
-<pinref part="L9" gate="G$1" pin="1"/>
-<pinref part="C66" gate="G$1" pin="P$1"/>
-<junction x="-58.42" y="185.42"/>
-<wire x1="-58.42" y1="177.8" x2="-58.42" y2="185.42" width="0.1524" layer="91"/>
-<wire x1="-58.42" y1="185.42" x2="-58.42" y2="193.04" width="0.1524" layer="91"/>
-<pinref part="C61" gate="G$1" pin="P$1"/>
-<junction x="-58.42" y="177.8"/>
-<pinref part="IC13" gate="G$1" pin="DVDD"/>
-<wire x1="-58.42" y1="177.8" x2="-58.42" y2="170.18" width="0.1524" layer="91"/>
-</segment>
-</net>

Commit message: with headphone wip
Parts:
- removed L7: ILHB1206ER601V, SparkFun-Passives:INDUCTOR1206H*
Connections:
- removed net N$34: C56.P$1, C57.P$1, IC12.OUT, L7.1
- net N$31: now also C56.P$1, C57.P$1, IC12.OUT; no longer L7.2
Changed lines of the file:
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@@
 <part name="U$48" library="microbuilder" deviceset="GND" device=""/>
 <part name="R49" library="microbuilder" deviceset="RESISTOR" device="_0805" value="270 270ohms 25ppm 0.5%  (ERA-6AED271V)"/>
-<part name="L7" library="SparkFun-Passives" deviceset="INDUCTOR" device="H*" technology="1206" value="ILHB1206ER601V"/>
 <part name="C56" library="microbuilder" deviceset="CAP_CERAMIC" device="1206" value="10uF"/>
 <part name="C57" library="microbuilder" deviceset="CAP_CERAMIC" device="0603" value="0.1uF"/>
@@
 <instance part="U$48" gate="G$1" x="101.6" y="254"/>
 <instance part="R49" gate="G$1" x="114.3" y="261.62"/>
-<instance part="L7" gate="G$1" x="152.4" y="271.78" rot="R90"/>
 <instance part="C56" gate="G$1" x="129.54" y="266.7"/>
 <instance part="C57" gate="G$1" x="139.7" y="266.7"/>
@@
 <wire x1="160.02" y1="271.78" x2="175.26" y2="271.78" width="0.1524" layer="91"/>
 <pinref part="X1" gate="-1" pin="1"/>
-<pinref part="L7" gate="G$1" pin="2"/>
-<junction x="160.02" y="271.78"/>
-</segment>
-</net>
-<net name="CAN_H" class="0">
-<segment>
-<wire x1="175.26" y1="266.7" x2="160.02" y2="266.7" width="0.1524" layer="91"/>
-<pinref part="X2" gate="-3" pin="1"/>
-<pinref part="X1" gate="-3" pin="1"/>
-</segment>
-</net>
-<net name="CAN_L" class="0">
-<segment>
-<wire x1="175.26" y1="269.24" x2="160.02" y2="269.24" width="0.1524" layer="91"/>
-<pinref part="X2" gate="-2" pin="1"/>
-<pinref part="X1" gate="-2" pin="1"/>
-</segment>
-</net>
-<net name="N$33" class="0">
-<segment>
-<pinref part="R49" gate="G$1" pin="1"/>
-<pinref part="IC12" gate="G$1" pin="TRIM"/>
-<wire x1="109.22" y1="261.62" x2="106.68" y2="261.62" width="0.1524" layer="91"/>
-</segment>
-</net>
-<net name="N$34" class="0">
-<segment>
-<pinref part="L7" gate="G$1" pin="1"/>
-<wire x1="144.78" y1="271.78" x2="139.7" y2="271.78" width="0.1524" layer="91"/>
 <pinref part="IC12" gate="G$1" pin="OUT"/>
 <pinref part="C56" gate="G$1" pin="P$1"/>
@@
 <junction x="129.54" y="271.78"/>
 <pinref part="C57" gate="G$1" pin="P$1"/>
+<wire x1="160.02" y1="271.78" x2="139.7" y2="271.78" width="0.1524" layer="91"/>
 <junction x="139.7" y="271.78"/>
 </segment>
 </net>
+<net name="CAN_H" class="0">
+<segment>
+<wire x1="175.26" y1="266.7" x2="160.02" y2="266.7" width="0.1524" layer="91"/>
+<pinref part="X2" gate="-3" pin="1"/>
+<pinref part="X1" gate="-3" pin="1"/>
+</segment>
+</net>
+<net name="CAN_L" class="0">
+<segment>
+<wire x1="175.26" y1="269.24" x2="160.02" y2="269.24" width="0.1524" layer="91"/>
+<pinref part="X2" gate="-2" pin="1"/>
+<pinref part="X1" gate="-2" pin="1"/>
+</segment>
+</net>
+<net name="N$33" class="0">
+<segment>
+<pinref part="R49" gate="G$1" pin="1"/>
+<pinref part="IC12" gate="G$1" pin="TRIM"/>
+<wire x1="109.22" y1="261.62" x2="106.68" y2="261.62" width="0.1524" layer="91"/>
+</segment>
+</net>

Commit message: with headphone wip
Parts:
- L1, L2, L3, L4, L5, L6, L8: value ILHB1206ER601V -> ILHB0805ER601V; device SparkFun-Passives:INDUCTOR1206H* -> microbuilder:INDUCTOR_0805
Other:
- moved on the sheet: C19, C21, C23

Commit message: wip
Connections:
- net N$69 renamed HP_R_OUT
- net N$70 renamed HP_L_OUT
Changed lines of the file:
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@@
 </segment>
 </net>
-<net name="N$69" class="0">
+<net name="HP_R_OUT" class="0">
 <segment>
 <pinref part="R36" gate="G$1" pin="1"/>
@@
 </segment>
 </net>
-<net name="N$70" class="0">
+<net name="HP_L_OUT" class="0">
 <segment>
 <pinref part="R35" gate="G$1" pin="1"/>
