File: phi-brain4ch/phi-brain4ch.sch (EAGLE design)
At the start: 41 parts, among them IC1 STM32F427VGT6, U1 LM1117MPX-3.3/NOPB or AP2114H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, U2 PRTR5V0U2X, X1 ABM7-8.000MHZ-D2Y-T, X2 04-JST-B4B-XH-A, X3 04-JST-B4B-XH-A

Commit message: wip
Parts:
- added IC2: PCM5102, PCM5102:PCM5102
Changed lines of the file:
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@@
 <part name="X3" library="bt_con-jst-xh" deviceset="04-JST" device="-B4B-XH-A"/>
 <part name="CAN_TERM" library="pinhead" deviceset="PINHD-2X2" device=""/>
+<part name="IC2" library="PCM5102" deviceset="PCM5102" device=""/>
 </parts>
 <sheets>
@@
 </nets>
 </sheet>
+<sheet>
+<plain>
+</plain>
+<instances>
+<instance part="IC2" gate="G$1" x="66.04" y="35.56"/>
+</instances>
+<busses>
+</busses>
+<nets>
+</nets>
+</sheet>

Commit message: wip
Other:
- note added: "TODO: - Verify USB connection - Add MIDI IN/OUT - Add user LEDs - Verify xtal is solderable - Add I2S+SPI connector - Add control interface connector (LCD + ROT ENCS + SPI? + CAN?)"
Changed lines of the file:
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@@
 <sheet>
 <plain>
+<text x="96.52" y="172.72" size="1.778" layer="91">TODO:
+- Verify USB connection
+- Add MIDI IN/OUT
+- Add user LEDs
+- Verify xtal is solderable
+- Add I2S+SPI connector
+- Add control interface connector (LCD + ROT ENCS + SPI? + CAN?)</text>
 </plain>
 <instances>
@@
 </schematic>
 </drawing>
+<compatibility>
+<note version="6.3" minversion="6.2.2" severity="warning">
+Since Version 6.2.2 text objects can contain more than one line,
+which will not be processed correctly with this version.
+</note>
+</compatibility>
 </eagle>

Commit message: wip
Parts:
- removed X1: ABM7-8.000MHZ-D2Y-T, keves:ABM7-8.000MHZ-D2Y-T
- added C23: 0.1uF, microbuilder:CAP_CERAMIC0603
- added CTRL, DAC: (no value), con-harting-ml:ML20
- added IC3: AT45DB161D-SU, atmel:AT45DB161D-SU
- added Y1: 8MHz, microbuilder:CRYSTALSMD
Connections:
- new net FLASH_CS: IC1.PC9, IC3.!CS
- new net I2S_BCK: DAC.7, IC1.PE5
- new net I2S_DATA: DAC.5, IC1.PE6
- new net I2S_DATA2: DAC.1, IC1.PE3
- new net I2S_LRCK: DAC.3, IC1.PE4
- new net I2S_MCK: DAC.9, IC1.PA5, IC1.PE2
- new net LCD_CLK: CTRL.2
- new net LCD_D0: CTRL.8
- new net LCD_D1: CTRL.7
- new net LCD_D2: CTRL.6
- new net LCD_D3: CTRL.5
- new net LCD_D4: CTRL.4
- new net LCD_D5: CTRL.3
- new net LCD_MOSI: CTRL.1
- new net ROT1_A: CTRL.14
- new net ROT1_B: CTRL.13
- new net ROT1_SW: CTRL.12
- new net ROT2_A: CTRL.10
- new net ROT2_B: CTRL.9
- new net ROT2_SW: CTRL.11
- new net SPI3_CLK: IC1.PC10, IC3.SCK
- new net SPI3_MISO: IC1.PC11, IC3.SO
- new net SPI3_MOSI: IC1.PC12, IC3.SI
- new net SPI_CLK: DAC.17
- new net SPI_CS: DAC.11
- new net SPI_MISO: DAC.15
- new net SPI_MOSI: DAC.13
- net 3.3V: now also C23.P$1, CTRL.17, CTRL.18, IC3.!RESET, IC3.!WP, IC3.VCC
- net 5.0V: now also CTRL.15, CTRL.16
- net GND: now also C23.P$2, CTRL.19, CTRL.20, DAC.10, DAC.12, DAC.14, DAC.16, DAC.18, DAC.19, DAC.2, DAC.20, DAC.4, DAC.6, DAC.8, IC3.GND
- net N$4: now also Y1.2; no longer X1.1
- net N$5: now also Y1.1; no longer X1.2
Other:
- note added: "TODO: - Add MIDI IN/OUT - Add user LEDs - Connect I2S+SPI connector to MCU - Connect CTRL connector - Validate I2S pins compared to current setup - Validate PA5<=>MCK connection"
- note removed: "TODO: - Verify USB connection - Add MIDI IN/OUT - Add user LEDs - Verify xtal is solderable - Add I2S+SPI connector - Add control interface connector (LCD + ROT ENCS + SPI? + CAN?)"

Commit message: wip
Parts:
- removed IC2: PCM5102, PCM5102:PCM5102
- C11, C12, C19, C2, C24, C3: device microbuilder:CAP_CERAMIC0603 -> microbuilder:CAP_CERAMIC0805
- C13, C23: value 0.1uF -> 0.1u
- C14, C15: value 10uF TANT -> 10u; device SparkFun-Capacitors:10UF-6.3V-20%(0603)(TANT)" -> microbuilder:CAP_CERAMIC0805
- LED1: device microbuilder:LED0603 -> microbuilder:LED0805
- R1, R15, R16, R23, R24, R25, R9: device microbuilder:RESISTOR0603 -> microbuilder:RESISTOR0805
Connections:
- removed net LCD_CLK: CTRL.2
- removed net LCD_D5: CTRL.3
- removed net LCD_MOSI: CTRL.1
- removed net SPI_CLK: DAC.17
- removed net SPI_CS: DAC.11
- removed net SPI_MISO: DAC.15
- removed net SPI_MOSI: DAC.13
- new net DAC_CS: DAC.11, IC1.PC8
- new net SPI4_CLK: CTRL.2, IC1.PE12
- new net SPI4_MISO: CTRL.3, IC1.PE13
- new net SPI4_MOSI: CTRL.1, IC1.PE14
- net 3.3V: now also C15.P$1; no longer C15.+
- net 5.0V: now also C14.P$1; no longer C14.+
- net GND: now also C14.P$2, C15.P$2; no longer C14.-, C15.-
- net SPI3_CLK: now also DAC.17
- net SPI3_MISO: now also DAC.15
- net SPI3_MOSI: now also DAC.13
Other:
- note added: "TODO: - Add MIDI IN/OUT - Add user LEDs - Connect CTRL connector: ROT*, LCD_D* - Validate I2S pins compared to current setup - Validate PA5<=>MCK connection"
- note removed: "TODO: - Add MIDI IN/OUT - Add user LEDs - Connect I2S+SPI connector to MCU - Connect CTRL connector - Validate I2S pins compared to current setup - Validate PA5<=>MCK connection"

Commit message: wip
Parts:
- added C16, C17, C21: 0.1u, microbuilder:CAP_CERAMIC0603
- added D4: (no value), microbuilder:DIODESOD-123
- added IC2: 6N138S-TA1, 6n138:6N138SMD
- added L1, L2, L3, L5: (no value), microbuilder:INDUCTOR0805
- added LED2, LED3: (no value), microbuilder:LED0805
- added MIDI_IN, MIDI_OUT: MIDIJACK, keves:MIDIJACK
- added R2, R3: 330, microbuilder:RESISTOR0805
- added R4, R6: 220, microbuilder:RESISTOR0805
- added R5: 220, microbuilder:RESISTOR_0603
- added R7: 10k, microbuilder:RESISTOR0805
- added R8: 1k, microbuilder:RESISTOR0805
Connections:
- new net MIDI_IN: IC1.PC7, IC2.VO, R8.1
- new net MIDI_OUT: IC1.PC6, R5.1
- new net N$10: IC1.PD10, R2.2
- new net N$11: IC1.PD9, R3.2
- new net N$12: LED2.A, R2.1
- new net N$13: LED3.A, R3.1
- new net N$14: L3.2, MIDI_OUT.5
- new net N$15: L3.1, R5.2
- new net N$16: L2.1, MIDI_IN.4
- new net N$17: D4.C, IC2.A, R4.1
- new net N$21: D4.A, IC2.C, L1.1
- new net N$22: IC2.VB, R7.1
- new net N$23: C21.P$1, MIDI_OUT.2
- new net N$24: C17.P$1, MIDI_IN.2
- new net N$25: L1.2, MIDI_IN.5
- new net N$26: L2.2, R4.2
- new net N$27: L5.2, R6.2
- new net N$28: L5.1, MIDI_OUT.4
- net 3.3V: now also R6.1, R8.2
- net 5.0V: now also C16.P$2, IC2.VCC
- net GND: now also C16.P$1, C17.P$2, C21.P$2, IC2.GND, LED2.C, LED3.C, R7.2
- net UART_RX: now also IC1.PD7
- net UART_TX: now also IC1.PD8
Other:
- note added: "TODO: - Connect CTRL connector: ROT*, LCD_D* - Validate I2S pins compared to current setup - Validate PA5<=>MCK connection"
- note removed: "TODO: - Add MIDI IN/OUT - Add user LEDs - Connect CTRL connector: ROT*, LCD_D* - Validate I2S pins compared to current setup - Validate PA5<=>MCK connection"

Commit message: wip
Other:
- note added: "TODO: - Connect CTRL connector: ROT*, LCD_D*"
- note removed: "TODO: - Connect CTRL connector: ROT*, LCD_D* - Validate I2S pins compared to current setup - Validate PA5<=>MCK connection"
Changed lines of the file:
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@@
 <text x="96.52" y="172.72" size="1.778" layer="91">TODO:
 - Connect CTRL connector: ROT*, LCD_D*
-- Validate I2S pins compared to current setup
-- Validate PA5&lt;=&gt;MCK connection</text>
+</text>
 </plain>
 <instances>

Commit message: wip
Parts:
- removed H5, H6: MOUNT-HOLE3.2, holes:MOUNT-HOLE3.2
- R5: device microbuilder:RESISTOR_0603 -> microbuilder:RESISTOR0805
- renumbered D1 to U5
Changed lines of the file:
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@@
 <part name="H1" library="holes" deviceset="MOUNT-HOLE" device="3.2"/>
 <part name="H2" library="holes" deviceset="MOUNT-HOLE" device="3.2"/>
-<part name="H5" library="holes" deviceset="MOUNT-HOLE" device="3.2"/>
-<part name="H6" library="holes" deviceset="MOUNT-HOLE" device="3.2"/>
 <part name="TC1" library="TagConnect" deviceset="TC2050-IDC" device="-NL"/>
 <part name="U$55" library="microbuilder" deviceset="3.3V" device=""/>
@@
 <part name="U2" library="Volks73-NXPSemiconductors" deviceset="PRTR5V0U2X?" device=""/>
 <part name="GND33" library="microbuilder" deviceset="GND" device=""/>
-<part name="D1" library="omc" deviceset="SN65HVD230" device="" value="SN65HVD230"/>
+<part name="U5" library="omc" deviceset="SN65HVD230" device="" value="SN65HVD230"/>
 <part name="GND12" library="microbuilder" deviceset="GND" device=""/>
 <part name="GND22" library="microbuilder" deviceset="GND" device=""/>
@@
 <part name="MIDI_OUT" library="keves" deviceset="MIDIJACK" device=""/>
 <part name="R4" library="microbuilder" deviceset="RESISTOR" device="0805" value="220"/>
-<part name="R5" library="microbuilder" deviceset="RESISTOR" device="_0603" value="220"/>
+<part name="R5" library="microbuilder" deviceset="RESISTOR" device="0805" value="220"/>
 <part name="R6" library="microbuilder" deviceset="RESISTOR" device="0805" value="220"/>
 <part name="IC2" library="6n138" deviceset="6N138" device="SMD" value="6N138S-TA1"/>
@@
 <instance part="H1" gate="G$1" x="-73.66" y="147.32"/>
 <instance part="H2" gate="G$1" x="-73.66" y="142.24"/>
-<instance part="H5" gate="G$1" x="-73.66" y="137.16"/>
-<instance part="H6" gate="G$1" x="-68.58" y="139.7"/>
 <instance part="TC1" gate="A" x="-7.62" y="142.24" rot="R180"/>
 <instance part="U$55" gate="G$1" x="-20.32" y="147.32" rot="R90"/>
@@
 <instance part="U2" gate="-SUPPLY" x="-22.86" y="114.3" rot="R270"/>
 <instance part="GND33" gate="G$1" x="-35.56" y="106.68"/>
-<instance part="D1" gate="G$1" x="-30.48" y="20.32"/>
+<instance part="U5" gate="G$1" x="-30.48" y="20.32"/>
 <instance part="GND12" gate="G$1" x="-48.26" y="10.16" rot="R270"/>
 <instance part="GND22" gate="G$1" x="-15.24" y="30.48" rot="R90"/>
@@
 </segment>
 <segment>
-<pinref part="D1" gate="G$1" pin="VCC"/>
+<pinref part="U5" gate="G$1" pin="VCC"/>
 <pinref part="3.3V8" gate="G$1" pin="3.3V"/>
 <pinref part="C13" gate="G$1" pin="P$1"/>
@@
 </segment>
 <segment>
-<pinref part="D1" gate="G$1" pin="GND"/>
+<pinref part="U5" gate="G$1" pin="GND"/>
 <pinref part="GND22" gate="G$1" pin="GND"/>
 <pinref part="C13" gate="G$1" pin="P$2"/>
@@
 </segment>
 <segment>
-<pinref part="D1" gate="G$1" pin="RS"/>
+<pinref part="U5" gate="G$1" pin="RS"/>
 <wire x1="-45.72" y1="10.16" x2="-43.18" y2="10.16" width="0.1524" layer="91"/>
 <pinref part="GND12" gate="G$1" pin="GND"/>
@@
 <net name="CAN_H" class="0">
 <segment>
-<pinref part="D1" gate="G$1" pin="CANH"/>
+<pinref part="U5" gate="G$1" pin="CANH"/>
 <wire x1="-17.78" y1="22.86" x2="-7.62" y2="22.86" width="0.1524" layer="91"/>
 <wire x1="-7.62" y1="22.86" x2="-7.62" y2="40.64" width="0.1524" layer="91"/>
@@
 <net name="CAN_L" class="0">
 <segment>
-<pinref part="D1" gate="G$1" pin="CANL"/>
+<pinref part="U5" gate="G$1" pin="CANL"/>
 <wire x1="-17.78" y1="17.78" x2="-10.16" y2="17.78" width="0.1524" layer="91"/>
 <wire x1="-10.16" y1="17.78" x2="-10.16" y2="2.54" width="0.1524" layer="91"/>
@@
 <segment>
 <label x="-58.42" y="22.86" size="1.778" layer="95"/>
-<pinref part="D1" gate="G$1" pin="TXD"/>
+<pinref part="U5" gate="G$1" pin="TXD"/>
 <wire x1="-53.34" y1="22.86" x2="-43.18" y2="22.86" width="0.1524" layer="91"/>
 </segment>
@@
 <segment>
 <label x="-58.42" y="17.78" size="1.778" layer="95"/>
-<pinref part="D1" gate="G$1" pin="RXD"/>
+<pinref part="U5" gate="G$1" pin="RXD"/>
 <wire x1="-43.18" y1="17.78" x2="-53.34" y2="17.78" width="0.1524" layer="91"/>
 </segment>
@@
 <net name="N$9" class="0">
 <segment>
-<pinref part="D1" gate="G$1" pin="VREF"/>
+<pinref part="U5" gate="G$1" pin="VREF"/>
 <wire x1="-17.78" y1="10.16" x2="15.24" y2="10.16" width="0.1524" layer="91"/>
 <wire x1="15.24" y1="10.16" x2="15.24" y2="15.24" width="0.1524" layer="91"/>

Commit message: wip
Connections:
- net 3.3V: now also IC1.VREF_PLUS
- net GND: no longer IC1.VREF_PLUS
Changed lines of the file:
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@@
 <junction x="147.32" y="127"/>
 <junction x="142.24" y="127"/>
+<pinref part="IC1" gate="G$1" pin="VREF_PLUS"/>
+<wire x1="129.54" y1="129.54" x2="129.54" y2="127" width="0.1524" layer="91"/>
 </segment>
 <segment>
@@
 <pinref part="IC1" gate="G$1" pin="VSS@1"/>
 <junction x="129.54" y="134.62"/>
-<pinref part="IC1" gate="G$1" pin="VREF_PLUS"/>
-<wire x1="129.54" y1="129.54" x2="129.54" y2="132.08" width="0.1524" layer="91"/>
-<junction x="129.54" y="132.08"/>
 <pinref part="C10" gate="G$1" pin="P$2"/>
 <wire x1="172.72" y1="137.16" x2="172.72" y2="142.24" width="0.1524" layer="91"/>
