File: phi-brain4ch/phi-brain4ch.sch (EAGLE design)
At the start: 63 parts, among them IC1 STM32F427VGT6, IC2 6N138S-TA1, IC3 AT45DB161D-SU, U1 LM1117MPX-3.3/NOPB or AP2114H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, U2 PRTR5V0U2X, U5 SN65HVD230, X2 04-JST-B4B-XH-A, X3 04-JST-B4B-XH-A, Y1 8MHz

Commit message: wip
Connections:
- removed net N$10: IC1.PD10, R2.2
- removed net N$11: IC1.PD9, R3.2
- net DAC_CS: now also IC1.PD3; no longer IC1.PC8
- net FLASH_CS: now also IC1.PD4; no longer IC1.PC9
- net I2S_DATA: now also IC1.PE3; no longer IC1.PE6
- net I2S_DATA2: now also IC1.PE6; no longer IC1.PE3
- net LCD_D0: now also IC1.PE7
- net LCD_D1: now also IC1.PE8
- net LCD_D2: now also IC1.PE10
- net LCD_D3: now also IC1.PE9
- net LCD_D4: now also IC1.PE11
- net SPI4_CLK: now also CTRL.3; no longer CTRL.2
- net SPI4_MISO: now also CTRL.1; no longer CTRL.3
- net SPI4_MOSI: now also CTRL.2; no longer CTRL.1
Other:
- note added: "TODO: - Connect CTRL connector: ROT*, LCD_D* - USER LEDs"
- note removed: "TODO: - Connect CTRL connector: ROT*, LCD_D*"
Changed lines of the file:
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@@
 <text x="96.52" y="172.72" size="1.778" layer="91">TODO:
 - Connect CTRL connector: ROT*, LCD_D*
-</text>
+- USER LEDs</text>
 </plain>
 <instances>
@@
 </segment>
 <segment>
-<pinref part="IC1" gate="G$1" pin="PC8"/>
-<wire x1="68.58" y1="20.32" x2="53.34" y2="20.32" width="0.1524" layer="91"/>
-<label x="50.8" y="20.32" size="1.778" layer="95"/>
+<pinref part="IC1" gate="G$1" pin="PD3"/>
+<wire x1="129.54" y1="10.16" x2="144.78" y2="10.16" width="0.1524" layer="91"/>
+<label x="142.24" y="10.16" size="1.778" layer="95"/>
 </segment>
 </net>
@@
 </segment>
 <segment>
+<pinref part="IC1" gate="G$1" pin="PE3"/>
+<wire x1="129.54" y1="53.34" x2="144.78" y2="53.34" width="0.1524" layer="91"/>
+<label x="139.7" y="53.34" size="1.778" layer="95"/>
+</segment>
+</net>
+<net name="I2S_LRCK" class="0">
+<segment>
+<wire x1="2.54" y1="-33.02" x2="-20.32" y2="-33.02" width="0.1524" layer="91"/>
+<label x="-10.16" y="-33.02" size="1.778" layer="95"/>
+<pinref part="DAC" gate="1" pin="3"/>
+</segment>
+<segment>
+<pinref part="IC1" gate="G$1" pin="PE4"/>
+<wire x1="129.54" y1="55.88" x2="144.78" y2="55.88" width="0.1524" layer="91"/>
+<label x="139.7" y="55.88" size="1.778" layer="95"/>
+</segment>
+</net>
+<net name="I2S_DATA2" class="0">
+<segment>
+<pinref part="DAC" gate="1" pin="1"/>
+<wire x1="-20.32" y1="-35.56" x2="-2.54" y2="-35.56" width="0.1524" layer="91"/>
+<label x="-10.16" y="-35.56" size="1.778" layer="95"/>
+</segment>
+<segment>
 <pinref part="IC1" gate="G$1" pin="PE6"/>
 <wire x1="129.54" y1="60.96" x2="144.78" y2="60.96" width="0.1524" layer="91"/>
@@
 </segment>
 </net>
-<net name="I2S_LRCK" class="0">
-<segment>
-<wire x1="2.54" y1="-33.02" x2="-20.32" y2="-33.02" width="0.1524" layer="91"/>
-<label x="-10.16" y="-33.02" size="1.778" layer="95"/>
-<pinref part="DAC" gate="1" pin="3"/>
-</segment>
-<segment>
-<pinref part="IC1" gate="G$1" pin="PE4"/>
-<wire x1="129.54" y1="55.88" x2="144.78" y2="55.88" width="0.1524" layer="91"/>
-<label x="139.7" y="55.88" size="1.778" layer="95"/>
-</segment>
-</net>
-<net name="I2S_DATA2" class="0">
-<segment>
-<pinref part="DAC" gate="1" pin="1"/>
-<wire x1="-20.32" y1="-35.56" x2="-2.54" y2="-35.56" width="0.1524" layer="91"/>
-<label x="-10.16" y="-35.56" size="1.778" layer="95"/>
-</segment>
-<segment>
-<pinref part="IC1" gate="G$1" pin="PE3"/>
-<wire x1="129.54" y1="53.34" x2="144.78" y2="53.34" width="0.1524" layer="91"/>
-<label x="139.7" y="53.34" size="1.778" layer="95"/>
-</segment>
-</net>
 <net name="SPI3_MOSI" class="0">
 <segment>
@@
 </segment>
 <segment>
-<pinref part="IC1" gate="G$1" pin="PC9"/>
-<wire x1="68.58" y1="17.78" x2="53.34" y2="17.78" width="0.1524" layer="91"/>
-<label x="50.8" y="17.78" size="1.778" layer="95"/>
+<pinref part="IC1" gate="G$1" pin="PD4"/>
+<wire x1="129.54" y1="12.7" x2="144.78" y2="12.7" width="0.1524" layer="91"/>
+<label x="142.24" y="12.7" size="1.778" layer="95"/>
 </segment>
 </net>
@@
 <label x="12.7" y="-27.94" size="1.778" layer="95"/>
 </segment>
+<segment>
+<pinref part="IC1" gate="G$1" pin="PE7"/>
+<wire x1="129.54" y1="63.5" x2="144.78" y2="63.5" width="0.1524" layer="91"/>
+<label x="142.24" y="63.5" size="1.778" layer="95"/>
+</segment>
 </net>
 <net name="LCD_D2" class="0">
@@
 <label x="12.7" y="-30.48" size="1.778" layer="95"/>
 </segment>
+<segment>
+<pinref part="IC1" gate="G$1" pin="PE10"/>
+<wire x1="129.54" y1="71.12" x2="144.78" y2="71.12" width="0.1524" layer="91"/>
+<label x="142.24" y="71.12" size="1.778" layer="95"/>
+</segment>
 </net>
 <net name="LCD_D4" class="0">
@@
 <label x="12.7" y="-33.02" size="1.778" layer="95"/>
 </segment>
+<segment>
+<pinref part="IC1" gate="G$1" pin="PE11"/>
+<wire x1="129.54" y1="73.66" x2="144.78" y2="73.66" width="0.1524" layer="91"/>
+<label x="142.24" y="73.66" size="1.778" layer="95"/>
+</segment>
 </net>
 <net name="SPI4_CLK" class="0">
+<segment>
+<pinref part="IC1" gate="G$1" pin="PE12"/>
+<wire x1="129.54" y1="76.2" x2="144.78" y2="76.2" width="0.1524" layer="91"/>
+<label x="142.24" y="76.2" size="1.778" layer="95"/>
+</segment>
+<segment>
+<pinref part="CTRL" gate="1" pin="3"/>
+<wire x1="43.18" y1="-33.02" x2="53.34" y2="-33.02" width="0.1524" layer="91"/>
+<label x="50.8" y="-33.02" size="1.778" layer="95"/>
+</segment>
+</net>
+<net name="SPI4_MOSI" class="0">
+<segment>
+<pinref part="IC1" gate="G$1" pin="PE14"/>
+<wire x1="129.54" y1="81.28" x2="144.78" y2="81.28" width="0.1524" layer="91"/>
+<label x="142.24" y="81.28" size="1.778" layer="95"/>
+</segment>
 <segment>
 <pinref part="CTRL" gate="1" pin="2"/>
@@
 <label x="12.7" y="-35.56" size="1.778" layer="95"/>
 </segment>
-<segment>
-<pinref part="IC1" gate="G$1" pin="PE12"/>
-<wire x1="129.54" y1="76.2" x2="144.78" y2="76.2" width="0.1524" layer="91"/>
-<label x="142.24" y="76.2" size="1.778" layer="95"/>
-</segment>
-</net>
-<net name="SPI4_MOSI" class="0">
+</net>
+<net name="SPI4_MISO" class="0">
+<segment>
+<pinref part="IC1" gate="G$1" pin="PE13"/>
+<wire x1="129.54" y1="78.74" x2="144.78" y2="78.74" width="0.1524" layer="91"/>
+<label x="142.24" y="78.74" size="1.778" layer="95"/>
+</segment>
 <segment>
 <pinref part="CTRL" gate="1" pin="1"/>
@@
 <label x="50.8" y="-35.56" size="1.778" layer="95"/>
 </segment>
-<segment>
-<pinref part="IC1" gate="G$1" pin="PE14"/>
-<wire x1="129.54" y1="81.28" x2="144.78" y2="81.28" width="0.1524" layer="91"/>
-<label x="142.24" y="81.28" size="1.778" layer="95"/>
-</segment>
-</net>
-<net name="SPI4_MISO" class="0">
-<segment>
-<pinref part="CTRL" gate="1" pin="3"/>
-<wire x1="43.18" y1="-33.02" x2="53.34" y2="-33.02" width="0.1524" layer="91"/>
-<label x="50.8" y="-33.02" size="1.778" layer="95"/>
-</segment>
-<segment>
-<pinref part="IC1" gate="G$1" pin="PE13"/>
-<wire x1="129.54" y1="78.74" x2="144.78" y2="78.74" width="0.1524" layer="91"/>
-<label x="142.24" y="78.74" size="1.778" layer="95"/>
-</segment>
 </net>
 <net name="LCD_D3" class="0">
@@
 <label x="50.8" y="-30.48" size="1.778" layer="95"/>
 </segment>
+<segment>
+<pinref part="IC1" gate="G$1" pin="PE9"/>
+<wire x1="129.54" y1="68.58" x2="144.78" y2="68.58" width="0.1524" layer="91"/>
+<label x="142.24" y="68.58" size="1.778" layer="95"/>
+</segment>
 </net>
 <net name="LCD_D1" class="0">
@@
 <label x="50.8" y="-27.94" size="1.778" layer="95"/>
 </segment>
+<segment>
+<pinref part="IC1" gate="G$1" pin="PE8"/>
+<wire x1="129.54" y1="66.04" x2="144.78" y2="66.04" width="0.1524" layer="91"/>
+<label x="142.24" y="66.04" size="1.778" layer="95"/>
+</segment>
 </net>
 <net name="ROT2_B" class="0">
@@
 </segment>
 </net>
-<net name="N$10" class="0">
-<segment>
-<pinref part="IC1" gate="G$1" pin="PD10"/>
-<pinref part="R2" gate="G$1" pin="2"/>
-<wire x1="137.16" y1="27.94" x2="129.54" y2="27.94" width="0.1524" layer="91"/>
-</segment>
-</net>
-<net name="N$11" class="0">
-<segment>
-<pinref part="IC1" gate="G$1" pin="PD9"/>
-<pinref part="R3" gate="G$1" pin="2"/>
-<wire x1="137.16" y1="25.4" x2="129.54" y2="25.4" width="0.1524" layer="91"/>
-</segment>
-</net>

Commit message: wip
Connections:
- net LCD_D2: now also IC1.PE9; no longer IC1.PE10
- net LCD_D3: now also IC1.PE10; no longer IC1.PE9
- net ROT1_A: now also IC1.PA7
- net ROT1_B: now also IC1.PC4
- net ROT1_SW: now also IC1.PC5
- net ROT2_A: now also IC1.PB1
- net ROT2_B: now also IC1.PB2
- net ROT2_SW: now also IC1.PB0
- net SPI4_MISO: now also CTRL.2; no longer CTRL.1
- net SPI4_MOSI: now also CTRL.1; no longer CTRL.2
Changed lines of the file:
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@@
 <label x="12.7" y="-20.32" size="1.778" layer="95"/>
+</segment>
+<segment>
+<pinref part="IC1" gate="G$1" pin="PA7"/>
+<wire x1="68.58" y1="96.52" x2="53.34" y2="96.52" width="0.1524" layer="91"/>
+<label x="53.34" y="96.52" size="1.778" layer="95"/>
 </segment>
 </net>
@@
 <label x="12.7" y="-22.86" size="1.778" layer="95"/>
 </segment>
+<segment>
+<pinref part="IC1" gate="G$1" pin="PC5"/>
+<wire x1="68.58" y1="27.94" x2="53.34" y2="27.94" width="0.1524" layer="91"/>
+<label x="50.8" y="27.94" size="1.778" layer="95"/>
+</segment>
 </net>
 <net name="ROT2_A" class="0">
@@
 <wire x1="27.94" y1="-25.4" x2="17.78" y2="-25.4" width="0.1524" layer="91"/>
 <label x="12.7" y="-25.4" size="1.778" layer="95"/>
+</segment>
+<segment>
+<pinref part="IC1" gate="G$1" pin="PB1"/>
+<wire x1="68.58" y1="76.2" x2="55.88" y2="76.2" width="0.1524" layer="91"/>
+<label x="53.34" y="76.2" size="1.778" layer="95"/>
 </segment>
 </net>
@@
 </segment>
 <segment>
-<pinref part="IC1" gate="G$1" pin="PE10"/>
-<wire x1="129.54" y1="71.12" x2="144.78" y2="71.12" width="0.1524" layer="91"/>
-<label x="142.24" y="71.12" size="1.778" layer="95"/>
+<pinref part="IC1" gate="G$1" pin="PE9"/>
+<wire x1="129.54" y1="68.58" x2="144.78" y2="68.58" width="0.1524" layer="91"/>
+<label x="142.24" y="68.58" size="1.778" layer="95"/>
 </segment>
 </net>
@@
 </segment>
 <segment>
-<pinref part="CTRL" gate="1" pin="2"/>
-<wire x1="27.94" y1="-35.56" x2="17.78" y2="-35.56" width="0.1524" layer="91"/>
-<label x="12.7" y="-35.56" size="1.778" layer="95"/>
+<pinref part="CTRL" gate="1" pin="1"/>
+<wire x1="43.18" y1="-35.56" x2="53.34" y2="-35.56" width="0.1524" layer="91"/>
+<label x="50.8" y="-35.56" size="1.778" layer="95"/>
 </segment>
 </net>
@@
 </segment>
 <segment>
-<pinref part="CTRL" gate="1" pin="1"/>
-<wire x1="43.18" y1="-35.56" x2="53.34" y2="-35.56" width="0.1524" layer="91"/>
-<label x="50.8" y="-35.56" size="1.778" layer="95"/>
+<pinref part="CTRL" gate="1" pin="2"/>
+<wire x1="27.94" y1="-35.56" x2="17.78" y2="-35.56" width="0.1524" layer="91"/>
+<label x="12.7" y="-35.56" size="1.778" layer="95"/>
 </segment>
 </net>
@@
 </segment>
 <segment>
-<pinref part="IC1" gate="G$1" pin="PE9"/>
-<wire x1="129.54" y1="68.58" x2="144.78" y2="68.58" width="0.1524" layer="91"/>
-<label x="142.24" y="68.58" size="1.778" layer="95"/>
+<pinref part="IC1" gate="G$1" pin="PE10"/>
+<wire x1="129.54" y1="71.12" x2="144.78" y2="71.12" width="0.1524" layer="91"/>
+<label x="142.24" y="71.12" size="1.778" layer="95"/>
 </segment>
 </net>
@@
 <label x="50.8" y="-25.4" size="1.778" layer="95"/>
 </segment>
+<segment>
+<pinref part="IC1" gate="G$1" pin="PB2"/>
+<wire x1="68.58" y1="73.66" x2="55.88" y2="73.66" width="0.1524" layer="91"/>
+<label x="53.34" y="73.66" size="1.778" layer="95"/>
+</segment>
 </net>
 <net name="ROT2_SW" class="0">
@@
 <wire x1="43.18" y1="-22.86" x2="53.34" y2="-22.86" width="0.1524" layer="91"/>
 <label x="50.8" y="-22.86" size="1.778" layer="95"/>
+</segment>
+<segment>
+<pinref part="IC1" gate="G$1" pin="PB0"/>
+<wire x1="68.58" y1="78.74" x2="55.88" y2="78.74" width="0.1524" layer="91"/>
+<label x="53.34" y="78.74" size="1.778" layer="95"/>
 </segment>
 </net>
@@
 <label x="50.8" y="-20.32" size="1.778" layer="95"/>
 </segment>
+<segment>
+<pinref part="IC1" gate="G$1" pin="PC4"/>
+<wire x1="68.58" y1="30.48" x2="53.34" y2="30.48" width="0.1524" layer="91"/>
+<label x="50.8" y="30.48" size="1.778" layer="95"/>
+</segment>
 </net>

Commit message: wip
Parts:
- removed LED3: (no value), microbuilder:LED0805
- removed R3: 330, microbuilder:RESISTOR0805
- added TP1, TP2, TP8: (no value), microbuilder:TESTPOINT0.1"
Connections:
- removed net N$13: LED3.A, R3.1
- new net N$10: IC1.PA2, R2.2
- new net N$11: IC1.PA3
- net 3.3V: now also TP2.P$1
- net GND: now also TP1.P$1, TP8.P$1; no longer LED3.C
Other:
- moved on the sheet: LED2, R2
Changed lines of the file:
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@@
-<attribute name="MPN" value="MF-RES-0603-330"/>
-</part>
-<part name="R3" library="microbuilder" deviceset="RESISTOR" device="0805" value="330">
 <attribute name="MPN" value="MF-RES-0603-330"/>
 </part>
 <part name="LED2" library="microbuilder" deviceset="LED" device="0805"/>
-<part name="LED3" library="microbuilder" deviceset="LED" device="0805"/>
-<part name="GND1" library="microbuilder" deviceset="GND" device=""/>
 <part name="GND2" library="microbuilder" deviceset="GND" device=""/>
 <part name="MIDI_IN" library="keves" deviceset="MIDIJACK" device=""/>
@@
 <part name="L3" library="microbuilder" deviceset="INDUCTOR" device="0805"/>
 <part name="L5" library="microbuilder" deviceset="INDUCTOR" device="0805"/>
+<part name="TP1" library="microbuilder" deviceset="TESTPOINT" device="0.1&quot;"/>
+<part name="U$60" library="microbuilder" deviceset="GND" device=""/>
+<part name="TP8" library="microbuilder" deviceset="TESTPOINT" device="0.1&quot;"/>
+<part name="TP2" library="microbuilder" deviceset="TESTPOINT" device="0.1&quot;"/>
+<part name="U$21" library="microbuilder" deviceset="3.3V" device=""/>
 </parts>
 <sheets>
@@
 <instance part="C14" gate="G$1" x="86.36" y="-22.86"/>
 <instance part="C15" gate="G$1" x="109.22" y="-22.86"/>
-<instance part="R2" gate="G$1" x="142.24" y="27.94" rot="R180">
-<attribute name="MPN" x="142.24" y="27.94" size="1.778" layer="96" rot="R180" display="off"/>
+<instance part="R2" gate="G$1" x="60.96" y="109.22">
+<attribute name="MPN" x="60.96" y="109.22" size="1.778" layer="96" display="off"/>
 </instance>
-<instance part="R3" gate="G$1" x="142.24" y="25.4" rot="R180">
-<attribute name="MPN" x="142.24" y="25.4" size="1.778" layer="96" rot="R180" display="off"/>
-</instance>
-<instance part="LED2" gate="G$1" x="157.48" y="27.94"/>
-<instance part="LED3" gate="G$1" x="157.48" y="25.4"/>
-<instance part="GND1" gate="G$1" x="165.1" y="25.4" rot="R90"/>
-<instance part="GND2" gate="G$1" x="165.1" y="27.94" rot="R90"/>
+<instance part="LED2" gate="G$1" x="45.72" y="109.22" rot="R180"/>
+<instance part="GND2" gate="G$1" x="38.1" y="109.22" rot="R270"/>
 <instance part="MIDI_IN" gate="G$1" x="304.8" y="142.24" rot="R270"/>
 <instance part="MIDI_OUT" gate="G$1" x="302.26" y="91.44" rot="R270"/>
@@
 <instance part="L3" gate="G$1" x="292.1" y="106.68"/>
 <instance part="L5" gate="G$1" x="299.72" y="71.12" rot="R270"/>
+<instance part="TP1" gate="G$1" x="200.66" y="86.36"/>
+<instance part="U$60" gate="G$1" x="200.66" y="83.82"/>
+<instance part="TP8" gate="G$1" x="205.74" y="86.36"/>
+<instance part="TP2" gate="G$1" x="213.36" y="86.36"/>
+<instance part="U$21" gate="G$1" x="213.36" y="81.28" rot="R180"/>
 </instances>
 <busses>
@@
 <pinref part="U$19" gate="G$1" pin="3.3V"/>
 </segment>
+<segment>
+<pinref part="TP2" gate="G$1" pin="P$1"/>
+<pinref part="U$21" gate="G$1" pin="3.3V"/>
+<wire x1="213.36" y1="83.82" x2="213.36" y2="86.36" width="0.1524" layer="91"/>
+</segment>
 </net>
 <net name="GND" class="0">
@@
 </segment>
 <segment>
-<pinref part="LED3" gate="G$1" pin="C"/>
-<pinref part="GND1" gate="G$1" pin="GND"/>
-<wire x1="162.56" y1="25.4" x2="160.02" y2="25.4" width="0.1524" layer="91"/>
-</segment>
-<segment>
 <pinref part="LED2" gate="G$1" pin="C"/>
 <pinref part="GND2" gate="G$1" pin="GND"/>
-<wire x1="162.56" y1="27.94" x2="160.02" y2="27.94" width="0.1524" layer="91"/>
+<wire x1="40.64" y1="109.22" x2="43.18" y2="109.22" width="0.1524" layer="91"/>
 </segment>
 <segment>
@@
 <pinref part="U$20" gate="G$1" pin="GND"/>
 <wire x1="287.02" y1="78.74" x2="287.02" y2="76.2" width="0.1524" layer="91"/>
+</segment>
+<segment>
+<pinref part="TP1" gate="G$1" pin="P$1"/>
+<pinref part="U$60" gate="G$1" pin="GND"/>
+<wire x1="200.66" y1="86.36" x2="205.74" y2="86.36" width="0.1524" layer="91"/>
+<pinref part="TP8" gate="G$1" pin="P$1"/>
+<junction x="200.66" y="86.36"/>
 </segment>
 </net>
@@
 <pinref part="R2" gate="G$1" pin="1"/>
 <pinref part="LED2" gate="G$1" pin="A"/>
-<wire x1="152.4" y1="27.94" x2="147.32" y2="27.94" width="0.1524" layer="91"/>
-</segment>
-</net>
-<net name="N$13" class="0">
-<segment>
-<pinref part="R3" gate="G$1" pin="1"/>
-<pinref part="LED3" gate="G$1" pin="A"/>
-<wire x1="152.4" y1="25.4" x2="147.32" y2="25.4" width="0.1524" layer="91"/>
+<wire x1="50.8" y1="109.22" x2="55.88" y2="109.22" width="0.1524" layer="91"/>
 </segment>
 </net>
@@
 </segment>
 </net>
+<net name="N$10" class="0">
+<segment>
+<pinref part="IC1" gate="G$1" pin="PA2"/>
+<pinref part="R2" gate="G$1" pin="2"/>
+<wire x1="68.58" y1="109.22" x2="66.04" y2="109.22" width="0.1524" layer="91"/>
+</segment>
+</net>
+<net name="N$11" class="0">
+<segment>
+<pinref part="IC1" gate="G$1" pin="PA3"/>
+<wire x1="68.58" y1="106.68" x2="66.04" y2="106.68" width="0.1524" layer="91"/>
+</segment>
+</net>

Commit message: wip
Parts:
- removed C24: 4.7nF, microbuilder:CAP_CERAMIC0805
- removed R15, R16: 60 1%, microbuilder:RESISTOR0805
- removed R23, R24: 22, microbuilder:RESISTOR0805
- removed U5: SN65HVD230, omc:SN65HVD230
- added C20: 0.1u, microbuilder:CAP_CERAMIC0603
- added R10: 10k, microbuilder:RESISTOR0805
- added R11, R12, R13: 220, microbuilder:RESISTOR0805
- added U3: LM1117MPX-3.3/NOPB or AP2114H-3.3TRG1, microbuilder:LM1117SOT223-REFLOW
- C10, C9: value 0.1u -> 18pf; device microbuilder:CAP_CERAMIC0603 -> microbuilder:CAP_CERAMIC0805
- C11: value 18pf -> 2.2u
- C12: value 18pf -> 0.1u; device microbuilder:CAP_CERAMIC0805 -> microbuilder:CAP_CERAMIC0603
- C14, C15: value 10u -> 0.1u; device microbuilder:CAP_CERAMIC0805 -> microbuilder:CAP_CERAMIC0603
- C19: value 4.7nF -> 0.1u; device microbuilder:CAP_CERAMIC0805 -> microbuilder:CAP_CERAMIC0603
- C2, C3: value 2.2u -> 4.7nF
- C5, C6: value 0.1u -> 10u; device microbuilder:CAP_CERAMIC0603 -> microbuilder:CAP_CERAMIC0805
- C7: value 0.1u -> 2.2u; device microbuilder:CAP_CERAMIC0603 -> microbuilder:CAP_CERAMIC0805
- IC2: value 6N138S-TA1 -> AT45DB161D-SU; device 6n138:6N138SMD -> atmel:AT45DB161D-SU; POPULATE (none) -> 0
- IC3: value AT45DB161D-SU -> 6N138S-TA1; device atmel:AT45DB161D-SU -> 6n138:6N138SMD; POPULATE 0 -> (none)
- R1: value 10k -> 22; MPN (none) -> MF-RES-0603-22
- R2: value 330 -> 22; MPN MF-RES-0603-330 -> MF-RES-0603-22
- R4, R5: value 220 -> 60 1%; MPN (none) -> MF-RES-0603-60.4
- R6: value 220 -> 10k
- R7: value 10k -> 330; MPN (none) -> MF-RES-0603-330
- R8: value 1k -> 330; MPN (none) -> MF-RES-0603-330
- R9: value 330 -> 1k; MPN MF-RES-0603-330 -> (none)
- U1: value LM1117MPX-3.3/NOPB or AP2114H-3.3TRG1 -> SN65HVD230; device microbuilder:LM1117SOT223-REFLOW -> omc:SN65HVD230
- renumbered C23 to C18, CAN_TERM to JP1, D4 to D1, L5 to L4, R25 to R3, TP1 to TP_GND1, TP2 to TP_3.3V, TP8 to TP_GND2, X3 to X1, X4 to USB
Connections:
- net 3.3V: now also C1.P$1, C12.P$1, C14.P$1, C16.P$1, C17.P$1, IC2.!RESET, IC2.!WP, IC2.VCC, R13.1, U1.VCC, U3.OUT; no longer C10.P$1, C4.P$1, C5.P$1, C7.P$1, C9.P$1, IC3.!RESET, IC3.!WP, IC3.VCC, R6.1, U1.OUT, U5.VCC
- net 5.0V: now also C19.P$2, C5.P$1, IC3.VCC, U3.IN; no longer C14.P$1, C16.P$2, IC2.VCC, U1.IN
- net CAN_H: now also U1.CANH; no longer U5.CANH
- net CAN_L: now also U1.CANL; no longer U5.CANL
- net CAN_RX: now also U1.RXD; no longer U5.RXD
- net CAN_TX: now also U1.TXD; no longer U5.TXD
- net FLASH_CS: now also IC2.!CS; no longer IC3.!CS
- net GND: now also C1.P$2, C10.P$1, C12.P$2, C16.P$2, C2.P$2, C20.P$2, C4.P$1, C7.P$1, C9.P$1, R10.2, R6.1, U1.GND, U1.RS, U3.ADJ; no longer C1.P$1, C10.P$2, C12.P$1, C16.P$1, C2.P$1, C24.P$2, C4.P$2, C7.P$2, C9.P$2, R1.1, R7.2, U1.ADJ, U5.GND, U5.RS
- net MIDI_IN: now also IC3.VO, R9.1; no longer IC2.VO, R8.1
- net MIDI_OUT: now also R11.1; no longer R5.1
- net N$1: now also R6.2; no longer R1.2
- net N$10: now also R7.2; no longer R2.2
- net N$12: now also LED1.A, R7.1; no longer LED2.A, R2.1
- net N$14: now also L1.2; no longer L3.2
- net N$15: now also L1.1, R11.2; no longer L3.1, R5.2
- net N$16: now also L3.1; no longer L2.1
- net N$17: now also IC3.A, R12.1; no longer IC2.A, R4.1
- net N$18: now also R2.1; no longer R24.1
- net N$19: now also R1.1; no longer R23.1
- net N$2: now also C11.P$2; no longer C2.P$2
- net N$20: now also C2.P$1; no longer C24.P$1
- net N$21: now also IC3.C, L2.1; no longer IC2.C, L1.1
- net N$22: now also IC3.VB, R10.1; no longer IC2.VB, R7.1
- net N$23: now also C20.P$1; no longer C21.P$1
- net N$24: now also C21.P$1; no longer C17.P$1
- net N$25: now also L2.2; no longer L1.2
- net N$26: now also L3.2, R12.2; no longer L2.2, R4.2
- net N$27: now also R13.2; no longer R6.2
- net N$3: now also C7.P$2; no longer C3.P$2
- net N$4: now also C9.P$2; no longer C12.P$2
- net N$5: now also C10.P$2; no longer C11.P$2
- net N$6: now also LED2.A, R8.1; no longer LED1.A, R9.1
- net N$7: now also R4.2; no longer R15.2
- net N$8: now also R5.1; no longer R16.1
- net N$9: now also C3.P$2, R4.1, R5.2, U1.VREF; no longer C19.P$2, R15.1, R16.2, U5.VREF
- net NRST: now also C4.P$2; no longer C1.P$2
- net SPI3_CLK: now also IC2.SCK; no longer IC3.SCK
- net SPI3_MISO: now also IC2.SO; no longer IC3.SO
- net SPI3_MOSI: now also IC2.SI; no longer IC3.SI
- net USB_DM: now also R2.2; no longer R24.2
- net USB_DP: now also R1.2; no longer R23.2
Other:
- note removed: "TODO: - Connect CTRL connector: ROT*, LCD_D* - USER LEDs"
- moved on the sheet: C1, C10, C11, C12, C13, C14, C15, C16, C17, C19, C2, C21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

Commit message: wip
Parts:
- C1, C12, C13, C14, C15, C16, C17, C18, C19, C20, C21, C4, C8: PARTNO (none) -> 0805DD104KAT2A
- C10, C9: PARTNO (none) -> C0805C180M3GACTU
- C11, C7: PARTNO (none) -> 581-08053D225MAT2A
- C2, C3: PARTNO (none) -> 885012207090
- C5, C6: PARTNO (none) -> 81-GRM21BR6YA106KE3L
- CTRL, DAC: PARTNO (none) -> 61202021621
- D1: PARTNO (none) -> MBR120
- IC1: PARTNO (none) -> STM32F427VGT6
- IC3: PARTNO (none) -> 6N138S
- L1, L2, L3, L4: PARTNO (none) -> 70-ILHB0805ER601V
- LED1, LED2: PARTNO (none) -> 604-APT2012YC
- R1, R2: PARTNO (none) -> ERJ-6ENF22R0V
- R10, R6: PARTNO (none) -> RC0805FR-0710KL
- R11, R12, R13: PARTNO (none) -> ERJ-6GEYJ221V
- R3: PARTNO (none) -> AS08J1004ET
- R4, R5: PARTNO (none) -> ERJ-6ENF60R4V
- R7, R8: PARTNO (none) -> CPF0805B330RE1
- R9: PARTNO (none) -> AS08J1001ET
- Y1: PARTNO (none) -> ABLS2-8.000MHz-B1U-T
Connections:
- removed net N$11: IC1.PA3
- net DAC_CS: now also IC1.PD4; no longer IC1.PD3
- net FLASH_CS: now also IC1.PD3; no longer IC1.PD4
