File: phi-brain4ch/phi-brain4ch.sch (EAGLE design)
At the start: 64 parts, among them IC1 STM32F427VGT6, IC2 AT45DB161D-SU, IC3 6N138S-TA1, U1 SN65HVD230, U2 PRTR5V0U2X, U3 LM1117MPX-3.3/NOPB or AP2114H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, X1 04-JST-B4B-XH-A, X2 04-JST-B4B-XH-A, Y1 8MHz

Commit message: wip
Parts:
- added C52: 0.1u, microbuilder:CAP_CERAMIC0603
- added OSC1: 12.288MHz C3391-12.288, microbuilder:OSCILLATOR
- added R14: 0, microbuilder:RESISTOR0805
- added R48: 0, microbuilder:RESISTOR_0805
- added TP18: (no value), microbuilder:TESTPOINT0.1"
Connections:
- new net I2S_CKIN: IC1.PC9, R14.1, R48.2, TP18.P$1
- new net N$11: IC1.PA0, R14.2
- new net N$32: OSC1.OUT, R48.1
- net 3.3V: now also C52.P$1, OSC1.VCC
- net GND: now also C52.P$2, OSC1.GND
- net UART_RX: now also IC1.PD6; no longer IC1.PD7
- net UART_TX: now also IC1.PD5; no longer IC1.PD8
Changed lines of the file:
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@@
 <part name="TP_3.3V" library="microbuilder" deviceset="TESTPOINT" device="0.1&quot;"/>
 <part name="3.3V11" library="microbuilder" deviceset="3.3V" device=""/>
+<part name="OSC1" library="microbuilder" deviceset="OSCILLATOR" device="" value="12.288MHz C3391-12.288"/>
+<part name="C52" library="microbuilder" deviceset="CAP_CERAMIC" device="0603" value="0.1u"/>
+<part name="U$45" library="microbuilder" deviceset="3.3V" device=""/>
+<part name="U$47" library="microbuilder" deviceset="GND" device=""/>
+<part name="R48" library="microbuilder" deviceset="RESISTOR" device="_0805" value="0"/>
+<part name="TP18" library="microbuilder" deviceset="TESTPOINT" device="0.1&quot;"/>
+<part name="R14" library="microbuilder" deviceset="RESISTOR" device="0805" value="0">
+<attribute name="MPN" value="MF-RES-0603-330"/>
+<attribute name="PARTNO" value="CPF0805B330RE1"/>
+</part>
 </parts>
 <sheets>
@@
 <instance part="TP_3.3V" gate="G$1" x="213.36" y="86.36"/>
 <instance part="3.3V11" gate="G$1" x="213.36" y="81.28" rot="R180"/>
+<instance part="OSC1" gate="G$1" x="218.44" y="48.26"/>
+<instance part="C52" gate="G$1" x="198.12" y="48.26"/>
+<instance part="U$45" gate="G$1" x="193.04" y="53.34" rot="R90"/>
+<instance part="U$47" gate="G$1" x="193.04" y="43.18" rot="R270"/>
+<instance part="R48" gate="G$1" x="236.22" y="48.26"/>
+<instance part="TP18" gate="G$1" x="246.38" y="48.26"/>
+<instance part="R14" gate="G$1" x="50.8" y="114.3">
+<attribute name="MPN" x="50.8" y="114.3" size="1.778" layer="96" display="off"/>
+<attribute name="PARTNO" x="50.8" y="114.3" size="1.778" layer="96" display="off"/>
+</instance>
 </instances>
 <busses>
@@
 <wire x1="213.36" y1="83.82" x2="213.36" y2="86.36" width="0.1524" layer="91"/>
 </segment>
+<segment>
+<pinref part="OSC1" gate="G$1" pin="VCC"/>
+<wire x1="208.28" y1="53.34" x2="198.12" y2="53.34" width="0.1524" layer="91"/>
+<pinref part="U$45" gate="G$1" pin="3.3V"/>
+<pinref part="C52" gate="G$1" pin="P$1"/>
+<junction x="198.12" y="53.34"/>
+<wire x1="198.12" y1="53.34" x2="195.58" y2="53.34" width="0.1524" layer="91"/>
+</segment>
 </net>
 <net name="GND" class="0">
@@
 <junction x="200.66" y="86.36"/>
 </segment>
+<segment>
+<pinref part="OSC1" gate="G$1" pin="GND"/>
+<pinref part="U$47" gate="G$1" pin="GND"/>
+<wire x1="208.28" y1="43.18" x2="198.12" y2="43.18" width="0.1524" layer="91"/>
+<junction x="198.12" y="43.18"/>
+<wire x1="198.12" y1="43.18" x2="195.58" y2="43.18" width="0.1524" layer="91"/>
+<pinref part="C52" gate="G$1" pin="P$2"/>
+<wire x1="198.12" y1="45.72" x2="198.12" y2="43.18" width="0.1524" layer="91"/>
+</segment>
 </net>
 <net name="NRST" class="0">
@@
 </segment>
 <segment>
-<pinref part="IC1" gate="G$1" pin="PD8"/>
-<wire x1="129.54" y1="22.86" x2="142.24" y2="22.86" width="0.1524" layer="91"/>
-<label x="142.24" y="22.86" size="1.778" layer="95"/>
+<pinref part="IC1" gate="G$1" pin="PD5"/>
+<wire x1="129.54" y1="15.24" x2="142.24" y2="15.24" width="0.1524" layer="91"/>
+<label x="142.24" y="15.24" size="1.778" layer="95"/>
 </segment>
 </net>
@@
 </segment>
 <segment>
-<pinref part="IC1" gate="G$1" pin="PD7"/>
-<wire x1="129.54" y1="20.32" x2="142.24" y2="20.32" width="0.1524" layer="91"/>
-<label x="139.7" y="20.32" size="1.778" layer="95"/>
+<pinref part="IC1" gate="G$1" pin="PD6"/>
+<wire x1="129.54" y1="17.78" x2="142.24" y2="17.78" width="0.1524" layer="91"/>
+<label x="142.24" y="17.78" size="1.778" layer="95"/>
 </segment>
 </net>
@@
 </segment>
 </net>
+<net name="I2S_CKIN" class="0">
+<segment>
+<pinref part="IC1" gate="G$1" pin="PC9"/>
+<wire x1="68.58" y1="17.78" x2="53.34" y2="17.78" width="0.1524" layer="91"/>
+<label x="50.8" y="17.78" size="1.778" layer="95"/>
+</segment>
+<segment>
+<pinref part="R48" gate="G$1" pin="2"/>
+<wire x1="241.3" y1="48.26" x2="246.38" y2="48.26" width="0.1524" layer="91"/>
+<label x="246.38" y="48.26" size="1.778" layer="95"/>
+<pinref part="TP18" gate="G$1" pin="P$1"/>
+<wire x1="246.38" y1="48.26" x2="251.46" y2="48.26" width="0.1524" layer="91"/>
+<junction x="246.38" y="48.26"/>
+</segment>
+<segment>
+<pinref part="R14" gate="G$1" pin="1"/>
+<wire x1="45.72" y1="114.3" x2="38.1" y2="114.3" width="0.1524" layer="91"/>
+<label x="33.02" y="114.3" size="1.778" layer="95"/>
+</segment>
+</net>
+<net name="N$32" class="0">
+<segment>
+<pinref part="R48" gate="G$1" pin="1"/>
+<pinref part="OSC1" gate="G$1" pin="OUT"/>
+<wire x1="231.14" y1="48.26" x2="228.6" y2="48.26" width="0.1524" layer="91"/>
+</segment>
+</net>
+<net name="N$11" class="0">
+<segment>
+<pinref part="IC1" gate="G$1" pin="PA0"/>
+<wire x1="68.58" y1="114.3" x2="55.88" y2="114.3" width="0.1524" layer="91"/>
+<pinref part="R14" gate="G$1" pin="2"/>
+</segment>
+</net>
