File: phi-brain4ch/phi-brain4ch.brd (EAGLE design)
At the start: 76.2 x 48.3 mm, 63 parts, among them IC1 STM32F427VGT6, IC2 6N138S-TA1, IC3 AT45DB161D-SU, U1 LM1117MPX-3.3/NOPB or AP2114H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, U2 PRTR5V0U2X, U5 SN65HVD230, X2 04-JST-B4B-XH-A, X3 04-JST-B4B-XH-A, Y1 8MHz

Commit message: wip
Parts:
- moved TC1 50.6 mm to (24.8, 26.4), turned to 180 degrees
- moved CTRL 37.8 mm to (71.1, 24.1), turned to 270 degrees
- moved C3 27.0 mm to (30.9, 32.6)
- moved C11 26.6 mm to (34.2, 4.45)
- moved C5 21.7 mm to (49.1, 8.51)
- moved C10 21.2 mm to (45.6, 8.51), turned to 180 degrees
- moved C8 20.6 mm to (36.4, 27.9), turned to 180 degrees
- moved C6 20.3 mm to (53.8, 13.1)
- moved C9 20.2 mm to (33.7, 11.6), turned to 270 degrees
- moved IC1 20.0 mm to (42.5, 16.9)
- moved C4 19.7 mm to (41.4, 8.51)
- moved C7 19.7 mm to (53.5, 25.5)
- moved Y1 19.3 mm to (43.9, 4.57)
- moved R1 18.4 mm to (32.4, 15.2)
- moved C2 17.7 mm to (55.8, 23.6), turned to 180 degrees
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Connections:
- net LCD_D2: now also IC1.40; no longer IC1.41
- net LCD_D3: now also IC1.41; no longer IC1.40
- net ROT1_A: now also IC1.32
- net ROT1_B: now also IC1.33
- net ROT1_SW: now also IC1.34
- net ROT2_A: now also IC1.36
- net ROT2_B: now also IC1.37
- net ROT2_SW: now also IC1.35
- net SPI4_MISO: now also CTRL.2; no longer CTRL.1
- net SPI4_MOSI: now also CTRL.1; no longer CTRL.2
Routing:
- net SPI3_MISO: track 79.3 -> 0.00 mm
- net SPI3_CLK: track 77.1 -> 0.00 mm
- net GND: track 69.8 -> 0.00 mm, vias 26 -> 0
- net SPI3_MOSI: track 67.0 -> 0.00 mm
- net FLASH_CS: track 58.7 -> 0.00 mm, vias 2 -> 0
- net DAC_CS: track 54.1 -> 0.00 mm, vias 2 -> 0
- net MIDI_IN: track 38.8 -> 0.00 mm, vias 2 -> 0
- net N$17: track 33.7 -> 0.00 mm
- net I2S_MCK: track 77.2 -> 45.3 mm, vias 1 -> 2
- net MIDI_OUT: track 31.1 -> 0.00 mm, vias 2 -> 0
- net SPI4_MISO: track 0.00 -> 27.4 mm
- net NRST: track 27.3 -> 0.00 mm, vias 2 -> 0
- net LCD_D4: track 0.00 -> 26.3 mm
- net LCD_D2: track 0.00 -> 25.3 mm
- net SPI4_MOSI: track 0.00 -> 24.7 mm
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Other:
- board text added: "GND AND 3.3V ARE HIDDEN"

Commit message: wip
Parts:
- moved C15 39.1 mm to (10.9, 11.9), turned to 90 degrees
- moved C14 38.6 mm to (10.9, 8.00), turned to 90 degrees
- moved C1 36.6 mm to (27.7, 24.4), turned to 0 degrees
- moved U1 35.8 mm to (16.9, 10.0), turned to 270 degrees
- moved C3 9.72 mm to (39.8, 28.7), turned to 180 degrees
- moved TC1 4.85 mm to (28.1, 30.0), turned to 270 degrees
- moved C23 2.90 mm to (17.9, 15.4)
- moved IC3 2.16 mm to (14.1, 18.8)
- moved C8 1.31 mm to (35.3, 27.3)
Routing:
- net 5.0V: track 50.0 -> 156.7 mm
- net SPI3_MISO: track 0.00 -> 79.7 mm
- net SPI3_CLK: track 0.00 -> 78.0 mm
- net SPI3_MOSI: track 0.00 -> 67.5 mm
- net DAC_CS: track 0.00 -> 35.6 mm, vias 0 -> 2
- net N$17: track 0.00 -> 32.5 mm
- net NRST: track 0.00 -> 32.2 mm, vias 0 -> 2
- net FLASH_CS: track 0.00 -> 26.3 mm, vias 0 -> 2
- net UART_TX: track 0.00 -> 22.4 mm, vias 0 -> 2
- net N$21: track 0.00 -> 22.3 mm
- net MIDI_IN: track 0.00 -> 22.2 mm
- net SWDIO: track 0.00 -> 17.7 mm
- net UART_RX: track 0.00 -> 17.7 mm, vias 0 -> 2
- net I2S_MCK: track 45.3 -> 62.6 mm, vias 2 -> 3
- net SWCLK: track 0.00 -> 13.5 mm
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
Commit message: wip
Parts:
- removed LED3: (no value), microbuilder:CHIPLED_0805
- removed R3: 330, microbuilder:0805
- added TP1, TP2, TP8: (no value), microbuilder:1X01_ROUND
- moved R9 82.6 mm to (63.5, 36.7)
- moved LED1 82.2 mm to (63.5, 34.0), turned to 270 degrees
- moved R2 81.9 mm to (52.2, 8.38), turned to 90 degrees
- moved LED2 75.1 mm to (55.4, 7.75), turned to 270 degrees
- moved R8 8.67 mm to (23.6, 41.4), turned to 180 degrees
- moved C8 0.74 mm to (35.7, 27.9), turned to 0 degrees
- moved C2 0.38 mm to (55.4, 23.6)
- moved C4 0.38 mm to (41.4, 8.13)
- moved C7 0.38 mm to (53.1, 25.5)
- moved C9 0.38 mm to (34.0, 11.6), turned to 90 degrees
- moved C5 0.13 mm to (49.1, 8.38), turned to 180 degrees
Connections:
- removed net N$13: LED3.A, R3.1
- new net N$10: IC1.25, R2.2
- new net N$11: IC1.26
- net 3.3V: now also TP2.1
- net GND: now also TP1.1, TP8.1; no longer LED3.C
Routing:
- net GND: track 0.00 -> 79.0 mm, vias 0 -> 31
- net MIDI_IN: track 22.2 -> 28.7 mm
- net 3.3V: track 0.00 -> 3.36 mm, vias 0 -> 1
- net 5.0V: track 156.7 -> 160.0 mm, vias 0 -> 7
- net N$10: track 0.00 -> 2.73 mm
- net N$6: track 0.00 -> 2.71 mm
- net N$2: track 0.00 -> 2.62 mm
- net N$12: track 0.00 -> 2.26 mm

Commit message: wip
Parts:
- removed C24: 4.7nF, microbuilder:0805
- removed R15, R16: 60 1%, microbuilder:0805
- removed R23, R24: 22, microbuilder:0805
- removed U5: SN65HVD230, omc:SO8
- added C20: 0.1u, microbuilder:0603
- added R10: 10k, microbuilder:0805
- added R11, R12, R13: 220, microbuilder:0805
- added U3: LM1117MPX-3.3/NOPB or AP2114H-3.3TRG1, microbuilder:SOT223-R
- C10, C9: value 0.1u -> 18pf; device microbuilder:0603 -> microbuilder:0805
- C11: value 18pf -> 2.2u
- C12: value 18pf -> 0.1u; device microbuilder:0805 -> microbuilder:0603
- C14, C15: value 10u -> 0.1u; device microbuilder:0805 -> microbuilder:0603
- C19: value 4.7nF -> 0.1u; device microbuilder:0805 -> microbuilder:0603
- C2, C3: value 2.2u -> 4.7nF
- C5, C6: value 0.1u -> 10u; device microbuilder:0603 -> microbuilder:0805
- C7: value 0.1u -> 2.2u; device microbuilder:0603 -> microbuilder:0805
- IC2: value 6N138S-TA1 -> AT45DB161D-SU; device 6n138:SO8-GW300 -> atmel:8S2
- IC3: value AT45DB161D-SU -> 6N138S-TA1; device atmel:8S2 -> 6n138:SO8-GW300
- R1: value 10k -> 22
- R2: value 330 -> 22
- R4, R5: value 220 -> 60 1%
- R6: value 220 -> 10k
- R7: value 10k -> 330
- R8: value 1k -> 330
- R9: value 330 -> 1k
- U1: value LM1117MPX-3.3/NOPB or AP2114H-3.3TRG1 -> SN65HVD230; device microbuilder:SOT223-R -> omc:SO8
- moved C14 45.7 mm to (53.1, 25.5), turned to 0 degrees
- moved C6 42.9 mm to (10.9, 11.9), turned to 90 degrees
- moved C17 41.9 mm to (45.6, 8.51), turned to 180 degrees
- moved R8 40.2 mm to (63.5, 36.7), turned to 0 degrees
- moved R9 40.2 mm to (23.6, 41.4), turned to 180 degrees
- moved C5 38.2 mm to (10.9, 8.00), turned to 90 degrees
- moved R7 36.8 mm to (52.2, 8.38), turned to 90 degrees
- moved R5 33.6 mm to (22.0, 6.22)
- moved C19 32.1 mm to (36.8, 39.1)
- moved R4 31.9 mm to (29.8, 6.22), turned to 270 degrees
- moved C15 29.5 mm to (35.7, 27.9), turned to 0 degrees
- moved IC2 28.8 mm to (14.1, 18.8)
- moved IC3 28.8 mm to (30.6, 42.4)
- moved C11 28.6 mm to (55.4, 23.6), turned to 180 degrees
- moved C16 27.7 mm to (34.0, 11.6), turned to 90 degrees
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- renumbered C23 to C18, CAN_TERM to JP1, D4 to D1, L5 to L4, R25 to R3, TP1 to TP_GND1, TP2 to TP_3.3V, TP8 to TP_GND2, X3 to X1, X4 to USB
Connections:
- net 3.3V: now also C1.1, C12.1, C14.1, C16.1, C17.1, IC2.3, IC2.5, IC2.6, R13.1, U1.3, U3.2; no longer C10.1, C4.1, C5.1, C7.1, C9.1, IC3.3, IC3.5, IC3.6, R6.1, U1.2, U5.3
- net 5.0V: now also C19.2, C5.1, IC3.8, U3.3; no longer C14.1, C16.2, IC2.8, U1.3
- net CAN_H: now also U1.7; no longer U5.7
- net CAN_L: now also U1.6; no longer U5.6
- net CAN_RX: now also U1.4; no longer U5.4
- net CAN_TX: now also U1.1; no longer U5.1
- net FLASH_CS: now also IC2.4; no longer IC3.4
- net GND: now also C1.2, C10.1, C12.2, C16.2, C2.2, C20.2, C4.1, C7.1, C9.1, IC2.7, IC3.5, R10.2, R6.1, U1.2, U1.8, U3.1; no longer C1.1, C10.2, C12.1, C16.1, C2.1, C24.2, C4.2, C7.2, C9.2, IC2.5, IC3.7, R1.1, R7.2, U1.1, U5.2, U5.8
- net MIDI_IN: now also IC3.6, R9.1; no longer IC2.6, R8.1
- net MIDI_OUT: now also R11.1; no longer R5.1
- net N$1: now also R6.2; no longer R1.2
- net N$10: now also R7.2; no longer R2.2
- net N$12: now also LED1.A, R7.1; no longer LED2.A, R2.1
- net N$14: now also L1.2; no longer L3.2
- net N$15: now also L1.1, R11.2; no longer L3.1, R5.2
- net N$16: now also L3.1; no longer L2.1
- net N$17: now also IC3.2, R12.1; no longer IC2.2, R4.1
- net N$18: now also R2.1; no longer R24.1
- net N$19: now also R1.1; no longer R23.1
- net N$2: now also C11.2; no longer C2.2
- net N$20: now also C2.1; no longer C24.1
- net N$21: now also IC3.3, L2.1; no longer IC2.3, L1.1
- net N$22: now also IC3.7, R10.1; no longer IC2.7, R7.1
- net N$23: now also C20.1; no longer C21.1
- net N$24: now also C21.1; no longer C17.1
- net N$25: now also L2.2; no longer L1.2
- net N$26: now also L3.2, R12.2; no longer L2.2, R4.2
- net N$27: now also R13.2; no longer R6.2
- net N$3: now also C7.2; no longer C3.2
- net N$4: now also C9.2; no longer C12.2
- net N$5: now also C10.2; no longer C11.2
- net N$6: now also LED2.A, R8.1; no longer LED1.A, R9.1
- net N$7: now also R4.2; no longer R15.2
- net N$8: now also R5.1; no longer R16.1
- net N$9: now also C3.2, R4.1, R5.2, U1.5; no longer C19.2, R15.1, R16.2, U5.5
- net NRST: now also C4.2; no longer C1.2
- net SPI3_CLK: now also IC2.2; no longer IC3.2
- net SPI3_MISO: now also IC2.8; no longer IC3.8
- net SPI3_MOSI: now also IC2.1; no longer IC3.1
- net USB_DM: now also R2.2; no longer R24.2
- net USB_DP: now also R1.2; no longer R23.2
Routing:
- net GND: track 79.0 -> 78.2 mm
Other:
- board text added: "Designed by Eran Rundstein"
- board text added: "Pulsar Heavy Industries"
- board text added: "phi-brain4ch"
- board text removed: "GND AND 3.3V ARE HIDDEN"

Commit message: wip
Parts:
- moved C18 15.6 mm to (16.5, 30.9), turned to 0 degrees
- moved IC2 9.38 mm to (18.5, 27.1), turned to 90 degrees
- moved DAC 0.13 mm to (4.70, 24.1), turned to 90 degrees
Connections:
- removed net N$11: IC1.26
- net DAC_CS: now also IC1.85; no longer IC1.84
- net FLASH_CS: now also IC1.84; no longer IC1.85
Routing:
- net SPI3_MISO: track 79.7 -> 35.2 mm
- net SPI3_CLK: track 78.0 -> 34.7 mm
- net SPI3_MOSI: track 67.5 -> 33.5 mm
- net I2S_DATA2: track 53.9 -> 39.2 mm
- net I2S_LRCK: track 51.7 -> 38.4 mm
- net I2S_DATA: track 49.3 -> 39.8 mm
- net I2S_BCK: track 47.9 -> 41.8 mm
- net I2S_MCK: track 62.6 -> 57.1 mm
- net FLASH_CS: track 26.3 -> 20.9 mm
- net DAC_CS: track 35.6 -> 32.5 mm
- net GND: track 78.2 -> 77.6 mm

Commit message: wip
Parts:
- added C52: 0.1u, microbuilder:0603
- added OSC1: 12.288MHz C3391-12.288, microbuilder:OSC_7X5MM
- added R14: 0, microbuilder:0805
- added R48: 0, microbuilder:_0805
- added TP18: (no value), microbuilder:1X01_ROUND
- moved C7 1.77 mm to (39.1, 30.4)
- moved C8 0.18 mm to (41.3, 8.26), turned to 0 degrees
Connections:
- new net I2S_CKIN: IC1.66, R14.1, R48.2, TP18.1
- new net N$11: IC1.23, R14.2
- new net N$32: OSC1.3, R48.1
- net 3.3V: now also C52.1, OSC1.4
- net GND: now also C52.2, OSC1.2
- net UART_RX: now also IC1.87; no longer IC1.88
- net UART_TX: now also IC1.86; no longer IC1.55
Routing:
- net UART_RX: track 17.7 -> 44.7 mm
- net UART_TX: track 22.4 -> 40.0 mm
- net N$11: track 0.00 -> 12.8 mm, vias 0 -> 1
- net I2S_CKIN: track 0.00 -> 9.36 mm, vias 0 -> 1
- net 3.3V: track 3.36 -> 6.61 mm, vias 1 -> 2
- net GND: track 77.6 -> 80.7 mm, vias 31 -> 33
- net N$32: track 0.00 -> 2.40 mm
- net N$3: track 2.55 -> 4.46 mm
- net DAC_CS: track 32.5 -> 33.2 mm
