File: phi-brain4ch/phi-brain4ch-ctrl.brd (EAGLE design)
At the start: 114.3 x 38.1 mm, 24 parts, among them U1 LCD-HD447804-HOLES16X2-4-HOLES

Commit message: wip
Parts:
- moved ROT1 96.5 mm to (8.89, 19.1)
- moved ROT2 96.5 mm to (105.4, 19.1)
- moved R2 55.1 mm to (18.8, 27.7), turned to 180 degrees
- moved SV1 25.1 mm to (82.3, 19.1), turned to 270 degrees
- moved C2 24.1 mm to (3.05, 10.4), turned to 270 degrees
- moved C4 22.5 mm to (100.1, 10.7), turned to 270 degrees
- moved R10 20.8 mm to (99.6, 32.3)
- moved C3 20.8 mm to (111.3, 10.2), turned to 270 degrees
- moved C1 20.6 mm to (14.7, 10.2), turned to 270 degrees
- moved R5 13.8 mm to (5.59, 14.2), turned to 180 degrees
- moved R9 11.5 mm to (102.9, 14.0), turned to 180 degrees
- moved R1 9.57 mm to (12.4, 14.0)
- moved R6 8.69 mm to (108.7, 13.7)
- moved R8 5.85 mm to (103.4, 9.14)
- moved R3 5.14 mm to (11.2, 9.40), turned to 180 degrees
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Connections:
- net LCD_D4: no longer SV1.4
- net LCD_RS: now also SV1.2
- net LCD_RW: no longer SV1.2
Routing:
- net N$15: track 0.00 -> 5.25 mm
- net N$14: track 0.00 -> 4.92 mm
- net ROT1_A: track 0.00 -> 3.49 mm
- net ROT1_B: track 0.00 -> 3.39 mm
- net 3.3V: track 0.00 -> 2.54 mm
- added copper zone on layer 16, net GND

Commit message: wip
Parts:
- added VR1: 3303W-3-103E, microbuilder:TRIMPOT_BOURNS3MM
- moved C1 5.04 mm to (11.4, 14.0), turned to 0 degrees
- moved C2 3.57 mm to (3.30, 14.0), turned to 180 degrees
- moved R1 3.42 mm to (15.0, 11.7)
- moved R5 3.42 mm to (3.30, 11.7)
- moved R9 2.03 mm to (100.8, 14.0)
- moved R10 1.37 mm to (100.1, 33.5), turned to 270 degrees
Connections:
- net GND: now also VR1.A
- net LCD_V0: now also VR1.S
- net LCD_VDD: now also VR1.E
Routing:
- net 3.3V: track 2.54 -> 171.5 mm, vias 0 -> 1
- net LCD_RS: track 0.00 -> 100.5 mm, vias 0 -> 1
- net LCD_VDD: track 0.00 -> 85.2 mm
- net ROT1_A: track 3.49 -> 81.7 mm
- net LCD_EN: track 0.00 -> 77.1 mm, vias 0 -> 2
- net LCD_D7: track 0.00 -> 76.8 mm, vias 0 -> 1
- net ROT1_B: track 3.39 -> 76.5 mm
- net LCD_V0: track 0.00 -> 71.8 mm
- net ROT1_SW: track 0.00 -> 71.0 mm
- net LCD_D5: track 0.00 -> 66.0 mm, vias 0 -> 2
- net LCD_D4: track 0.00 -> 59.1 mm, vias 0 -> 1
- net LCD_D6: track 0.00 -> 58.5 mm, vias 0 -> 2
- net LCD_RW: track 0.00 -> 45.1 mm, vias 0 -> 1
- net N$6: track 0.00 -> 41.3 mm
- net ROT2_SW: track 0.00 -> 33.1 mm
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Other:
- board text added: "Designed by Eran Rundstein"
- board text added: "phi-brain-4ch-ctrl revision 1"

Commit message: wip
Routing:
- net LCD_RS: track 100.5 -> 101.7 mm
- net LCD_D7: track 76.8 -> 75.9 mm, vias 1 -> 3

Commit message: bleh
Parts:
- R10: value 220 -> 750
Changed lines of the file:
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@@
 </element>
 <element name="JP1" library="pinhead+" package="1X03" value="" x="103.632" y="32.258" rot="MR270"/>
-<element name="R10" library="microbuilder" package="_0805" value="220" x="100.076" y="33.528" rot="MR270"/>
+<element name="R10" library="microbuilder" package="_0805" value="750" x="100.076" y="33.528" rot="MR270"/>
 <element name="R2" library="microbuilder" package="_0805" value="5" x="18.796" y="27.686" rot="MR180"/>
 <element name="VR1" library="microbuilder" package="TRIMPOT_BOURNS3MM" value="3303W-3-103E" x="29.21" y="30.48" rot="MR180"/>
