File: phi-brain4ch/phi-brain4ch-ctrl.sch (EAGLE design)
At the start: 24 parts, among them U1 LCD-HD447804-HOLES16X2-4-HOLES

Commit message: wip
Connections:
- net LCD_D4: no longer SV1.4
- net LCD_RS: now also SV1.2
- net LCD_RW: no longer SV1.2
Changed lines of the file:
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@@
 <net name="LCD_D4" class="0">
-<segment>
-<pinref part="SV1" gate="1" pin="4"/>
-<wire x1="15.24" y1="60.96" x2="5.08" y2="60.96" width="0.1524" layer="91"/>
-<label x="0" y="60.96" size="1.778" layer="95"/>
-</segment>
 <segment>
 <pinref part="U1" gate="G$1" pin="DB4"/>
@@
 <junction x="88.9" y="40.386"/>
 </segment>
+<segment>
+<pinref part="SV1" gate="1" pin="2"/>
+<wire x1="15.24" y1="58.42" x2="5.08" y2="58.42" width="0.1524" layer="91"/>
+<label x="0" y="58.42" size="1.778" layer="95"/>
+</segment>
 </net>
 <net name="LCD_D5" class="0">
@@
 <label x="38.1" y="60.96" size="1.778" layer="95"/>
 </segment>
-<segment>
-<pinref part="SV1" gate="1" pin="2"/>
-<wire x1="15.24" y1="58.42" x2="5.08" y2="58.42" width="0.1524" layer="91"/>
-<label x="0" y="58.42" size="1.778" layer="95"/>
-</segment>
-</net>
+</net>

Commit message: wip
Parts:
- added VR1: 3303W-3-103E, microbuilder:TRIMPOT10K_BOURNS
Connections:
- net GND: now also VR1.A
- net LCD_V0: now also VR1.S
- net LCD_VDD: now also VR1.E

Commit message: bleh
Parts:
- R10: value 220 -> 750
Changed lines of the file:
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@@
 <part name="3.3V9" library="microbuilder" deviceset="3.3V" device=""/>
 <part name="5.0V3" library="microbuilder" deviceset="5.0V" device=""/>
-<part name="R10" library="microbuilder" deviceset="RESISTOR" device="_0805" value="220"/>
+<part name="R10" library="microbuilder" deviceset="RESISTOR" device="_0805" value="750"/>
 <part name="3.3V3" library="microbuilder" deviceset="3.3V" device=""/>
 <part name="R2" library="microbuilder" deviceset="RESISTOR" device="_0805" value="5"/>
