File: cdf-driver/cdf-dual-driver.brd (EAGLE design)
At the start: 48.3 x 97.3 mm, 30 parts, among them IC1 R-789.0-0.5, IC2 UCC27423, Q1 FDD8424H, Q2 FDD8424H

Commit message: wip
Parts:
- added C13, C15: 1u, microbuilder:1206
- added C14, C16, C22: 0.1u, microbuilder:0805
- added C17, C18: 4.7u, rcl:C1210
- added C19: 2.2u, rcl:C1210
- added C20, C21: 330u (661-ELXZ250ELL331MH1), rcl:E3,5-8
- added D4, D5: MCL4148-TR, diode:MICROMELF-W
- added IC3: UCC27423, keves:SOIC8
- added IC4: 7805TV, linear:TO220V
- added IC5: 74AC14D, 74xx-eu:SO14
- added JP1, JP2: (no value), jumper:JP2Q
- added LED1: (no value), led:LED5MM
- added OUT1: (no value), con-ptr500:AK500/2
- added Q3, Q4: FDD8424H, keves:TO252-4
- added R5, R6: 1k, microbuilder:0805
- added R7: 15, rcl:R1210
- added R8: 470, rcl:0204/7
- GATE_IN: device con-ptr500:AK500/3 -> con-ptr500:AK500/4
- moved GATE_IN 139.4 mm to (-11.2, -60.2), turned to 0 degrees
Connections:
- new net +5V: C21.+, C22.1, IC4.3, IC5.14, R8.2
- new net N$1: C14.2, IC3.7, Q3.2
- new net N$12: C19.1, Q3.TAB, R7.1
- new net N$13: C15.2, R7.2
- new net N$14: C15.1, C19.2, OUT1.2
- new net N$15: C16.2, IC3.5, Q4.2
- new net N$16: C16.1, D5.A, Q4.5, R6.1
- new net N$17: OUT1.1, Q4.TAB
- new net N$18: LED1.A, R8.1
- new net N$19: IC2.2, JP1.3
- new net N$2: C14.1, D4.A, Q3.5, R5.1
- new net N$20: IC2.4, JP1.1
- new net N$21: IC3.2, JP2.3
- new net N$22: IC3.4, JP2.1
- new net N$23: GATE_IN.1, IC5.11
- new net N$24: IC5.10, JP1.4, JP2.4
- new net N$25: GATE_IN.3, IC5.13
- new net N$26: GATE_IN.4, IC5.12, IC5.9
- new net N$27: IC5.8, JP1.2, JP2.2
- net +24V: now also C17.1, C18.1, D4.C, D5.C, Q3.4, Q4.4, R5.2, R6.2
- net +9V: now also C13.2, C20.+, IC3.1, IC3.6, IC3.8, IC4.1
- net GND: now also C13.1, C17.2, C18.2, C20.-, C21.-, C22.2, IC3.3, IC4.2, IC5.1, IC5.3, IC5.5, IC5.7, LED1.K, Q3.1, Q4.1
Routing:
- net +9V: track 41.2 -> 102.6 mm
- net N$1: track 0.00 -> 34.1 mm
- net GND: track 24.1 -> 42.0 mm, vias 4 -> 8
- net N$17: track 0.00 -> 17.1 mm
- net N$14: track 0.00 -> 14.9 mm
- net N$15: track 0.00 -> 14.1 mm
- net N$2: track 0.00 -> 13.6 mm
- net N$16: track 0.00 -> 13.5 mm
- net +24V: track 6.14 -> 12.3 mm
- net N$13: track 0.00 -> 2.32 mm
- added copper zone on layer 1, net N$12
- added copper zone on layer 1, net N$17

Commit message: wip
Parts:
- removed LED1: (no value), led:LED5MM
- removed OUT, OUT1: (no value), con-ptr500:AK500/2
- added OUT_A, OUT_B: (no value), con-ptr500:AK500/2
- added PWR: (no value), led:LED5MM
- GATE_IN: device con-ptr500:AK500/4 -> con-ptr500:AK500/3
- R8: device rcl:0204/7 -> microbuilder:0805
- moved GATE_IN 116.6 mm to (4.06, 55.4), turned to 90 degrees
- moved JP1 114.8 mm to (16.5, 47.2)
- moved C20 99.7 mm to (21.8, 73.2), turned to 180 degrees
- moved C22 97.0 mm to (5.08, 41.7), turned to 270 degrees
- moved C21 90.6 mm to (12.7, 58.4)
- moved IC5 90.4 mm to (11.2, 39.6)
- moved JP2 90.1 mm to (15.5, 15.5)
- moved IC4 79.2 mm to (21.1, 64.3), turned to 180 degrees
- moved R8 69.2 mm to (1.78, 32.8), turned to 270 degrees
- moved C2 37.3 mm to (11.9, 70.1), turned to 0 degrees
- moved C4 31.7 mm to (34.8, 68.3)
- moved C1 25.5 mm to (13.0, 79.0), turned to 0 degrees
- moved C5 24.1 mm to (29.0, 71.5), turned to 90 degrees
- moved D1 23.2 mm to (42.8, 71.2), turned to 180 degrees
- moved IC1 18.5 mm to (36.3, 74.9), turned to 0 degrees
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Connections:
- removed net N$24 (its old number): IC5.10, JP1.4, JP2.4
- new net N$25: GATE_IN.1, IC5.9
- new net N$28: IC5.2, JP2.1
- net +5V: now also R8.1; no longer R8.2
- net GND: now also PWR.K; no longer IC5.1, LED1.K
- net N$10: now also OUT_A.1; no longer OUT.1
- net N$14: now also OUT_B.2; no longer OUT1.2
- net N$17: now also OUT_B.1; no longer OUT1.1
- net N$18: now also PWR.A, R8.2; no longer LED1.A, R8.1
- net N$19: now also JP1.4; no longer JP1.3
- net N$20: now also JP1.2; no longer JP1.1
- net N$21: now also JP2.4; no longer JP2.3
- net N$22: now also JP2.2; no longer JP2.1
- net N$23: now also IC5.12, JP1.3; no longer GATE_IN.1
- net N$26: now also IC5.10, JP1.1; no longer GATE_IN.4, IC5.12, IC5.9
- net N$27: now also IC5.1, JP2.3; no longer JP1.2, JP2.2
- net N$7: now also OUT_A.2; no longer OUT.2
Routing:
- net +5V: track 0.00 -> 47.2 mm, vias 0 -> 2
- net N$27: track 0.00 -> 45.4 mm
- net N$25: track 0.00 -> 26.0 mm
- net N$28: track 0.00 -> 24.6 mm
- net N$24: track 0.00 -> 19.6 mm
- net GND: track 42.0 -> 53.7 mm, vias 8 -> 12
- net N$23: track 0.00 -> 8.77 mm
- net +9V: track 102.6 -> 110.9 mm
- net N$26: track 0.00 -> 4.88 mm
- net N$18: track 0.00 -> 4.00 mm
- net N$22: track 0.00 -> 3.80 mm
- net N$21: track 0.00 -> 3.80 mm
- net N$17: track 17.1 -> 14.3 mm
- net N$20: track 0.00 -> 2.79 mm
- net N$19: track 0.00 -> 2.79 mm
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Other:
- board size 48.3 x 97.3 mm -> 48.3 x 83.3 mm
- board text added: "CDF Dual Driver"
- board text added: "Rev 1 - Jul 2017"
- board text removed: "CDF Single Driver"
- board text removed: "Rev 1 - Apr 2017"

Commit message: wip
Parts:
- C10, C9: value 4.7u -> 1u; device rcl:C1210 -> microbuilder:1206
- C11: value 2.2u -> 0.1u; device rcl:C1210 -> microbuilder:0805
- C12, C13: value 1u -> 0.1u; device microbuilder:1206 -> microbuilder:0805
- C15: value 1u -> 4.7u; device microbuilder:1206 -> rcl:C1210
- C16: value 0.1u -> 4.7u; device microbuilder:0805 -> rcl:C1210
- C20: value 330u (661-ELXZ250ELL331MH1) -> 2.2u; device rcl:E3,5-8 -> rcl:C1210
- C21: value 330u (661-ELXZ250ELL331MH1) -> 1u; device rcl:E3,5-8 -> microbuilder:1206
- C22: value 0.1u -> 1u; device microbuilder:0805 -> microbuilder:1206
- C3: value 4.7u -> 330u (661-ELXZ250ELL331MH1); device rcl:C1210 -> rcl:E3,5-8
- C4: value 330u (661-ELXZ250ELL331MH1) -> 4.7u; device rcl:E3,5-8 -> rcl:C1210
- C5: value 0.1u -> 330u (661-ELXZ250ELL331MH1); device microbuilder:0805 -> rcl:E3,5-8
- C6: value 1u -> 330u (661-ELXZ250ELL331MH1); device microbuilder:1206 -> rcl:E3,5-8
- IC2: value UCC27423 -> 7805TV; device keves:SOIC8 -> linear:TO220V
- IC3: value UCC27423 -> 74AC14D; device keves:SOIC8 -> 74xx-eu:SO14
- IC4: value 7805TV -> UCC27423; device linear:TO220V -> keves:SOIC8
- IC5: value 74AC14D -> UCC27423; device 74xx-eu:SO14 -> keves:SOIC8
- R2: value 1k -> 470
- R4: value 15 -> 1k; device rcl:R1210 -> microbuilder:0805
- R8: value 470 -> 15; device microbuilder:0805 -> rcl:R1210
- moved C11 54.7 mm to (21.2, 8.38)
- moved C18 51.2 mm to (26.4, 61.7)
- moved D5 50.9 mm to (23.9, 55.4)
- moved Q4 50.9 mm to (27.2, 56.9)
- moved R3 50.9 mm to (21.6, 4.95)
- moved R6 50.9 mm to (21.6, 55.9)
- moved IC4 48.3 mm to (23.1, 16.0), turned to 270 degrees
- moved C21 47.1 mm to (45.2, 24.4), turned to 270 degrees
- moved R8 45.8 mm to (41.7, 55.4), turned to 0 degrees
- moved C22 42.8 mm to (45.2, 56.4)
- moved C16 33.9 mm to (26.4, 41.9)
- moved C14 32.0 mm to (21.6, 60.2)
- moved C7 32.0 mm to (29.0, 71.5)
- moved D2 31.4 mm to (23.9, 4.45)
- moved Q1 31.4 mm to (27.2, 5.97)
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- renumbered OUT_A to X4, OUT_B to X3, X1 to X2
Connections:
- net +24V: now also C15.1, C16.1, C4.2, R4.2; no longer C10.1, C3.2, C9.1, R2.2
- net +5V: now also C6.+, C8.1, IC2.3, IC3.14, R2.1; no longer C21.+, C22.1, IC4.3, IC5.14, R8.1
- net +9V: now also C10.2, C3.+, C5.+, C7.1, C9.2, IC4.6, IC4.8, IC5.1, IC5.6, IC5.8; no longer C13.2, C20.+, C4.+, C5.1, C6.2, IC2.6, IC2.8, IC3.1, IC3.6, IC3.8
- net GND: now also C10.1, C15.2, C16.2, C3.-, C5.-, C6.-, C7.2, C8.2, C9.1, IC2.2, IC3.5, IC3.7, IC4.3; no longer C10.2, C13.1, C20.-, C21.-, C22.2, C4.-, C5.2, C6.1, C9.2, IC2.3, IC4.2, IC5.5, IC5.7
- net N$1: now also C13.2, IC4.7; no longer C14.2, IC3.7
- net N$10: now also Q2.TAB; no longer Q1.TAB
- net N$11: now also C4.1; no longer C3.1
- net N$13: now also C21.2; no longer C15.2
- net N$14: now also C21.1; no longer C15.1
- net N$15: now also C11.2, IC4.5, Q1.2; no longer C16.2, IC3.5, Q4.2
- net N$16: now also C11.1, D2.A, Q1.5, R3.1; no longer C16.1, D5.A, Q4.5, R6.1
- net N$17: now also Q1.TAB; no longer Q4.TAB
- net N$18: now also R2.2; no longer R8.2
- net N$19: now also IC5.2; no longer IC2.2
- net N$2: now also C13.1; no longer C14.1
- net N$20: now also IC5.4; no longer IC2.4
- net N$21: now also IC4.2; no longer IC3.2
- net N$22: now also IC4.4; no longer IC3.4
- net N$23: now also IC3.11, IC3.12; no longer IC5.11, IC5.12
- net N$24: now also GATE_IN.1, IC3.13; no longer GATE_IN.3, IC5.13
- net N$25: now also GATE_IN.3, IC3.9; no longer GATE_IN.1, IC5.9
- net N$26: now also IC3.10; no longer IC5.10
- net N$27: now also IC3.1, IC3.8; no longer IC5.1, IC5.8
- net N$28: now also IC3.2; no longer IC5.2
- net N$3: now also C14.2, IC5.7, Q4.2; no longer C8.2, IC2.7, Q2.2
- net N$4: now also C14.1, D5.A, Q4.5, R6.1; no longer C8.1, D3.A, Q2.5, R3.1
- net N$5: now also C20.1, Q4.TAB, R8.1; no longer C11.1, Q2.TAB, R4.1
- net N$6: now also C22.2, R8.2; no longer C12.2, R4.2
- net N$7: now also C20.2, C22.1; no longer C11.2, C12.1
- net N$8: now also C12.2, IC5.5, Q2.2; no longer C7.2, IC2.5, Q1.2
- net N$9: now also C12.1, D3.A, Q2.5, R4.1; no longer C7.1, D2.A, Q1.5, R2.1
Routing:
- net N$24: track 19.6 -> 20.5 mm
- net N$25: track 26.0 -> 26.5 mm
