File: cdf-driver/cdf-dual-driver.sch (EAGLE design)
At the start: 30 parts, among them IC1 R-789.0-0.5, IC2 UCC27423, Q1 FDD8424H, Q2 FDD8424H

Commit message: wip
Parts:
- added C13, C15: 1u, microbuilder:CAP_CERAMIC1206
- added C14, C16, C22: 0.1u, microbuilder:CAP_CERAMIC0805
- added C17, C18: 4.7u, rcl:C-EUC1210
- added C19: 2.2u, rcl:C-EUC1210
- added C20, C21: 330u (661-ELXZ250ELL331MH1), rcl:CPOL-USE3.5-8
- added D4, D5: MCL4148-TR, diode:DIODE-MICROMELF-W
- added IC3: UCC27423, keves:UCC27423
- added IC4: 7805TV, linear:7805TV
- added IC5: 74AC14D, 74xx-eu:74AC14D
- added JP1, JP2: (no value), jumper:JP2Q
- added LED1: (no value), led:LED5MM
- added OUT1: (no value), con-ptr500:AK500/2
- added Q3, Q4: FDD8424H, keves:FDD8424H
- added R5, R6: 1k, microbuilder:RESISTOR0805
- added R7: 15, rcl:R-US_R1210
- added R8: 470, rcl:R-US_0204/7
- GATE_IN: device con-ptr500:AK500/3 -> con-ptr500:AK500/4
Connections:
- new net +5V: C21.+, C22.P$1, IC4.VO, IC5P.VCC, R8.2
- new net N$1: C14.P$2, IC3.OUTA, Q3.LSG
- new net N$12: C19.1, Q3.TAB, R7.1
- new net N$13: C15.P$2, R7.2
- new net N$14: C15.P$1, C19.2, OUT1-2.KL
- new net N$15: C16.P$2, IC3.OUTB, Q4.LSG
- new net N$16: C16.P$1, D5.A, Q4.HSG, R6.1
- new net N$17: OUT1-1.KL, Q4.TAB
- new net N$18: LED1.A, R8.1
- new net N$19: IC2.INA, JP1.3
- new net N$2: C14.P$1, D4.A, Q3.HSG, R5.1
- new net N$20: IC2.INB, JP1.1
- new net N$21: IC3.INA, JP2.3
- new net N$22: IC3.INB, JP2.1
- new net N$23: GATE_IN-1.KL, IC5B.I
- new net N$24: IC5B.O, JP1.4, JP2.4
- new net N$25: GATE_IN-3.KL, IC5A.I
- new net N$26: GATE_IN-4.KL, IC5A.O, IC5C.I
- new net N$27: IC5C.O, JP1.2, JP2.2
- net +24V: now also C17.1, C18.1, D4.C, D5.C, Q3.VCC, Q4.VCC, R5.2, R6.2
- net +9V: now also C13.P$2, C20.+, IC3.ENA, IC3.ENB, IC3.VCC, IC4.VI
- net GND: now also C13.P$1, C17.2, C18.2, C20.-, C21.-, C22.P$2, IC3.GND, IC4.GND, IC5D.I, IC5E.I, IC5F.I, IC5P.GND, LED1.C, Q3.GND, Q4.GND
Other:
- moved on the sheet: GATE_IN-1, GATE_IN-2, GATE_IN-3

Commit message: wip
Parts:
- GATE_IN: device con-ptr500:AK500/4 -> con-ptr500:AK500/3
- R8: device rcl:R-US_0204/7 -> microbuilder:RESISTOR0805
- renumbered LED1 to PWR, OUT to OUT_A, OUT1 to OUT_B
Connections:
- removed net N$24 (its old number): IC5B.O, JP1.4, JP2.4
- new net N$25: GATE_IN-1.KL, IC5C.I
- new net N$28: IC5D.O, JP2.1
- net +5V: now also R8.1; no longer R8.2
- net GND: no longer IC5D.I
- net N$18: now also R8.2; no longer R8.1
- net N$19: now also JP1.4; no longer JP1.3
- net N$20: now also JP1.2; no longer JP1.1
- net N$21: now also JP2.4; no longer JP2.3
- net N$22: now also JP2.2; no longer JP2.1
- net N$23: now also IC5A.O, JP1.3; no longer GATE_IN-1.KL
- net N$26: now also IC5B.O, JP1.1; no longer GATE_IN-4.KL, IC5A.O, IC5C.I
- net N$27: now also IC5D.I, JP2.3; no longer JP1.2, JP2.2
Other:
- moved on the sheet: GATE_IN-1, GATE_IN-2, GATE_IN-3, IC5A, IC5B, IC5C, IC5D, JP1, JP2

Commit message: wip
Parts:
- C10, C9: value 4.7u -> 1u; device rcl:C-EUC1210 -> microbuilder:CAP_CERAMIC1206
- C11: value 2.2u -> 0.1u; device rcl:C-EUC1210 -> microbuilder:CAP_CERAMIC0805
- C12, C13: value 1u -> 0.1u; device microbuilder:CAP_CERAMIC1206 -> microbuilder:CAP_CERAMIC0805
- C15: value 1u -> 4.7u; device microbuilder:CAP_CERAMIC1206 -> rcl:C-EUC1210
- C16: value 0.1u -> 4.7u; device microbuilder:CAP_CERAMIC0805 -> rcl:C-EUC1210
- C20: value 330u (661-ELXZ250ELL331MH1) -> 2.2u; device rcl:CPOL-USE3.5-8 -> rcl:C-EUC1210
- C21: value 330u (661-ELXZ250ELL331MH1) -> 1u; device rcl:CPOL-USE3.5-8 -> microbuilder:CAP_CERAMIC1206
- C22: value 0.1u -> 1u; device microbuilder:CAP_CERAMIC0805 -> microbuilder:CAP_CERAMIC1206
- C3: value 4.7u -> 330u (661-ELXZ250ELL331MH1); device rcl:C-EUC1210 -> rcl:CPOL-USE3.5-8
- C4: value 330u (661-ELXZ250ELL331MH1) -> 4.7u; device rcl:CPOL-USE3.5-8 -> rcl:C-EUC1210
- C5: value 0.1u -> 330u (661-ELXZ250ELL331MH1); device microbuilder:CAP_CERAMIC0805 -> rcl:CPOL-USE3.5-8
- C6: value 1u -> 330u (661-ELXZ250ELL331MH1); device microbuilder:CAP_CERAMIC1206 -> rcl:CPOL-USE3.5-8
- IC2: value UCC27423 -> 7805TV; device keves:UCC27423 -> linear:7805TV
- IC3: value UCC27423 -> 74AC14D; device keves:UCC27423 -> 74xx-eu:74AC14D
- IC4: value 7805TV -> UCC27423; device linear:7805TV -> keves:UCC27423
- IC5: value 74AC14D -> UCC27423; device 74xx-eu:74AC14D -> keves:UCC27423
- R2: value 1k -> 470
- R4: value 15 -> 1k; device rcl:R-US_R1210 -> microbuilder:RESISTOR0805
- R8: value 470 -> 15; device microbuilder:RESISTOR0805 -> rcl:R-US_R1210
- renumbered OUT_A to X4, OUT_B to X3, X1 to X2
Connections:
- net +24V: now also C15.1, C16.1, C4.2, R4.2; no longer C10.1, C3.2, C9.1, R2.2
- net +5V: now also C6.+, C8.P$1, IC2.VO, IC3P.VCC, R2.1; no longer C21.+, C22.P$1, IC4.VO, IC5P.VCC, R8.1
- net +9V: now also C10.P$2, C3.+, C5.+, C7.P$1, C9.P$2, IC2.VI, IC4.ENA, IC4.ENB, IC4.VCC, IC5.ENA, IC5.ENB, IC5.VCC; no longer C13.P$2, C20.+, C4.+, C5.P$1, C6.P$2, IC2.ENA, IC2.ENB, IC2.VCC, IC3.ENA, IC3.ENB, IC3.VCC, IC4.VI
- net GND: now also C10.P$1, C15.2, C16.2, C3.-, C5.-, C6.-, C7.P$2, C8.P$2, C9.P$1, IC3E.I, IC3F.I, IC3P.GND, IC5.GND; no longer C10.2, C13.P$1, C20.-, C21.-, C22.P$2, C4.-, C5.P$2, C6.P$1, C9.2, IC3.GND, IC5E.I, IC5F.I, IC5P.GND
- net N$1: now also C13.P$2, IC4.OUTA; no longer C14.P$2, IC3.OUTA
- net N$10: now also Q2.TAB; no longer Q1.TAB
- net N$11: now also C4.1; no longer C3.1
- net N$13: now also C21.P$2; no longer C15.P$2
- net N$14: now also C21.P$1; no longer C15.P$1
- net N$15: now also C11.P$2, IC4.OUTB, Q1.LSG; no longer C16.P$2, IC3.OUTB, Q4.LSG
- net N$16: now also C11.P$1, D2.A, Q1.HSG, R3.1; no longer C16.P$1, D5.A, Q4.HSG, R6.1
- net N$17: now also Q1.TAB; no longer Q4.TAB
- net N$18: now also R2.2; no longer R8.2
- net N$19: now also IC5.INA; no longer IC2.INA
- net N$2: now also C13.P$1; no longer C14.P$1
- net N$20: now also IC5.INB; no longer IC2.INB
- net N$21: now also IC4.INA; no longer IC3.INA
- net N$22: now also IC4.INB; no longer IC3.INB
- net N$23: now also IC3A.O, IC3B.I; no longer IC5A.O, IC5B.I
- net N$24: now also GATE_IN-1.KL, IC3A.I; no longer GATE_IN-3.KL, IC5A.I
- net N$25: now also GATE_IN-3.KL, IC3C.I; no longer GATE_IN-1.KL, IC5C.I
- net N$26: now also IC3B.O; no longer IC5B.O
- net N$27: now also IC3C.O, IC3D.I; no longer IC5C.O, IC5D.I
- net N$28: now also IC3D.O; no longer IC5D.O
- net N$3: now also C14.P$2, IC5.OUTA, Q4.LSG; no longer C8.P$2, IC2.OUTA, Q2.LSG
- net N$4: now also C14.P$1, D5.A, Q4.HSG, R6.1; no longer C8.P$1, D3.A, Q2.HSG, R3.1
- net N$5: now also C20.1, Q4.TAB, R8.1; no longer C11.1, Q2.TAB, R4.1
- net N$6: now also C22.P$2, R8.2; no longer C12.P$2, R4.2
- net N$7: now also C20.2, C22.P$1; no longer C11.2, C12.P$1
- net N$8: now also C12.P$2, IC5.OUTB, Q2.LSG; no longer C7.P$2, IC2.OUTB, Q1.LSG
- net N$9: now also C12.P$1, D3.A, Q2.HSG, R4.1; no longer C7.P$1, D2.A, Q1.HSG, R2.1
Other:
- moved on the sheet: C10, C11, C12, C13, C14, C15, C16, C18, C22, C7, C8, C9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
