File: dual-led-wireless-dimmer/dual-led-wireless-dimmer-tx.brd (EAGLE design)
At the start: 100 x 80 mm, 17 parts, among them J1 AVR_SPI_PRG_6PTH, U1 ATMEGA328P_TQFP, X1 PTL45, X2 PTL45, Y1 8MHz

Commit message: wip
Parts:
- added C10: 100uF, microbuilder:PANASONIC_D
- added C11: 10uF, microbuilder:0805
- added C12: 0.1uF, microbuilder:0805
- added C6: 4.7uF, microbuilder:0805
- added D1: 17V (1N5247B), diode:ZDIO-5
- added D2: 24v 1N5359B, diode:ZDIO-10
- added F1: KEYSTONE-3557-2, keves-ng:KEYSTONE-3557-2
- added IC1: LM2937IMP-3.3, linear:TO263-3
- added JP1: (no value), pinhead:2X04
- added JP2: (no value), pinhead:1X03
- added L1: 5248-RC, rcl:0207/5V
- added Q1: DN2625K4-G, SparkFun-DiscreteSemi:DPAK
- added Q2: SI2323DS-T1-E3, SparkFun-DiscreteSemi:SOT23-3
- added Q3, Q4: IRF520NPBF, Seeed-Transistor-2016:TO-220
- added R10, R11, R9: 10k, microbuilder:0805
- added R4, R5, R6: 220, microbuilder:0805
- added R7: 100k, microbuilder:0805
- added R8: 39k, microbuilder:0805
- added SJ1, SJ2, SJ3: (no value), jumper:SJW
- added X3, X4, X5: AK550/2, con-ptr500:AK550/2
- added ZD1: 7.5v BZT52C7V5-7-F, diodes:SOD123
Connections:
- new net 12V: F1.R1, F1.R2, Q1.4, R7.2, X4.2, X5.2
- new net ADC0: U1.23, X1.2
- new net ADC1: U1.24, X2.2
- new net CE: JP1.3, U1.1
- new net CSN: JP1.4, R9.1, U1.2
- new net IRQ: JP1.8, U1.32
- new net N$10: JP1.5, R4.2
- new net N$11: D1.C, Q1.1, R7.1
- new net N$12: SJ1.1, U1.27
- new net N$13: Q1.3, Q2.3
- new net N$14: Q2.1, R8.1, ZD1.A
- new net N$15: D2.C, L1.1, Q2.2, ZD1.C
- new net N$16: SJ2.1, U1.28
- new net N$17: C10.+, C12.1, IC1.1, L1.2
- new net N$18: SJ3.1, U1.19
- new net N$19: JP2.3, U1.31
- new net N$20: JP2.2, U1.30
- new net N$5: F1.L1, F1.L2, X3.2
- new net N$6: Q3.3, X4.1
- new net N$7: JP1.6, R5.1
- new net N$8: Q4.3, X5.1
- new net N$9: JP1.7, R6.2
- new net PWM1: Q3.1, R10.1, U1.13
- new net PWM2: Q4.1, R11.1, U1.14
- net 3.3V: now also C11.1, C6.2, IC1.3, JP1.2, R9.2
- net GND: now also C10.-, C11.2, C12.2, C6.1, D1.A, D2.A, IC1.2, JP1.1, JP2.1, Q3.2, Q3.HEAT, Q4.2, Q4.HEAT, R10.2, R11.2, R8.2, SJ1.2, SJ2.2, SJ3.2, X3.1
- net MISO: now also R6.1
- net MOSI: now also R5.2
- net SCK: now also R4.1

Commit message: wip
Parts:
- removed C10: 100uF, microbuilder:PANASONIC_D
- removed C11: 10uF, microbuilder:0805
- removed C12, C3: 0.1uF, microbuilder:0805
- removed JP1: (no value), pinhead:2X04
- removed X1, X2: PTL45, keves-ng:BOURNS-PTL45
- removed X3, X4, X5: AK550/2, con-ptr500:AK550/2
- added C7: 100uF, microbuilder:PANASONIC_D
- added C8: 0.1uF, microbuilder:0805
- added C9: 10uF, microbuilder:0805
- added CH1, CH2: PTL45, keves-ng:BOURNS-PTL45
- added IN, OUT1, OUT2: AK550/2, con-ptr500:AK550/2
- added NRF24L01: (no value), pinhead:2X04
- C1, C2: value 22pF -> 0.1uF
- C4, C5: value 0.1uF -> 22pF
- R1: value 10k -> 150
- R3: value 150 -> 100k
- R4: value 220 -> 39k
- R5: value 220 -> 10k
- R7: value 100k -> 10k
- R8: value 39k -> 220
- R9: value 10k -> 220
- moved SJ3 599.4 mm to (30.0, 47.2), flipped to the bottom, turned to 180 degrees
- moved SJ2 593.7 mm to (30.0, 43.4), flipped to the bottom, turned to 180 degrees
- moved R11 590.8 mm to (24.1, 57.1), flipped to the bottom, turned to 180 degrees
- moved JP2 589.4 mm to (8.64, 31.5), turned to 90 degrees
- moved SJ1 588.1 mm to (30.0, 39.6), flipped to the bottom, turned to 180 degrees
- moved Q4 561.9 mm to (25.4, 64.8)
- moved R10 512.6 mm to (11.4, 57.1), flipped to the bottom, turned to 180 degrees
- moved Q3 464.6 mm to (12.7, 64.8)
- moved R9 399.8 mm to (20.6, 34.0), turned to 90 degrees
- moved IC1 372.3 mm to (31.8, 29.2), flipped to the bottom
- moved L1 342.0 mm to (21.6, 21.6), flipped to the bottom, turned to 180 degrees
- moved R8 328.1 mm to (22.9, 34.0), turned to 270 degrees
- moved ZD1 319.8 mm to (5.08, 26.7), flipped to the bottom
- moved D2 315.3 mm to (1.27, 15.2), flipped to the bottom, turned to 270 degrees
- moved Q2 303.3 mm to (5.08, 20.3), flipped to the bottom, turned to 180 degrees
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Connections:
- removed net N$10: JP1.5, R4.2
- new net JP1: NRF24L01.5, R9.2
- net 12V: now also OUT1.2, OUT2.2, R3.2; no longer R7.2, X4.2, X5.2
- net 3.3V: now also C1.2, C2.2, C9.1, CH1.1, CH2.1, NRF24L01.2, R1.1, R5.2, R7.2; no longer C11.1, C3.2, C4.2, C5.2, JP1.2, R1.2, R3.1, R9.2, X1.1, X2.1
- net ADC0: now also CH1.2; no longer X1.2
- net ADC1: now also CH2.2; no longer X2.2
- net CE: now also NRF24L01.3; no longer JP1.3
- net CSN: now also NRF24L01.4, R7.1; no longer JP1.4, R9.1
- net GND: now also C2.1, C4.2, C7.-, C8.2, C9.2, CH1.3, CH1.E, CH2.3, CH2.E, IN.1, NRF24L01.1, R4.2; no longer C10.-, C11.2, C12.2, C2.2, C3.1, C4.1, JP1.1, R8.2, X1.3, X1.E, X2.3, X2.E, X3.1
- net IRQ: now also NRF24L01.8; no longer JP1.8
- net MISO: now also R8.1; no longer R6.1
- net MOSI: now also R6.2; no longer R5.2
- net N$1: now also C5.2; no longer C1.2
- net N$11: now also R3.1; no longer R7.1
- net N$14: now also R4.1; no longer R8.1
- net N$17: now also C7.+, C8.1; no longer C10.+, C12.1
- net N$2: now also C4.1; no longer C2.1
- net N$3: now also CH1.B, R1.2; no longer R2.2, X1.B
- net N$4: now also CH2.B, R2.2; no longer R3.2, X2.B
- net N$5: now also IN.2; no longer X3.2
- net N$6: now also OUT1.1; no longer X4.1
- net N$7: now also NRF24L01.6, R6.1; no longer JP1.6, R5.1
- net N$8: now also OUT2.1; no longer X5.1
- net N$9: now also NRF24L01.7, R8.2; no longer JP1.7, R6.2
- net RESET: now also R5.1; no longer R1.1
- net SCK: now also R9.1; no longer R4.1
Routing:
- added copper zone on layer 16, net GND
Other:
- board size 100 x 80 mm -> 38.1 x 76.2 mm

Commit message: wip
Parts:
- moved C5 10.7 mm to (1.52, 39.6), turned to 270 degrees
- moved Y1 5.38 mm to (4.32, 43.2)
- moved C4 2.29 mm to (1.52, 47.0), turned to 270 degrees
- moved C1 1.63 mm to (8.64, 36.8), turned to 90 degrees
- moved JP2 1.44 mm to (9.65, 30.5)
- moved R3 0.25 mm to (11.2, 20.3), turned to 0 degrees
Changed lines of the file:
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@@
 </variantdefs>
 <classes>
-<class number="0" name="default" width="0" drill="0">
+<class number="0" name="default" width="0.254" drill="0">
+</class>
+<class number="1" name="3.3v" width="0.4064" drill="0">
 </class>
 </classes>
@@
 <param name="RoutingGrid" value="50mil"/>
 <param name="AutoGrid" value="1"/>
-<param name="Efforts" value="0"/>
+<param name="Efforts" value="2"/>
 <param name="TopRouterVariant" value="1"/>
 <param name="tpViaShape" value="round"/>
@@
 <attribute name="PROD_ID" value="IC-09069" x="15.24" y="38.1" size="1.778" layer="28" rot="MR180" display="off"/>
 </element>
-<element name="Y1" library="SparkFun-FreqCtrl" package="HC49UP" value="8MHz" x="2.54" y="38.1" rot="MR270"/>
-<element name="C5" library="microbuilder" package="0805" value="22pF" x="3.81" y="29.21" rot="MR0"/>
-<element name="C4" library="microbuilder" package="0805" value="22pF" x="3.81" y="46.99" rot="MR180"/>
+<element name="Y1" library="SparkFun-FreqCtrl" package="HC49UP" value="8MHz" x="4.318" y="43.18" rot="MR270"/>
+<element name="C5" library="microbuilder" package="0805" value="22pF" x="1.524" y="39.624" rot="MR270"/>
+<element name="C4" library="microbuilder" package="0805" value="22pF" x="1.524" y="46.99" rot="MR270"/>
 <element name="R5" library="microbuilder" package="0805" value="10k" x="25.146" y="47.498" rot="MR90"/>
 <element name="J1" library="SparkFun-Connectors" package="2X3" value="AVR_SPI_PRG_6PTH" x="17.018" y="46.482"/>
-<element name="C1" library="microbuilder" package="0805" value="0.1uF" x="7.62" y="38.1" rot="MR180"/>
+<element name="C1" library="microbuilder" package="0805" value="0.1uF" x="8.636" y="36.83" rot="MR90"/>
 <element name="C2" library="microbuilder" package="0805" value="0.1uF" x="22.86" y="39.37" rot="MR270"/>
 <element name="R1" library="microbuilder" package="0805" value="150" x="11.684" y="62.738" rot="MR180"/>
@@
 <attribute name="PROD_ID" value="TRANS-09984" x="11.43" y="15.24" size="1.778" layer="28" rot="MR90" display="off"/>
 </element>
-<element name="R3" library="microbuilder" package="0805" value="100k" x="11.43" y="20.32" rot="MR180"/>
+<element name="R3" library="microbuilder" package="0805" value="100k" x="11.176" y="20.32" rot="MR0"/>
 <element name="D1" library="diode" library_urn="urn:adsk.eagle:library:210" package="ZDIO-5" package3d_urn="urn:adsk.eagle:package:43412/1" value="17V (1N5247B)" x="14.732" y="22.86" rot="MR90"/>
 <element name="Q2" library="SparkFun-DiscreteSemi" package="SOT23-3" value="SI2323DS-T1-E3" x="5.08" y="20.32" rot="MR180">
@@
 <element name="SJ2" library="jumper" library_urn="urn:adsk.eagle:library:252" package="SJW" package3d_urn="urn:adsk.eagle:package:15507/1" value="" x="29.972" y="43.434" rot="MR180"/>
 <element name="SJ3" library="jumper" library_urn="urn:adsk.eagle:library:252" package="SJW" package3d_urn="urn:adsk.eagle:package:15507/1" value="" x="29.972" y="47.244" rot="MR180"/>
-<element name="JP2" library="pinhead" library_urn="urn:adsk.eagle:library:325" package="1X03" package3d_urn="urn:adsk.eagle:package:22458/2" value="" x="8.636" y="31.496" rot="R90"/>
+<element name="JP2" library="pinhead" library_urn="urn:adsk.eagle:library:325" package="1X03" package3d_urn="urn:adsk.eagle:package:22458/2" value="" x="9.652" y="30.48" rot="R90"/>
 </elements>
 <signals>
@@
 <contactref element="Y1" pad="2"/>
 <contactref element="C5" pad="2"/>
-<wire x1="2.54" y1="33.274" x2="10.9474" y2="40.1" width="0" layer="19" extent="16-16"/>
-<wire x1="2.86" y1="29.21" x2="2.54" y2="33.274" width="0" layer="19" extent="16-16"/>
+<wire x1="4.318" y1="38.354" x2="10.9474" y2="40.1" width="0" layer="19" extent="16-16"/>
+<wire x1="1.524" y1="38.674" x2="4.318" y2="38.354" width="0" layer="19" extent="16-16"/>
 </signal>
 <signal name="N$2">
@@
 <contactref element="Y1" pad="1"/>
 <contactref element="C4" pad="1"/>
-<wire x1="2.54" y1="42.926" x2="10.9474" y2="40.9" width="0" layer="19" extent="16-16"/>
-<wire x1="2.86" y1="46.99" x2="2.54" y2="42.926" width="0" layer="19" extent="16-16"/>
+<wire x1="4.318" y1="48.006" x2="10.9474" y2="40.9" width="0" layer="19" extent="16-16"/>
+<wire x1="1.524" y1="47.94" x2="4.318" y2="48.006" width="0" layer="19" extent="16-16"/>
 </signal>
 <signal name="GND">
@@
 <contactref element="SJ3" pad="2"/>
 <contactref element="JP2" pad="1"/>
-<polygon width="0.1524" layer="16">
+<polygon width="0.254" layer="16">
 <vertex x="-3.81" y="77.47"/>
 <vertex x="41.91" y="77.47"/>
@@
 <vertex x="-2.54" y="76.2"/>
 </polygon>
-<wire x1="31.242" y1="43.434" x2="31.242" y2="39.624" width="0" layer="19" extent="1-1"/>
-<wire x1="31.242" y1="47.244" x2="31.242" y2="43.434" width="0" layer="19" extent="1-1"/>
-<wire x1="8.636" y1="28.956" x2="31.242" y2="43.434" width="0" layer="19" extent="1-1"/>
-<wire x1="27.96" y1="65.6" x2="31.242" y2="47.244" width="0" layer="19" extent="1-1"/>
 </signal>
 <signal name="3.3V">
@@
 <wire x1="10.9474" y1="39.3" x2="19.5326" y2="40.1" width="0" layer="19" extent="16-16"/>
 <wire x1="10.9474" y1="37.7" x2="10.9474" y2="39.3" width="0" layer="19" extent="16-16"/>
-<wire x1="8.57" y1="38.1" x2="10.9474" y2="37.7" width="0" layer="19" extent="16-16"/>
+<wire x1="8.636" y1="37.78" x2="10.9474" y2="37.7" width="0" layer="19" extent="16-16"/>
 <wire x1="12.446" y1="28.006" x2="10.9474" y2="37.7" width="0" layer="19" extent="16-16"/>
 <wire x1="15.24" y1="27.94" x2="12.446" y2="28.006" width="0" layer="19" extent="16-16"/>
@@
 <contactref element="Q1" pad="1"/>
 <contactref element="D1" pad="C"/>
-<wire x1="10.48" y1="20.32" x2="14.732" y2="20.32" width="0" layer="19" extent="16-16"/>
-<wire x1="6.12" y1="12.96" x2="10.48" y2="20.32" width="0" layer="19" extent="16-16"/>
+<wire x1="12.126" y1="20.32" x2="14.732" y2="20.32" width="0" layer="19" extent="16-16"/>
+<wire x1="6.12" y1="12.96" x2="12.126" y2="20.32" width="0" layer="19" extent="16-16"/>
 </signal>
 <signal name="N$13">
@@
 <contactref element="OUT2" pad="2"/>
 <wire x1="2.54" y1="56.36" x2="35.56" y2="52.86" width="0" layer="19" extent="1-1"/>
-<wire x1="12.38" y1="20.32" x2="2.54" y2="56.36" width="0" layer="19" extent="16-16"/>
-<wire x1="13.018" y1="15.24" x2="12.38" y2="20.32" width="0" layer="19" extent="16-16"/>
+<wire x1="10.226" y1="20.32" x2="2.54" y2="56.36" width="0" layer="19" extent="16-16"/>
+<wire x1="13.018" y1="15.24" x2="10.226" y2="20.32" width="0" layer="19" extent="16-16"/>
 <wire x1="18.6182" y1="16.891" x2="13.018" y2="15.24" width="0" layer="19" extent="16-16"/>
 <wire x1="22.0218" y1="16.891" x2="18.6182" y2="16.891" width="0" layer="19" extent="1-1"/>
@@
 <contactref element="SJ1" pad="1"/>
 <contactref element="U1" pad="27"/>
-<wire x1="16.44" y1="33.8074" x2="28.702" y2="39.624" width="0" layer="19" extent="1-16"/>
+<wire x1="16.44" y1="33.8074" x2="28.702" y2="39.624" width="0" layer="19" extent="16-16"/>
 </signal>
 <signal name="N$16">
 <contactref element="SJ2" pad="1"/>
 <contactref element="U1" pad="28"/>
-<wire x1="15.64" y1="33.8074" x2="28.702" y2="43.434" width="0" layer="19" extent="1-16"/>
+<wire x1="15.64" y1="33.8074" x2="28.702" y2="43.434" width="0" layer="19" extent="16-16"/>
 </signal>
 <signal name="N$18">
 <contactref element="SJ3" pad="1"/>
 <contactref element="U1" pad="19"/>
-<wire x1="19.5326" y1="39.3" x2="28.702" y2="47.244" width="0" layer="19" extent="1-16"/>
+<wire x1="19.5326" y1="39.3" x2="28.702" y2="47.244" width="0" layer="19" extent="16-16"/>
 </signal>
 <signal name="N$19">
 <contactref element="U1" pad="31"/>
 <contactref element="JP2" pad="3"/>
-<wire x1="13.24" y1="33.8074" x2="8.636" y2="34.036" width="0" layer="19" extent="16-16"/>
+<wire x1="9.652" y1="33.02" x2="13.24" y2="33.8074" width="0" layer="19" extent="16-16"/>
 </signal>
 <signal name="N$20">
 <contactref element="U1" pad="30"/>
 <contactref element="JP2" pad="2"/>
-<wire x1="14.04" y1="33.8074" x2="8.636" y2="31.496" width="0" layer="19" extent="16-16"/>
+<wire x1="9.652" y1="30.48" x2="14.04" y2="33.8074" width="0" layer="19" extent="16-16"/>
 </signal>
 </signals>

Commit message: routed
Parts:
- removed C4, C5: 22pF, microbuilder:0805
- removed SJ3: (no value), jumper:SJW
- removed Y1: 8MHz, SparkFun-FreqCtrl:HC49UP
- added SJ4: SOLDERJUMPERNO, SparkFun-Retired:SJ_2S-NO
- SJ1, SJ2: value (none) -> SOLDERJUMPERNO; device jumper:SJW -> SparkFun-Retired:SJ_2S-NO
- moved SJ1 22.6 mm to (7.62, 36.1), turned to 270 degrees
- moved C2 20.9 mm to (2.03, 41.0), turned to 90 degrees
- moved SJ2 19.2 mm to (12.2, 36.1), turned to 270 degrees
- moved JP2 18.2 mm to (1.91, 47.0)
- moved J1 13.0 mm to (17.8, 33.5), turned to 90 degrees
- moved C1 9.18 mm to (15.5, 42.9)
- moved R5 8.98 mm to (20.8, 39.6)
- moved U1 7.98 mm to (8.89, 42.9)
- moved R7 7.95 mm to (10.4, 29.0), flipped to the bottom, turned to 270 degrees
- moved R6 2.29 mm to (19.3, 25.4), turned to 180 degrees
- moved C8 2.16 mm to (34.3, 18.2), turned to 270 degrees
- moved D2 1.28 mm to (2.54, 15.1)
- moved ZD1 0.65 mm to (4.45, 26.5), turned to 180 degrees
- moved R9 0.25 mm to (20.3, 34.0), turned to 270 degrees
- moved C6 0.25 mm to (12.7, 29.0)
Connections:
- removed net N$1: C5.2, U1.7, Y1.2
- removed net N$18: SJ3.1, U1.19
- removed net N$2: C4.1, U1.8, Y1.1
- new net N$10: SJ2.1, U1.26
- net ADC0: now also U1.24; no longer U1.23
- net ADC1: now also U1.23; no longer U1.24
- net GND: now also SJ4.2; no longer C4.2, C5.1, SJ3.2
- net N$12: now also SJ4.1; no longer SJ1.1
- net N$16: now also SJ1.1; no longer SJ2.1
Routing:
- net 12V: track 0.00 -> 100.1 mm
- net ADC1: track 0.00 -> 64.2 mm, vias 0 -> 1
- net ADC0: track 0.00 -> 41.0 mm, vias 0 -> 1
- net 3.3V: track 0.00 -> 40.9 mm, vias 0 -> 10
- net MISO: track 0.00 -> 39.1 mm, vias 0 -> 1
- net MOSI: track 0.00 -> 37.0 mm, vias 0 -> 2
- net IRQ: track 0.00 -> 30.3 mm, vias 0 -> 1
- net N$15: track 0.00 -> 24.0 mm
- net CSN: track 0.00 -> 23.5 mm, vias 0 -> 2
- net CE: track 0.00 -> 20.9 mm, vias 0 -> 1
- net PWM2: track 0.00 -> 19.6 mm
- net SCK: track 0.00 -> 19.4 mm, vias 0 -> 1
- net RESET: track 0.00 -> 17.6 mm, vias 0 -> 2
- net N$6: track 0.00 -> 16.8 mm
- net N$11: track 0.00 -> 15.7 mm
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- added copper zone on layer 1, net 3.3V

Commit message: wip
Parts:
- removed SJ4: SOLDERJUMPERNO, SparkFun-Retired:SJ_2S-NO
- added SJ3: SOLDERJUMPERNO, SparkFun-Retired:SJ_2S-NO
- moved SJ1 4.57 mm to (12.2, 36.1)
- moved SJ2 2.29 mm to (9.91, 36.1)
- moved IN 1.09 mm to (12.1, 2.92), flipped to the bottom, turned to 180 degrees
- renumbered J1 to ISP
Connections:
- net GND: now also SJ3.2; no longer SJ4.2
- net N$10: now also SJ1.1; no longer SJ2.1
- net N$12: now also SJ2.1; no longer SJ4.1
- net N$16: now also SJ3.1; no longer SJ1.1
Routing:
- net N$5: track 7.73 -> 8.42 mm
Other:
- board text added: "12V"
- board text added: "Dual LED Wireless Dimmer Rev A / Eran Rundstein, 2017"
- board text added: "GND"

Commit message: wip
Parts:
- added R12, R13: 150, microbuilder:0805
- Q3, Q4: value IRF520NPBF -> IRL520
- moved R10 4.72 mm to (7.11, 59.1), turned to 0 degrees
- moved R11 4.66 mm to (19.9, 59.2), turned to 0 degrees
Connections:
- new net N$1: Q3.1, R12.2
- new net N$2: Q4.1, R13.2
- net PWM1: now also R12.1; no longer Q3.1
- net PWM2: now also R13.1; no longer Q4.1
Routing:
- net N$2: track 0.00 -> 3.58 mm
- net N$1: track 0.00 -> 3.51 mm
- net PWM1: track 10.4 -> 12.3 mm
- net PWM2: track 19.6 -> 20.3 mm
Changed lines of the file:
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@@
 <?xml version="1.0" encoding="utf-8"?>
 <!DOCTYPE eagle SYSTEM "eagle.dtd">
-<eagle version="8.5.0">
+<eagle version="8.5.1">
 <drawing>
 <settings>
@@
 <element name="C8" library="microbuilder" package="0805" value="0.1uF" x="34.29" y="18.161" rot="MR270"/>
 <element name="R7" library="microbuilder" package="0805" value="10k" x="10.414" y="28.956" rot="MR270"/>
-<element name="Q3" library="Seeed-Transistor-2016" package="TO-220" value="IRF520NPBF" x="12.7" y="64.77">
+<element name="Q3" library="Seeed-Transistor-2016" package="TO-220" value="IRL520" x="12.7" y="64.77">
 <attribute name="MPN" value="IRF520NPBF" x="12.7" y="64.77" size="1.778" layer="27" display="off"/>
 </element>
@@
 <attribute name="OC_NEWARK" value="unknown" x="2.54" y="54.61" size="1.778" layer="28" rot="MR90" display="off"/>
 </element>
-<element name="R10" library="microbuilder" package="0805" value="10k" x="11.43" y="57.15" rot="MR180"/>
-<element name="Q4" library="Seeed-Transistor-2016" package="TO-220" value="IRF520NPBF" x="25.4" y="64.77">
+<element name="R10" library="microbuilder" package="0805" value="10k" x="7.112" y="59.055" rot="MR0"/>
+<element name="Q4" library="Seeed-Transistor-2016" package="TO-220" value="IRL520" x="25.4" y="64.77">
 <attribute name="MPN" value="IRF520NPBF" x="25.4" y="64.77" size="1.778" layer="27" display="off"/>
 </element>
@@
 <attribute name="OC_NEWARK" value="unknown" x="35.56" y="54.61" size="1.778" layer="28" rot="MR270" display="off"/>
 </element>
-<element name="R11" library="microbuilder" package="0805" value="10k" x="24.13" y="57.15" rot="MR180"/>
+<element name="R11" library="microbuilder" package="0805" value="10k" x="19.939" y="59.182" rot="MR0"/>
 <element name="JP2" library="pinhead" library_urn="urn:adsk.eagle:library:325" package="1X03" package3d_urn="urn:adsk.eagle:package:22458/2" value="" x="1.905" y="46.99" rot="R90"/>
 <element name="SJ2" library="SparkFun-Retired" package="SJ_2S-NO" value="SOLDERJUMPERNO" x="9.906" y="36.068" smashed="yes" rot="MR270">
@@
 <attribute name="VALUE" x="13.843" y="36.976" size="0.4064" layer="28" rot="MR270"/>
 </element>
+<element name="R12" library="microbuilder" package="0805" value="150" x="9.017" y="56.769" rot="MR180"/>
+<element name="R13" library="microbuilder" package="0805" value="150" x="21.844" y="56.896" rot="MR180"/>
 </elements>
 <signals>
@@
 <wire x1="35.56" y1="52.86" x2="33.754" y2="52.86" width="1.27" layer="1"/>
 <wire x1="33.754" y1="52.86" x2="29.972" y2="56.642" width="1.27" layer="1"/>
-<wire x1="29.972" y1="56.642" x2="2.822" y2="56.642" width="1.27" layer="1"/>
+<wire x1="29.972" y1="56.642" x2="10.033" y2="56.642" width="1.27" layer="1"/>
+<wire x1="10.033" y1="56.642" x2="2.822" y2="56.642" width="1.27" layer="1"/>
 <wire x1="2.822" y1="56.642" x2="2.54" y2="56.36" width="1.27" layer="1"/>
 <wire x1="18.6182" y1="16.891" x2="16.9672" y2="15.24" width="0.508" layer="16"/>
@@
 </signal>
 <signal name="PWM1">
-<contactref element="Q3" pad="1"/>
 <contactref element="R10" pad="1"/>
 <contactref element="U1" pad="13"/>
-<wire x1="10.48" y1="57.15" x2="10.16" y2="56.83" width="0.4064" layer="16"/>
-<wire x1="10.16" y1="56.83" x2="10.16" y2="53.34" width="0.4064" layer="16"/>
-<wire x1="10.16" y1="53.34" x2="9.29" y2="52.47" width="0.4064" layer="16"/>
-<wire x1="9.29" y1="52.47" x2="9.29" y2="47.2186" width="0.4064" layer="16"/>
+<contactref element="R12" pad="1"/>
+<wire x1="8.062" y1="59.055" x2="8.062" y2="56.774" width="0.4064" layer="16"/>
+<wire x1="8.062" y1="56.774" x2="8.067" y2="56.769" width="0.4064" layer="16"/>
+<wire x1="9.29" y1="47.2186" x2="9.29" y2="49.892" width="0.4064" layer="16"/>
+<wire x1="9.29" y1="49.892" x2="8.128" y2="51.054" width="0.4064" layer="16"/>
+<wire x1="8.128" y1="51.054" x2="8.128" y2="56.708" width="0.4064" layer="16"/>
+<wire x1="8.128" y1="56.708" x2="8.067" y2="56.769" width="0.4064" layer="16"/>
 </signal>
 <signal name="N$8">
@@
 </signal>
 <signal name="PWM2">
-<contactref element="Q4" pad="1"/>
 <contactref element="R11" pad="1"/>
 <contactref element="U1" pad="14"/>
+<contactref element="R13" pad="1"/>
 <wire x1="10.09" y1="47.2186" x2="10.255" y2="47.3836" width="0.4064" layer="16"/>
 <wire x1="10.255" y1="47.3836" x2="10.255" y2="48.00089375" width="0.4064" layer="16"/>
-<wire x1="10.255" y1="48.00089375" x2="12.80010625" y2="50.546" width="0.4064" layer="16"/>
-<wire x1="20.066" y1="50.546" x2="22.86" y2="53.34" width="0.4064" layer="16"/>
-<wire x1="12.80010625" y1="50.546" x2="20.066" y2="50.546" width="0.4064" layer="16"/>
-<wire x1="22.86" y1="53.34" x2="23.18" y2="53.66" width="0.4064" layer="16"/>
-<wire x1="23.18" y1="53.66" x2="23.18" y2="57.15" width="0.4064" layer="16"/>
+<wire x1="10.255" y1="48.00089375" x2="12.54610625" y2="50.292" width="0.4064" layer="16"/>
+<wire x1="12.54610625" y1="50.292" x2="19.05" y2="50.292" width="0.4064" layer="16"/>
+<wire x1="19.05" y1="50.292" x2="20.894" y2="52.136" width="0.4064" layer="16"/>
+<wire x1="20.894" y1="52.136" x2="20.894" y2="56.896" width="0.4064" layer="16"/>
+<wire x1="20.894" y1="56.896" x2="20.894" y2="59.177" width="0.4064" layer="16"/>
+<wire x1="20.894" y1="59.177" x2="20.889" y2="59.182" width="0.4064" layer="16"/>
 </signal>
 <signal name="N$12">
@@
 <wire x1="10.89" y1="37.82" x2="10.89" y2="38.6334" width="0.254" layer="16"/>
 </signal>
+<signal name="N$1">
+<contactref element="Q3" pad="1"/>
+<contactref element="R12" pad="2"/>
+<wire x1="10.16" y1="53.34" x2="10.16" y2="56.576" width="0.4064" layer="16"/>
+<wire x1="10.16" y1="56.576" x2="9.967" y2="56.769" width="0.4064" layer="16"/>
+</signal>
+<signal name="N$2">
+<contactref element="Q4" pad="1"/>
+<contactref element="R13" pad="2"/>
+<wire x1="22.86" y1="53.34" x2="22.86" y2="56.83" width="0.4064" layer="16"/>
+<wire x1="22.86" y1="56.83" x2="22.794" y2="56.896" width="0.4064" layer="16"/>
+</signal>
 </signals>
