File: dual-led-wireless-dimmer/dual-led-wireless-dimmer-tx.brd (EAGLE design)
At the start: 38.1 x 76.2 mm, 45 parts, among them IC1 LM2937IMP-3.3, Q1 DN2625K4-G, Q2 SI2323DS-T1-E3, Q3 IRL520, Q4 IRL520, U1 ATMEGA328P_TQFP

Commit message: wip
Parts:
- moved IN 1.02 mm to (11.0, 2.92)
Routing:
- net N$5: track 8.42 -> 9.43 mm
Changed lines of the file:
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@@
 <layer number="42" name="bRestrict" color="1" fill="10" visible="yes" active="yes"/>
 <layer number="43" name="vRestrict" color="2" fill="10" visible="no" active="yes"/>
-<layer number="44" name="Drills" color="7" fill="1" visible="no" active="yes"/>
+<layer number="44" name="Drills" color="7" fill="1" visible="yes" active="yes"/>
 <layer number="45" name="Holes" color="7" fill="1" visible="yes" active="yes"/>
 <layer number="46" name="Milling" color="3" fill="1" visible="no" active="yes"/>
@@
 <element name="H3" library="holes" library_urn="urn:adsk.eagle:library:237" package="3,2" package3d_urn="urn:adsk.eagle:package:14275/1" value="MOUNT-HOLE3.2" x="2.54" y="73.66"/>
 <element name="H4" library="holes" library_urn="urn:adsk.eagle:library:237" package="3,2" package3d_urn="urn:adsk.eagle:package:14275/1" value="MOUNT-HOLE3.2" x="35.56" y="73.66"/>
-<element name="IN" library="con-ptr500" library_urn="urn:adsk.eagle:library:181" package="AK550/2" package3d_urn="urn:adsk.eagle:package:9907/1" value="AK550/2" x="12.065" y="2.921" smashed="yes" rot="MR180">
-<attribute name="MF" value="" x="12.065" y="2.921" size="1.778" layer="28" rot="MR180" display="off"/>
-<attribute name="MPN" value="" x="12.065" y="2.921" size="1.778" layer="28" rot="MR180" display="off"/>
-<attribute name="NAME" x="6.731" y="3.81" size="1.778" layer="26" rot="MR90"/>
-<attribute name="OC_FARNELL" value="unknown" x="12.065" y="2.921" size="1.778" layer="28" rot="MR180" display="off"/>
-<attribute name="OC_NEWARK" value="unknown" x="12.065" y="2.921" size="1.778" layer="28" rot="MR180" display="off"/>
-<attribute name="VALUE" x="8.89" y="8.636" size="1.778" layer="28" rot="MR180"/>
+<element name="IN" library="con-ptr500" library_urn="urn:adsk.eagle:library:181" package="AK550/2" package3d_urn="urn:adsk.eagle:package:9907/1" value="AK550/2" x="11.049" y="2.921" smashed="yes" rot="MR180">
+<attribute name="MF" value="" x="11.049" y="2.921" size="1.778" layer="28" rot="MR180" display="off"/>
+<attribute name="MPN" value="" x="11.049" y="2.921" size="1.778" layer="28" rot="MR180" display="off"/>
+<attribute name="NAME" x="5.715" y="3.81" size="1.778" layer="26" rot="MR90"/>
+<attribute name="OC_FARNELL" value="unknown" x="11.049" y="2.921" size="1.778" layer="28" rot="MR180" display="off"/>
+<attribute name="OC_NEWARK" value="unknown" x="11.049" y="2.921" size="1.778" layer="28" rot="MR180" display="off"/>
+<attribute name="VALUE" x="7.874" y="8.636" size="1.778" layer="28" rot="MR180"/>
 </element>
 <element name="NRF24L01" library="pinhead" library_urn="urn:adsk.eagle:library:325" package="2X04" package3d_urn="urn:adsk.eagle:package:22461/2" value="" x="19.05" y="29.21" rot="MR180"/>
@@
 <contactref element="F1" pad="L2"/>
 <wire x1="18.6182" y1="3.429" x2="22.0218" y2="3.429" width="1.778" layer="1"/>
-<wire x1="13.815" y1="2.921" x2="18.1102" y2="2.921" width="1.778" layer="1"/>
+<wire x1="12.799" y1="2.921" x2="18.1102" y2="2.921" width="1.778" layer="1"/>
 <wire x1="18.1102" y1="2.921" x2="18.6182" y2="3.429" width="1.778" layer="1"/>
 </signal>

Commit message: wip
Other:
- board text added: "IRQ"
Changed lines of the file:
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@@
 <layers>
 <layer number="1" name="Top" color="4" fill="1" visible="yes" active="yes"/>
-<layer number="16" name="Bottom" color="1" fill="1" visible="yes" active="yes"/>
+<layer number="16" name="Bottom" color="1" fill="1" visible="no" active="yes"/>
 <layer number="17" name="Pads" color="2" fill="1" visible="yes" active="yes"/>
 <layer number="18" name="Vias" color="2" fill="1" visible="yes" active="yes"/>
@@
 <layer number="20" name="Dimension" color="24" fill="1" visible="yes" active="yes"/>
 <layer number="21" name="tPlace" color="7" fill="1" visible="yes" active="yes"/>
-<layer number="22" name="bPlace" color="7" fill="1" visible="yes" active="yes"/>
+<layer number="22" name="bPlace" color="7" fill="1" visible="no" active="yes"/>
 <layer number="23" name="tOrigins" color="15" fill="1" visible="yes" active="yes"/>
-<layer number="24" name="bOrigins" color="15" fill="1" visible="yes" active="yes"/>
+<layer number="24" name="bOrigins" color="15" fill="1" visible="no" active="yes"/>
 <layer number="25" name="tNames" color="7" fill="1" visible="yes" active="yes"/>
-<layer number="26" name="bNames" color="7" fill="1" visible="yes" active="yes"/>
-<layer number="27" name="tValues" color="7" fill="1" visible="yes" active="yes"/>
-<layer number="28" name="bValues" color="7" fill="1" visible="yes" active="yes"/>
+<layer number="26" name="bNames" color="7" fill="1" visible="no" active="yes"/>
+<layer number="27" name="tValues" color="7" fill="1" visible="no" active="yes"/>
+<layer number="28" name="bValues" color="7" fill="1" visible="no" active="yes"/>
 <layer number="29" name="tStop" color="7" fill="3" visible="no" active="yes"/>
 <layer number="30" name="bStop" color="7" fill="6" visible="no" active="yes"/>
@@
 <layer number="38" name="bTest" color="7" fill="1" visible="no" active="yes"/>
 <layer number="39" name="tKeepout" color="4" fill="11" visible="yes" active="yes"/>
-<layer number="40" name="bKeepout" color="1" fill="11" visible="yes" active="yes"/>
+<layer number="40" name="bKeepout" color="1" fill="11" visible="no" active="yes"/>
 <layer number="41" name="tRestrict" color="4" fill="10" visible="yes" active="yes"/>
-<layer number="42" name="bRestrict" color="1" fill="10" visible="yes" active="yes"/>
+<layer number="42" name="bRestrict" color="1" fill="10" visible="no" active="yes"/>
 <layer number="43" name="vRestrict" color="2" fill="10" visible="no" active="yes"/>
-<layer number="44" name="Drills" color="7" fill="1" visible="yes" active="yes"/>
+<layer number="44" name="Drills" color="7" fill="1" visible="no" active="yes"/>
 <layer number="45" name="Holes" color="7" fill="1" visible="yes" active="yes"/>
 <layer number="46" name="Milling" color="3" fill="1" visible="no" active="yes"/>
@@
 <layer number="50" name="dxf" color="7" fill="1" visible="no" active="no"/>
 <layer number="51" name="tDocu" color="7" fill="1" visible="yes" active="yes"/>
-<layer number="52" name="bDocu" color="7" fill="1" visible="yes" active="yes"/>
+<layer number="52" name="bDocu" color="7" fill="1" visible="no" active="yes"/>
 <layer number="53" name="tGND_GNDA" color="7" fill="9" visible="no" active="no"/>
 <layer number="54" name="bGND_GNDA" color="1" fill="9" visible="no" active="no"/>
@@
 </layers>
 <board>
+<fusionsync huburn="a.cGVyc29uYWw6dWUyYWI1OThm" projecturn="a.cGVyc29uYWw6dWUyYWI1OThmIzIwMTcxMjE5MTA5MDk2NTMx" f3durn="urn:adsk.wipprod:dm.lineage:nHyQx4NYSI-B4NU9s-gEEQ" pcbguid="547d86a4-2050-44a8-95dd-225fd4500e45" lastpulledtime="" lastsyncedchangeguid="22225110-515c-72f5-8785-f8839dc68c2f"/>
 <plain>
 <wire x1="0" y1="0" x2="38.1" y2="0" width="0" layer="20"/>
@@
 <text x="11.176" y="7.112" size="0.762" layer="26" rot="MR0">GND</text>
 <text x="15.113" y="6.858" size="0.762" layer="26" rot="MR0">12V</text>
+<text x="14.224" y="31.623" size="0.4064" layer="22" rot="MR0">GND</text>
+<text x="25.019" y="26.797" size="0.4064" layer="22" rot="MR0">IRQ</text>
 </plain>
 <attributes>
@@
 </autorouter>
 <elements>
-<element name="CH1" library="keves-ng" package="BOURNS-PTL45" value="PTL45" x="8.89" y="38.1" smashed="yes" rot="R90">
+<element name="CH1" library="keves-ng" library_urn="urn:adsk.eagle:library:1429743" package="BOURNS-PTL45" package3d_urn="urn:adsk.eagle:package:1429786/2" value="PTL45" x="8.89" y="38.1" smashed="yes" rot="R90">
 <attribute name="NAME" x="13.97" y="11.303" size="1.27" layer="25"/>
-</element>
-<element name="CH2" library="keves-ng" package="BOURNS-PTL45" value="PTL45" x="29.21" y="38.1" smashed="yes" rot="R90">
+<attribute name="SPICEPREFIX" value="C" x="8.89" y="38.1" size="1.778" layer="27" rot="R90" display="off"/>
+</element>
+<element name="CH2" library="keves-ng" library_urn="urn:adsk.eagle:library:1429743" package="BOURNS-PTL45" package3d_urn="urn:adsk.eagle:package:1429786/2" value="PTL45" x="29.21" y="38.1" smashed="yes" rot="R90">
 <attribute name="NAME" x="24.13" y="12.446" size="1.27" layer="25" rot="R180"/>
 </element>
@@
 <attribute name="VALUE" x="22.098" y="32.004" size="0.4064" layer="27" ratio="10" rot="R270"/>
 </element>
-<element name="F1" library="keves-ng" package="KEYSTONE-3557-2" value="KEYSTONE-3557-2" x="20.32" y="10.16" rot="MR90"/>
+<element name="F1" library="keves-ng" library_urn="urn:adsk.eagle:library:1429743" package="KEYSTONE-3557-2" package3d_urn="urn:adsk.eagle:package:1429787/2" value="KEYSTONE-3557-2" x="20.32" y="10.16" rot="MR90"/>
 <element name="Q1" library="SparkFun-DiscreteSemi" package="DPAK" value="DN2625K4-G" x="11.43" y="15.24" rot="MR90">
 <attribute name="PROD_ID" value="TRANS-09984" x="11.43" y="15.24" size="1.778" layer="28" rot="MR90" display="off"/>
@@
 </note>
 <note version="8.3" severity="warning">
+Since Version 8.3, EAGLE supports Fusion synchronisation.
+This feature will not be available in this version and saving
+the document will break the link to the Fusion PCB feature.
+</note>
+<note version="8.3" severity="warning">
