File: dual-led-wireless-dimmer/dual-led-wireless-dimmer-tx.sch (EAGLE design)
At the start: 17 parts, among them J1 AVR_SPI_PRG_6PTH, U1 ATMEGA328P_TQFP, X1 PTL45, X2 PTL45, Y1 8MHz

Commit message: wip
Parts:
- added C10: 100uF, microbuilder:CAP_ELECTROLYTICPANASONIC_D
- added C11: 10uF, microbuilder:CAP_CERAMIC0805
- added C12: 0.1uF, microbuilder:CAP_CERAMIC0805
- added C6: 4.7uF, microbuilder:CAP_CERAMIC0805
- added D1: 17V (1N5247B), diode:ZENER-DIODEZD-5
- added D2: 24v 1N5359B, diode:ZENER-DIODEZD-10
- added F1: KEYSTONE-3557-2, keves-ng:KEYSTONE-3557-2
- added IC1: LM2937IMP-3.3, linear:LM2937
- added JP1: (no value), pinhead:PINHD-2X4
- added JP2: (no value), pinhead:PINHD-1X3
- added L1: 5248-RC, rcl:L-US0207/5V
- added Q1: DN2625K4-G, SparkFun-DiscreteSemi:MOSFET-NCHANNELFDD8780
- added Q2: SI2323DS-T1-E3, SparkFun-DiscreteSemi:MOSFET-PCHANNEL
- added Q3, Q4: IRF520NPBF, Seeed-Transistor-2016:DIP-MOSFET-N-CH-100V-9.7A-IRF520NPBF(TO-220AB)
- added R10, R11, R9: 10k, microbuilder:RESISTOR0805
- added R4, R5, R6: 220, microbuilder:RESISTOR0805
- added R7: 100k, microbuilder:RESISTOR0805
- added R8: 39k, microbuilder:RESISTOR0805
- added SJ1, SJ2, SJ3: (no value), jumper:SJW
- added X3, X4, X5: AK550/2, con-ptr500:AK550/2
- added ZD1: 7.5v BZT52C7V5-7-F, diodes:ZD-SOD123
Connections:
- new net 12V: F1.2, Q1.D, R7.2, X4-2.KL, X5-2.KL
- new net ADC0: U1.PC0(ADC0), X1.S
- new net ADC1: U1.PC1(ADC1), X2.S
- new net CE: JP1.3, U1.PD3(INT1)
- new net CSN: JP1.4, R9.1, U1.PD4(XCK/T0)
- new net IRQ: JP1.8, U1.PD2(INT0)
- new net N$10: JP1.5, R4.2
- new net N$11: D1.C, Q1.G, R7.1
- new net N$12: SJ1.1, U1.PC4(ADC4/SDA)
- new net N$13: Q1.S, Q2.D
- new net N$14: Q2.G, R8.1, ZD1.A
- new net N$15: D2.C, L1.1, Q2.S, ZD1.C
- new net N$16: SJ2.1, U1.PC5(ADC5/SCL)
- new net N$17: C10.+, C12.P$1, IC1.VI, L1.2
- new net N$18: SJ3.1, U1.ADC6
- new net N$19: JP2.3, U1.PD1(TXD)
- new net N$20: JP2.2, U1.PD0(RXD)
- new net N$5: F1.1, X3-2.KL
- new net N$6: Q3.D, X4-1.KL
- new net N$7: JP1.6, R5.1
- new net N$8: Q4.D, X5-1.KL
- new net N$9: JP1.7, R6.2
- new net PWM1: Q3.G, R10.1, U1.PB1(OC1A)
- new net PWM2: Q4.G, R11.1, U1.PB2(SS/OC1B)
- net 3.3V: now also C11.P$1, C6.P$2, IC1.VO, JP1.2, R9.2
- net GND: now also C10.-, C11.P$2, C12.P$2, C6.P$1, D1.A, D2.A, IC1.GND, JP1.1, JP2.1, Q3.S, Q4.S, R10.2, R11.2, R8.2, SJ1.2, SJ2.2, SJ3.2, X3-1.KL
- net MISO: now also R6.1
- net MOSI: now also R5.2
- net SCK: now also R4.1
Other:
- note added: "https://rusefi.com/wiki/index.php?title=Manual:Hardware_Frankenso_board"

Commit message: wip
Parts:
- removed C3: 0.1uF, microbuilder:CAP_CERAMIC0805
- C1, C2: value 22pF -> 0.1uF
- C4, C5: value 0.1uF -> 22pF
- R1: value 10k -> 150
- R3: value 150 -> 100k
- R4: value 220 -> 39k
- R5: value 220 -> 10k
- R7: value 100k -> 10k
- R8: value 39k -> 220
- R9: value 10k -> 220
- renumbered C10 to C7, C11 to C9, C12 to C8, JP1 to NRF24L01, X1 to CH1, X2 to CH2, X3 to IN, X4 to OUT1, X5 to OUT2
Connections:
- removed net N$10: NRF24L01.5, R4.2
- new net JP1: NRF24L01.5, R9.2
- net 12V: now also R3.2; no longer R7.2
- net 3.3V: now also C1.P$2, C2.P$2, R1.1, R5.2, R7.2; no longer C3.P$2, C4.P$2, C5.P$2, R1.2, R3.1, R9.2
- net CSN: now also R7.1; no longer R9.1
- net GND: now also C2.P$1, C4.P$2, R4.2; no longer C2.P$2, C3.P$1, C4.P$1, R8.2
- net MISO: now also R8.1; no longer R6.1
- net MOSI: now also R6.2; no longer R5.2
- net N$1: now also C5.P$2; no longer C1.P$2
- net N$11: now also R3.1; no longer R7.1
- net N$14: now also R4.1; no longer R8.1
- net N$2: now also C4.P$1; no longer C2.P$1
- net N$3: now also R1.2; no longer R2.2
- net N$4: now also R2.2; no longer R3.2
- net N$7: now also R6.1; no longer R5.1
- net N$9: now also R8.2; no longer R6.2
- net RESET: now also R5.1; no longer R1.1
- net SCK: now also R9.1; no longer R4.1
Other:
- note removed: "TODO: 1) 12V input 2) Connect POTs to ADC 3) Put Wireless module"
- moved on the sheet: C1, C2, C4, C5, R1, R2, R3, R4, R5, R6, R7, R8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

Commit message: routed
Parts:
- removed C4, C5: 22pF, microbuilder:CAP_CERAMIC0805
- removed SJ3: (no value), jumper:SJW
- removed Y1: 8MHz, SparkFun-FreqCtrl:CRYSTALSMD
- added SJ4: SOLDERJUMPERNO, SparkFun-Retired:SOLDERJUMPERNO
- SJ1, SJ2: value (none) -> SOLDERJUMPERNO; device jumper:SJW -> SparkFun-Retired:SOLDERJUMPERNO
Connections:
- removed net N$1: C5.P$2, U1.PB6(XTAL1/TOSC1), Y1.2
- removed net N$18: SJ3.1, U1.ADC6
- removed net N$2: C4.P$1, U1.PB7(XTAL2/TOSC2), Y1.1
- new net N$10: SJ2.1, U1.PC3(ADC3)
- net ADC0: now also U1.PC1(ADC1); no longer U1.PC0(ADC0)
- net ADC1: now also U1.PC0(ADC0); no longer U1.PC1(ADC1)
- net GND: now also SJ4.2; no longer C4.P$2, C5.P$1, SJ3.2
- net N$12: now also SJ4.1; no longer SJ1.1
- net N$16: now also SJ1.1; no longer SJ2.1
Changed lines of the file:
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@@
 <part name="CH2" library="keves-ng" deviceset="PTL45" device=""/>
 <part name="U1" library="SparkFun-DigitalIC" deviceset="ATMEGA328P_TQFP" device="" value="ATMEGA328P_TQFP"/>
-<part name="Y1" library="SparkFun-FreqCtrl" deviceset="CRYSTAL" device="SMD" value="8MHz"/>
-<part name="C5" library="microbuilder" deviceset="CAP_CERAMIC" device="0805" value="22pF"/>
-<part name="C4" library="microbuilder" deviceset="CAP_CERAMIC" device="0805" value="22pF"/>
-<part name="GND7" library="microbuilder" deviceset="GND" device=""/>
-<part name="GND8" library="microbuilder" deviceset="GND" device=""/>
 <part name="GND9" library="microbuilder" deviceset="GND" device=""/>
 <part name="3.3V6" library="microbuilder" deviceset="3.3V" device=""/>
@@
 <part name="R11" library="microbuilder" deviceset="RESISTOR" device="0805" value="10k"/>
 <part name="GND17" library="microbuilder" deviceset="GND" device=""/>
-<part name="SJ1" library="jumper" library_urn="urn:adsk.eagle:library:252" deviceset="SJ" device="W" package3d_urn="urn:adsk.eagle:package:15507/1"/>
-<part name="SJ2" library="jumper" library_urn="urn:adsk.eagle:library:252" deviceset="SJ" device="W" package3d_urn="urn:adsk.eagle:package:15507/1"/>
-<part name="SJ3" library="jumper" library_urn="urn:adsk.eagle:library:252" deviceset="SJ" device="W" package3d_urn="urn:adsk.eagle:package:15507/1"/>
 <part name="GND12" library="microbuilder" deviceset="GND" device=""/>
 <part name="GND13" library="microbuilder" deviceset="GND" device=""/>
@@
 <part name="JP2" library="pinhead" library_urn="urn:adsk.eagle:library:325" deviceset="PINHD-1X3" device="" package3d_urn="urn:adsk.eagle:package:22458/2"/>
 <part name="GND15" library="microbuilder" deviceset="GND" device=""/>
+<part name="SJ4" library="SparkFun-Retired" deviceset="SOLDERJUMPER" device="NO"/>
+<part name="SJ1" library="SparkFun-Retired" deviceset="SOLDERJUMPER" device="NO"/>
+<part name="SJ2" library="SparkFun-Retired" deviceset="SOLDERJUMPER" device="NO"/>
 </parts>
 <sheets>
@@
 <instance part="CH2" gate="G$1" x="78.74" y="78.74" rot="R270"/>
 <instance part="U1" gate="U$1" x="167.64" y="93.98"/>
-<instance part="Y1" gate="G$1" x="137.16" y="96.52" rot="R90"/>
-<instance part="C5" gate="G$1" x="129.54" y="99.06" rot="R90"/>
-<instance part="C4" gate="G$1" x="127" y="93.98" rot="R270"/>
-<instance part="GND7" gate="G$1" x="119.38" y="99.06" rot="R270"/>
-<instance part="GND8" gate="G$1" x="119.38" y="93.98" rot="R270"/>
 <instance part="GND9" gate="G$1" x="137.16" y="68.58" rot="R270"/>
 <instance part="3.3V6" gate="G$1" x="124.46" y="124.46" rot="R90"/>
@@
 <instance part="R11" gate="G$1" x="238.76" y="55.88" rot="R270"/>
 <instance part="GND17" gate="G$1" x="238.76" y="48.26"/>
-<instance part="SJ1" gate="1" x="198.12" y="114.3"/>
-<instance part="SJ2" gate="1" x="198.12" y="111.76"/>
-<instance part="SJ3" gate="1" x="198.12" y="109.22"/>
 <instance part="GND12" gate="G$1" x="205.74" y="114.3" rot="R90"/>
 <instance part="GND13" gate="G$1" x="205.74" y="111.76" rot="R90"/>
-<instance part="GND14" gate="G$1" x="205.74" y="109.22" rot="R90"/>
+<instance part="GND14" gate="G$1" x="205.74" y="116.84" rot="R90"/>
 <instance part="JP2" gate="A" x="220.98" y="101.6"/>
 <instance part="GND15" gate="G$1" x="218.44" y="111.76" rot="R180"/>
+<instance part="SJ4" gate="1" x="198.12" y="114.3"/>
+<instance part="SJ1" gate="1" x="198.12" y="111.76"/>
+<instance part="SJ2" gate="1" x="198.12" y="116.84"/>
 </instances>
 <busses>
 </busses>
 <nets>
-<net name="N$1" class="0">
-<segment>
-<pinref part="U1" gate="U$1" pin="PB6(XTAL1/TOSC1)"/>
-<pinref part="Y1" gate="G$1" pin="2"/>
-<wire x1="137.16" y1="99.06" x2="142.24" y2="99.06" width="0.1524" layer="91"/>
-<pinref part="C5" gate="G$1" pin="P$2"/>
-<wire x1="132.08" y1="99.06" x2="137.16" y2="99.06" width="0.1524" layer="91"/>
-<junction x="137.16" y="99.06"/>
-</segment>
-</net>
-<net name="N$2" class="0">
-<segment>
-<pinref part="U1" gate="U$1" pin="PB7(XTAL2/TOSC2)"/>
-<pinref part="Y1" gate="G$1" pin="1"/>
-<wire x1="137.16" y1="93.98" x2="142.24" y2="93.98" width="0.1524" layer="91"/>
-<pinref part="C4" gate="G$1" pin="P$1"/>
-<wire x1="132.08" y1="93.98" x2="137.16" y2="93.98" width="0.1524" layer="91"/>
-<junction x="137.16" y="93.98"/>
-</segment>
-</net>
 <net name="GND" class="0">
-<segment>
-<pinref part="C5" gate="G$1" pin="P$1"/>
-<pinref part="GND7" gate="G$1" pin="GND"/>
-<wire x1="121.92" y1="99.06" x2="124.46" y2="99.06" width="0.1524" layer="91"/>
-</segment>
-<segment>
-<pinref part="C4" gate="G$1" pin="P$2"/>
-<pinref part="GND8" gate="G$1" pin="GND"/>
-<wire x1="121.92" y1="93.98" x2="124.46" y2="93.98" width="0.1524" layer="91"/>
-</segment>
 <segment>
 <pinref part="U1" gate="U$1" pin="AGND"/>
@@
 </segment>
 <segment>
-<pinref part="SJ1" gate="1" pin="2"/>
-<pinref part="GND12" gate="G$1" pin="GND"/>
-</segment>
-<segment>
-<pinref part="SJ2" gate="1" pin="2"/>
-<pinref part="GND13" gate="G$1" pin="GND"/>
-</segment>
-<segment>
-<pinref part="SJ3" gate="1" pin="2"/>
-<pinref part="GND14" gate="G$1" pin="GND"/>
-</segment>
-<segment>
 <pinref part="GND15" gate="G$1" pin="GND"/>
 <pinref part="JP2" gate="A" pin="1"/>
 <wire x1="218.44" y1="109.22" x2="218.44" y2="104.14" width="0.1524" layer="91"/>
+</segment>
+<segment>
+<pinref part="GND12" gate="G$1" pin="GND"/>
+<pinref part="SJ4" gate="1" pin="2"/>
+</segment>
+<segment>
+<pinref part="GND13" gate="G$1" pin="GND"/>
+<pinref part="SJ1" gate="1" pin="2"/>
+</segment>
+<segment>
+<pinref part="GND14" gate="G$1" pin="GND"/>
+<pinref part="SJ2" gate="1" pin="2"/>
 </segment>
 </net>
@@
 </segment>
 <segment>
+<pinref part="U1" gate="U$1" pin="PC1(ADC1)"/>
+<wire x1="190.5" y1="121.92" x2="203.2" y2="121.92" width="0.1524" layer="91"/>
+<label x="200.66" y="121.92" size="1.778" layer="95"/>
+</segment>
+</net>
+<net name="ADC1" class="0">
+<segment>
+<pinref part="CH2" gate="G$1" pin="S"/>
+<wire x1="78.74" y1="66.04" x2="78.74" y2="55.88" width="0.1524" layer="91"/>
+<label x="78.74" y="55.88" size="1.778" layer="95"/>
+</segment>
+<segment>
 <pinref part="U1" gate="U$1" pin="PC0(ADC0)"/>
 <wire x1="190.5" y1="124.46" x2="203.2" y2="124.46" width="0.1524" layer="91"/>
 <label x="200.66" y="124.46" size="1.778" layer="95"/>
-</segment>
-</net>
-<net name="ADC1" class="0">
-<segment>
-<pinref part="CH2" gate="G$1" pin="S"/>
-<wire x1="78.74" y1="66.04" x2="78.74" y2="55.88" width="0.1524" layer="91"/>
-<label x="78.74" y="55.88" size="1.778" layer="95"/>
-</segment>
-<segment>
-<pinref part="U1" gate="U$1" pin="PC1(ADC1)"/>
-<wire x1="190.5" y1="121.92" x2="203.2" y2="121.92" width="0.1524" layer="91"/>
-<label x="200.66" y="121.92" size="1.778" layer="95"/>
 </segment>
 </net>
@@
 <net name="N$12" class="0">
 <segment>
-<pinref part="SJ1" gate="1" pin="1"/>
 <pinref part="U1" gate="U$1" pin="PC4(ADC4/SDA)"/>
 <wire x1="193.04" y1="114.3" x2="190.5" y2="114.3" width="0.1524" layer="91"/>
+<pinref part="SJ4" gate="1" pin="1"/>
 </segment>
 </net>
 <net name="N$16" class="0">
 <segment>
-<pinref part="SJ2" gate="1" pin="1"/>
 <pinref part="U1" gate="U$1" pin="PC5(ADC5/SCL)"/>
 <wire x1="193.04" y1="111.76" x2="190.5" y2="111.76" width="0.1524" layer="91"/>
-</segment>
-</net>
-<net name="N$18" class="0">
-<segment>
-<pinref part="SJ3" gate="1" pin="1"/>
-<pinref part="U1" gate="U$1" pin="ADC6"/>
-<wire x1="193.04" y1="109.22" x2="190.5" y2="109.22" width="0.1524" layer="91"/>
+<pinref part="SJ1" gate="1" pin="1"/>
 </segment>
 </net>
@@
 </segment>
 </net>
+<net name="N$10" class="0">
+<segment>
+<pinref part="SJ2" gate="1" pin="1"/>
+<pinref part="U1" gate="U$1" pin="PC3(ADC3)"/>
+<wire x1="193.04" y1="116.84" x2="190.5" y2="116.84" width="0.1524" layer="91"/>
+</segment>
+</net>

Commit message: wip
Parts:
- removed SJ4: SOLDERJUMPERNO, SparkFun-Retired:SOLDERJUMPERNO
- added SJ3: SOLDERJUMPERNO, SparkFun-Retired:SOLDERJUMPERNO
- renumbered J1 to ISP
Connections:
- net GND: now also SJ3.2; no longer SJ4.2
- net N$10: now also SJ1.1; no longer SJ2.1
- net N$12: now also SJ2.1; no longer SJ4.1
- net N$16: now also SJ3.1; no longer SJ1.1
Other:
- moved on the sheet: SJ1, SJ2
Changed lines of the file:
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@@
 <part name="3.3V6" library="microbuilder" deviceset="3.3V" device=""/>
 <part name="R5" library="microbuilder" deviceset="RESISTOR" device="0805" value="10k"/>
-<part name="J1" library="SparkFun-Connectors" deviceset="AVR_SPI_PRG_6" device="PTH"/>
+<part name="ISP" library="SparkFun-Connectors" deviceset="AVR_SPI_PRG_6" device="PTH"/>
 <part name="GND10" library="microbuilder" deviceset="GND" device=""/>
 <part name="3.3V9" library="microbuilder" deviceset="3.3V" device=""/>
@@
 <part name="JP2" library="pinhead" library_urn="urn:adsk.eagle:library:325" deviceset="PINHD-1X3" device="" package3d_urn="urn:adsk.eagle:package:22458/2"/>
 <part name="GND15" library="microbuilder" deviceset="GND" device=""/>
-<part name="SJ4" library="SparkFun-Retired" deviceset="SOLDERJUMPER" device="NO"/>
+<part name="SJ2" library="SparkFun-Retired" deviceset="SOLDERJUMPER" device="NO"/>
+<part name="SJ3" library="SparkFun-Retired" deviceset="SOLDERJUMPER" device="NO"/>
 <part name="SJ1" library="SparkFun-Retired" deviceset="SOLDERJUMPER" device="NO"/>
-<part name="SJ2" library="SparkFun-Retired" deviceset="SOLDERJUMPER" device="NO"/>
 </parts>
 <sheets>
@@
 <instance part="3.3V6" gate="G$1" x="124.46" y="124.46" rot="R90"/>
 <instance part="R5" gate="G$1" x="134.62" y="124.46" rot="R180"/>
-<instance part="J1" gate="G$1" x="152.4" y="43.18"/>
+<instance part="ISP" gate="G$1" x="152.4" y="43.18"/>
 <instance part="GND10" gate="G$1" x="167.64" y="40.64" rot="R90"/>
 <instance part="3.3V9" gate="G$1" x="167.64" y="45.72" rot="R270"/>
@@
 <instance part="JP2" gate="A" x="220.98" y="101.6"/>
 <instance part="GND15" gate="G$1" x="218.44" y="111.76" rot="R180"/>
-<instance part="SJ4" gate="1" x="198.12" y="114.3"/>
-<instance part="SJ1" gate="1" x="198.12" y="111.76"/>
-<instance part="SJ2" gate="1" x="198.12" y="116.84"/>
+<instance part="SJ2" gate="1" x="198.12" y="114.3"/>
+<instance part="SJ3" gate="1" x="198.12" y="111.76"/>
+<instance part="SJ1" gate="1" x="198.12" y="116.84"/>
 </instances>
 <busses>
@@
 </segment>
 <segment>
-<pinref part="J1" gate="G$1" pin="6"/>
+<pinref part="ISP" gate="G$1" pin="6"/>
 <pinref part="GND10" gate="G$1" pin="GND"/>
 <wire x1="165.1" y1="40.64" x2="162.56" y2="40.64" width="0.1524" layer="91"/>
@@
 <segment>
 <pinref part="GND12" gate="G$1" pin="GND"/>
-<pinref part="SJ4" gate="1" pin="2"/>
+<pinref part="SJ2" gate="1" pin="2"/>
 </segment>
 <segment>
 <pinref part="GND13" gate="G$1" pin="GND"/>
+<pinref part="SJ3" gate="1" pin="2"/>
+</segment>
+<segment>
+<pinref part="GND14" gate="G$1" pin="GND"/>
 <pinref part="SJ1" gate="1" pin="2"/>
-</segment>
-<segment>
-<pinref part="GND14" gate="G$1" pin="GND"/>
-<pinref part="SJ2" gate="1" pin="2"/>
 </segment>
 </net>
@@
 </segment>
 <segment>
-<pinref part="J1" gate="G$1" pin="2"/>
+<pinref part="ISP" gate="G$1" pin="2"/>
 <pinref part="3.3V9" gate="G$1" pin="3.3V"/>
 <wire x1="165.1" y1="45.72" x2="162.56" y2="45.72" width="0.1524" layer="91"/>
@@
 <net name="MISO" class="0">
 <segment>
-<pinref part="J1" gate="G$1" pin="1"/>
+<pinref part="ISP" gate="G$1" pin="1"/>
 <wire x1="144.78" y1="45.72" x2="132.08" y2="45.72" width="0.1524" layer="91"/>
 <label x="132.08" y="45.72" size="1.778" layer="95" rot="R180"/>
@@
 <net name="SCK" class="0">
 <segment>
-<pinref part="J1" gate="G$1" pin="3"/>
+<pinref part="ISP" gate="G$1" pin="3"/>
 <wire x1="144.78" y1="43.18" x2="132.08" y2="43.18" width="0.1524" layer="91"/>
 <label x="132.08" y="43.18" size="1.778" layer="95" rot="R180"/>
@@
 <net name="RESET" class="0">
 <segment>
-<pinref part="J1" gate="G$1" pin="5"/>
+<pinref part="ISP" gate="G$1" pin="5"/>
 <wire x1="144.78" y1="40.64" x2="132.08" y2="40.64" width="0.1524" layer="91"/>
 <label x="132.08" y="40.64" size="1.778" layer="95" rot="R180"/>
@@
 <net name="MOSI" class="0">
 <segment>
-<pinref part="J1" gate="G$1" pin="4"/>
+<pinref part="ISP" gate="G$1" pin="4"/>
 <wire x1="162.56" y1="43.18" x2="175.26" y2="43.18" width="0.1524" layer="91"/>
 <label x="180.34" y="43.18" size="1.778" layer="95" rot="R180"/>
@@
 <pinref part="U1" gate="U$1" pin="PC4(ADC4/SDA)"/>
 <wire x1="193.04" y1="114.3" x2="190.5" y2="114.3" width="0.1524" layer="91"/>
-<pinref part="SJ4" gate="1" pin="1"/>
+<pinref part="SJ2" gate="1" pin="1"/>
 </segment>
 </net>
@@
 <pinref part="U1" gate="U$1" pin="PC5(ADC5/SCL)"/>
 <wire x1="193.04" y1="111.76" x2="190.5" y2="111.76" width="0.1524" layer="91"/>
-<pinref part="SJ1" gate="1" pin="1"/>
+<pinref part="SJ3" gate="1" pin="1"/>
 </segment>
 </net>
@@
 <net name="N$10" class="0">
 <segment>
-<pinref part="SJ2" gate="1" pin="1"/>
+<pinref part="SJ1" gate="1" pin="1"/>
 <pinref part="U1" gate="U$1" pin="PC3(ADC3)"/>
 <wire x1="193.04" y1="116.84" x2="190.5" y2="116.84" width="0.1524" layer="91"/>
