File: dt/dt.sch (EAGLE design)
At the start: 253 parts, among them IC1 TL072D, IC10 LM317, IC11 LM337, IC2 TL072D, IC3 TL072D, IC4 TL072D, IC5 TL072D, IC6 TL072D, U2 PCN2-S5-D12-S, U3 STM32F7X3ZXT, U4 USBLC6-2SC6YSOT23-6L_STM-M, U5 USBLC6-2SC6YSOT23-6L_STM-M, U6 PCM1681PWPPWP28_6P46X2P4-M, U7 PCM1681PWPPWP28_6P46X2P4-M, Y1 ABLS7M2-25.000MHZ-D2Y-T

Commit message: wip
Parts:
- added R100, R98, R99: 1k, keves-ng:RESISTOR0603
Connections:
- new net LED1: R98.2, U3A.PC12
- new net LED2: R99.2, U3A.PC11
- new net LED3: R100.2, U3A.PC10
- new net N$119: LED1.A_3, R100.1
- new net N$120: LED1.A_1, R98.1
- new net N$96: LED1.A_2, R99.1
- net DAC_OUT10: now also U7A.VOUT3; no longer U7A.VOUT2
- net DAC_OUT11: now also U7A.VOUT2; no longer U7A.VOUT3
- net DAC_OUT12: now also U7A.VOUT1; no longer U7A.VOUT4
- net DAC_OUT9: now also U7A.VOUT4; no longer U7A.VOUT1
- net EXT_OUT10: now also PL5.TB
- net EXT_OUT11: now also PL6.TT
- net EXT_OUT12: now also PL6.TB
- net EXT_OUT2: now also PL1.TB; no longer PL1.RT
- net EXT_OUT3: now also PL2.TT
- net EXT_OUT4: now also PL2.TB
- net EXT_OUT5: now also PL3.TT
- net EXT_OUT6: now also PL3.TB
- net EXT_OUT7: now also PL4.TT
- net EXT_OUT8: now also PL4.TB
- net EXT_OUT9: now also PL5.TT
- net GND: now also LED1.K_1, LED1.K_2, LED1.K_3
Changed lines of the file:
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@@
 <part name="P-8" library="supply1" library_urn="urn:adsk.eagle:library:371" deviceset="-12V" device=""/>
 <part name="P-9" library="supply1" library_urn="urn:adsk.eagle:library:371" deviceset="-12V" device=""/>
+<part name="R98" library="keves-ng" library_urn="urn:adsk.eagle:library:1429743" deviceset="RESISTOR" device="0603" package3d_urn="urn:adsk.eagle:package:23799129/3" value="1k"/>
+<part name="R99" library="keves-ng" library_urn="urn:adsk.eagle:library:1429743" deviceset="RESISTOR" device="0603" package3d_urn="urn:adsk.eagle:package:23799129/3" value="1k"/>
+<part name="R100" library="keves-ng" library_urn="urn:adsk.eagle:library:1429743" deviceset="RESISTOR" device="0603" package3d_urn="urn:adsk.eagle:package:23799129/3" value="1k"/>
+<part name="GND79" library="supply1" library_urn="urn:adsk.eagle:library:371" deviceset="GND" device=""/>
 </parts>
 <sheets>
@@
 <attribute name="VALUE" x="246.38" y="-185.42" size="1.778" layer="96" rot="R180"/>
 </instance>
+<instance part="R98" gate="G$1" x="129.54" y="81.28" smashed="yes">
+<attribute name="NAME" x="127" y="83.312" size="1.27" layer="95" font="vector"/>
+<attribute name="VALUE" x="127" y="78.105" size="1.27" layer="96" font="vector"/>
+</instance>
+<instance part="R99" gate="G$1" x="129.54" y="76.2" smashed="yes">
+<attribute name="NAME" x="127" y="78.232" size="1.27" layer="95" font="vector"/>
+<attribute name="VALUE" x="127" y="73.025" size="1.27" layer="96" font="vector"/>
+</instance>
+<instance part="R100" gate="G$1" x="129.54" y="71.12" smashed="yes">
+<attribute name="NAME" x="127" y="73.152" size="1.27" layer="95" font="vector"/>
+<attribute name="VALUE" x="127" y="67.945" size="1.27" layer="96" font="vector"/>
+</instance>
+<instance part="GND79" gate="1" x="104.14" y="66.04" smashed="yes">
+<attribute name="VALUE" x="101.6" y="63.5" size="1.778" layer="96"/>
+</instance>
 </instances>
 <busses>
@@
 </segment>
 </net>
-<net name="EXT_OUT2" class="0">
-<segment>
-<pinref part="PL1" gate="G$1" pin="RT"/>
-<wire x1="27.94" y1="147.32" x2="38.1" y2="147.32" width="0.1524" layer="91"/>
-<label x="38.1" y="147.32" size="1.778" layer="95"/>
-</segment>
-</net>
 <net name="GND" class="0">
 <segment>
@@
 <junction x="198.12" y="-157.48"/>
 </segment>
+<segment>
+<pinref part="GND79" gate="1" pin="GND"/>
+<pinref part="LED1" gate="G$1" pin="K_1"/>
+<wire x1="104.14" y1="68.58" x2="104.14" y2="71.12" width="0.1524" layer="91"/>
+<wire x1="104.14" y1="71.12" x2="104.14" y2="76.2" width="0.1524" layer="91"/>
+<wire x1="104.14" y1="76.2" x2="104.14" y2="81.28" width="0.1524" layer="91"/>
+<wire x1="104.14" y1="81.28" x2="109.22" y2="81.28" width="0.1524" layer="91"/>
+<pinref part="LED1" gate="G$1" pin="K_2"/>
+<wire x1="109.22" y1="76.2" x2="104.14" y2="76.2" width="0.1524" layer="91"/>
+<pinref part="LED1" gate="G$1" pin="K_3"/>
+<wire x1="109.22" y1="71.12" x2="104.14" y2="71.12" width="0.1524" layer="91"/>
+<junction x="104.14" y="76.2"/>
+<junction x="104.14" y="71.12"/>
+</segment>
 </net>
 <net name="N$49" class="0">
@@
 </segment>
 </net>
+<net name="EXT_OUT3" class="0">
+<segment>
+<pinref part="PL2" gate="G$1" pin="TT"/>
+<wire x1="27.94" y1="111.76" x2="38.1" y2="111.76" width="0.1524" layer="91"/>
+<label x="38.1" y="111.76" size="1.778" layer="95"/>
+</segment>
+</net>
+<net name="EXT_OUT5" class="0">
+<segment>
+<pinref part="PL3" gate="G$1" pin="TT"/>
+<wire x1="27.94" y1="73.66" x2="38.1" y2="73.66" width="0.1524" layer="91"/>
+<label x="38.1" y="73.66" size="1.778" layer="95"/>
+</segment>
+</net>
+<net name="EXT_OUT2" class="0">
+<segment>
+<pinref part="PL1" gate="G$1" pin="TB"/>
+<wire x1="27.94" y1="139.7" x2="38.1" y2="139.7" width="0.1524" layer="91"/>
+<label x="35.56" y="139.7" size="1.778" layer="95"/>
+</segment>
+</net>
+<net name="EXT_OUT4" class="0">
+<segment>
+<pinref part="PL2" gate="G$1" pin="TB"/>
+<wire x1="27.94" y1="101.6" x2="38.1" y2="101.6" width="0.1524" layer="91"/>
+<label x="38.1" y="101.6" size="1.778" layer="95"/>
+</segment>
+</net>
+<net name="EXT_OUT6" class="0">
+<segment>
+<pinref part="PL3" gate="G$1" pin="TB"/>
+<wire x1="27.94" y1="63.5" x2="38.1" y2="63.5" width="0.1524" layer="91"/>
+<label x="38.1" y="63.5" size="1.778" layer="95"/>
+</segment>
+</net>
+<net name="EXT_OUT7" class="0">
+<segment>
+<pinref part="PL4" gate="G$1" pin="TT"/>
+<wire x1="27.94" y1="35.56" x2="38.1" y2="35.56" width="0.1524" layer="91"/>
+<label x="38.1" y="35.56" size="1.778" layer="95"/>
+</segment>
+</net>
+<net name="EXT_OUT8" class="0">
+<segment>
+<pinref part="PL4" gate="G$1" pin="TB"/>
+<wire x1="27.94" y1="25.4" x2="38.1" y2="25.4" width="0.1524" layer="91"/>
+<label x="35.56" y="25.4" size="1.778" layer="95"/>
+</segment>
+</net>
+<net name="EXT_OUT9" class="0">
+<segment>
+<pinref part="PL5" gate="G$1" pin="TT"/>
+<wire x1="27.94" y1="-2.54" x2="38.1" y2="-2.54" width="0.1524" layer="91"/>
+<label x="35.56" y="-2.54" size="1.778" layer="95"/>
+</segment>
+</net>
+<net name="EXT_OUT10" class="0">
+<segment>
+<pinref part="PL5" gate="G$1" pin="TB"/>
+<wire x1="27.94" y1="-12.7" x2="38.1" y2="-12.7" width="0.1524" layer="91"/>
+<label x="35.56" y="-12.7" size="1.778" layer="95"/>
+</segment>
+</net>
+<net name="EXT_OUT11" class="0">
+<segment>
+<pinref part="PL6" gate="G$1" pin="TT"/>
+<wire x1="27.94" y1="-40.64" x2="38.1" y2="-40.64" width="0.1524" layer="91"/>
+<label x="38.1" y="-40.64" size="1.778" layer="95"/>
+</segment>
+</net>
+<net name="EXT_OUT12" class="0">
+<segment>
+<pinref part="PL6" gate="G$1" pin="TB"/>
+<wire x1="27.94" y1="-50.8" x2="38.1" y2="-50.8" width="0.1524" layer="91"/>
+<label x="38.1" y="-50.8" size="1.778" layer="95"/>
+</segment>
+</net>
+<net name="N$96" class="0">
+<segment>
+<pinref part="LED1" gate="G$1" pin="A_2"/>
+<pinref part="R99" gate="G$1" pin="1"/>
+<wire x1="124.46" y1="76.2" x2="121.92" y2="76.2" width="0.1524" layer="91"/>
+</segment>
+</net>
+<net name="N$119" class="0">
+<segment>
+<pinref part="LED1" gate="G$1" pin="A_3"/>
+<pinref part="R100" gate="G$1" pin="1"/>
+<wire x1="124.46" y1="71.12" x2="121.92" y2="71.12" width="0.1524" layer="91"/>
+</segment>
+</net>
+<net name="N$120" class="0">
+<segment>
+<pinref part="LED1" gate="G$1" pin="A_1"/>
+<pinref part="R98" gate="G$1" pin="1"/>
+<wire x1="124.46" y1="81.28" x2="121.92" y2="81.28" width="0.1524" layer="91"/>
+</segment>
+</net>
+<net name="LED1" class="0">
+<segment>
+<pinref part="R98" gate="G$1" pin="2"/>
+<wire x1="134.62" y1="81.28" x2="144.78" y2="81.28" width="0.1524" layer="91"/>
+<label x="142.24" y="81.28" size="1.778" layer="95"/>
+</segment>
+</net>
+<net name="LED2" class="0">
+<segment>
+<pinref part="R99" gate="G$1" pin="2"/>
+<wire x1="134.62" y1="76.2" x2="144.78" y2="76.2" width="0.1524" layer="91"/>
+<label x="142.24" y="76.2" size="1.778" layer="95"/>
+</segment>
+</net>
+<net name="LED3" class="0">
+<segment>
+<pinref part="R100" gate="G$1" pin="2"/>
+<wire x1="134.62" y1="71.12" x2="144.78" y2="71.12" width="0.1524" layer="91"/>
+<label x="142.24" y="71.12" size="1.778" layer="95"/>
+</segment>
+</net>
 </nets>
 </sheet>
@@
 </segment>
 </net>
+<net name="LED2" class="0">
+<segment>
+<pinref part="U3" gate="A" pin="PC11"/>
+<wire x1="99.06" y1="20.32" x2="109.22" y2="20.32" width="0.1524" layer="91"/>
+<label x="109.22" y="20.32" size="1.778" layer="95"/>
+</segment>
+</net>
+<net name="LED3" class="0">
+<segment>
+<pinref part="U3" gate="A" pin="PC10"/>
+<wire x1="99.06" y1="22.86" x2="109.22" y2="22.86" width="0.1524" layer="91"/>
+<label x="109.22" y="22.86" size="1.778" layer="95"/>
+</segment>
+</net>
+<net name="LED1" class="0">
+<segment>
+<pinref part="U3" gate="A" pin="PC12"/>
+<wire x1="99.06" y1="17.78" x2="109.22" y2="17.78" width="0.1524" layer="91"/>
+<label x="109.22" y="17.78" size="1.778" layer="95"/>
+</segment>
+</net>
 </nets>
 </sheet>
@@
 <net name="DAC_OUT9" class="0">
 <segment>
-<pinref part="U7" gate="A" pin="VOUT1"/>
-<wire x1="119.38" y1="76.2" x2="127" y2="76.2" width="0.1524" layer="91"/>
-<label x="127" y="76.2" size="1.778" layer="95"/>
+<pinref part="U7" gate="A" pin="VOUT4"/>
+<wire x1="119.38" y1="83.82" x2="127" y2="83.82" width="0.1524" layer="91"/>
+<label x="127" y="83.82" size="1.778" layer="95"/>
 </segment>
 </net>
 <net name="DAC_OUT10" class="0">
 <segment>
-<pinref part="U7" gate="A" pin="VOUT2"/>
-<wire x1="119.38" y1="78.74" x2="127" y2="78.74" width="0.1524" layer="91"/>
-<label x="127" y="78.74" size="1.778" layer="95"/>
-</segment>
-</net>
-<net name="DAC_OUT11" class="0">
-<segment>
 <pinref part="U7" gate="A" pin="VOUT3"/>
 <wire x1="119.38" y1="81.28" x2="127" y2="81.28" width="0.1524" layer="91"/>
@@
 </segment>
 </net>
-<net name="DAC_OUT12" class="0">
-<segment>
-<pinref part="U7" gate="A" pin="VOUT4"/>
-<wire x1="119.38" y1="83.82" x2="127" y2="83.82" width="0.1524" layer="91"/>
-<label x="127" y="83.82" size="1.778" layer="95"/>
-</segment>
-</net>
 <net name="N$97" class="0">
 <segment>
@@
 </segment>
 </net>
+<net name="DAC_OUT11" class="0">
+<segment>
+<pinref part="U7" gate="A" pin="VOUT2"/>
+<wire x1="119.38" y1="78.74" x2="127" y2="78.74" width="0.1524" layer="91"/>
+<label x="127" y="78.74" size="1.778" layer="95"/>
+</segment>
+</net>
+<net name="DAC_OUT12" class="0">
+<segment>
+<pinref part="U7" gate="A" pin="VOUT1"/>
+<wire x1="119.38" y1="76.2" x2="127" y2="76.2" width="0.1524" layer="91"/>
+<label x="127" y="76.2" size="1.778" layer="95"/>
+</segment>
+</net>

Commit message: wip
Parts:
- added C102: 0.1u, keves-ng:CAP_CERAMIC0603
- added C103: 100n, keves-ng:CAP_CERAMIC0603
- added IC7: AT45DB161D-SU, atmel:AT45DB161D-SU
- added R101: 1k, keves-ng:RESISTOR0603
- C95, C99: device microbuilder:CAP_CERAMIC0603 -> keves-ng:CAP_CERAMIC0603
- L5, L6: device microbuilder:INDUCTOR_0805 -> keves-ng:INDUCTOR_0603
- R94, R95, R96, R97: device microbuilder:RESISTOR_0805 -> keves-ng:RESISTOR0603
Connections:
- new net LED4: R101.1, U3A.PD0
- new net N$121: R101.2, U$1.LED+
- new net PUSHBTN: C102.P$1, U$1.IN1, U$1.IN2, U3A.PD1
- net +3V3: now also C103.P$1, IC7.!RESET, IC7.!WP, IC7.VCC
- net GND: now also C102.P$2, C103.P$2, IC7.GND, U$1.LED-, U$1.OUT1_NO, U$1.OUT2_NO
- net SPI_CLK: now also IC7.SCK
- net SPI_MISO: now also IC7.SO
- net SPI_MOSI: now also IC7.SI

Commit message: wip
Connections:
- new net SPI_CS_FLASH: IC7.!CS, U3A.PC4
Changed lines of the file:
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@@
 <junction x="106.68" y="15.24"/>
 <label x="91.44" y="15.24" size="1.778" layer="95"/>
+<junction x="114.3" y="15.24"/>
 </segment>
 </net>
@@
 </segment>
 </net>
+<net name="SPI_CS_FLASH" class="0">
+<segment>
+<pinref part="U3" gate="A" pin="PC4"/>
+<wire x1="99.06" y1="38.1" x2="116.84" y2="38.1" width="0.1524" layer="91"/>
+<label x="111.76" y="38.1" size="1.778" layer="95"/>
+</segment>
+<segment>
+<pinref part="IC7" gate="G$1" pin="!CS"/>
+<wire x1="139.7" y1="0" x2="116.84" y2="0" width="0.1524" layer="91"/>
+<label x="111.76" y="0" size="1.778" layer="95"/>
+</segment>
+</net>
 </nets>
 </sheet>
@@
 </sheet>
 </sheets>
+<errors>
+</errors>
 </schematic>
 </drawing>

Commit message: wip
Parts:
- added R102, R103, R104, R105: 1k, keves-ng:RESISTOR0603
Connections:
- net +5V: now also U4.VBUS
- net GND: now also R102.2, R103.2, R104.2, R105.2
- net N$100: now also R105.1
- net N$97: now also R102.1
- net N$98: now also R103.1
- net N$99: now also R104.1
Changed lines of the file:
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@@
 <part name="+3V19" library="supply1" library_urn="urn:adsk.eagle:library:371" deviceset="+3V3" device=""/>
 <part name="+3V20" library="supply1" library_urn="urn:adsk.eagle:library:371" deviceset="+3V3" device=""/>
+<part name="P+19" library="supply1" library_urn="urn:adsk.eagle:library:371" deviceset="+5V" device=""/>
+<part name="R102" library="keves-ng" library_urn="urn:adsk.eagle:library:1429743" deviceset="RESISTOR" device="0603" package3d_urn="urn:adsk.eagle:package:23799129/3" value="1k"/>
+<part name="R103" library="keves-ng" library_urn="urn:adsk.eagle:library:1429743" deviceset="RESISTOR" device="0603" package3d_urn="urn:adsk.eagle:package:23799129/3" value="1k"/>
+<part name="R104" library="keves-ng" library_urn="urn:adsk.eagle:library:1429743" deviceset="RESISTOR" device="0603" package3d_urn="urn:adsk.eagle:package:23799129/3" value="1k"/>
+<part name="R105" library="keves-ng" library_urn="urn:adsk.eagle:library:1429743" deviceset="RESISTOR" device="0603" package3d_urn="urn:adsk.eagle:package:23799129/3" value="1k"/>
+<part name="GND91" library="supply1" library_urn="urn:adsk.eagle:library:371" deviceset="GND" device=""/>
+<part name="GND92" library="supply1" library_urn="urn:adsk.eagle:library:371" deviceset="GND" device=""/>
+<part name="GND93" library="supply1" library_urn="urn:adsk.eagle:library:371" deviceset="GND" device=""/>
+<part name="GND94" library="supply1" library_urn="urn:adsk.eagle:library:371" deviceset="GND" device=""/>
 </parts>
 <sheets>
@@
 <attribute name="VALUE" x="104.14" y="-2.54" size="1.778" layer="96"/>
 </instance>
+<instance part="P+19" gate="1" x="111.76" y="142.24" smashed="yes" rot="R270">
+<attribute name="VALUE" x="106.68" y="144.78" size="1.778" layer="96"/>
+</instance>
 </instances>
 <busses>
@@
 <wire x1="142.24" y1="101.6" x2="139.7" y2="101.6" width="0.1524" layer="91"/>
 </segment>
+<segment>
+<pinref part="U4" gate="A" pin="VBUS"/>
+<pinref part="P+19" gate="1" pin="+5V"/>
+<wire x1="109.22" y1="142.24" x2="106.68" y2="142.24" width="0.1524" layer="91"/>
+</segment>
 </net>
 <net name="N$50" class="0">
@@
 <net name="USB_DEV_P" class="1">
 <segment>
-<wire x1="109.22" y1="142.24" x2="109.22" y2="139.7" width="0.1524" layer="91"/>
+<wire x1="114.3" y1="142.24" x2="114.3" y2="139.7" width="0.1524" layer="91"/>
 <pinref part="R62" gate="G$1" pin="1"/>
-<wire x1="109.22" y1="142.24" x2="116.84" y2="142.24" width="0.1524" layer="91"/>
+<wire x1="114.3" y1="142.24" x2="116.84" y2="142.24" width="0.1524" layer="91"/>
 <pinref part="U4" gate="A" pin="I/O1"/>
-<wire x1="109.22" y1="139.7" x2="106.68" y2="139.7" width="0.1524" layer="91"/>
+<wire x1="114.3" y1="139.7" x2="106.68" y2="139.7" width="0.1524" layer="91"/>
 </segment>
 </net>
@@
 <attribute name="VALUE" x="58.42" y="111.76" size="1.778" layer="96"/>
 </instance>
+<instance part="R102" gate="G$1" x="132.08" y="86.36" smashed="yes">
+<attribute name="NAME" x="129.54" y="88.392" size="1.27" layer="95" font="vector"/>
+<attribute name="VALUE" x="129.54" y="83.185" size="1.27" layer="96" font="vector"/>
+</instance>
+<instance part="R103" gate="G$1" x="132.08" y="88.9" smashed="yes">
+<attribute name="NAME" x="129.54" y="90.932" size="1.27" layer="95" font="vector"/>
+<attribute name="VALUE" x="129.54" y="85.725" size="1.27" layer="96" font="vector"/>
+</instance>
+<instance part="R104" gate="G$1" x="132.08" y="91.44" smashed="yes">
+<attribute name="NAME" x="129.54" y="93.472" size="1.27" layer="95" font="vector"/>
+<attribute name="VALUE" x="129.54" y="88.265" size="1.27" layer="96" font="vector"/>
+</instance>
+<instance part="R105" gate="G$1" x="132.08" y="93.98" smashed="yes">
+<attribute name="NAME" x="129.54" y="96.012" size="1.27" layer="95" font="vector"/>
+<attribute name="VALUE" x="129.54" y="90.805" size="1.27" layer="96" font="vector"/>
+</instance>
+<instance part="GND91" gate="1" x="142.24" y="93.98" smashed="yes" rot="R90">
+<attribute name="VALUE" x="144.78" y="91.44" size="1.778" layer="96" rot="R90"/>
+</instance>
+<instance part="GND92" gate="1" x="142.24" y="91.44" smashed="yes" rot="R90">
+<attribute name="VALUE" x="144.78" y="88.9" size="1.778" layer="96" rot="R90"/>
+</instance>
+<instance part="GND93" gate="1" x="142.24" y="88.9" smashed="yes" rot="R90">
+<attribute name="VALUE" x="144.78" y="86.36" size="1.778" layer="96" rot="R90"/>
+</instance>
+<instance part="GND94" gate="1" x="142.24" y="86.36" smashed="yes" rot="R90">
+<attribute name="VALUE" x="144.78" y="83.82" size="1.778" layer="96" rot="R90"/>
+</instance>
 </instances>
 <busses>
@@
 <wire x1="-10.16" y1="83.82" x2="-2.54" y2="83.82" width="0.1524" layer="91"/>
 </segment>
+<segment>
+<pinref part="R105" gate="G$1" pin="2"/>
+<pinref part="GND91" gate="1" pin="GND"/>
+<wire x1="139.7" y1="93.98" x2="137.16" y2="93.98" width="0.1524" layer="91"/>
+</segment>
+<segment>
+<pinref part="R104" gate="G$1" pin="2"/>
+<pinref part="GND92" gate="1" pin="GND"/>
+<wire x1="139.7" y1="91.44" x2="137.16" y2="91.44" width="0.1524" layer="91"/>
+</segment>
+<segment>
+<pinref part="R103" gate="G$1" pin="2"/>
+<pinref part="GND93" gate="1" pin="GND"/>
+<wire x1="139.7" y1="88.9" x2="137.16" y2="88.9" width="0.1524" layer="91"/>
+</segment>
+<segment>
+<pinref part="R102" gate="G$1" pin="2"/>
+<pinref part="GND94" gate="1" pin="GND"/>
+<wire x1="139.7" y1="86.36" x2="137.16" y2="86.36" width="0.1524" layer="91"/>
+</segment>
 </net>
 <net name="N$79" class="0">
@@
 <pinref part="U7" gate="A" pin="VOUT5"/>
 <wire x1="119.38" y1="86.36" x2="127" y2="86.36" width="0.1524" layer="91"/>
+<pinref part="R102" gate="G$1" pin="1"/>
 </segment>
 </net>
@@
 <pinref part="U7" gate="A" pin="VOUT6"/>
 <wire x1="119.38" y1="88.9" x2="127" y2="88.9" width="0.1524" layer="91"/>
+<pinref part="R103" gate="G$1" pin="1"/>
 </segment>
 </net>
@@
 <pinref part="U7" gate="A" pin="VOUT7"/>
 <wire x1="119.38" y1="91.44" x2="127" y2="91.44" width="0.1524" layer="91"/>
+<pinref part="R104" gate="G$1" pin="1"/>
 </segment>
 </net>
@@
 <pinref part="U7" gate="A" pin="VOUT8"/>
 <wire x1="119.38" y1="93.98" x2="127" y2="93.98" width="0.1524" layer="91"/>
+<pinref part="R105" gate="G$1" pin="1"/>
 </segment>
 </net>
