File: dt/dt.sch (EAGLE design)
At the start: 264 parts, among them IC1 TL072D, IC10 LM317, IC11 LM337, IC2 TL072D, IC3 TL072D, IC4 TL072D, IC5 TL072D, IC6 TL072D, IC7 AT45DB161D-SU, U2 PCN2-S5-D12-S, U3 STM32F7X3ZXT, U4 USBLC6-2SC6YSOT23-6L_STM-M, U5 USBLC6-2SC6YSOT23-6L_STM-M, U6 PCM1681PWPPWP28_6P46X2P4-M, U7 PCM1681PWPPWP28_6P46X2P4-M, Y1 ABLS7M2-25.000MHZ-D2Y-T

Commit message: wip
Parts:
- D1, D2, D3, D4: value (none) -> MBR120LSFT3G
- OSC1: value (none) -> 12.288MHz; PARTNO (none) -> C3391-12.288
- U1: value (none) -> LM1117DTX-3.3; PARTNO (none) -> LM1117DTX-3.3/NOPB
Connections:
- net UART_RX: now also U3A.PD6
- net UART_TX: now also U3A.PD5
Changed lines of the file:
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@@
 <part name="GND35" library="supply1" library_urn="urn:adsk.eagle:library:371" deviceset="GND" device=""/>
 <part name="GND36" library="supply1" library_urn="urn:adsk.eagle:library:371" deviceset="GND" device=""/>
-<part name="U1" library="keves-ng" library_urn="urn:adsk.eagle:library:1429743" deviceset="LM1117" device="TO252" package3d_urn="urn:adsk.eagle:package:23807383/2"/>
+<part name="U1" library="keves-ng" library_urn="urn:adsk.eagle:library:1429743" deviceset="LM1117" device="TO252" package3d_urn="urn:adsk.eagle:package:23807383/2" value="LM1117DTX-3.3">
+<attribute name="PARTNO" value="LM1117DTX-3.3/NOPB"/>
+</part>
 <part name="P+1" library="supply1" library_urn="urn:adsk.eagle:library:371" deviceset="+5V" device=""/>
 <part name="GND37" library="supply1" library_urn="urn:adsk.eagle:library:371" deviceset="GND" device=""/>
@@
 <part name="GND54" library="supply1" library_urn="urn:adsk.eagle:library:371" deviceset="GND" device=""/>
 <part name="C75" library="keves-ng" library_urn="urn:adsk.eagle:library:1429743" deviceset="CAP_CERAMIC" device="0603" package3d_urn="urn:adsk.eagle:package:23799129/3" value="4.7uF"/>
-<part name="OSC1" library="keves-ng" library_urn="urn:adsk.eagle:library:1429743" deviceset="OSCILLATOR" device="" package3d_urn="urn:adsk.eagle:package:23815268/1"/>
+<part name="OSC1" library="keves-ng" library_urn="urn:adsk.eagle:library:1429743" deviceset="OSCILLATOR" device="" package3d_urn="urn:adsk.eagle:package:23815268/1" value="12.288MHz">
+<attribute name="PARTNO" value="C3391-12.288"/>
+</part>
 <part name="GND55" library="supply1" library_urn="urn:adsk.eagle:library:371" deviceset="GND" device=""/>
 <part name="+3V9" library="supply1" library_urn="urn:adsk.eagle:library:371" deviceset="+3V3" device=""/>
@@
 </part>
 <part name="C94" library="microbuilder" deviceset="CAP_CERAMIC" device="_0805" value="2.2uF"/>
-<part name="D1" library="microbuilder" deviceset="DIODE" device="SOD-123"/>
+<part name="D1" library="microbuilder" deviceset="DIODE" device="SOD-123" value="MBR120LSFT3G"/>
 <part name="R94" library="keves-ng" library_urn="urn:adsk.eagle:library:1429743" deviceset="RESISTOR" device="0603" package3d_urn="urn:adsk.eagle:package:23799129/3" value="240 0.1%"/>
 <part name="R95" library="keves-ng" library_urn="urn:adsk.eagle:library:1429743" deviceset="RESISTOR" device="0603" package3d_urn="urn:adsk.eagle:package:23799129/3" value="2.2k 0.1%"/>
@@
 <part name="C96" library="microbuilder" deviceset="CAP_CERAMIC" device="0805" value="10uF"/>
 <part name="C97" library="microbuilder" deviceset="CAP_CERAMIC" device="1206" value="1uF 12065C105M4Z2A"/>
-<part name="D2" library="microbuilder" deviceset="DIODE" device="SOD-123"/>
+<part name="D2" library="microbuilder" deviceset="DIODE" device="SOD-123" value="MBR120LSFT3G"/>
 <part name="U$27" library="microbuilder" deviceset="GND" device=""/>
 <part name="L5" library="keves-ng" library_urn="urn:adsk.eagle:library:1429743" deviceset="INDUCTOR" device="_0603" package3d_urn="urn:adsk.eagle:package:23799135/2" value="ILHB0805ER601V"/>
@@
 <attribute name="PARTNO" value="LM337IMPX/NOPB"/>
 </part>
-<part name="D3" library="microbuilder" deviceset="DIODE" device="SOD-123"/>
+<part name="D3" library="microbuilder" deviceset="DIODE" device="SOD-123" value="MBR120LSFT3G"/>
 <part name="C98" library="microbuilder" deviceset="CAP_CERAMIC" device="_0805" value="2.2uF"/>
 <part name="C99" library="keves-ng" library_urn="urn:adsk.eagle:library:1429743" deviceset="CAP_CERAMIC" device="0603" package3d_urn="urn:adsk.eagle:package:23799129/3" value="0.1u"/>
@@
 <part name="U$29" library="microbuilder" deviceset="GND" device=""/>
 <part name="C100" library="microbuilder" deviceset="CAP_CERAMIC" device="0805" value="10uF"/>
-<part name="D4" library="microbuilder" deviceset="DIODE" device="SOD-123"/>
+<part name="D4" library="microbuilder" deviceset="DIODE" device="SOD-123" value="MBR120LSFT3G"/>
 <part name="L6" library="keves-ng" library_urn="urn:adsk.eagle:library:1429743" deviceset="INDUCTOR" device="_0603" package3d_urn="urn:adsk.eagle:package:23799135/2" value="ILHB0805ER601V"/>
 <part name="C101" library="microbuilder" deviceset="CAP_CERAMIC" device="1206" value="1uF 12065C105M4Z2A"/>
@@
 <attribute name="NAME" x="147.32" y="-54.864" size="1.27" layer="95"/>
 <attribute name="VALUE" x="153.416" y="-66.04" size="1.27" layer="96"/>
+<attribute name="PARTNO" x="152.4" y="-58.42" size="1.778" layer="96" display="off"/>
 </instance>
 <instance part="P+1" gate="1" x="129.54" y="-58.42" smashed="yes" rot="R90">
@@
 <attribute name="NAME" x="124.46" y="137.795" size="1.27" layer="95"/>
 <attribute name="VALUE" x="124.46" y="119.38" size="1.27" layer="96"/>
+<attribute name="PARTNO" x="132.08" y="129.54" size="1.778" layer="96" display="off"/>
 </instance>
 <instance part="GND55" gate="1" x="114.3" y="121.92" smashed="yes">
@@
 <label x="60.96" y="134.62" size="1.778" layer="95"/>
 </segment>
+<segment>
+<pinref part="U3" gate="A" pin="PD6"/>
+<wire x1="27.94" y1="30.48" x2="12.7" y2="30.48" width="0.1524" layer="91"/>
+<label x="10.16" y="30.48" size="1.778" layer="95"/>
+</segment>
 </net>
 <net name="SWCLK" class="0">
@@
 <label x="27.94" y="134.62" size="1.778" layer="95"/>
 </segment>
+<segment>
+<pinref part="U3" gate="A" pin="PD5"/>
+<wire x1="27.94" y1="33.02" x2="12.7" y2="33.02" width="0.1524" layer="91"/>
+<label x="10.16" y="33.02" size="1.778" layer="95"/>
+</segment>
 </net>

Commit message: wip
Parts:
- added U$2: PHI-LOGO, keves-ng:PHI-LOGO
Changed lines of the file:
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@@
 <part name="GND93" library="supply1" library_urn="urn:adsk.eagle:library:371" deviceset="GND" device=""/>
 <part name="GND94" library="supply1" library_urn="urn:adsk.eagle:library:371" deviceset="GND" device=""/>
+<part name="U$2" library="keves-ng" library_urn="urn:adsk.eagle:library:1429743" deviceset="PHI-LOGO" device="" package3d_urn="urn:adsk.eagle:package:24014368/1"/>
 </parts>
 <sheets>
@@
 <attribute name="VALUE" x="106.68" y="144.78" size="1.778" layer="96"/>
 </instance>
+<instance part="U$2" gate="G$1" x="182.88" y="147.32" smashed="yes"/>
 </instances>
 <busses>

Commit message: wip
Parts:
- C100, C96: value 10uF -> 10u; device microbuilder:CAP_CERAMIC0805 -> keves-ng:CAP_CERAMIC0805
- C101, C97: device microbuilder:CAP_CERAMIC1206 -> keves-ng:CAP_CERAMIC1206
- C102, C95, C99: value 0.1u -> 100n
- C77: value 100uF -> 100u
- C94, C98: value 2.2uF -> 2.2u; device microbuilder:CAP_CERAMIC_0805 -> keves-ng:CAP_CERAMIC0805
- D1, D2, D3, D4: device microbuilder:DIODESOD-123 -> keves-ng:DIODESOD-123
Changed lines of the file:
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@@
 <part name="GND56" library="supply1" library_urn="urn:adsk.eagle:library:371" deviceset="GND" device=""/>
 <part name="P+4" library="supply1" library_urn="urn:adsk.eagle:library:371" deviceset="+5V" device=""/>
-<part name="C77" library="keves-ng" library_urn="urn:adsk.eagle:library:1429743" deviceset="CAP_ELECTROLYTIC" device="PANASONIC_D" package3d_urn="urn:adsk.eagle:package:23799140/1" value="100uF"/>
+<part name="C77" library="keves-ng" library_urn="urn:adsk.eagle:library:1429743" deviceset="CAP_ELECTROLYTIC" device="PANASONIC_D" package3d_urn="urn:adsk.eagle:package:23799140/1" value="100u"/>
 <part name="GND57" library="supply1" library_urn="urn:adsk.eagle:library:371" deviceset="GND" device=""/>
 <part name="R57" library="keves-ng" library_urn="urn:adsk.eagle:library:1429743" deviceset="RESISTOR" device="0603" package3d_urn="urn:adsk.eagle:package:23799129/3" value="1M"/>
@@
 <attribute name="PARTNO" value="LM317MBSTT3G"/>
 </part>
-<part name="C94" library="microbuilder" deviceset="CAP_CERAMIC" device="_0805" value="2.2uF"/>
-<part name="D1" library="microbuilder" deviceset="DIODE" device="SOD-123" value="MBR120LSFT3G"/>
+<part name="C94" library="keves-ng" library_urn="urn:adsk.eagle:library:1429743" deviceset="CAP_CERAMIC" device="0805" package3d_urn="urn:adsk.eagle:package:23799128/2" value="2.2u"/>
+<part name="D1" library="keves-ng" library_urn="urn:adsk.eagle:library:1429743" deviceset="DIODE" device="SOD-123" value="MBR120LSFT3G"/>
 <part name="R94" library="keves-ng" library_urn="urn:adsk.eagle:library:1429743" deviceset="RESISTOR" device="0603" package3d_urn="urn:adsk.eagle:package:23799129/3" value="240 0.1%"/>
 <part name="R95" library="keves-ng" library_urn="urn:adsk.eagle:library:1429743" deviceset="RESISTOR" device="0603" package3d_urn="urn:adsk.eagle:package:23799129/3" value="2.2k 0.1%"/>
-<part name="C95" library="keves-ng" library_urn="urn:adsk.eagle:library:1429743" deviceset="CAP_CERAMIC" device="0603" package3d_urn="urn:adsk.eagle:package:23799129/3" value="0.1u"/>
-<part name="C96" library="microbuilder" deviceset="CAP_CERAMIC" device="0805" value="10uF"/>
-<part name="C97" library="microbuilder" deviceset="CAP_CERAMIC" device="1206" value="1uF 12065C105M4Z2A"/>
-<part name="D2" library="microbuilder" deviceset="DIODE" device="SOD-123" value="MBR120LSFT3G"/>
-<part name="U$27" library="microbuilder" deviceset="GND" device=""/>
+<part name="C95" library="keves-ng" library_urn="urn:adsk.eagle:library:1429743" deviceset="CAP_CERAMIC" device="0603" package3d_urn="urn:adsk.eagle:package:23799129/3" value="100n"/>
+<part name="C96" library="keves-ng" library_urn="urn:adsk.eagle:library:1429743" deviceset="CAP_CERAMIC" device="0805" package3d_urn="urn:adsk.eagle:package:23799128/2" value="10u"/>
+<part name="C97" library="keves-ng" library_urn="urn:adsk.eagle:library:1429743" deviceset="CAP_CERAMIC" device="1206" package3d_urn="urn:adsk.eagle:package:23799125/1" value="1uF 12065C105M4Z2A"/>
+<part name="D2" library="keves-ng" library_urn="urn:adsk.eagle:library:1429743" deviceset="DIODE" device="SOD-123" value="MBR120LSFT3G"/>
+<part name="U$27" library="supply1" library_urn="urn:adsk.eagle:library:371" deviceset="GND" device=""/>
 <part name="L5" library="keves-ng" library_urn="urn:adsk.eagle:library:1429743" deviceset="INDUCTOR" device="_0603" package3d_urn="urn:adsk.eagle:package:23799135/2" value="ILHB0805ER601V"/>
 <part name="APWR_EN" library="jumper" deviceset="JP2QE" device=""/>
@@
 <attribute name="PARTNO" value="LM337IMPX/NOPB"/>
 </part>
-<part name="D3" library="microbuilder" deviceset="DIODE" device="SOD-123" value="MBR120LSFT3G"/>
-<part name="C98" library="microbuilder" deviceset="CAP_CERAMIC" device="_0805" value="2.2uF"/>
-<part name="C99" library="keves-ng" library_urn="urn:adsk.eagle:library:1429743" deviceset="CAP_CERAMIC" device="0603" package3d_urn="urn:adsk.eagle:package:23799129/3" value="0.1u"/>
+<part name="D3" library="keves-ng" library_urn="urn:adsk.eagle:library:1429743" deviceset="DIODE" device="SOD-123" value="MBR120LSFT3G"/>
+<part name="C98" library="keves-ng" library_urn="urn:adsk.eagle:library:1429743" deviceset="CAP_CERAMIC" device="0805" package3d_urn="urn:adsk.eagle:package:23799128/2" value="2.2u"/>
+<part name="C99" library="keves-ng" library_urn="urn:adsk.eagle:library:1429743" deviceset="CAP_CERAMIC" device="0603" package3d_urn="urn:adsk.eagle:package:23799129/3" value="100n"/>
 <part name="R96" library="keves-ng" library_urn="urn:adsk.eagle:library:1429743" deviceset="RESISTOR" device="0603" package3d_urn="urn:adsk.eagle:package:23799129/3" value="2.2k 0.1%"/>
 <part name="R97" library="keves-ng" library_urn="urn:adsk.eagle:library:1429743" deviceset="RESISTOR" device="0603" package3d_urn="urn:adsk.eagle:package:23799129/3" value="240 0.1%"/>
-<part name="U$29" library="microbuilder" deviceset="GND" device=""/>
-<part name="C100" library="microbuilder" deviceset="CAP_CERAMIC" device="0805" value="10uF"/>
-<part name="D4" library="microbuilder" deviceset="DIODE" device="SOD-123" value="MBR120LSFT3G"/>
+<part name="U$29" library="supply1" library_urn="urn:adsk.eagle:library:371" deviceset="GND" device=""/>
+<part name="C100" library="keves-ng" library_urn="urn:adsk.eagle:library:1429743" deviceset="CAP_CERAMIC" device="0805" package3d_urn="urn:adsk.eagle:package:23799128/2" value="10u"/>
+<part name="D4" library="keves-ng" library_urn="urn:adsk.eagle:library:1429743" deviceset="DIODE" device="SOD-123" value="MBR120LSFT3G"/>
 <part name="L6" library="keves-ng" library_urn="urn:adsk.eagle:library:1429743" deviceset="INDUCTOR" device="_0603" package3d_urn="urn:adsk.eagle:package:23799135/2" value="ILHB0805ER601V"/>
-<part name="C101" library="microbuilder" deviceset="CAP_CERAMIC" device="1206" value="1uF 12065C105M4Z2A"/>
+<part name="C101" library="keves-ng" library_urn="urn:adsk.eagle:library:1429743" deviceset="CAP_CERAMIC" device="1206" package3d_urn="urn:adsk.eagle:package:23799125/1" value="1uF 12065C105M4Z2A"/>
 <part name="P+3" library="supply1" library_urn="urn:adsk.eagle:library:371" deviceset="+15V" device=""/>
 <part name="P+11" library="supply1" library_urn="urn:adsk.eagle:library:371" deviceset="+15V" device=""/>
@@
 <part name="R101" library="keves-ng" library_urn="urn:adsk.eagle:library:1429743" deviceset="RESISTOR" device="0603" package3d_urn="urn:adsk.eagle:package:23799129/3" value="1k"/>
 <part name="GND86" library="supply1" library_urn="urn:adsk.eagle:library:371" deviceset="GND" device=""/>
-<part name="C102" library="keves-ng" library_urn="urn:adsk.eagle:library:1429743" deviceset="CAP_CERAMIC" device="0603" package3d_urn="urn:adsk.eagle:package:23799129/3" value="0.1u"/>
+<part name="C102" library="keves-ng" library_urn="urn:adsk.eagle:library:1429743" deviceset="CAP_CERAMIC" device="0603" package3d_urn="urn:adsk.eagle:package:23799129/3" value="100n"/>
 <part name="GND87" library="supply1" library_urn="urn:adsk.eagle:library:371" deviceset="GND" device=""/>
 <part name="GND88" library="supply1" library_urn="urn:adsk.eagle:library:371" deviceset="GND" device=""/>
@@
 <attribute name="VALUE" x="172.72" y="-105.41" size="1.27" layer="96" rot="R180"/>
 </instance>
-<instance part="U$27" gate="G$1" x="165.1" y="-152.4" smashed="yes">
+<instance part="U$27" gate="1" x="165.1" y="-152.4" smashed="yes">
 <attribute name="VALUE" x="163.576" y="-154.94" size="1.27" layer="96"/>
 </instance>
@@
 <attribute name="VALUE" x="193.675" y="-180.34" size="1.27" layer="96" font="vector" rot="R90"/>
 </instance>
-<instance part="U$29" gate="G$1" x="180.34" y="-152.4" smashed="yes" rot="R180">
+<instance part="U$29" gate="1" x="180.34" y="-152.4" smashed="yes" rot="R180">
 <attribute name="VALUE" x="181.864" y="-149.86" size="1.27" layer="96" rot="R180"/>
 </instance>
@@
 <segment>
 <pinref part="R95" gate="G$1" pin="1"/>
-<pinref part="U$27" gate="G$1" pin="GND"/>
+<pinref part="U$27" gate="1" pin="GND"/>
 <wire x1="165.1" y1="-149.86" x2="165.1" y2="-147.32" width="0.1524" layer="91"/>
 <pinref part="C97" gate="G$1" pin="P$2"/>
@@
 </segment>
 <segment>
-<pinref part="U$29" gate="G$1" pin="GND"/>
+<pinref part="U$29" gate="1" pin="GND"/>
 <pinref part="R96" gate="G$1" pin="2"/>
 <wire x1="180.34" y1="-154.94" x2="180.34" y2="-157.48" width="0.1524" layer="91"/>
