File: dt/dt.brd (EAGLE design)
At the start: 148.6 x 101.6 mm, 260 parts, among them IC1 TL072D, IC10 LM317, IC11 LM337, IC2 TL072D, IC3 TL072D, IC4 TL072D, IC5 TL072D, IC6 TL072D, IC7 AT45DB161D-SU, U2 PCN2-S5-D12-S, U3 STM32F7X3ZXT, U4 USBLC6-2SC6YSOT23-6L_STM-M, U5 USBLC6-2SC6YSOT23-6L_STM-M, U6 PCM1681PWPPWP28_6P46X2P4-M, U7 PCM1681PWPPWP28_6P46X2P4-M, Y1 ABLS7M2-25.000MHZ-D2Y-T

Commit message: wip
Routing:
- added copper zone on layer 2, net GND
- removed copper zone on layer 1, net GND

Commit message: wip
Parts:
- moved C68 1.30 mm to (83.3, 62.2)
- moved C84 1.27 mm to (8.00, 55.8), turned to 90 degrees
- moved C90 1.27 mm to (41.9, 55.6), turned to 90 degrees
- moved C83 1.05 mm to (4.19, 57.9), turned to 90 degrees
- moved C87 0.80 mm to (21.7, 58.8)
- moved C81 0.80 mm to (54.6, 58.7)
- moved C86 0.80 mm to (54.1, 54.1), turned to 0 degrees
- moved C55 0.51 mm to (110.5, 77.0)
- moved C75 0.51 mm to (97.8, 53.3)
- moved C80 0.25 mm to (21.0, 54.5), turned to 0 degrees
Routing:
- net GND: track 0.62 -> 277.3 mm, vias 0 -> 113
- net N$80: track 21.7 -> 27.5 mm
- net +3V3: track 218.2 -> 222.2 mm
- net USB_DEV_P: track 0.09 -> 2.03 mm
- net USB_DEV_N: track 0.09 -> 2.03 mm
- net N$104: track 20.6 -> 21.6 mm
- net N$84: track 16.6 -> 17.2 mm
- net N$58: track 2.54 -> 3.04 mm

Commit message: wip
Connections:
- new net SPI_CS_FLASH: IC7.4, U3.44
Routing:
- net SPI_CS_FLASH: track 0.00 -> 10.00 mm
- net +3V3: track 222.2 -> 220.7 mm
Changed lines of the file:
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@@
 <via x="93.726" y="97.536" extent="1-16" drill="0.35"/>
 <wire x1="91.186" y1="96.647" x2="91.186" y2="97.5007" width="0.3556" layer="1"/>
-<wire x1="91.186" y1="97.5007" x2="91.186" y2="97.536" width="0.3556" layer="1"/>
 <via x="91.186" y="97.5007" extent="1-16" drill="0.35"/>
-<wire x1="91.186" y1="97.5007" x2="91.186" y2="97.536" width="0.3556" layer="2"/>
 <wire x1="18.63" y1="79.248" x2="20.066" y2="79.248" width="0.3556" layer="1"/>
 <via x="20.066" y="79.248" extent="1-16" drill="0.35"/>
@@
 <contactref element="C87" pad="+"/>
 <contactref element="JP7" pad="3"/>
-<wire x1="54.61" y1="55.46" x2="54.61" y2="56.624" width="0.3556" layer="1"/>
 <contactref element="JP8" pad="3"/>
 <contactref element="R92" pad="2"/>
@@
 <wire x1="100.778" y1="54.25" x2="100.778" y2="56.685" width="0.3556" layer="1"/>
 <wire x1="95.886" y1="54.102" x2="95.778" y2="54.21" width="0.3556" layer="1"/>
-<wire x1="97.878" y1="54.102" x2="97.79" y2="54.19" width="0.3556" layer="1"/>
 <wire x1="100.838" y1="54.19" x2="100.778" y2="54.25" width="0.3556" layer="1"/>
 <wire x1="100.63" y1="54.102" x2="100.778" y2="54.25" width="0.3556" layer="1"/>
@@
 <wire x1="84.162" y1="63.412" x2="84.162" y2="62.23" width="0.3556" layer="1"/>
 <wire x1="84.832" y1="61.56" x2="84.162" y2="62.23" width="0.3556" layer="1"/>
-<wire x1="21.58605" y1="54.483" x2="21.805" y2="54.483" width="0.3556" layer="1"/>
 <wire x1="17.3228" y1="53.680015625" x2="19.426934375" y2="53.680015625" width="0.3556" layer="1"/>
 <wire x1="19.426934375" y1="53.680015625" x2="19.42875" y2="53.6782" width="0.3556" layer="1"/>
@@
 <wire x1="68.6562" y1="56.52328125" x2="68.6562" y2="56.40511875" width="0.254" layer="15"/>
 <wire x1="68.6562" y1="56.40511875" x2="67.44528125" y2="55.1942" width="0.254" layer="15"/>
-<wire x1="67.44528125" y1="55.1942" x2="28.8798" y2="55.1942" width="0.254" layer="15"/>
+<wire x1="67.44528125" y1="55.1942" x2="54.864" y2="55.1942" width="0.254" layer="15"/>
+<wire x1="54.864" y1="55.1942" x2="28.8798" y2="55.1942" width="0.254" layer="15"/>
 <wire x1="28.8798" y1="55.1942" x2="26.67" y2="57.404" width="0.254" layer="15"/>
 <wire x1="87.376" y1="55.372" x2="71.882" y2="55.372" width="0.254" layer="16"/>
@@
 <wire x1="64.516" y1="62.484" x2="28.448" y2="62.484" width="0.3556" layer="16"/>
 <wire x1="28.448" y1="62.484" x2="26.67" y2="60.706" width="0.3556" layer="16"/>
-<wire x1="64.516" y1="62.484" x2="64.516" y2="62.738" width="0.254" layer="15"/>
 <wire x1="91.186" y1="75.692" x2="91.694" y2="76.2" width="0.254" layer="15"/>
 <via x="91.694" y="76.2" extent="1-16" drill="0.35"/>
@@
 <contactref element="C91" pad="2"/>
 <contactref element="C92" pad="+"/>
-<wire x1="37.154" y1="55.538" x2="36.83" y2="55.862" width="0.3556" layer="1"/>
 <wire x1="36.83" y1="50.818" x2="36.83" y2="51.308" width="0.3556" layer="1"/>
 <wire x1="40.894" y1="51.65" x2="40.552" y2="51.308" width="0.3556" layer="1"/>
@@
 <wire x1="44.2722" y1="51.602984375" x2="40.941015625" y2="51.602984375" width="0.3556" layer="1"/>
 <wire x1="40.941015625" y1="51.602984375" x2="40.894" y2="51.65" width="0.3556" layer="1"/>
-<wire x1="36.83" y1="55.862" x2="37.25" y2="55.442" width="1.016" layer="1"/>
-<wire x1="37.25" y1="55.442" x2="37.25" y2="53.594" width="1.016" layer="1"/>
 <wire x1="37.25" y1="53.594" x2="37.25" y2="51.728" width="1.016" layer="1"/>
 <wire x1="37.25" y1="51.728" x2="36.83" y2="51.308" width="1.016" layer="1"/>
 <wire x1="44.2722" y1="55.50305" x2="42.88295" y2="55.50305" width="0.3556" layer="1"/>
 <wire x1="42.88295" y1="55.50305" x2="41.91" y2="56.476" width="0.3556" layer="1"/>
-<wire x1="36.83" y1="55.862" x2="37.444" y2="56.476" width="1.016" layer="1"/>
-<wire x1="37.444" y1="56.476" x2="41.91" y2="56.476" width="1.016" layer="1"/>
+<wire x1="37.25" y1="53.594" x2="36.83" y2="54.014" width="1.016" layer="1"/>
+<wire x1="36.83" y1="54.014" x2="36.83" y2="55.862" width="1.016" layer="1"/>
+<wire x1="41.91" y1="56.476" x2="37.444" y2="56.476" width="1.016" layer="1"/>
+<wire x1="37.444" y1="56.476" x2="36.83" y2="55.862" width="1.016" layer="1"/>
 </signal>
 <signal name="N$105">
@@
 <wire x1="12.168" y1="79.248" x2="16.93" y2="79.248" width="0.254" layer="1"/>
 </signal>
+<signal name="SPI_CS_FLASH">
+<contactref element="U3" pad="44"/>
+<contactref element="IC7" pad="4"/>
+<wire x1="91.778" y1="56.685" x2="91.7098" y2="56.7532" width="0.254" layer="1"/>
+<wire x1="91.7098" y1="56.7532" x2="91.7098" y2="57.4633125" width="0.254" layer="1"/>
+<wire x1="86.8454" y1="54.6024" x2="85.954" y2="53.711" width="0.254" layer="1"/>
+<wire x1="91.7098" y1="57.4633125" x2="91.1341125" y2="58.039" width="0.254" layer="1"/>
+<wire x1="91.1341125" y1="58.039" x2="87.88306875" y2="58.039" width="0.254" layer="1"/>
+<wire x1="87.88306875" y1="58.039" x2="86.8454" y2="57.00133125" width="0.254" layer="1"/>
+<wire x1="86.8454" y1="57.00133125" x2="86.8454" y2="54.6024" width="0.254" layer="1"/>
+</signal>
 </signals>

Commit message: wip
Parts:
- added R102, R103, R104, R105: 1k, keves-ng:0603
Connections:
- removed net VBUS: U4.5
- net +5V: now also U4.5
- net GND: now also R102.2, R103.2, R104.2, R105.2
- net N$100: now also R105.1
- net N$97: now also R102.1
- net N$98: now also R103.1
- net N$99: now also R104.1
Routing:
- net N$97: track 0.00 -> 11.3 mm, vias 0 -> 3
- net N$98: track 0.00 -> 10.7 mm, vias 0 -> 2
- net N$99: track 0.00 -> 8.72 mm
- net N$100: track 0.00 -> 7.74 mm
- net GND: track 277.2 -> 282.0 mm, vias 113 -> 117
- net +5V: track 290.0 -> 291.6 mm, vias 9 -> 10
- net +3V3: track 220.7 -> 219.9 mm

Commit message: wip
Parts:
- D1, D2, D3, D4: value (none) -> MBR120LSFT3G
- OSC1: value (none) -> 12.288MHz
- U1: value (none) -> LM1117DTX-3.3
- moved C48 0.36 mm to (135.1, 33.0)
Connections:
- net UART_RX: now also U3.122
- net UART_TX: now also U3.119
Routing:
- net UART_TX: track 0.00 -> 25.9 mm, vias 0 -> 2
- net UART_RX: track 0.00 -> 20.3 mm, vias 0 -> 2

Commit message: wip
Parts:
- added U$2: PHI-LOGO, keves-ng:PHI-LOGO
Other:
- board text added: "DT Breakout Box"
- board text added: "Designed by:"
- board text added: "Eran Rundstein"
- board text added: "Pulsar Heavy Industries"
- board text added: "Rev A, Nov 2020"
Changed lines of the file:
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@@
 <grid distance="10" unitdist="mil" unit="mil" style="lines" multiple="1" display="no" altdistance="5" altunitdist="mil" altunit="mil"/>
 <layers>
-<layer number="1" name="Top" color="4" fill="1" visible="no" active="yes"/>
-<layer number="2" name="Route2" color="16" fill="1" visible="no" active="yes"/>
+<layer number="1" name="Top" color="4" fill="1" visible="yes" active="yes"/>
+<layer number="2" name="Route2" color="16" fill="1" visible="yes" active="yes"/>
 <layer number="3" name="Route3" color="17" fill="1" visible="no" active="no"/>
 <layer number="4" name="Route4" color="18" fill="1" visible="no" active="no"/>
@@
 <layer number="13" name="Route13" color="21" fill="1" visible="no" active="no"/>
 <layer number="14" name="Route14" color="22" fill="1" visible="no" active="no"/>
-<layer number="15" name="Route15" color="23" fill="1" visible="no" active="yes"/>
-<layer number="16" name="Bottom" color="1" fill="1" visible="no" active="yes"/>
+<layer number="15" name="Route15" color="23" fill="1" visible="yes" active="yes"/>
+<layer number="16" name="Bottom" color="1" fill="1" visible="yes" active="yes"/>
 <layer number="17" name="Pads" color="2" fill="1" visible="yes" active="yes"/>
 <layer number="18" name="Vias" color="2" fill="1" visible="yes" active="yes"/>
@@
 <wire x1="148.59" y1="101.6" x2="0" y2="101.6" width="0" layer="20"/>
 <wire x1="0" y1="101.6" x2="0" y2="0" width="0" layer="20"/>
+<text x="42.926" y="88.392" size="1.778" layer="25" font="vector">DT Breakout Box</text>
+<text x="42.926" y="83.82" size="1.016" layer="25" font="vector">Designed by:</text>
+<text x="44.45" y="81.28" size="1.778" layer="25" font="vector">Eran Rundstein</text>
+<text x="43.18" y="79.248" size="1.27" layer="25" font="vector">Pulsar Heavy Industries</text>
+<text x="42.926" y="86.36" size="1.27" layer="25" font="vector">Rev A, Nov 2020</text>
 </plain>
 <attributes>
@@
 <attribute name="VALUE" x="44.45" y="66.548" size="0.4064" layer="27" font="vector" ratio="10" rot="R90"/>
 </element>
+<element name="U$2" library="keves-ng" library_urn="urn:adsk.eagle:library:1429743" package="PHI-LOGO" package3d_urn="urn:adsk.eagle:package:24014368/1" value="PHI-LOGO" x="32.512" y="86.106" smashed="yes" rot="R90"/>
 </elements>
 <signals>

Commit message: wip
Parts:
- C100, C96: value 10uF -> 10u; device microbuilder:0805 -> keves-ng:0805
- C101, C97: device microbuilder:1206 -> keves-ng:1206
- C102, C95, C99: value 0.1u -> 100n
- C77: value 100uF -> 100u
- C94, C98: value 2.2uF -> 2.2u; device microbuilder:_0805 -> keves-ng:0805
- D1, D2, D3, D4: device microbuilder:SOD-123 -> keves-ng:SOD-123
Routing:
- net PUSHBTN: track 117.6 -> 119.6 mm
- net N$73: track 9.50 -> 10.3 mm

Commit message: wip
Parts:
- C101, C97: value 1uF 12065C105M4Z2A -> 1u 12065C105M4Z2A
- C75: value 4.7uF -> 4.7u
- C80, C84, C85, C86, C90, C91: value 1uF Ceramic -> 1u Ceramic
- C81, C82, C83, C87, C88, C89, C92, C93: value 10uF Electrolyte -> 10u Electrolyte
Routing:
- net N$73: track 10.3 -> 9.65 mm
