File: dt/dt-rev-b.brd (EAGLE design)
At the start: 148.6 x 101.6 mm, 261 parts, among them IC1 TL072D, IC10 LM317, IC11 LM337, IC2 TL072D, IC3 TL072D, IC4 TL072D, IC5 TL072D, IC6 TL072D, IC7 AT45DB161D-SU, U1 LM1117DTX-3.3, U2 PCN2-S5-D15-S, U3 STM32F7X3ZXT, U4 USBLC6-2SC6YSOT23-6L_STM-M, U5 USBLC6-2SC6YSOT23-6L_STM-M, U6 PCM1681PWPPWP28_6P46X2P4-M, U7 PCM1681PWPPWP28_6P46X2P4-M, Y1 ABLS7M2-25.000MHZ-D2Y-T

Commit message: dt rev b: new layout wip
Parts:
- moved C102 267.7 mm to (284.5, 102.1)
- moved TP16 267.7 mm to (332.2, 104.1)
- moved R100 267.7 mm to (291.8, 122.7)
- moved R101 267.7 mm to (281.2, 105.4)
- moved R98 267.7 mm to (291.8, 117.6)
- moved R99 267.7 mm to (291.8, 120.1)
- moved U$2 267.7 mm to (299.2, 109.0)
- moved U$1 185.4 mm to (193.0, 76.2)
- moved R49 165.5 mm to (224.5, 145.3)
- moved TP1 165.5 mm to (237.5, 140.0)
- moved TP2 165.5 mm to (237.5, 135.4)
- moved U1 165.5 mm to (229.6, 143.5)
- moved C49 165.5 mm to (234.2, 140.0)
- moved C50 165.5 mm to (234.2, 145.0)
- moved C77 165.5 mm to (231.1, 134.1)
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Routing:
- net +5V: track 294.1 -> 115.4 mm, vias 10 -> 9
- net -12V: track 176.1 -> 19.6 mm, vias 10 -> 4
- net +12V: track 171.3 -> 27.0 mm, vias 9 -> 4
- net DAC_OUT12: track 105.4 -> 2.31 mm
- net DAC_OUT11: track 93.1 -> 2.96 mm
- net PUSHBTN: track 119.6 -> 31.3 mm, vias 2 -> 0
- net DAC_OUT8: track 90.9 -> 2.89 mm
- net LED3: track 91.6 -> 6.34 mm, vias 2 -> 0
- net DAC_OUT10: track 86.7 -> 3.82 mm
- net LED2: track 91.8 -> 9.36 mm, vias 2 -> 0
- net LED1: track 92.8 -> 11.8 mm, vias 2 -> 0
- net LED4: track 106.7 -> 29.7 mm, vias 2 -> 0
- net DAC_OUT7: track 79.1 -> 4.35 mm
- net DAC_OUT9: track 74.0 -> 4.55 mm
- net DAC_OUT6: track 70.1 -> 5.23 mm
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Other:
- board size 148.6 x 101.6 mm -> 199.4 x 101.6 mm

Commit message: dt rev b: new layout wip
Parts:
- moved TP4 156.9 mm to (99.2, 44.3), turned to 180 degrees
- moved TP5 153.7 mm to (99.2, 40.8), turned to 180 degrees
- moved TP3 150.7 mm to (99.2, 37.2), turned to 180 degrees
- moved JP6 148.0 mm to (106.6, 43.3), turned to 180 degrees
- moved C52 147.8 mm to (103.5, 39.5), turned to 180 degrees
- moved U2 144.0 mm to (115.4, 48.4), turned to 180 degrees
- moved C53 143.1 mm to (107.8, 39.5), turned to 0 degrees
- moved C51 141.6 mm to (113.2, 43.8), turned to 90 degrees
- moved C100 141.4 mm to (121.0, 50.9), turned to 0 degrees
- moved C101 138.7 mm to (126.4, 52.7), turned to 0 degrees
- moved L7 138.1 mm to (116.5, 43.6), turned to 90 degrees
- moved R96 137.6 mm to (122.6, 48.6), turned to 180 degrees
- moved D4 136.7 mm to (126.1, 50.7), turned to 0 degrees
- moved L6 134.8 mm to (130.9, 51.6), turned to 0 degrees
- moved R97 133.7 mm to (126.9, 48.6), turned to 180 degrees
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Routing:
- net +5V: track 115.4 -> 391.3 mm, vias 9 -> 10
- net +12V: track 27.0 -> 179.9 mm, vias 4 -> 6
- net -12V: track 19.6 -> 164.8 mm, vias 4 -> 9
- net N$71: track 11.0 -> 115.0 mm
- net N$70: track 12.3 -> 115.2 mm
- net N$68: track 13.5 -> 115.4 mm
- net N$66: track 14.8 -> 115.3 mm
- net I2C_SDA: track 69.5 -> 161.1 mm
- net I2C_SCL: track 73.7 -> 160.5 mm
- net +3V3: track 193.7 -> 277.5 mm, vias 39 -> 40
- net EXT_OUT2: track 0.04 -> 18.4 mm
- net EXT_OUT4: track 0.00 -> 17.1 mm
- net EXT_OUT10: track 0.00 -> 17.1 mm
- net EXT_OUT8: track 0.00 -> 17.0 mm
- net EXT_OUT12: track 0.00 -> 16.7 mm
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
Commit message: dt rev b: new layout wip
Parts:
- moved U$2 245.9 mm to (9.53, 11.6), turned to 180 degrees
- moved TP16 200.5 mm to (87.0, 17.1)
- moved R100 96.9 mm to (149.0, 69.5), turned to 270 degrees
- moved R99 95.4 mm to (150.7, 69.5), turned to 270 degrees
- moved R98 94.0 mm to (152.5, 69.5), turned to 270 degrees
- moved TP18 78.5 mm to (192.3, 15.2)
- moved R53 72.4 mm to (191.3, 25.4), turned to 90 degrees
- moved C71 69.9 mm to (193.0, 25.4), turned to 90 degrees
- moved TC1 66.0 mm to (195.6, 26.7), turned to 270 degrees
- moved C102 46.3 mm to (191.9, 38.7)
- moved R101 43.3 mm to (191.6, 40.5), turned to 0 degrees
- moved C19 21.0 mm to (52.7, 39.6), turned to 90 degrees
- moved C11 20.6 mm to (27.8, 40.5), turned to 90 degrees
- moved C27 20.6 mm to (78.0, 39.9), turned to 90 degrees
- moved C7 20.6 mm to (20.8, 40.6), turned to 90 degrees
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Connections:
- net DAC_OUT1: now also U6.27; no longer U6.15
- net DAC_OUT10: now also U7.26; no longer U7.22
- net DAC_OUT11: now also U7.22; no longer U7.26
- net DAC_OUT12: now also U7.21; no longer U7.27
- net DAC_OUT2: now also U6.26; no longer U6.16
- net DAC_OUT3: now also U6.22; no longer U6.19
- net DAC_OUT4: now also U6.21; no longer U6.20
- net DAC_OUT5: now also U6.20; no longer U6.21
- net DAC_OUT6: now also U6.19; no longer U6.22
- net DAC_OUT7: now also U6.16; no longer U6.26
- net DAC_OUT8: now also U6.15; no longer U6.27
- net DAC_OUT9: now also U7.27; no longer U7.21
- net LED1: now also U3.111; no longer U3.113
- net LED3: now also U3.113; no longer U3.111
- net LED4: now also U3.47; no longer U3.114
- net PUSHBTN: now also U3.46; no longer U3.115
Routing:
- net DAC_OUT8: track 2.89 -> 82.7 mm
- net DAC_OUT7: track 4.35 -> 68.5 mm
- net DAC_OUT6: track 5.23 -> 64.4 mm
- net UART_TX: track 1.10 -> 54.5 mm, vias 1 -> 2
- net UART_RX: track 0.10 -> 49.1 mm, vias 0 -> 2
- net SWCLK: track 0.00 -> 47.7 mm, vias 0 -> 2
- net DAC_OUT5: track 5.76 -> 50.7 mm
- net SWDIO: track 1.38 -> 45.9 mm, vias 0 -> 2
- net SWO: track 0.07 -> 44.2 mm, vias 0 -> 2
- net DAC_OUT4: track 6.29 -> 46.2 mm
- net DAC_OUT1: track 8.82 -> 45.2 mm
- net LED3: track 6.34 -> 33.1 mm
- net DAC_OUT2: track 7.98 -> 34.4 mm
- net DAC_OUT3: track 6.93 -> 31.7 mm
- net LED2: track 9.36 -> 32.9 mm
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Other:
- board size 199.4 x 101.6 mm -> 199.4 x 81.3 mm

Commit message: dt rev b: new layout wip
Parts:
- moved C35 1.78 mm to (104.1, 40.9)
- moved C31 1.55 mm to (95.2, 41.0)
- moved C23 1.27 mm to (69.7, 41.0)
- moved C39 1.27 mm to (121.7, 41.0)
- moved C27 0.76 mm to (78.0, 40.6)
Routing:
- net DAC_OUT12: track 9.93 -> 98.2 mm, vias 1 -> 2
- net DAC_OUT11: track 11.3 -> 92.3 mm, vias 1 -> 2
- net DAC_OUT10: track 14.1 -> 86.6 mm
- net DAC_OUT9: track 16.1 -> 69.7 mm
- net +12V: track 179.9 -> 202.2 mm, vias 6 -> 10
- net N$48: track 0.53 -> 7.61 mm
- net +3V3: track 284.5 -> 279.3 mm, vias 41 -> 33
- net N$36: track 0.00 -> 4.84 mm
- net N$38: track 7.70 -> 10.7 mm
- net N$40: track 0.53 -> 3.19 mm
- net N$44: track 0.00 -> 2.48 mm
- net +5V: track 391.3 -> 389.6 mm
- net N$32: track 4.72 -> 3.26 mm
- net -12V: track 164.8 -> 163.4 mm
- net N$24: track 4.61 -> 3.34 mm
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
Commit message: dt rev b
Parts:
- added H1, H2, H3, H4, H5, H6, H7: MOUNT-HOLE3.3, holes:3,3
- moved C78 5.48 mm to (173.5, 70.4)
- moved R57 5.48 mm to (171.7, 70.4)
- moved U$2 2.75 mm to (11.0, 13.8)
Routing:
- net N$67: track 17.7 -> 20.0 mm
- net GND: track 286.0 -> 287.5 mm
- net +5V: track 389.6 -> 390.5 mm

Commit message: wip
Parts:
- R12, R15, R20, R23, R28, R31, R36, R39, R4, R44, R47, R7: value 5.1k -> 51k
