File: dt/dt-rev-b.sch (EAGLE design)
At the start: 261 parts, among them IC1 TL072D, IC10 LM317, IC11 LM337, IC2 TL072D, IC3 TL072D, IC4 TL072D, IC5 TL072D, IC6 TL072D, IC7 AT45DB161D-SU, U1 LM1117DTX-3.3, U2 PCN2-S5-D15-S, U3 STM32F7X3ZXT, U4 USBLC6-2SC6YSOT23-6L_STM-M, U5 USBLC6-2SC6YSOT23-6L_STM-M, U6 PCM1681PWPPWP28_6P46X2P4-M, U7 PCM1681PWPPWP28_6P46X2P4-M, Y1 ABLS7M2-25.000MHZ-D2Y-T

Commit message: dt rev b: new layout wip
Connections:
- net DAC_OUT1: now also U6A.VOUT1; no longer U6A.VOUT8
- net DAC_OUT10: now also U7A.VOUT2; no longer U7A.VOUT3
- net DAC_OUT11: now also U7A.VOUT3; no longer U7A.VOUT2
- net DAC_OUT12: now also U7A.VOUT4; no longer U7A.VOUT1
- net DAC_OUT2: now also U6A.VOUT2; no longer U6A.VOUT7
- net DAC_OUT3: now also U6A.VOUT3; no longer U6A.VOUT6
- net DAC_OUT4: now also U6A.VOUT4; no longer U6A.VOUT5
- net DAC_OUT5: now also U6A.VOUT5; no longer U6A.VOUT4
- net DAC_OUT6: now also U6A.VOUT6; no longer U6A.VOUT3
- net DAC_OUT7: now also U6A.VOUT7; no longer U6A.VOUT2
- net DAC_OUT8: now also U6A.VOUT8; no longer U6A.VOUT1
- net DAC_OUT9: now also U7A.VOUT1; no longer U7A.VOUT4
- net LED1: now also U3A.PC10; no longer U3A.PC12
- net LED3: now also U3A.PC12; no longer U3A.PC10
- net LED4: now also U3A.PB1; no longer U3A.PD0
- net PUSHBTN: now also U3A.PB0; no longer U3A.PD1
Changed lines of the file:
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@@
 </segment>
 </net>
-<net name="LED3" class="0">
+<net name="LED1" class="0">
 <segment>
 <pinref part="U3" gate="A" pin="PC10"/>
@@
 </segment>
 </net>
-<net name="LED1" class="0">
-<segment>
-<pinref part="U3" gate="A" pin="PC12"/>
-<wire x1="99.06" y1="17.78" x2="109.22" y2="17.78" width="0.1524" layer="91"/>
-<label x="109.22" y="17.78" size="1.778" layer="95"/>
-</segment>
-</net>
 <net name="LED4" class="0">
 <segment>
-<pinref part="U3" gate="A" pin="PD0"/>
-<wire x1="27.94" y1="45.72" x2="10.16" y2="45.72" width="0.1524" layer="91"/>
-<label x="10.16" y="45.72" size="1.778" layer="95"/>
+<pinref part="U3" gate="A" pin="PB1"/>
+<wire x1="27.94" y1="88.9" x2="12.7" y2="88.9" width="0.1524" layer="91"/>
+<label x="10.16" y="88.9" size="1.778" layer="95"/>
 </segment>
 </net>
 <net name="PUSHBTN" class="0">
 <segment>
-<pinref part="U3" gate="A" pin="PD1"/>
-<wire x1="27.94" y1="43.18" x2="10.16" y2="43.18" width="0.1524" layer="91"/>
-<label x="10.16" y="43.18" size="1.778" layer="95"/>
+<pinref part="U3" gate="A" pin="PB0"/>
+<wire x1="27.94" y1="91.44" x2="12.7" y2="91.44" width="0.1524" layer="91"/>
+<label x="10.16" y="91.44" size="1.778" layer="95"/>
 </segment>
 </net>
@@
 <wire x1="266.7" y1="91.44" x2="279.4" y2="91.44" width="0.1524" layer="91"/>
 <junction x="266.7" y="91.44"/>
+</segment>
+</net>
+<net name="LED3" class="0">
+<segment>
+<pinref part="U3" gate="A" pin="PC12"/>
+<wire x1="99.06" y1="17.78" x2="109.22" y2="17.78" width="0.1524" layer="91"/>
+<label x="109.22" y="17.78" size="1.778" layer="95"/>
 </segment>
 </net>
@@
 </busses>
 <nets>
-<net name="DAC_OUT1" class="0">
-<segment>
-<pinref part="U6" gate="A" pin="VOUT8"/>
-<wire x1="119.38" y1="231.14" x2="127" y2="231.14" width="0.1524" layer="91"/>
-<label x="127" y="231.14" size="1.778" layer="95"/>
-</segment>
-</net>
-<net name="DAC_OUT2" class="0">
-<segment>
-<pinref part="U6" gate="A" pin="VOUT7"/>
-<wire x1="119.38" y1="228.6" x2="127" y2="228.6" width="0.1524" layer="91"/>
-<label x="127" y="228.6" size="1.778" layer="95"/>
-</segment>
-</net>
-<net name="DAC_OUT3" class="0">
-<segment>
-<pinref part="U6" gate="A" pin="VOUT6"/>
-<wire x1="119.38" y1="226.06" x2="127" y2="226.06" width="0.1524" layer="91"/>
-<label x="127" y="226.06" size="1.778" layer="95"/>
-</segment>
-</net>
-<net name="DAC_OUT4" class="0">
-<segment>
-<pinref part="U6" gate="A" pin="VOUT5"/>
-<wire x1="119.38" y1="223.52" x2="127" y2="223.52" width="0.1524" layer="91"/>
-<label x="127" y="223.52" size="1.778" layer="95"/>
-</segment>
-</net>
 <net name="N$75" class="0">
 <segment>
@@
 <net name="DAC_OUT9" class="0">
 <segment>
-<pinref part="U7" gate="A" pin="VOUT4"/>
-<wire x1="119.38" y1="83.82" x2="127" y2="83.82" width="0.1524" layer="91"/>
-<label x="127" y="83.82" size="1.778" layer="95"/>
+<pinref part="U7" gate="A" pin="VOUT1"/>
+<wire x1="119.38" y1="76.2" x2="127" y2="76.2" width="0.1524" layer="91"/>
+<label x="127" y="76.2" size="1.778" layer="95"/>
 </segment>
 </net>
 <net name="DAC_OUT10" class="0">
 <segment>
-<pinref part="U7" gate="A" pin="VOUT3"/>
-<wire x1="119.38" y1="81.28" x2="127" y2="81.28" width="0.1524" layer="91"/>
-<label x="127" y="81.28" size="1.778" layer="95"/>
+<pinref part="U7" gate="A" pin="VOUT2"/>
+<wire x1="119.38" y1="78.74" x2="127" y2="78.74" width="0.1524" layer="91"/>
+<label x="127" y="78.74" size="1.778" layer="95"/>
 </segment>
 </net>
@@
 <net name="DAC_OUT5" class="0">
 <segment>
+<pinref part="U6" gate="A" pin="VOUT5"/>
+<wire x1="119.38" y1="223.52" x2="127" y2="223.52" width="0.1524" layer="91"/>
+<label x="127" y="223.52" size="1.778" layer="95"/>
+</segment>
+</net>
+<net name="DAC_OUT6" class="0">
+<segment>
+<pinref part="U6" gate="A" pin="VOUT6"/>
+<wire x1="119.38" y1="226.06" x2="127" y2="226.06" width="0.1524" layer="91"/>
+<label x="127" y="226.06" size="1.778" layer="95"/>
+</segment>
+</net>
+<net name="DAC_OUT7" class="0">
+<segment>
+<pinref part="U6" gate="A" pin="VOUT7"/>
+<wire x1="119.38" y1="228.6" x2="127" y2="228.6" width="0.1524" layer="91"/>
+<label x="127" y="228.6" size="1.778" layer="95"/>
+</segment>
+</net>
+<net name="DAC_OUT8" class="0">
+<segment>
+<pinref part="U6" gate="A" pin="VOUT8"/>
+<wire x1="119.38" y1="231.14" x2="127" y2="231.14" width="0.1524" layer="91"/>
+<label x="127" y="231.14" size="1.778" layer="95"/>
+</segment>
+</net>
+<net name="DAC_OUT4" class="0">
+<segment>
 <pinref part="U6" gate="A" pin="VOUT4"/>
 <wire x1="119.38" y1="220.98" x2="127" y2="220.98" width="0.1524" layer="91"/>
@@
 </segment>
 </net>
-<net name="DAC_OUT6" class="0">
+<net name="DAC_OUT3" class="0">
 <segment>
 <pinref part="U6" gate="A" pin="VOUT3"/>
@@
 </segment>
 </net>
-<net name="DAC_OUT7" class="0">
+<net name="DAC_OUT2" class="0">
 <segment>
 <pinref part="U6" gate="A" pin="VOUT2"/>
@@
 </segment>
 </net>
-<net name="DAC_OUT8" class="0">
+<net name="DAC_OUT1" class="0">
 <segment>
 <pinref part="U6" gate="A" pin="VOUT1"/>
@@
 <net name="DAC_OUT11" class="0">
 <segment>
-<pinref part="U7" gate="A" pin="VOUT2"/>
-<wire x1="119.38" y1="78.74" x2="127" y2="78.74" width="0.1524" layer="91"/>
-<label x="127" y="78.74" size="1.778" layer="95"/>
+<pinref part="U7" gate="A" pin="VOUT3"/>
+<wire x1="119.38" y1="81.28" x2="127" y2="81.28" width="0.1524" layer="91"/>
+<label x="127" y="81.28" size="1.778" layer="95"/>
 </segment>
 </net>
 <net name="DAC_OUT12" class="0">
 <segment>
-<pinref part="U7" gate="A" pin="VOUT1"/>
-<wire x1="119.38" y1="76.2" x2="127" y2="76.2" width="0.1524" layer="91"/>
-<label x="127" y="76.2" size="1.778" layer="95"/>
-</segment>
-</net>
+<pinref part="U7" gate="A" pin="VOUT4"/>
+<wire x1="119.38" y1="83.82" x2="127" y2="83.82" width="0.1524" layer="91"/>
+<label x="127" y="83.82" size="1.778" layer="95"/>
+</segment>
+</net>

Commit message: dt rev b
Parts:
- added H1, H2, H3, H4, H5, H6, H7: MOUNT-HOLE3.3, holes:MOUNT-HOLE3.3
- TP10, TP16, TP17, TP18, TP7, TP8, TP9: PARTNO (none) -> 5001
Changed lines of the file:
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@@
 <attribute name="PARTNO" value="PM1812-5R6J-RC"/>
 </part>
-<part name="TP7" library="keves-ng" library_urn="urn:adsk.eagle:library:1429743" deviceset="TP" device="PAD1-13" package3d_urn="urn:adsk.eagle:package:24104776/2" value="TPPAD1-13"/>
-<part name="TP8" library="keves-ng" library_urn="urn:adsk.eagle:library:1429743" deviceset="TP" device="PAD1-13" package3d_urn="urn:adsk.eagle:package:24104776/2" value="TPPAD1-13"/>
-<part name="TP9" library="keves-ng" library_urn="urn:adsk.eagle:library:1429743" deviceset="TP" device="PAD1-13" package3d_urn="urn:adsk.eagle:package:24104776/2" value="TPPAD1-13"/>
-<part name="TP10" library="keves-ng" library_urn="urn:adsk.eagle:library:1429743" deviceset="TP" device="PAD1-13" package3d_urn="urn:adsk.eagle:package:24104776/2" value="TPPAD1-13"/>
-<part name="TP16" library="keves-ng" library_urn="urn:adsk.eagle:library:1429743" deviceset="TP" device="PAD1-13" package3d_urn="urn:adsk.eagle:package:24104776/2" value="TPPAD1-13"/>
-<part name="TP17" library="keves-ng" library_urn="urn:adsk.eagle:library:1429743" deviceset="TP" device="PAD1-13" package3d_urn="urn:adsk.eagle:package:24104776/2" value="TPPAD1-13"/>
-<part name="TP18" library="keves-ng" library_urn="urn:adsk.eagle:library:1429743" deviceset="TP" device="PAD1-13" package3d_urn="urn:adsk.eagle:package:24104776/2" value="TPPAD1-13"/>
+<part name="TP7" library="keves-ng" library_urn="urn:adsk.eagle:library:1429743" deviceset="TP" device="PAD1-13" package3d_urn="urn:adsk.eagle:package:24104776/2" value="TPPAD1-13">
+<attribute name="PARTNO" value="5001"/>
+</part>
+<part name="TP8" library="keves-ng" library_urn="urn:adsk.eagle:library:1429743" deviceset="TP" device="PAD1-13" package3d_urn="urn:adsk.eagle:package:24104776/2" value="TPPAD1-13">
+<attribute name="PARTNO" value="5001"/>
+</part>
+<part name="TP9" library="keves-ng" library_urn="urn:adsk.eagle:library:1429743" deviceset="TP" device="PAD1-13" package3d_urn="urn:adsk.eagle:package:24104776/2" value="TPPAD1-13">
+<attribute name="PARTNO" value="5001"/>
+</part>
+<part name="TP10" library="keves-ng" library_urn="urn:adsk.eagle:library:1429743" deviceset="TP" device="PAD1-13" package3d_urn="urn:adsk.eagle:package:24104776/2" value="TPPAD1-13">
+<attribute name="PARTNO" value="5001"/>
+</part>
+<part name="TP16" library="keves-ng" library_urn="urn:adsk.eagle:library:1429743" deviceset="TP" device="PAD1-13" package3d_urn="urn:adsk.eagle:package:24104776/2" value="TPPAD1-13">
+<attribute name="PARTNO" value="5001"/>
+</part>
+<part name="TP17" library="keves-ng" library_urn="urn:adsk.eagle:library:1429743" deviceset="TP" device="PAD1-13" package3d_urn="urn:adsk.eagle:package:24104776/2" value="TPPAD1-13">
+<attribute name="PARTNO" value="5001"/>
+</part>
+<part name="TP18" library="keves-ng" library_urn="urn:adsk.eagle:library:1429743" deviceset="TP" device="PAD1-13" package3d_urn="urn:adsk.eagle:package:24104776/2" value="TPPAD1-13">
+<attribute name="PARTNO" value="5001"/>
+</part>
 <part name="GND95" library="supply1" library_urn="urn:adsk.eagle:library:371" deviceset="GND" device=""/>
 <part name="GND96" library="supply1" library_urn="urn:adsk.eagle:library:371" deviceset="GND" device=""/>
@@
 <part name="GND78" library="supply1" library_urn="urn:adsk.eagle:library:371" deviceset="GND" device=""/>
 <part name="GND67" library="supply1" library_urn="urn:adsk.eagle:library:371" deviceset="GND" device=""/>
+<part name="H1" library="holes" library_urn="urn:adsk.eagle:library:237" deviceset="MOUNT-HOLE" device="3.3" package3d_urn="urn:adsk.eagle:package:14278/1">
+<attribute name="PARTNO" value="*"/>
+</part>
+<part name="H2" library="holes" library_urn="urn:adsk.eagle:library:237" deviceset="MOUNT-HOLE" device="3.3" package3d_urn="urn:adsk.eagle:package:14278/1">
+<attribute name="PARTNO" value="*"/>
+</part>
+<part name="H3" library="holes" library_urn="urn:adsk.eagle:library:237" deviceset="MOUNT-HOLE" device="3.3" package3d_urn="urn:adsk.eagle:package:14278/1">
+<attribute name="PARTNO" value="*"/>
+</part>
+<part name="H4" library="holes" library_urn="urn:adsk.eagle:library:237" deviceset="MOUNT-HOLE" device="3.3" package3d_urn="urn:adsk.eagle:package:14278/1">
+<attribute name="PARTNO" value="*"/>
+</part>
+<part name="H5" library="holes" library_urn="urn:adsk.eagle:library:237" deviceset="MOUNT-HOLE" device="3.3" package3d_urn="urn:adsk.eagle:package:14278/1">
+<attribute name="PARTNO" value="*"/>
+</part>
+<part name="H6" library="holes" library_urn="urn:adsk.eagle:library:237" deviceset="MOUNT-HOLE" device="3.3" package3d_urn="urn:adsk.eagle:package:14278/1">
+<attribute name="PARTNO" value="*"/>
+</part>
+<part name="H7" library="holes" library_urn="urn:adsk.eagle:library:237" deviceset="MOUNT-HOLE" device="3.3" package3d_urn="urn:adsk.eagle:package:14278/1">
+<attribute name="PARTNO" value="*"/>
+</part>
 </parts>
 <sheets>
@@
 <attribute name="NAME" x="260.35" y="100.33" size="1.778" layer="95"/>
 <attribute name="TP_SIGNAL_NAME" x="262.89" y="97.79" size="1.778" layer="97"/>
+<attribute name="PARTNO" x="261.62" y="99.06" size="1.778" layer="96" display="off"/>
 </instance>
 <instance part="TP8" gate="G$1" x="264.16" y="96.52" smashed="yes">
 <attribute name="NAME" x="262.89" y="97.79" size="1.778" layer="95"/>
 <attribute name="TP_SIGNAL_NAME" x="265.43" y="95.25" size="1.778" layer="97"/>
+<attribute name="PARTNO" x="264.16" y="96.52" size="1.778" layer="96" display="off"/>
 </instance>
 <instance part="TP9" gate="G$1" x="266.7" y="93.98" smashed="yes">
 <attribute name="NAME" x="265.43" y="95.25" size="1.778" layer="95"/>
 <attribute name="TP_SIGNAL_NAME" x="267.97" y="92.71" size="1.778" layer="97"/>
+<attribute name="PARTNO" x="266.7" y="93.98" size="1.778" layer="96" display="off"/>
 </instance>
 <instance part="TP10" gate="G$1" x="269.24" y="91.44" smashed="yes">
 <attribute name="NAME" x="267.97" y="92.71" size="1.778" layer="95"/>
 <attribute name="TP_SIGNAL_NAME" x="270.51" y="90.17" size="1.778" layer="97"/>
+<attribute name="PARTNO" x="269.24" y="91.44" size="1.778" layer="96" display="off"/>
 </instance>
 <instance part="TP16" gate="G$1" x="22.86" y="-10.16" smashed="yes">
 <attribute name="NAME" x="21.59" y="-8.89" size="1.778" layer="95"/>
 <attribute name="TP_SIGNAL_NAME" x="24.13" y="-11.43" size="1.778" layer="97"/>
+<attribute name="PARTNO" x="22.86" y="-10.16" size="1.778" layer="96" display="off"/>
 </instance>
 <instance part="TP17" gate="G$1" x="27.94" y="-10.16" smashed="yes">
 <attribute name="NAME" x="26.67" y="-8.89" size="1.778" layer="95"/>
 <attribute name="TP_SIGNAL_NAME" x="29.21" y="-11.43" size="1.778" layer="97"/>
+<attribute name="PARTNO" x="27.94" y="-10.16" size="1.778" layer="96" display="off"/>
 </instance>
 <instance part="TP18" gate="G$1" x="33.02" y="-10.16" smashed="yes">
 <attribute name="NAME" x="31.75" y="-8.89" size="1.778" layer="95"/>
 <attribute name="TP_SIGNAL_NAME" x="34.29" y="-11.43" size="1.778" layer="97"/>
+<attribute name="PARTNO" x="33.02" y="-10.16" size="1.778" layer="96" display="off"/>
 </instance>
 <instance part="GND95" gate="1" x="22.86" y="-17.78" smashed="yes">
 <attribute name="VALUE" x="20.32" y="-20.32" size="1.778" layer="96"/>
 </instance>
+<instance part="H1" gate="G$1" x="256.54" y="193.04" smashed="yes">
+<attribute name="NAME" x="258.572" y="193.6242" size="1.778" layer="95"/>
+<attribute name="VALUE" x="258.572" y="190.5762" size="1.778" layer="96"/>
+<attribute name="PARTNO" x="256.54" y="193.04" size="1.778" layer="96" display="off"/>
+</instance>
+<instance part="H2" gate="G$1" x="256.54" y="185.42" smashed="yes">
+<attribute name="NAME" x="258.572" y="186.0042" size="1.778" layer="95"/>
+<attribute name="VALUE" x="258.572" y="182.9562" size="1.778" layer="96"/>
+<attribute name="PARTNO" x="256.54" y="185.42" size="1.778" layer="96" display="off"/>
+</instance>
+<instance part="H3" gate="G$1" x="256.54" y="177.8" smashed="yes">
+<attribute name="NAME" x="258.572" y="178.3842" size="1.778" layer="95"/>
+<attribute name="VALUE" x="258.572" y="175.3362" size="1.778" layer="96"/>
+<attribute name="PARTNO" x="256.54" y="177.8" size="1.778" layer="96" display="off"/>
+</instance>
+<instance part="H4" gate="G$1" x="256.54" y="170.18" smashed="yes">
+<attribute name="NAME" x="258.572" y="170.7642" size="1.778" layer="95"/>
+<attribute name="VALUE" x="258.572" y="167.7162" size="1.778" layer="96"/>
+<attribute name="PARTNO" x="256.54" y="170.18" size="1.778" layer="96" display="off"/>
+</instance>
+<instance part="H5" gate="G$1" x="256.54" y="162.56" smashed="yes">
+<attribute name="NAME" x="258.572" y="163.1442" size="1.778" layer="95"/>
+<attribute name="VALUE" x="258.572" y="160.0962" size="1.778" layer="96"/>
+<attribute name="PARTNO" x="256.54" y="162.56" size="1.778" layer="96" display="off"/>
+</instance>
+<instance part="H6" gate="G$1" x="256.54" y="154.94" smashed="yes">
+<attribute name="NAME" x="258.572" y="155.5242" size="1.778" layer="95"/>
+<attribute name="VALUE" x="258.572" y="152.4762" size="1.778" layer="96"/>
+<attribute name="PARTNO" x="256.54" y="154.94" size="1.778" layer="96" display="off"/>
+</instance>
+<instance part="H7" gate="G$1" x="256.54" y="147.32" smashed="yes">
+<attribute name="NAME" x="258.572" y="147.9042" size="1.778" layer="95"/>
+<attribute name="VALUE" x="258.572" y="144.8562" size="1.778" layer="96"/>
+<attribute name="PARTNO" x="256.54" y="147.32" size="1.778" layer="96" display="off"/>
+</instance>
 </instances>
