File: dt/dt-rev-b.sch (EAGLE design)
At the start: 268 parts, among them IC1 TL072D, IC10 LM317, IC11 LM337, IC2 TL072D, IC3 TL072D, IC4 TL072D, IC5 TL072D, IC6 TL072D, IC7 AT45DB161D-SU, U1 LM1117DTX-3.3, U2 PCN2-S5-D15-S, U3 STM32F7X3ZXT, U4 USBLC6-2SC6YSOT23-6L_STM-M, U5 USBLC6-2SC6YSOT23-6L_STM-M, U6 PCM1681PWPPWP28_6P46X2P4-M, U7 PCM1681PWPPWP28_6P46X2P4-M, Y1 ABLS7M2-25.000MHZ-D2Y-T

Commit message: wip
Parts:
- R12, R15, R20, R23, R28, R31, R36, R39, R4, R44, R47, R7: value 5.1k -> 51k; PARTNO CRCW06035K10FKEAC -> RC0603FR-0751KL
Changed lines of the file:
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@@
 <attribute name="PARTNO" value="ERJ-3EKF8201V"/>
 </part>
-<part name="R4" library="keves-ng" library_urn="urn:adsk.eagle:library:1429743" deviceset="RESISTOR" device="0603" package3d_urn="urn:adsk.eagle:package:23799129/3" value="5.1k">
-<attribute name="PARTNO" value="CRCW06035K10FKEAC"/>
+<part name="R4" library="keves-ng" library_urn="urn:adsk.eagle:library:1429743" deviceset="RESISTOR" device="0603" package3d_urn="urn:adsk.eagle:package:23799129/3" value="51k">
+<attribute name="PARTNO" value="RC0603FR-0751KL"/>
 </part>
 <part name="C2" library="keves-ng" library_urn="urn:adsk.eagle:library:1429743" deviceset="CAP_CERAMIC" device="0603" package3d_urn="urn:adsk.eagle:package:23799129/3" value="4700pF">
@@
 <attribute name="PARTNO" value="ERJ-3EKF8201V"/>
 </part>
-<part name="R7" library="keves-ng" library_urn="urn:adsk.eagle:library:1429743" deviceset="RESISTOR" device="0603" package3d_urn="urn:adsk.eagle:package:23799129/3" value="5.1k">
-<attribute name="PARTNO" value="CRCW06035K10FKEAC"/>
+<part name="R7" library="keves-ng" library_urn="urn:adsk.eagle:library:1429743" deviceset="RESISTOR" device="0603" package3d_urn="urn:adsk.eagle:package:23799129/3" value="51k">
+<attribute name="PARTNO" value="RC0603FR-0751KL"/>
 </part>
 <part name="C6" library="keves-ng" library_urn="urn:adsk.eagle:library:1429743" deviceset="CAP_CERAMIC" device="0603" package3d_urn="urn:adsk.eagle:package:23799129/3" value="4700pF">
@@
 <attribute name="PARTNO" value="ERJ-3EKF8201V"/>
 </part>
-<part name="R12" library="keves-ng" library_urn="urn:adsk.eagle:library:1429743" deviceset="RESISTOR" device="0603" package3d_urn="urn:adsk.eagle:package:23799129/3" value="5.1k">
-<attribute name="PARTNO" value="CRCW06035K10FKEAC"/>
+<part name="R12" library="keves-ng" library_urn="urn:adsk.eagle:library:1429743" deviceset="RESISTOR" device="0603" package3d_urn="urn:adsk.eagle:package:23799129/3" value="51k">
+<attribute name="PARTNO" value="RC0603FR-0751KL"/>
 </part>
 <part name="C10" library="keves-ng" library_urn="urn:adsk.eagle:library:1429743" deviceset="CAP_CERAMIC" device="0603" package3d_urn="urn:adsk.eagle:package:23799129/3" value="4700pF">
@@
 <attribute name="PARTNO" value="ERJ-3EKF8201V"/>
 </part>
-<part name="R15" library="keves-ng" library_urn="urn:adsk.eagle:library:1429743" deviceset="RESISTOR" device="0603" package3d_urn="urn:adsk.eagle:package:23799129/3" value="5.1k">
-<attribute name="PARTNO" value="CRCW06035K10FKEAC"/>
+<part name="R15" library="keves-ng" library_urn="urn:adsk.eagle:library:1429743" deviceset="RESISTOR" device="0603" package3d_urn="urn:adsk.eagle:package:23799129/3" value="51k">
+<attribute name="PARTNO" value="RC0603FR-0751KL"/>
 </part>
 <part name="C14" library="keves-ng" library_urn="urn:adsk.eagle:library:1429743" deviceset="CAP_CERAMIC" device="0603" package3d_urn="urn:adsk.eagle:package:23799129/3" value="4700pF">
@@
 <attribute name="PARTNO" value="ERJ-3EKF8201V"/>
 </part>
-<part name="R20" library="keves-ng" library_urn="urn:adsk.eagle:library:1429743" deviceset="RESISTOR" device="0603" package3d_urn="urn:adsk.eagle:package:23799129/3" value="5.1k">
-<attribute name="PARTNO" value="CRCW06035K10FKEAC"/>
+<part name="R20" library="keves-ng" library_urn="urn:adsk.eagle:library:1429743" deviceset="RESISTOR" device="0603" package3d_urn="urn:adsk.eagle:package:23799129/3" value="51k">
+<attribute name="PARTNO" value="RC0603FR-0751KL"/>
 </part>
 <part name="C18" library="keves-ng" library_urn="urn:adsk.eagle:library:1429743" deviceset="CAP_CERAMIC" device="0603" package3d_urn="urn:adsk.eagle:package:23799129/3" value="4700pF">
@@
 <attribute name="PARTNO" value="ERJ-3EKF8201V"/>
 </part>
-<part name="R23" library="keves-ng" library_urn="urn:adsk.eagle:library:1429743" deviceset="RESISTOR" device="0603" package3d_urn="urn:adsk.eagle:package:23799129/3" value="5.1k">
-<attribute name="PARTNO" value="CRCW06035K10FKEAC"/>
+<part name="R23" library="keves-ng" library_urn="urn:adsk.eagle:library:1429743" deviceset="RESISTOR" device="0603" package3d_urn="urn:adsk.eagle:package:23799129/3" value="51k">
+<attribute name="PARTNO" value="RC0603FR-0751KL"/>
 </part>
 <part name="C22" library="keves-ng" library_urn="urn:adsk.eagle:library:1429743" deviceset="CAP_CERAMIC" device="0603" package3d_urn="urn:adsk.eagle:package:23799129/3" value="4700pF">
@@
 <attribute name="PARTNO" value="ERJ-3EKF8201V"/>
 </part>
-<part name="R28" library="keves-ng" library_urn="urn:adsk.eagle:library:1429743" deviceset="RESISTOR" device="0603" package3d_urn="urn:adsk.eagle:package:23799129/3" value="5.1k">
-<attribute name="PARTNO" value="CRCW06035K10FKEAC"/>
+<part name="R28" library="keves-ng" library_urn="urn:adsk.eagle:library:1429743" deviceset="RESISTOR" device="0603" package3d_urn="urn:adsk.eagle:package:23799129/3" value="51k">
+<attribute name="PARTNO" value="RC0603FR-0751KL"/>
 </part>
 <part name="C26" library="keves-ng" library_urn="urn:adsk.eagle:library:1429743" deviceset="CAP_CERAMIC" device="0603" package3d_urn="urn:adsk.eagle:package:23799129/3" value="4700pF">
@@
 <attribute name="PARTNO" value="ERJ-3EKF8201V"/>
 </part>
-<part name="R31" library="keves-ng" library_urn="urn:adsk.eagle:library:1429743" deviceset="RESISTOR" device="0603" package3d_urn="urn:adsk.eagle:package:23799129/3" value="5.1k">
-<attribute name="PARTNO" value="CRCW06035K10FKEAC"/>
+<part name="R31" library="keves-ng" library_urn="urn:adsk.eagle:library:1429743" deviceset="RESISTOR" device="0603" package3d_urn="urn:adsk.eagle:package:23799129/3" value="51k">
+<attribute name="PARTNO" value="RC0603FR-0751KL"/>
 </part>
 <part name="C30" library="keves-ng" library_urn="urn:adsk.eagle:library:1429743" deviceset="CAP_CERAMIC" device="0603" package3d_urn="urn:adsk.eagle:package:23799129/3" value="4700pF">
@@
 <attribute name="PARTNO" value="ERJ-3EKF8201V"/>
 </part>
-<part name="R36" library="keves-ng" library_urn="urn:adsk.eagle:library:1429743" deviceset="RESISTOR" device="0603" package3d_urn="urn:adsk.eagle:package:23799129/3" value="5.1k">
-<attribute name="PARTNO" value="CRCW06035K10FKEAC"/>
+<part name="R36" library="keves-ng" library_urn="urn:adsk.eagle:library:1429743" deviceset="RESISTOR" device="0603" package3d_urn="urn:adsk.eagle:package:23799129/3" value="51k">
+<attribute name="PARTNO" value="RC0603FR-0751KL"/>
 </part>
 <part name="C34" library="keves-ng" library_urn="urn:adsk.eagle:library:1429743" deviceset="CAP_CERAMIC" device="0603" package3d_urn="urn:adsk.eagle:package:23799129/3" value="4700pF">
@@
 <attribute name="PARTNO" value="ERJ-3EKF8201V"/>
 </part>
-<part name="R39" library="keves-ng" library_urn="urn:adsk.eagle:library:1429743" deviceset="RESISTOR" device="0603" package3d_urn="urn:adsk.eagle:package:23799129/3" value="5.1k">
-<attribute name="PARTNO" value="CRCW06035K10FKEAC"/>
+<part name="R39" library="keves-ng" library_urn="urn:adsk.eagle:library:1429743" deviceset="RESISTOR" device="0603" package3d_urn="urn:adsk.eagle:package:23799129/3" value="51k">
+<attribute name="PARTNO" value="RC0603FR-0751KL"/>
 </part>
 <part name="C38" library="keves-ng" library_urn="urn:adsk.eagle:library:1429743" deviceset="CAP_CERAMIC" device="0603" package3d_urn="urn:adsk.eagle:package:23799129/3" value="4700pF">
@@
 <attribute name="PARTNO" value="ERJ-3EKF8201V"/>
 </part>
-<part name="R44" library="keves-ng" library_urn="urn:adsk.eagle:library:1429743" deviceset="RESISTOR" device="0603" package3d_urn="urn:adsk.eagle:package:23799129/3" value="5.1k">
-<attribute name="PARTNO" value="CRCW06035K10FKEAC"/>
+<part name="R44" library="keves-ng" library_urn="urn:adsk.eagle:library:1429743" deviceset="RESISTOR" device="0603" package3d_urn="urn:adsk.eagle:package:23799129/3" value="51k">
+<attribute name="PARTNO" value="RC0603FR-0751KL"/>
 </part>
 <part name="C42" library="keves-ng" library_urn="urn:adsk.eagle:library:1429743" deviceset="CAP_CERAMIC" device="0603" package3d_urn="urn:adsk.eagle:package:23799129/3" value="4700pF">
@@
 <attribute name="PARTNO" value="ERJ-3EKF8201V"/>
 </part>
-<part name="R47" library="keves-ng" library_urn="urn:adsk.eagle:library:1429743" deviceset="RESISTOR" device="0603" package3d_urn="urn:adsk.eagle:package:23799129/3" value="5.1k">
-<attribute name="PARTNO" value="CRCW06035K10FKEAC"/>
+<part name="R47" library="keves-ng" library_urn="urn:adsk.eagle:library:1429743" deviceset="RESISTOR" device="0603" package3d_urn="urn:adsk.eagle:package:23799129/3" value="51k">
+<attribute name="PARTNO" value="RC0603FR-0751KL"/>
 </part>
 <part name="C46" library="keves-ng" library_urn="urn:adsk.eagle:library:1429743" deviceset="CAP_CERAMIC" device="0603" package3d_urn="urn:adsk.eagle:package:23799129/3" value="4700pF">
